Commit message: Update pre-generated URDF of HSR-B.

File: tmc_hsrb_description/robots/hsrb.urdf (robot description, URDF)
Before this commit: robot hsrb, 36 links, 35 joints
Links:
- link hsrb/arm_flex_link: geometry collision mesh filename=package://tmc_hsrb_description/meshes/arm_v0/arm_flex.stl; visual mesh filename=package://tmc_hsrb_description/meshes/arm_v0/arm_flex.dae
- link hsrb/arm_lift_link: geometry collision mesh filename=package://tmc_hsrb_description/meshes/arm_v0/shoulder.stl; visual mesh filename=package://tmc_hsrb_description/meshes/arm_v0/shoulder.dae
- link hsrb/arm_roll_link: geometry collision mesh filename=package://tmc_hsrb_description/meshes/arm_v0/arm_roll.stl; visual mesh filename=package://tmc_hsrb_description/meshes/arm_v0/arm_roll.dae
- link hsrb/base_laser_link: geometry collision mesh filename=package://tmc_hsrb_description/meshes/sensors/laser.stl; visual mesh filename=package://tmc_hsrb_description/meshes/sensors/laser.dae
- link hsrb/base_link: geometry collision mesh filename=package://tmc_hsrb_description/meshes/base_v0/base.stl; visual mesh filename=package://tmc_hsrb_description/meshes/base_v0/base.dae
- link hsrb/hand_palm_link: geometry collision mesh filename=package://tmc_hsrb_description/meshes/hand_v0/palm.stl; visual mesh filename=package://tmc_hsrb_description/meshes/hand_v0/palm.dae
- link hsrb/head_depth_camera_link: geometry collision mesh filename=package://tmc_hsrb_description/meshes/sensors/xtion.stl; visual mesh filename=package://tmc_hsrb_description/meshes/sensors/xtion.dae
- link hsrb/head_left_camera_link: geometry visual mesh filename=package://tmc_hsrb_description/meshes/sensors/head_camera.d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
- link hsrb/head_pan_link: geometry collision mesh filename=package://tmc_hsrb_description/meshes/head_v0/head_pan.stl; visual mesh filename=package://tmc_hsrb_description/meshes/head_v0/head_pan.dae
- link hsrb/head_right_camera_link: geometry visual mesh filename=package://tmc_hsrb_description/meshes/sensors/head_camera.d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
- link hsrb/head_tilt_link: geometry collision mesh filename=package://tmc_hsrb_description/meshes/head_v0/head.stl; collision mesh filename=package://tmc_hsrb_description/meshes/head_v0/tablet.stl
- link hsrb/left_distal_link: geometry collision mesh filename=package://tmc_hsrb_description/meshes/hand_v0/left_distal.s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; visual mesh filename=package://tmc_hsrb_description/meshes/hand_v0/left_distal.d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
- link hsrb/left_proximal_link: geometry collision mesh filename=package://tmc_hsrb_description/meshes/hand_v0/left_proximal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; visual mesh filename=package://tmc_hsrb_description/meshes/hand_v0/left_proximal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
- link hsrb/right_distal_link: geometry collision mesh filename=package://tmc_hsrb_description/meshes/hand_v0/right_distal.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; visual mesh filename=package://tmc_hsrb_description/meshes/hand_v0/right_distal.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
- link hsrb/right_proximal_link: geometry collision mesh filename=package://tmc_hsrb_description/meshes/hand_v0/right_proxima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; visual mesh filename=package://tmc_hsrb_description/meshes/hand_v0/right_proxima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
- link hsrb/torso_lift_link: geometry collision mesh filename=package://tmc_hsrb_description/meshes/torso_v0/torso.stl; visual mesh filename=package://tmc_hsrb_description/meshes/torso_v0/torso.dae
- link hsrb/wrist_flex_link: geometry collision cylinder length=0.04 radius=0.017; visual cylinder length=0.02 radius=0.017
- link hsrb/wrist_roll_link: geometry collision mesh filename=package://tmc_hsrb_description/meshes/wrist_v0/wrist_roll.s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; visual mesh filename=package://tmc_hsrb_description/meshes/wrist_v0/wrist_roll.d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

Commit message: Update model parameters to make odom_base_trajectory_controllr work.

File: tmc_hsrb_description/robots/hsrb.urdf (robot description, URDF)
Before this commit: robot hsrb, 36 links, 35 joints
Links:
- link hsrb/left_drive_wheel_link: mass 1 -> 0.1
- link hsrb/right_drive_wheel_link: mass 1 -> 0.1
Joints:
- joint hsrb/base_roll_joint: limit effort=100.0 velocity=1.0 -> effort=1000.0 velocity=1.0
- joint hsrb/left_drive_wheel_joint: limit effort=100.0 velocity=10.0 -> effort=1000.0 velocity=10.0
- joint hsrb/right_drive_wheel_joint: limit effort=100.0 velocity=10.0 -> effort=1000.0 velocity=10.0

File: tmc_hsrb_description/robots/hsrb_sim.urdf.xacro (robot description, xacro)
@@ -35,7 +35,6 @@
     </xacro:hsrb_hand_base>
     <gazebo>
-        <plugin name="gazebo_ros_control" filename="libgazebo_ros_control.so">
+        <plugin name="hsrb_ros_control" filename="libgazebo_ros_control.so">
             <robotNamespace>${robot_name}</robotNamespace>
-            <robotSimType>gazebo_ros_control/DefaultRobotHWSim</robotSimType>
         </plugin>
     </gazebo>

File: tmc_hsrb_description/urdf/arm_v0/arm.transmission.xacro (robot description, xacro)
@@ -1,5 +1,5 @@
 <?xml version="1.0"?>
 <robot xmlns:xacro="http://ros.org/wiki/xacro">
-    <xacro:macro naem="hsrb_arm_transmission" params="robot_name">
+    <xacro:macro name="hsrb_arm_transmission" params="robot_name">
         <hsrb_trans joint="${robot_name}/arm_lift_joint" reduction="1"/>
         <hsrb_trans joint="${robot_name}/arm_flex_joint" reduction="1"/>

File: tmc_hsrb_description/urdf/base_v0/base.transmission.xacro (robot description, xacro)
@@ -2,7 +2,33 @@
 <robot xmlns:xacro="http://ros.org/wiki/xacro">
     <xacro:macro name="hsrb_base_transmission" params="robot_name">
+        <!--
         <hsrb_trans joint="${robot_name}/base_roll_joint" reduction="1"/>
         <hsrb_trans joint="${robot_name}/left_drive_wheel_joint" reduction="1"/>
         <hsrb_trans joint="${robot_name}/right_drive_wheel_joint" reduction="1"/>
+        -->
+        <transmission name="${robot_name}/base_roll_joint_trans">
+            <type>transmission_interface/SimpleTransmission</type>
+            <joint name="${robot_name}/base_roll_joint"/>
+            <actuator name="${robot_name}/base_roll_joint_motor">
+                <hardwareInterface>VelocityJointInterface</hardwareInterface>
+                <mechanicalReduction>1</mechanicalReduction>
+            </actuator>
+        </transmission>
+        <transmission name="${robot_name}/left_drive_wheel_joint_trans">
+            <type>transmission_interface/SimpleTransmission</type>
+            <joint name="${robot_name}/left_drive_wheel_joint"/>
+            <actuator name="${robot_name}/left_drive_wheel_joint_motor">
+                <hardwareInterface>VelocityJointInterface</hardwareInterface>
+                <mechanicalReduction>1</mechanicalReduction>
+            </actuator>
+        </transmission>
+        <transmission name="${robot_name}/right_drive_wheel_joint_trans">
+            <type>transmission_interface/SimpleTransmission</type>
+            <joint name="${robot_name}/right_drive_wheel_joint"/>
+            <actuator name="${robot_name}/right_drive_wheel_joint_motor">
+                <hardwareInterface>VelocityJointInterface</hardwareInterface>
+                <mechanicalReduction>1</mechanicalReduction>
+            </actuator>
+        </transmission>
     </xacro:macro>
 </robot>

File: tmc_hsrb_description/urdf/base_v0/base.urdf.xacro (robot description, xacro)
@@ -18,5 +18,5 @@
             <insert_block name="origin" />
             <axis xyz="0.0 1.0 0.0" />
-            <limit effort="100.0" velocity="10.0" />
+            <limit effort="1000.0" velocity="10.0" />
             <parent link="${parent}" />
             <child link="${prefix}_drive_wheel_link" />
@@ -38,7 +38,7 @@
             </collision>
             <inertial>
-                <mass value="1"/>
+                <mass value="0.1"/>
                 <origin xyz="0 0 0"/>
-                <inertia ixx="1" ixy="0" ixz="0" iyy="1" iyz="0" izz="1"/>
+                <inertia ixx="0.001" ixy="0" ixz="0" iyy="0.001" iyz="0" izz="0.001"/>
             </inertial>
         </link>
@@ -57,5 +57,5 @@
                 <mass value="0.3"/>
                 <origin xyz="0 0 0"/>
-                <inertia ixx="1" ixy="0" ixz="0" iyy="1" iyz="0" izz="1"/>
+                <inertia ixx="0.001" ixy="0" ixz="0" iyy="0.001" iyz="0" izz="0.001"/>
             </inertial>
         </link>
@@ -70,5 +70,5 @@
                 <mass value="0.3"/>
                 <origin xyz="0 0 0"/>
-                <inertia ixx="1" ixy="0" ixz="0" iyy="1" iyz="0" izz="1"/>
+                <inertia ixx="0.001" ixy="0" ixz="0" iyy="0.001" iyz="0" izz="0.001"/>
             </inertial>
         </link>
@@ -95,5 +95,5 @@
                 <mass value="0.3"/>
                 <origin xyz="0 0 0"/>
-                <inertia ixx="1" ixy="0" ixz="0" iyy="1" iyz="0" izz="1"/>
+                <inertia ixx="0.001" ixy="0" ixz="0" iyy="0.001" iyz="0" izz="0.001"/>
             </inertial>
         </link>
@@ -142,8 +142,7 @@
             <origin xyz="0.0 0.0 0.0" rpy="0.0 0.0 0.0" />
             <axis xyz="0.0 0.0 1.0" />
-            <limit effort="100.0" velocity="1.0" />
+            <limit effort="1000.0" velocity="1.0" />
             <parent link="${name}_body_link" />
             <child link="${name}_roll_link" />
-            <limit effort="1.0" velocity="1.0"/>
         </joint>
         <link name="${name}_roll_link">

File: tmc_hsrb_description/urdf/common.xacro (robot description, xacro)
@@ -24,11 +24,13 @@
       <selfCollide>false</selfCollide>
       <gravity>true</gravity>
+      <turnGravityOff>false</turnGravityOff>
       <kp>1000000.0</kp>
-      <kd>100.0</kd>
-      <mu1>1.5</mu1>
-      <mu2>1.5</mu2>
+      <kd>10.0</kd>
+      <mu1>1.0</mu1>
+      <mu2>1.0</mu2>
       <fdir1>1 0 0</fdir1>
       <maxVel>1.0</maxVel>
       <minDepth>0.00</minDepth>
+      <material value="Gazebo/Black"/>
     </gazebo>
   </macro>
