Commit message: Add missing robot namspace to some sensors.

File: tmc_hsrb_description/robots/hsrb1s.urdf.xacro (robot description, xacro)
@@ -16,22 +16,33 @@
     <xacro:include filename="$(find tmc_hsrb_description)/urdf/hand_v0/hand.urdf.xacro" />
     <!-- constant -->
-    <!-- constant -->
     <xacro:property name="robot_name" value= "hsrb"/>
     <!-- create robot -->
-    <xacro:hsrb_base name="${robot_name}/base" />
-    <xacro:hsrb_torso name="${robot_name}/torso" parent="${robot_name}/base_body_link" robot="${robot_name}">
+    <xacro:hsrb_base prefix="base" robot_namespace="${robot_name}"/>
+    <xacro:hsrb_torso prefix="torso" parent="base_body_link" mimic_joint="arm_lift_joint">
         <origin xyz="0.0 0.0 0.752" rpy="0.0 0.0 0.0"/>
     </xacro:hsrb_torso>
-    <xacro:hsrb_head name="${robot_name}/head" parent="${robot_name}/torso_lift_link">
+    <xacro:hsrb_head prefix="head" parent="torso_lift_link">
         <origin xyz="0.0 0.0 0.0" rpy="0.0 0.0 0.0"/>
     </xacro:hsrb_head>
-    <xacro:hsrb_arm name="${robot_name}/arm" parent="${robot_name}/base_body_link">
+    <xacro:hsrb_arm prefix="arm" parent="base_body_link">
         <origin xyz="0.0 0.0 0.340" rpy="0.0 0.0 0.0"/>
     </xacro:hsrb_arm>
-    <xacro:hsrb_wrist name="${robot_name}/wrist" parent="${robot_name}/arm_roll_link">
+    <xacro:hsrb_wrist prefix="wrist" parent="arm_roll_link" robot_namespace="${robot_name}">
         <origin xyz="0.0 0.0 0.0" rpy="0.0 0.0 0.0"/>
     </xacro:hsrb_wrist>
-    <xacro:hsrb_hand_base name="${robot_name}/hand" parent="${robot_name}/wrist_roll_link">
+    <xacro:hsrb_hand prefix="hand" parent="wrist_roll_link">
         <origin xyz="0.012 0.0 0.1405" rpy="0.0 0.0 ${pi}"/>
-    </xacro:hsrb_hand_base>
+    </xacro:hsrb_hand>
+    <gazebo>
+        <plugin name="${robot_name}_ros_control" filename="libgazebo_ros_control.so">
+            <robotNamespace>${robot_name}</robotNamespace>
+        </plugin>
+        <plugin name="${robot_name}_p3d_ground_truth" filename="libgazebo_ros_p3d.so">
+            <robotNamespace>${robot_name}</robotNamespace>
+            <bodyName>base_footprint</bodyName>
+            <topicName>odom_ground_truth</topicName>
+            <frameName>map</frameName>
+            <updateRate>30</updateRate>
+        </plugin>
+    </gazebo>
 </robot>

File: tmc_hsrb_description/robots/hsrb1s_sim.urdf.xacro (robot description, xacro)
@@ -16,8 +16,8 @@
     <xacro:include filename="$(find tmc_hsrb_description)/urdf/hand_v0/hand.urdf.xacro" />
     <!-- constant -->
-    <xacro:property name="robot_name" value= "hsrb"/>
+    <xacro:property name="robot_name" value="hsrb"/>
     <!-- create robot -->
-    <xacro:hsrb_base prefix="base" />
-    <xacro:hsrb_torso prefix="torso" parent="base_body_link" mimic="arm_lift_joint">
+    <xacro:hsrb_base prefix="base" robot_namespace="${robot_name}"/>
+    <xacro:hsrb_torso prefix="torso" parent="base_body_link" mimic_joint="arm_lift_joint">
         <origin xyz="0.0 0.0 0.752" rpy="0.0 0.0 0.0"/>
     </xacro:hsrb_torso>
@@ -28,5 +28,5 @@
         <origin xyz="0.0 0.0 0.340" rpy="0.0 0.0 0.0"/>
     </xacro:hsrb_arm>
-    <xacro:hsrb_wrist prefix="wrist" parent="arm_roll_link">
+    <xacro:hsrb_wrist prefix="wrist" parent="arm_roll_link" robot_namespace="${robot_name}">
         <origin xyz="0.0 0.0 0.0" rpy="0.0 0.0 0.0"/>
     </xacro:hsrb_wrist>

File: tmc_hsrb_description/urdf/base_v0/base.urdf.xacro (robot description, xacro)
@@ -100,5 +100,5 @@
     </xacro:macro>
     <!-- base -->
-    <xacro:macro name="hsrb_base" params="prefix">
+    <xacro:macro name="hsrb_base" params="prefix robot_namespace">
         <link name="base_footprint"/>
         <joint name="${prefix}_joint" type="fixed">
@@ -185,8 +185,8 @@
         </xacro:hsrb_passive_wheel>
         <!-- sensors -->
-        <xacro:hokuyo_laser prefix="${prefix}" parent="${prefix}_link">
+        <xacro:hokuyo_laser prefix="${prefix}" robot_namespace="${robot_namespace}" parent="${prefix}_link">
             <origin xyz="0.1375 0.0 0.1895" rpy="0.0 0.0 0.0" />
         </xacro:hokuyo_laser>
-        <xacro:imu_sensor prefix="${prefix}" parent="${prefix}_link">
+        <xacro:imu_sensor prefix="${prefix}" robot_namespace="${robot_namespace}" parent="${prefix}_link">
             <origin xyz="0.0005 0.1296 0.181" rpy="${pi} 0.0 0.0" />
         </xacro:imu_sensor>

File: tmc_hsrb_description/urdf/sensors/hokuyo_laser.gazebo.xacro (robot description, xacro)
@@ -1,5 +1,5 @@
 <?xml version="1.0" ?>
 <robot name="hsrb" xmlns:xacro="http://www.ros.org/wiki/xacro">
-    <xacro:macro name="hokuyo_laser_gazebo" params="sensor_name ros_topic frame_name min_angle max_angle">
+    <xacro:macro name="hokuyo_laser_gazebo" params="sensor_name robot_namespace ros_topic frame_name min_angle max_angle">
         <gazebo reference="${frame_name}">
             <sensor type="ray" name="${sensor_name}">
@@ -23,5 +23,5 @@
                 </ray>
                 <plugin name="hokuyo_laser" filename="libgazebo_ros_laser.so">
-                    <robotNamespace>${robot_name}</robotNamespace>
+                    <robotNamespace>${robot_namespace}</robotNamespace>
                     <topicName>${ros_topic}</topicName>
                     <frameName>${frame_name}</frameName>

File: tmc_hsrb_description/urdf/sensors/hokuyo_laser.urdf.xacro (robot description, xacro)
@@ -2,5 +2,5 @@
     <xacro:include filename="$(find tmc_hsrb_description)/urdf/sensors/hokuyo_laser.gazebo.xacro"/>
     <!-- range sensor -->
-    <xacro:macro name="hokuyo_laser" params="prefix parent *origin">
+    <xacro:macro name="hokuyo_laser" params="prefix robot_namespace parent *origin">
         <joint name="${prefix}_laser_joint" type="fixed">
             <insert_block name="origin" />
@@ -24,4 +24,5 @@
         <xacro:hokuyo_laser_gazebo
             sensor_name="${prefix}_laser"
+            robot_namespace="${robot_namespace}"
             ros_topic="${prefix}_scan"
             frame_name="${prefix}_laser_link"

File: tmc_hsrb_description/urdf/sensors/imu.gazebo.xacro (robot description, xacro)
@@ -1,5 +1,5 @@
 <?xml version="1.0" ?>
 <robot name="hsrb" xmlns:xacro="http://www.ros.org/wiki/xacro">
-    <xacro:macro name="imu_gazebo" params="sensor_name frame_name">
+    <xacro:macro name="imu_gazebo" params="sensor_name frame_name robot_namespace">
         <gazebo reference="${frame_name}">
             <sensor type="imu" name="${sensor_name}">
@@ -30,4 +30,5 @@
                 <frameName>${frame_name}</frameName>
                 <bodyName>base_link</bodyName>
+                <robotNamespace>${robot_namespace}</robotNamespace>
             </plugin>
         </gazebo>

File: tmc_hsrb_description/urdf/sensors/imu.urdf.xacro (robot description, xacro)
@@ -3,5 +3,5 @@
     <xacro:include filename="$(find tmc_hsrb_description)/urdf/sensors/imu.gazebo.xacro"/>
     <!-- imu sensor -->
-    <xacro:macro name="imu_sensor" params="prefix parent *origin">
+    <xacro:macro name="imu_sensor" params="prefix parent robot_namespace *origin">
         <joint name="${prefix}_imu_joint" type="fixed">
             <insert_block name="origin" />
@@ -10,5 +10,5 @@
         </joint>
         <link name="${prefix}_imu_link"/>
-        <xacro:imu_gazebo sensor_name="${prefix}_imu" frame_name="${prefix}_imu_link"/>
+        <xacro:imu_gazebo sensor_name="${prefix}_imu" robot_namespace="${robot_namespace}" frame_name="${prefix}_imu_link"/>
     </xacro:macro>
 </robot>

File: tmc_hsrb_description/urdf/sensors/minebea_ft_sensor.gazebo.xacro (robot description, xacro)
@@ -1,5 +1,5 @@
 <?xml version="1.0" ?>
 <robot name="hsrb" xmlns:xacro="http://www.ros.org/wiki/xacro">
-    <xacro:macro name="minebea_ft_sensor_gazebo" params="sensor_name joint_name ros_topic">
+    <xacro:macro name="minebea_ft_sensor_gazebo" params="sensor_name robot_namespace joint_name ros_topic">
         <gazebo reference="${joint_name}">
             <provideFeedback>true</provideFeedback>
@@ -11,4 +11,5 @@
                 <jointName>${joint_name}</jointName>
                 <bodyName>wrist_roll_link</bodyName>
+                <robotNamespace>${robot_namespace}</robotNamespace>
             </plugin>
         </gazebo>

File: tmc_hsrb_description/urdf/sensors/minebea_ft_sensor.urdf.xacro (robot description, xacro)
@@ -2,5 +2,5 @@
 <robot name="hsrb" xmlns:xacro="http://www.ros.org/wiki/xacro">
     <xacro:include filename="$(find tmc_hsrb_description)/urdf/sensors/minebea_ft_sensor.gazebo.xacro"/>
-    <xacro:macro name="minebea_ft_sensor" params="prefix parent joint_name *origin">
+    <xacro:macro name="minebea_ft_sensor" params="prefix robot_namespace parent joint_name *origin">
         <joint name="${prefix}_ft_sensor_joint" type="fixed">
             <insert_block name="origin"/>
@@ -9,5 +9,5 @@
         </joint>
         <link name="${prefix}_ft_sensor_frame"/>
-        <xacro:minebea_ft_sensor_gazebo sensor_name="${prefix}_ft_sensor" joint_name="${joint_name}" ros_topic="${prefix}_wrench" />
+        <xacro:minebea_ft_sensor_gazebo sensor_name="${prefix}_ft_sensor" robot_namespace="${robot_namespace}" joint_name="${joint_name}" ros_topic="${prefix}_wrench" />
     </xacro:macro>
 </robot>

File: tmc_hsrb_description/urdf/torso_v0/torso.gazebo.xacro (robot description, xacro)
@@ -1,5 +1,5 @@
 <?xml version="1.0"?>
 <robot xmlns:xacro="http://ros.org/wiki/xacro">
-    <xacro:macro name="hsrb_torso_gazebo" params="prefix">
+    <xacro:macro name="hsrb_torso_gazebo" params="prefix mimic_joint">
         <gazebo_link name="${prefix}_lift_link" gravity="true" collide="false" friction="0.9"/>
         <gazebo_joint name="${prefix}_lift_joint"/>
@@ -7,5 +7,5 @@
             <plugin name="torso_mimic_plugin" filename="libtmc_gazebo_mimic_plugin.so">
                 <joint>${prefix}_lift_joint</joint>
-                <mimicJoint>${prefix}_lift_joint</mimicJoint>
+                <mimicJoint>${mimic_joint}</mimicJoint>
                 <multiplier>0.5</multiplier>
                 <p>900.0</p>

File: tmc_hsrb_description/urdf/torso_v0/torso.urdf.xacro (robot description, xacro)
@@ -4,5 +4,5 @@
     <xacro:include filename="$(find tmc_hsrb_description)/urdf/torso_v0/torso.gazebo.xacro"/>
     <!-- torso -->
-    <xacro:macro name="hsrb_torso" params="prefix parent mimic *origin">
+    <xacro:macro name="hsrb_torso" params="prefix parent mimic_joint *origin">
         <joint name="${prefix}_lift_joint" type="prismatic">
             <insert_block name="origin" />
@@ -12,5 +12,5 @@
             <parent link="${parent}" />
             <child link="${prefix}_lift_link" />
-            <mimic joint="${mimic}" multiplier="0.5" />
+            <mimic joint="${mimic_joint}" multiplier="0.5" />
         </joint>
         <link name="${prefix}_lift_link">
@@ -34,5 +34,5 @@
             </collision>
         </link>
-        <xacro:hsrb_torso_gazebo prefix="${prefix}"/>
+        <xacro:hsrb_torso_gazebo prefix="${prefix}" mimic_joint="${mimic_joint}"/>
         <xacro:hsrb_torso_transmission prefix="${prefix}"/>
     </xacro:macro>

File: tmc_hsrb_description/urdf/wrist_v0/wrist.urdf.xacro (robot description, xacro)
@@ -5,5 +5,5 @@
     <xacro:include filename="$(find tmc_hsrb_description)/urdf/sensors/minebea_ft_sensor.urdf.xacro"/>
     <!-- wrist -->
-    <xacro:macro name="hsrb_wrist" params="prefix parent *origin">
+    <xacro:macro name="hsrb_wrist" params="prefix robot_namespace parent *origin">
         <joint name="${prefix}_flex_joint" type="revolute">
             <origin xyz="0.0 0.0 0.0" rpy="0.0 0.0 0.0" />
@@ -68,5 +68,5 @@
             </collision>
         </link>
-        <xacro:minebea_ft_sensor prefix="${prefix}" parent="${prefix}_roll_link" joint_name="${prefix}_roll_joint">
+        <xacro:minebea_ft_sensor prefix="${prefix}" robot_namespace="${robot_namespace}" parent="${prefix}_roll_link" joint_name="${prefix}_roll_joint">
             <origin xyz="0.0 0.0 0.0735" rpy="${pi} 0.0 0.0"/>
         </xacro:minebea_ft_sensor>

Commit message: Unify hsrb1s_sim and hsrb1s to hsrb1s. Rewrite URDF generation command.

File: tmc_hsrb_description/robots/hsrb1s.urdf.xacro (robot description, xacro)
@@ -16,5 +16,5 @@
     <xacro:include filename="$(find tmc_hsrb_description)/urdf/hand_v0/hand.urdf.xacro" />
     <!-- constant -->
-    <xacro:property name="robot_name" value= "hsrb"/>
+    <xacro:property name="robot_name" value="hsrb"/>
     <!-- create robot -->
     <xacro:hsrb_base prefix="base" robot_namespace="${robot_name}"/>
