Commit message: Rearrange frame/joint/link structure

File: tmc_hsrb_description/robots/hsrb1s.urdf.xacro (robot description, xacro)
@@ -19,5 +19,5 @@
     <!-- create robot -->
     <xacro:hsrb_base prefix="base" robot_namespace="${robot_name}"/>
-    <xacro:hsrb_torso prefix="torso" parent="base_body_link" mimic_joint="arm_lift_joint">
+    <xacro:hsrb_torso prefix="torso" parent="base_link" mimic_joint="arm_lift_joint">
         <origin xyz="0.0 0.0 0.752" rpy="0.0 0.0 0.0"/>
     </xacro:hsrb_torso>
@@ -25,5 +25,5 @@
         <origin xyz="0.0 0.0 0.0" rpy="0.0 0.0 0.0"/>
     </xacro:hsrb_head>
-    <xacro:hsrb_arm prefix="arm" parent="base_body_link">
+    <xacro:hsrb_arm prefix="arm" parent="base_link">
         <origin xyz="0.0 0.0 0.340" rpy="0.0 0.0 0.0"/>
     </xacro:hsrb_arm>

File: tmc_hsrb_description/robots/hsrb2s.urdf.xacro (robot description, xacro)
@@ -19,5 +19,5 @@
     <!-- create robot -->
     <xacro:hsrb_base prefix="base" robot_namespace="${robot_name}"/>
-    <xacro:hsrb_torso prefix="torso" parent="base_body_link" mimic_joint="arm_lift_joint">
+    <xacro:hsrb_torso prefix="torso" parent="base_link" mimic_joint="arm_lift_joint">
         <origin xyz="0.0 0.0 0.752" rpy="0.0 0.0 0.0"/>
     </xacro:hsrb_torso>
@@ -25,5 +25,5 @@
         <origin xyz="0.0 0.0 0.0" rpy="0.0 0.0 0.0"/>
     </xacro:hsrb_head>
-    <xacro:hsrb_arm prefix="arm" parent="base_body_link">
+    <xacro:hsrb_arm prefix="arm" parent="base_link">
         <origin xyz="0.0 0.0 0.340" rpy="0.0 0.0 0.0"/>
     </xacro:hsrb_arm>

File: tmc_hsrb_description/urdf/base_v0/base.gazebo.xacro (robot description, xacro)
@@ -3,10 +3,9 @@
     <xacro:macro name="hsrb_base_gazebo" params="prefix">
         <gazebo_link name="${prefix}_link" gravity="true" collide="false" friction="0.9"/>
-        <gazebo_link name="${prefix}_body_link" gravity="true" collide="false" friction="0.9"/>
         <gazebo_link name="${prefix}_roll_link" gravity="true" collide="false" friction="0.9"/>
-        <gazebo_link_rubber name="${prefix}_right_drive_wheel_link"/>
-        <gazebo_link_rubber name="${prefix}_left_drive_wheel_link"/>
-        <gazebo_link_rubber name="${prefix}_right_passive_wheel_z_link"/>
-        <gazebo_link_rubber name="${prefix}_left_passive_wheel_z_link"/>
+        <gazebo_link_rubber name="${prefix}_r_drive_wheel_link"/>
+        <gazebo_link_rubber name="${prefix}_l_drive_wheel_link"/>
+        <gazebo_link_rubber name="${prefix}_r_passive_wheel_z_link"/>
+        <gazebo_link_rubber name="${prefix}_l_passive_wheel_z_link"/>
         <gazebo_link name="${prefix}_range_sensor_link" gravity="true" collide="false" friction="0.9"/>
         <gazebo_link name="${prefix}_imu_sensor_link" gravity="true" collide="false" friction="0.9"/>

File: tmc_hsrb_description/urdf/base_v0/base.transmission.xacro (robot description, xacro)
@@ -2,6 +2,6 @@
 <robot xmlns:xacro="http://ros.org/wiki/xacro">
     <xacro:macro name="hsrb_base_transmission" params="prefix">
-        <hsrb_velocity_joint_transmission joint="${prefix}_right_drive_wheel_joint" reduction="1"/>
-        <hsrb_velocity_joint_transmission joint="${prefix}_left_drive_wheel_joint" reduction="1"/>
+        <hsrb_velocity_joint_transmission joint="${prefix}_r_drive_wheel_joint" reduction="1"/>
+        <hsrb_velocity_joint_transmission joint="${prefix}_l_drive_wheel_joint" reduction="1"/>
         <hsrb_velocity_joint_transmission joint="${prefix}_roll_joint" reduction="1"/>
     </xacro:macro>

File: tmc_hsrb_description/urdf/base_v0/base.urdf.xacro (robot description, xacro)
@@ -109,4 +109,10 @@
         </joint>
         <link name="${prefix}_link">
+            <inertial>
+                <mass value="11.017971"/>
+                <origin xyz="-0.025978 -0.005498 0.17633"/>
+                <inertia ixx="0.3742" ixy="0.000434172172" ixz="0.03088"
+                    iyy="0.3436" iyz="0.01775" izz="0.1509"/>
+            </inertial>
             <visual>
                 <geometry>
@@ -134,21 +140,9 @@
             </collision>
         </link>
-        <joint name="${prefix}_body_joint" type="fixed">
-            <parent link="${prefix}_link" />
-            <child link="${prefix}_body_link" />
-        </joint>
-        <link name="${prefix}_body_link">
-            <inertial>
-                <mass value="11.017971"/>
-                <origin xyz="-0.025978 -0.005498 0.17633"/>
-                <inertia ixx="0.3742" ixy="0.000434172172" ixz="0.03088"
-                    iyy="0.3436" iyz="0.01775" izz="0.1509"/>
-            </inertial>
-        </link>
         <joint name="${prefix}_roll_joint" type="continuous">
             <origin xyz="0.0 0.0 0.0" rpy="0.0 0.0 0.0" />
             <axis xyz="0.0 0.0 1.0" />
             <limit effort="1000.0" velocity="1.0" />
-            <parent link="${prefix}_body_link" />
+            <parent link="${prefix}_link" />
             <child link="${prefix}_roll_link" />
             <dynamics damping="0.7"/>
@@ -163,5 +157,5 @@
         </link>
         <!-- wheels -->
-        <xacro:hsrb_drive_wheel prefix="${prefix}" suffix="right" parent="${prefix}_roll_link">
+        <xacro:hsrb_drive_wheel prefix="${prefix}" suffix="r" parent="${prefix}_roll_link">
             <origin xyz="${drive_wheel_offset_x}
                 ${-drive_wheel_offset_y}
@@ -169,5 +163,5 @@
                 rpy="0.0 0.0 0.0" />
         </xacro:hsrb_drive_wheel>
-        <xacro:hsrb_drive_wheel prefix="${prefix}" suffix="left" parent="${prefix}_roll_link">
+        <xacro:hsrb_drive_wheel prefix="${prefix}" suffix="l" parent="${prefix}_roll_link">
             <origin xyz="${drive_wheel_offset_x}
                 ${drive_wheel_offset_y}
@@ -175,5 +169,5 @@
                 rpy="0.0 0.0 0.0" />
         </xacro:hsrb_drive_wheel>
-        <xacro:hsrb_passive_wheel prefix="${prefix}" suffix="right" parent="${prefix}_roll_link">
+        <xacro:hsrb_passive_wheel prefix="${prefix}" suffix="r" parent="${prefix}_roll_link">
             <origin xyz="${passive_wheel_offset_x}
                 ${-passive_wheel_offset_y}
@@ -181,5 +175,5 @@
                 rpy="0.0 0.0 0.0" />
         </xacro:hsrb_passive_wheel>
-        <xacro:hsrb_passive_wheel prefix="${prefix}" suffix="left" parent="${prefix}_roll_link">
+        <xacro:hsrb_passive_wheel prefix="${prefix}" suffix="l" parent="${prefix}_roll_link">
             <origin xyz="${passive_wheel_offset_x}
                 ${passive_wheel_offset_y}

File: tmc_hsrb_description/urdf/base_v1/base.urdf.xacro (robot description, xacro)
@@ -109,4 +109,10 @@
         </joint>
         <link name="${prefix}_link">
+            <inertial>
+                <mass value="11.017971"/>
+                <origin xyz="-0.025978 -0.005498 0.17633"/>
+                <inertia ixx="0.3742" ixy="0.000434172172" ixz="0.03088"
+                    iyy="0.3436" iyz="0.01775" izz="0.1509"/>
+            </inertial>
             <visual>
                 <geometry>
@@ -133,21 +139,9 @@
             </collision>
         </link>
-        <joint name="${prefix}_body_joint" type="fixed">
-            <parent link="${prefix}_link" />
-            <child link="${prefix}_body_link" />
-        </joint>
-        <link name="${prefix}_body_link">
-            <inertial>
-                <mass value="11.017971"/>
-                <origin xyz="-0.025978 -0.005498 0.17633"/>
-                <inertia ixx="0.3742" ixy="0.000434172172" ixz="0.03088"
-                    iyy="0.3436" iyz="0.01775" izz="0.1509"/>
-            </inertial>
-        </link>
         <joint name="${prefix}_roll_joint" type="continuous">
             <origin xyz="0.0 0.0 0.0" rpy="0.0 0.0 0.0" />
             <axis xyz="0.0 0.0 1.0" />
             <limit effort="1000.0" velocity="1.0" />
-            <parent link="${prefix}_body_link" />
+            <parent link="${prefix}_link" />
             <child link="${prefix}_roll_link" />
             <dynamics damping="0.7"/>
@@ -163,15 +157,15 @@
         </link>
         <!-- wheels -->
-        <xacro:hsrb_drive_wheel prefix="${prefix}" suffix="right" parent="${prefix}_roll_link">
+        <xacro:hsrb_drive_wheel prefix="${prefix}" suffix="r" parent="${prefix}_roll_link">
             <origin
                 xyz="${-drive_wheel_offset_x} ${-drive_wheel_offset_y} ${drive_wheel_radius}"
                 rpy="0.0 0.0 0.0" />
         </xacro:hsrb_drive_wheel>
-        <xacro:hsrb_drive_wheel prefix="${prefix}" suffix="left" parent="${prefix}_roll_link">
+        <xacro:hsrb_drive_wheel prefix="${prefix}" suffix="l" parent="${prefix}_roll_link">
             <origin
                 xyz="${-drive_wheel_offset_x} ${drive_wheel_offset_y} ${drive_wheel_radius}"
                 rpy="0.0 0.0 0.0" />
         </xacro:hsrb_drive_wheel>
-        <xacro:hsrb_passive_wheel prefix="${prefix}" suffix="right" parent="${prefix}_roll_link">
+        <xacro:hsrb_passive_wheel prefix="${prefix}" suffix="r" parent="${prefix}_roll_link">
             <origin xyz="${passive_wheel_offset_x}
                 ${-passive_wheel_offset_y}
@@ -179,5 +173,5 @@
                 rpy="0.0 0.0 0.0" />
         </xacro:hsrb_passive_wheel>
-        <xacro:hsrb_passive_wheel prefix="${prefix}" suffix="left" parent="${prefix}_roll_link">
+        <xacro:hsrb_passive_wheel prefix="${prefix}" suffix="l" parent="${prefix}_roll_link">
             <origin xyz="${passive_wheel_offset_x}
                 ${passive_wheel_offset_y}

File: tmc_hsrb_description/urdf/hand_v0/hand.gazebo.xacro (robot description, xacro)
@@ -4,26 +4,26 @@
         <gazebo_link name="${prefix}_palm_link" gravity="true" collide="false" friction="0.9"/>
         <gazebo_link name="${prefix}_camera_link" gravity="true" collide="false" friction="0.9"/>
-        <gazebo_link name="${prefix}_left_actuated_proximal_link" gravity="true" collide="false" friction="1.0"/>
-        <gazebo_link name="${prefix}_left_spring_proximal_link" gravity="true" collide="false" friction="1.0"/>
-        <gazebo_link name="${prefix}_left_mimic_link" gravity="true" collide="false" friction="1.0"/>
-        <gazebo_link name="${prefix}_left_distal_link" gravity="true" collide="false" friction="1.0"/>
-        <gazebo_link name="${prefix}_left_finger_tip_frame" gravity="true" collide="false" friction="1.0"/>
-        <gazebo_link name="${prefix}_left_finger_vacuum_frame" gravity="true" collide="false" friction="1.0"/>
-        <gazebo_link name="${prefix}_right_actuated_proximal_link" gravity="true" collide="false" friction="1.0"/>
-        <gazebo_link name="${prefix}_right_spring_proximal_link" gravity="true" collide="false" friction="1.0"/>
-        <gazebo_link name="${prefix}_right_mimic_link" gravity="true" collide="false" friction="1.0"/>
-        <gazebo_link name="${prefix}_right_distal_link" gravity="true" collide="false" friction="1.0"/>
-        <gazebo_link name="${prefix}_right_finger_tip_frame" gravity="true" collide="false" friction="1.0"/>
-        <gazebo_link name="${prefix}_right_finger_vacuum_frame" gravity="true" collide="false" friction="1.0"/>
+        <gazebo_link name="${prefix}_l_actuated_proximal_link" gravity="true" collide="false" friction="1.0"/>
+        <gazebo_link name="${prefix}_l_spring_proximal_link" gravity="true" collide="false" friction="1.0"/>
+        <gazebo_link name="${prefix}_l_mimic_link" gravity="true" collide="false" friction="1.0"/>
+        <gazebo_link name="${prefix}_l_distal_link" gravity="true" collide="false" friction="1.0"/>
+        <gazebo_link name="${prefix}_l_finger_tip_frame" gravity="true" collide="false" friction="1.0"/>
+        <gazebo_link name="${prefix}_l_finger_vacuum_frame" gravity="true" collide="false" friction="1.0"/>
+        <gazebo_link name="${prefix}_r_actuated_proximal_link" gravity="true" collide="false" friction="1.0"/>
+        <gazebo_link name="${prefix}_r_spring_proximal_link" gravity="true" collide="false" friction="1.0"/>
+        <gazebo_link name="${prefix}_r_mimic_link" gravity="true" collide="false" friction="1.0"/>
+        <gazebo_link name="${prefix}_r_distal_link" gravity="true" collide="false" friction="1.0"/>
+        <gazebo_link name="${prefix}_r_finger_tip_frame" gravity="true" collide="false" friction="1.0"/>
+        <gazebo_link name="${prefix}_r_finger_vacuum_frame" gravity="true" collide="false" friction="1.0"/>
         <gazebo_joint name="${prefix}_palm_joint"/>
         <gazebo_joint name="${prefix}_motor_joint"/>
-        <gazebo_joint name="${prefix}_left_actuated_proximal_joint"/>
-        <gazebo_joint name="${prefix}_left_spring_proximal_joint"/>
-        <gazebo_joint name="${prefix}_left_mimic_distal_joint"/>
-        <gazebo_joint name="${prefix}_left_distal_joint"/>
-        <gazebo_joint name="${prefix}_right_actuated_proximal_joint"/>
-        <gazebo_joint name="${prefix}_right_spring_proximal_joint"/>
-        <gazebo_joint name="${prefix}_right_mimic_distal_joint"/>
-        <gazebo_joint name="${prefix}_right_distal_joint"/>
+        <gazebo_joint name="${prefix}_l_actuated_proximal_joint"/>
+        <gazebo_joint name="${prefix}_l_spring_proximal_joint"/>
+        <gazebo_joint name="${prefix}_l_mimic_distal_joint"/>
+        <gazebo_joint name="${prefix}_l_distal_joint"/>
+        <gazebo_joint name="${prefix}_r_actuated_proximal_joint"/>
+        <gazebo_joint name="${prefix}_r_spring_proximal_joint"/>
+        <gazebo_joint name="${prefix}_r_mimic_distal_joint"/>
+        <gazebo_joint name="${prefix}_r_distal_joint"/>
         <gazebo>
             <plugin name="hsrb_hrh_gripper_plugin" filename="libtmc_gazebo_hrh_gripper.so">
@@ -35,8 +35,8 @@
                     <min_contact_count>1</min_contact_count>
                 </grasp_check>
-                <gripper_link>${prefix}_right_distal_link</gripper_link>
-                <gripper_link>${prefix}_left_distal_link</gripper_link>
-                <gripper_link>${prefix}_right_spring_proximal_link</gripper_link>
-                <gripper_link>${prefix}_left_spring_proximal_link</gripper_link>
+                <gripper_link>${prefix}_r_distal_link</gripper_link>
+                <gripper_link>${prefix}_l_distal_link</gripper_link>
+                <gripper_link>${prefix}_r_spring_proximal_link</gripper_link>
+                <gripper_link>${prefix}_l_spring_proximal_link</gripper_link>
                 <palm_link>${prefix}_palm_link</palm_link>
             </gripper>

File: tmc_hsrb_description/urdf/hand_v0/hand.transmission.xacro (robot description, xacro)
@@ -3,12 +3,12 @@
     <xacro:macro name="hsrb_hand_transmission" params="prefix">
         <hsrb_effort_joint_transmission joint="${prefix}_motor_joint" reduction="1"/>
-        <hsrb_effort_joint_transmission joint="${prefix}_left_actuated_proximal_joint" reduction="1"/>
-        <hsrb_effort_joint_transmission joint="${prefix}_left_spring_proximal_joint" reduction="1"/>
-        <hsrb_effort_joint_transmission joint="${prefix}_left_mimic_distal_joint" reduction="1"/>
-        <hsrb_effort_joint_transmission joint="${prefix}_left_distal_joint" reduction="1"/>
-        <hsrb_effort_joint_transmission joint="${prefix}_right_actuated_proximal_joint" reduction="1"/>
-        <hsrb_effort_joint_transmission joint="${prefix}_right_spring_proximal_joint" reduction="1"/>
-        <hsrb_effort_joint_transmission joint="${prefix}_right_mimic_distal_joint" reduction="1"/>
-        <hsrb_effort_joint_transmission joint="${prefix}_right_distal_joint" reduction="1"/>
+        <hsrb_effort_joint_transmission joint="${prefix}_l_actuated_proximal_joint" reduction="1"/>
+        <hsrb_effort_joint_transmission joint="${prefix}_l_spring_proximal_joint" reduction="1"/>
+        <hsrb_effort_joint_transmission joint="${prefix}_l_mimic_distal_joint" reduction="1"/>
+        <hsrb_effort_joint_transmission joint="${prefix}_l_distal_joint" reduction="1"/>
+        <hsrb_effort_joint_transmission joint="${prefix}_r_actuated_proximal_joint" reduction="1"/>
+        <hsrb_effort_joint_transmission joint="${prefix}_r_spring_proximal_joint" reduction="1"/>
+        <hsrb_effort_joint_transmission joint="${prefix}_r_mimic_distal_joint" reduction="1"/>
+        <hsrb_effort_joint_transmission joint="${prefix}_r_distal_joint" reduction="1"/>
     </xacro:macro>
 </robot>

File: tmc_hsrb_description/urdf/hand_v0/hand.urdf.xacro (robot description, xacro)
@@ -58,9 +58,9 @@
                 upper="${actuated_proximal_joint_angle_range_max}" />
             <parent link="${prefix}_palm_link" />
-            <child link="${prefix}_motor_link" />
+            <child link="${prefix}_motor_frame" />
             <dynamics damping="1.0"/>
         </joint>
         <!-- dummy link -->
-        <xacro:hsrb_gripper_dummy_link name="${prefix}_motor_link" />
+        <xacro:hsrb_gripper_dummy_link name="${prefix}_motor_frame" />
     </xacro:macro>
     <xacro:macro name="hsrb_hand" params="prefix parent *origin">
@@ -68,9 +68,9 @@
             <insert_block name="origin" />
         </xacro:hsrb_gripper_base>
-        <xacro:hsrb_finger_with_vacuum prefix="${prefix}" suffix="left" parent="${prefix}_palm_link">
+        <xacro:hsrb_finger_with_vacuum prefix="${prefix}" suffix="l" parent="${prefix}_palm_link">
             <origin xyz="${palm_to_proximal_x} ${palm_to_proximal_y} ${palm_to_proximal_z}"
                 rpy="0.0 0.0 0.0" />
         </xacro:hsrb_finger_with_vacuum>
-        <xacro:hsrb_finger_without_vacuum prefix="${prefix}" suffix="right" parent="${prefix}_palm_link">
+        <xacro:hsrb_finger_without_vacuum prefix="${prefix}" suffix="r" parent="${prefix}_palm_link">
             <origin xyz="${palm_to_proximal_x} ${-palm_to_proximal_y} ${palm_to_proximal_z}"
                 rpy="0.0 0.0 0.0" />
@@ -150,11 +150,11 @@
             <visual>
                 <geometry>
-                    <mesh filename="package://tmc_hsrb_description/meshes/hand_v0/left_proximal.dae" />
-                </geometry>
-                <material name="body_sub" />
-            </visual>
-            <collision>
-                <geometry>
-                    <mesh filename="package://tmc_hsrb_description/meshes/hand_v0/left_proximal.stl" />
+                    <mesh filename="package://tmc_hsrb_description/meshes/hand_v0/l_proximal.dae" />
+                </geometry>
+                <material name="body_sub" />
+            </visual>
+            <collision>
+                <geometry>
+                    <mesh filename="package://tmc_hsrb_description/meshes/hand_v0/l_proximal.stl" />
                 </geometry>
                 <material name="body_sub" />
@@ -175,11 +175,11 @@
             <visual>
                 <geometry>
-                    <mesh filename="package://tmc_hsrb_description/meshes/hand_v0/left_distal.dae" />
-                </geometry>
-                <material name="body_sub" />
-            </visual>
-            <collision>
-                <geometry>
-                    <mesh filename="package://tmc_hsrb_description/meshes/hand_v0/left_distal.stl" />
+                    <mesh filename="package://tmc_hsrb_description/meshes/hand_v0/l_distal.dae" />
+                </geometry>
+                <material name="body_sub" />
+            </visual>
+            <collision>
+                <geometry>
+                    <mesh filename="package://tmc_hsrb_description/meshes/hand_v0/l_distal.stl" />
                 </geometry>
                 <material name="body_sub" />
@@ -229,11 +229,11 @@
             <visual>
                 <geometry>
-                    <mesh filename="package://tmc_hsrb_description/meshes/hand_v0/right_proximal.dae" />
-                </geometry>
-                <material name="body_sub" />
-            </visual>
-            <collision>
-                <geometry>
-                    <mesh filename="package://tmc_hsrb_description/meshes/hand_v0/right_proximal.stl" />
+                    <mesh filename="package://tmc_hsrb_description/meshes/hand_v0/r_proximal.dae" />
+                </geometry>
+                <material name="body_sub" />
+            </visual>
+            <collision>
+                <geometry>
+                    <mesh filename="package://tmc_hsrb_description/meshes/hand_v0/r_proximal.stl" />
                 </geometry>
                 <material name="body_sub" />
@@ -254,11 +254,11 @@
             <visual>
                 <geometry>
-                    <mesh filename="package://tmc_hsrb_description/meshes/hand_v0/right_distal.dae" />
-                </geometry>
-                <material name="body_sub" />
-            </visual>
-            <collision>
-                <geometry>
-                    <mesh filename="package://tmc_hsrb_description/meshes/hand_v0/right_distal.stl" />
+                    <mesh filename="package://tmc_hsrb_description/meshes/hand_v0/r_distal.dae" />
+                </geometry>
+                <material name="body_sub" />
+            </visual>
+            <collision>
+                <geometry>
+                    <mesh filename="package://tmc_hsrb_description/meshes/hand_v0/r_distal.stl" />
                 </geometry>
                 <material name="body_sub" />

File: tmc_hsrb_description/urdf/head_v0/head.gazebo.xacro (robot description, xacro)
@@ -4,6 +4,6 @@
         <gazebo_link name="${prefix}_pan_link" gravity="true" collide="false" friction="0.9"/>
         <gazebo_link name="${prefix}_tilt_link" gravity="true" collide="false" friction="0.9"/>
-        <gazebo_link name="${prefix}_left_camera_link" gravity="true" collide="false" friction="0.9"/>
-        <gazebo_link name="${prefix}_right_camera_link" gravity="true" collide="false" friction="0.9"/>
+        <gazebo_link name="${prefix}_l_camera_link" gravity="true" collide="false" friction="0.9"/>
+        <gazebo_link name="${prefix}_r_camera_link" gravity="true" collide="false" friction="0.9"/>
         <gazebo_link name="${prefix}_center_camera_link" gravity="true" collide="false" friction="0.9"/>
         <gazebo_link name="${prefix}_xtion_link" gravity="true" collide="false" friction="0.9"/>
