Commit message: Rearrange frame/joint/link structure

File: tmc_hsrb_description/urdf/head_v0/head.urdf.xacro (robot description, xacro)
@@ -3,6 +3,6 @@
     <xacro:include filename="$(find tmc_hsrb_description)/urdf/head_v0/head.transmission.xacro"/>
     <xacro:include filename="$(find tmc_hsrb_description)/urdf/head_v0/head.gazebo.xacro"/>
-    <xacro:include filename="$(find tmc_hsrb_description)/urdf/sensors/depth_camera.urdf.xacro"/>
-    <xacro:include filename="$(find tmc_hsrb_description)/urdf/sensors/stereo_camera.urdf.xacro"/>
+    <xacro:include filename="$(find tmc_hsrb_description)/urdf/sensors/asus_xtion.urdf.xacro"/>
+    <xacro:include filename="$(find tmc_hsrb_description)/urdf/sensors/pointgrey_chameleon.urdf.xacro"/>
     <xacro:include filename="$(find tmc_hsrb_description)/urdf/sensors/wide_camera.urdf.xacro"/>
     <!-- head -->
@@ -89,8 +89,8 @@
         </link>
         <!-- cameras -->
-        <xacro:pointgrey_chameleon prefix="${prefix}_left" parent="${prefix}_tilt_link" robot_namespace="${robot_name}">
+        <xacro:pointgrey_chameleon prefix="${prefix}_l_stereo" parent="${prefix}_tilt_link" robot_namespace="${robot_name}">
             <origin xyz="0.02 0.07 0.061" rpy="0 0 0"/>
         </xacro:pointgrey_chameleon>
-        <xacro:pointgrey_chameleon prefix="${prefix}_right" parent="${prefix}_tilt_link" robot_namespace="${robot_name}">
+        <xacro:pointgrey_chameleon prefix="${prefix}_r_stereo" parent="${prefix}_tilt_link" robot_namespace="${robot_name}">
             <origin xyz="0.02 -0.07 0.061" rpy="0 0 0"/>
         </xacro:pointgrey_chameleon>
@@ -98,7 +98,7 @@
             <origin xyz="0.0195 0.0 0.061" rpy="0 0 0"/>
         </xacro:wide_camera>
-        <xacro:depth_camera1 prefix="${prefix}" parent="${prefix}_tilt_link" robot_namespace="${robot_name}">
+        <xacro:asus_xtion prefix="${prefix}" parent="${prefix}_tilt_link" robot_namespace="${robot_name}">
             <origin xyz="-0.079796 0.022 0.215172" rpy="0 0 0"/>
-        </xacro:depth_camera1>
+        </xacro:asus_xtion>
         <xacro:hsrb_head_gazebo prefix="${prefix}"/>
         <xacro:hsrb_head_transmission prefix="${prefix}"/>

File: tmc_hsrb_description/urdf/sensors/asus_xtion.urdf.xacro (robot description, xacro)
@@ -1,13 +1,13 @@
 <?xml version="1.0" ?>
 <robot name="hsrb" xmlns:xacro="http://www.ros.org/wiki/xacro">
-    <xacro:include filename="$(find tmc_hsrb_description)/urdf/sensors/depth_camera.gazebo.xacro"/>
-    <!-- depth_camera -->
-    <xacro:macro name="depth_camera1" params="prefix parent robot_namespace *origin">
-        <joint name="${prefix}_depth_camera_joint" type="fixed">
+    <xacro:include filename="$(find tmc_hsrb_description)/urdf/sensors/asus_xtion.gazebo.xacro"/>
+    <!-- rgbd_sensor -->
+    <xacro:macro name="asus_xtion" params="prefix parent robot_namespace *origin">
+        <joint name="${prefix}_rgbd_sensor_joint" type="fixed">
             <insert_block name="origin" />
             <parent link="${parent}"/>
-            <child link="${prefix}_depth_camera_link"/>
+            <child link="${prefix}_rgbd_sensor_link"/>
         </joint>
-        <link name="${prefix}_depth_camera_link">
+        <link name="${prefix}_rgbd_sensor_link">
             <visual>
                 <origin xyz="0 0 0" rpy="${-pi/2.0} 0.0 ${-pi/2.0}"/>
@@ -25,16 +25,16 @@
             </collision>
         </link>
-        <joint name="${prefix}_depth_camera_pointcloud_frame_joint" type="fixed">
+        <joint name="${prefix}_rgbd_sensor_pointcloud_frame_joint" type="fixed">
             <origin xyz="0 0 0" rpy="${-pi/2.0} 0.0 ${-pi/2.0}"/>
-            <parent link="${prefix}_depth_camera_link"/>
-            <child link="${prefix}_depth_camera_pointcloud_frame"/>
+            <parent link="${prefix}_rgbd_sensor_link"/>
+            <child link="${prefix}_rgbd_sensor_pointcloud_frame"/>
         </joint>
         `
-        <link name="${prefix}_depth_camera_pointcloud_frame"></link>
-        <xacro:depth_camera_gazebo
+        <link name="${prefix}_rgbd_sensor_pointcloud_frame"></link>
+        <xacro:rgbd_sensor_gazebo
             robot_namespace="${robot_namespace}"
-            sensor_name="${prefix}_depth_camera"
-            parent_camera_link="${prefix}_depth_camera_link"
-            parent_depth_link="${prefix}_depth_camera_pointcloud_frame"/>
+            sensor_name="${prefix}_rgbd_sensor"
+            parent_camera_link="${prefix}_rgbd_sensor_link"
+            parent_depth_link="${prefix}_rgbd_sensor_pointcloud_frame"/>
     </xacro:macro>
 </robot>

File: tmc_hsrb_description/urdf/sensors/hokuyo_laser.urdf.xacro (robot description, xacro)
@@ -3,10 +3,10 @@
     <!-- range sensor -->
     <xacro:macro name="hokuyo_laser" params="prefix robot_namespace parent *origin">
-        <joint name="${prefix}_laser_joint" type="fixed">
+        <joint name="${prefix}_range_sensor_joint" type="fixed">
             <insert_block name="origin" />
             <parent link="${parent}" />
-            <child link="${prefix}_laser_link" />
+            <child link="${prefix}_range_sensor_link" />
         </joint>
-        <link name="${prefix}_laser_link">
+        <link name="${prefix}_range_sensor_link">
             <visual>
                 <geometry>
@@ -23,8 +23,8 @@
         </link>
         <xacro:hokuyo_laser_gazebo
-            sensor_name="${prefix}_laser"
+            sensor_name="${prefix}_range_sensor"
             robot_namespace="${robot_namespace}"
             ros_topic="${prefix}_scan"
-            frame_name="${prefix}_laser_link"
+            frame_name="${prefix}_range_sensor_link"
             min_angle="-2.3562" max_angle="2.3562" />
     </xacro:macro>

File: tmc_hsrb_description/urdf/sensors/imu.urdf.xacro (robot description, xacro)
@@ -7,8 +7,8 @@
             <insert_block name="origin" />
             <parent link="${parent}" />
-            <child link="${prefix}_imu_link" />
+            <child link="${prefix}_imu_frame" />
         </joint>
-        <link name="${prefix}_imu_link"/>
-        <xacro:imu_gazebo sensor_name="${prefix}_imu" robot_namespace="${robot_namespace}" frame_name="${prefix}_imu_link"/>
+        <link name="${prefix}_imu_frame"/>
+        <xacro:imu_gazebo sensor_name="${prefix}_imu" robot_namespace="${robot_namespace}" frame_name="${prefix}_imu_frame"/>
     </xacro:macro>
 </robot>

File: tmc_hsrb_description/urdf/sensors/pointgrey_chameleon.urdf.xacro (robot description, xacro)
@@ -1,5 +1,5 @@
 <?xml version="1.0"?>
 <robot xmlns:xacro="http://ros.org/wiki/xacro">
-    <xacro:include filename="$(find tmc_hsrb_description)/urdf/sensors/stereo_camera.gazebo.xacro"/>
+    <xacro:include filename="$(find tmc_hsrb_description)/urdf/sensors/pointgrey_chameleon.gazebo.xacro"/>
     <xacro:macro name="pointgrey_chameleon" params="prefix parent robot_namespace *origin">
         <joint name="${prefix}_camera_joint" type="fixed">

File: tmc_hsrb_description/urdf/sensors/wide_camera.urdf.xacro (robot description, xacro)
@@ -7,10 +7,10 @@
             <insert_block name="origin" />
             <parent link="${parent}" />
-            <child link="${prefix}_camera_link" />
+            <child link="${prefix}_camera_frame" />
         </joint>
-        <link name="${prefix}_camera_link"></link>
+        <link name="${prefix}_camera_frame"></link>
         <xacro:wide_camera_gazebo
             sensor_name="${prefix}_camera"
-            frame_name="${prefix}_camera_link"
+            frame_name="${prefix}_camera_frame"
             robot_namespace="${robot_namespace}"
             />
