Commit message: Split meshes into vesioned layout.

File: tmc_hsrb_description/urdf/arm_v0/arm.urdf.xacro (robot description, xacro)
@@ -21,5 +21,5 @@
             <visual>
                 <geometry>
-                    <mesh filename="package://tmc_hsrb_description/meshes/visual/shoulder.dae" />
+                    <mesh filename="package://tmc_hsrb_description/meshes/arm_v0/shoulder.dae" />
                 </geometry>
                 <material name="body_sub" />
@@ -27,5 +27,5 @@
             <collision>
                 <geometry>
-                    <mesh filename="package://tmc_hsrb_description/meshes/collision/shoulder.stl" />
+                    <mesh filename="package://tmc_hsrb_description/meshes/arm_v0/shoulder.stl" />
                 </geometry>
                 <material name="body_sub" />
@@ -48,5 +48,5 @@
             <visual>
                 <geometry>
-                    <mesh filename="package://tmc_hsrb_description/meshes/visual/arm_flex.dae" />
+                    <mesh filename="package://tmc_hsrb_description/meshes/arm_v0/arm_flex.dae" />
                 </geometry>
                 <material name="body_main" />
@@ -54,5 +54,5 @@
             <collision>
                 <geometry>
-                    <mesh filename="package://tmc_hsrb_description/meshes/collision/arm_flex.stl" />
+                    <mesh filename="package://tmc_hsrb_description/meshes/arm_v0/arm_flex.stl" />
                 </geometry>
                 <material name="body_main" />
@@ -75,5 +75,5 @@
             <visual>
                 <geometry>
-                    <mesh filename="package://tmc_hsrb_description/meshes/visual/arm_roll.dae" />
+                    <mesh filename="package://tmc_hsrb_description/meshes/arm_v0/arm_roll.dae" />
                 </geometry>
                 <material name="body_main" />
@@ -81,5 +81,5 @@
             <collision>
                 <geometry>
-                    <mesh filename="package://tmc_hsrb_description/meshes/collision/arm_roll.stl" />
+                    <mesh filename="package://tmc_hsrb_description/meshes/arm_v0/arm_roll.stl" />
                 </geometry>
                 <material name="body_main" />

File: tmc_hsrb_description/urdf/base_v0/base.urdf.xacro (robot description, xacro)
@@ -104,5 +104,5 @@
             <visual>
                 <geometry>
-                    <mesh filename="package://tmc_hsrb_description/meshes/visual/base.dae" />
+                    <mesh filename="package://tmc_hsrb_description/meshes/base_v0/base.dae" />
                 </geometry>
                 <material name="body_main" />
@@ -110,5 +110,5 @@
             <visual>
                 <geometry>
-                    <mesh filename="package://tmc_hsrb_description/meshes/visual/body.dae" />
+                    <mesh filename="package://tmc_hsrb_description/meshes/base_v0/body.dae" />
                 </geometry>
                 <material name="body_main" />
@@ -116,5 +116,5 @@
             <visual>
                 <geometry>
-                    <mesh filename="package://tmc_hsrb_description/meshes/visual/torso_base.dae" />
+                    <mesh filename="package://tmc_hsrb_description/meshes/base_v0/torso_base.dae" />
                 </geometry>
                 <material name="body_sub" />
@@ -122,5 +122,5 @@
             <collision>
                 <geometry>
-                    <mesh filename="package://tmc_hsrb_description/meshes/collision/base.stl" />
+                    <mesh filename="package://tmc_hsrb_description/meshes/base_v0/base.stl" />
                 </geometry>
                 <material name="body_sub" />

File: tmc_hsrb_description/urdf/hand_v0/hand.urdf.xacro (robot description, xacro)
@@ -22,11 +22,11 @@
             <visual>
                 <geometry>
-                    <mesh filename="package://tmc_hsrb_description/meshes/visual/palm.dae" />
-                </geometry>
-                <material name="body_sub" />
-            </visual>
-            <collision>
-                <geometry>
-                    <mesh filename="package://tmc_hsrb_description/meshes/collision/palm.stl" />
+                    <mesh filename="package://tmc_hsrb_description/meshes/hand_v0/palm.dae" />
+                </geometry>
+                <material name="body_sub" />
+            </visual>
+            <collision>
+                <geometry>
+                    <mesh filename="package://tmc_hsrb_description/meshes/hand_v0/palm.stl" />
                 </geometry>
                 <material name="body_sub" />
@@ -74,11 +74,11 @@
             <visual>
                 <geometry>
-                    <mesh filename="package://tmc_hsrb_description/meshes/visual/left_proximal.dae" />
-                </geometry>
-                <material name="body_sub" />
-            </visual>
-            <collision>
-                <geometry>
-                    <mesh filename="package://tmc_hsrb_description/meshes/collision/left_proximal.stl" />
+                    <mesh filename="package://tmc_hsrb_description/meshes/hand_v0/left_proximal.dae" />
+                </geometry>
+                <material name="body_sub" />
+            </visual>
+            <collision>
+                <geometry>
+                    <mesh filename="package://tmc_hsrb_description/meshes/hand_v0/left_proximal.stl" />
                 </geometry>
                 <material name="body_sub" />
@@ -103,11 +103,11 @@
             <visual>
                 <geometry>
-                    <mesh filename="package://tmc_hsrb_description/meshes/visual/left_distal.dae" />
-                </geometry>
-                <material name="body_sub" />
-            </visual>
-            <collision>
-                <geometry>
-                    <mesh filename="package://tmc_hsrb_description/meshes/collision/left_distal.stl" />
+                    <mesh filename="package://tmc_hsrb_description/meshes/hand_v0/left_distal.dae" />
+                </geometry>
+                <material name="body_sub" />
+            </visual>
+            <collision>
+                <geometry>
+                    <mesh filename="package://tmc_hsrb_description/meshes/hand_v0/left_distal.stl" />
                 </geometry>
                 <material name="body_sub" />
@@ -156,11 +156,11 @@
             <visual>
                 <geometry>
-                    <mesh filename="package://tmc_hsrb_description/meshes/visual/right_proximal.dae" />
-                </geometry>
-                <material name="body_sub" />
-            </visual>
-            <collision>
-                <geometry>
-                    <mesh filename="package://tmc_hsrb_description/meshes/collision/right_proximal.stl" />
+                    <mesh filename="package://tmc_hsrb_description/meshes/hand_v0/right_proximal.dae" />
+                </geometry>
+                <material name="body_sub" />
+            </visual>
+            <collision>
+                <geometry>
+                    <mesh filename="package://tmc_hsrb_description/meshes/hand_v0/right_proximal.stl" />
                 </geometry>
                 <material name="body_sub" />
@@ -185,11 +185,11 @@
             <visual>
                 <geometry>
-                    <mesh filename="package://tmc_hsrb_description/meshes/visual/right_distal.dae" />
-                </geometry>
-                <material name="body_sub" />
-            </visual>
-            <collision>
-                <geometry>
-                    <mesh filename="package://tmc_hsrb_description/meshes/collision/right_distal.stl" />
+                    <mesh filename="package://tmc_hsrb_description/meshes/hand_v0/right_distal.dae" />
+                </geometry>
+                <material name="body_sub" />
+            </visual>
+            <collision>
+                <geometry>
+                    <mesh filename="package://tmc_hsrb_description/meshes/hand_v0/right_distal.stl" />
                 </geometry>
                 <material name="body_sub" />

File: tmc_hsrb_description/urdf/head_v0/head.urdf.xacro (robot description, xacro)
@@ -24,5 +24,5 @@
             <visual>
                 <geometry>
-                    <mesh filename="package://tmc_hsrb_description/meshes/visual/head_pan.dae" />
+                    <mesh filename="package://tmc_hsrb_description/meshes/head_v0/head_pan.dae" />
                 </geometry>
                 <material name="body_main" />
@@ -30,5 +30,5 @@
             <collision>
                 <geometry>
-                    <mesh filename="package://tmc_hsrb_description/meshes/collision/head_pan.stl" />
+                    <mesh filename="package://tmc_hsrb_description/meshes/head_v0/head_pan.stl" />
                 </geometry>
                 <material name="body_main" />
@@ -51,5 +51,5 @@
             <visual>
                 <geometry>
-                    <mesh filename="package://tmc_hsrb_description/meshes/visual/head_upper.dae" />
+                    <mesh filename="package://tmc_hsrb_description/meshes/head_v0/head_upper.dae" />
                 </geometry>
                 <material name="body_sub" />
@@ -57,5 +57,5 @@
             <visual>
                 <geometry>
-                    <mesh filename="package://tmc_hsrb_description/meshes/visual/head_tilt.dae" />
+                    <mesh filename="package://tmc_hsrb_description/meshes/head_v0/head_tilt.dae" />
                 </geometry>
                 <material name="body_main" />
@@ -63,5 +63,5 @@
             <visual>
                 <geometry>
-                    <mesh filename="package://tmc_hsrb_description/meshes/visual/tablet_base.dae" />
+                    <mesh filename="package://tmc_hsrb_description/meshes/head_v0/tablet_base.dae" />
                 </geometry>
                 <material name="body_sub" />
@@ -69,5 +69,5 @@
             <visual>
                 <geometry>
-                    <mesh filename="package://tmc_hsrb_description/meshes/visual/tablet.dae" />
+                    <mesh filename="package://tmc_hsrb_description/meshes/head_v0/tablet.dae" />
                 </geometry>
                 <material name="tablet" />
@@ -75,5 +75,5 @@
             <collision>
                 <geometry>
-                    <mesh filename="package://tmc_hsrb_description/meshes/collision/head.stl" />
+                    <mesh filename="package://tmc_hsrb_description/meshes/head_v0/head.stl" />
                 </geometry>
                 <material name="body_main" />
@@ -81,5 +81,5 @@
             <collision>
                 <geometry>
-                    <mesh filename="package://tmc_hsrb_description/meshes/collision/tablet.stl" />
+                    <mesh filename="package://tmc_hsrb_description/meshes/head_v0/tablet.stl" />
                 </geometry>
                 <material name="tablet" />

File: tmc_hsrb_description/urdf/sensors/depth_camera.urdf.xacro (robot description, xacro)
@@ -13,5 +13,5 @@
                 <origin xyz="0 0 0" rpy="${-pi/2.0} 0.0 ${-pi/2.0}"/>
                 <geometry>
-                    <mesh filename="package://tmc_hsrb_description/meshes/visual/xtion.dae" />
+                    <mesh filename="package://tmc_hsrb_description/meshes/sensors/xtion.dae" />
                 </geometry>
                 <material name="black" />
@@ -20,5 +20,5 @@
                 <origin xyz="0 0 0" rpy="${-pi/2.0} 0.0 ${-pi/2.0}"/>
                 <geometry>
-                    <mesh filename="package://tmc_hsrb_description/meshes/collision/xtion.stl" />
+                    <mesh filename="package://tmc_hsrb_description/meshes/sensors/xtion.stl" />
                 </geometry>
                 <material name="black" />

File: tmc_hsrb_description/urdf/sensors/hokuyo_laser.urdf.xacro (robot description, xacro)
@@ -11,5 +11,5 @@
             <visual>
                 <geometry>
-                    <mesh filename="package://tmc_hsrb_description/meshes/visual/laser.dae" />
+                    <mesh filename="package://tmc_hsrb_description/meshes/sensors/laser.dae" />
                 </geometry>
                 <material name="black" />
@@ -17,5 +17,5 @@
             <collision>
                 <geometry>
-                    <mesh filename="package://tmc_hsrb_description/meshes/collision/laser.stl" />
+                    <mesh filename="package://tmc_hsrb_description/meshes/sensors/laser.stl" />
                 </geometry>
                 <material name="black" />

File: tmc_hsrb_description/urdf/sensors/stereo_camera.urdf.xacro (robot description, xacro)
@@ -12,5 +12,5 @@
                 <origin xyz="0 0 0" rpy="${-pi/2.0} 0.0 ${-pi/2.0}"/>
                 <geometry>
-                    <mesh filename="package://tmc_hsrb_description/meshes/visual/head_camera.dae" />
+                    <mesh filename="package://tmc_hsrb_description/meshes/sensors/head_camera.dae" />
                 </geometry>
                 <material name="black" />

File: tmc_hsrb_description/urdf/torso_v0/torso.urdf.xacro (robot description, xacro)
@@ -23,5 +23,5 @@
             <visual>
                 <geometry>
-                    <mesh filename="package://tmc_hsrb_description/meshes/visual/torso.dae" />
+                    <mesh filename="package://tmc_hsrb_description/meshes/torso_v0/torso.dae" />
                 </geometry>
                 <material name="body_sub" />
@@ -29,5 +29,5 @@
             <collision>
                 <geometry>
-                    <mesh filename="package://tmc_hsrb_description/meshes/collision/torso.stl" />
+                    <mesh filename="package://tmc_hsrb_description/meshes/torso_v0/torso.stl" />
                 </geometry>
                 <material name="body_sub" />

File: tmc_hsrb_description/urdf/wrist_v0/wrist.urdf.xacro (robot description, xacro)
@@ -22,5 +22,5 @@
             <visual>
                 <geometry>
-                    <mesh filename="package://tmc_hsrb_description/meshes/visual/wrist_flex.dae" />
+                    <mesh filename="package://tmc_hsrb_description/meshes/wrist_v0/wrist_flex.dae" />
                 </geometry>
                 <material name="body_sub" />
@@ -57,5 +57,5 @@
             <visual>
                 <geometry>
-                    <mesh filename="package://tmc_hsrb_description/meshes/visual/wrist_roll.dae" />
+                    <mesh filename="package://tmc_hsrb_description/meshes/wrist_v0/wrist_roll.dae" />
                 </geometry>
                 <material name="body_main" />
@@ -63,5 +63,5 @@
             <collision>
                 <geometry>
-                    <mesh filename="package://tmc_hsrb_description/meshes/collision/wrist_roll.stl" />
+                    <mesh filename="package://tmc_hsrb_description/meshes/wrist_v0/wrist_roll.stl" />
                 </geometry>
                 <material name="body_main" />
