Commit message: Add prefix to depth camera, stereo camera, and wide cameras.

File: tmc_hsrb_description/urdf/arm_v0/arm.urdf.xacro (robot description, xacro)
@@ -11,4 +11,5 @@
             <parent link="${parent}" />
             <child link="${prefix}_lift_link" />
+            <dynamics damping="1.0"/>
         </joint>
         <link name="${prefix}_lift_link">
@@ -38,4 +39,5 @@
             <parent link="${prefix}_lift_link" />
             <child link="${prefix}_flex_link" />
+            <dynamics damping="1.0"/>
         </joint>
         <link name="${prefix}_flex_link">
@@ -65,4 +67,5 @@
             <parent link="${prefix}_flex_link" />
             <child link="${prefix}_roll_link" />
+            <dynamics damping="0.1"/>
         </joint>
         <link name="${prefix}_roll_link">

File: tmc_hsrb_description/urdf/base_v0/base.urdf.xacro (robot description, xacro)
@@ -21,4 +21,5 @@
             <parent link="${parent}" />
             <child link="${prefix}_${suffix}_drive_wheel_link" />
+            <dynamics damping="1.0"/>
         </joint>
         <link name="${prefix}_${suffix}_drive_wheel_link">
@@ -52,4 +53,5 @@
             <parent link="${parent}" />
             <child link="${prefix}_${suffix}_passive_wheel_x_frame" />
+            <dynamics damping="1.0"/>
         </joint>
         <link name="${prefix}_${suffix}_passive_wheel_x_frame">
@@ -150,4 +152,5 @@
             <parent link="${prefix}_body_link" />
             <child link="${prefix}_roll_link" />
+            <dynamics damping="0.7"/>
         </joint>
         <link name="${prefix}_roll_link">
@@ -185,5 +188,8 @@
         </xacro:hsrb_passive_wheel>
         <!-- sensors -->
-        <xacro:hokuyo_laser prefix="${prefix}" robot_namespace="${robot_namespace}" parent="${prefix}_link">
+        <xacro:hokuyo_laser
+            prefix="${prefix}"
+            robot_namespace="${robot_namespace}"
+            parent="${prefix}_link">
             <origin xyz="0.1375 0.0 0.1895" rpy="0.0 0.0 0.0" />
         </xacro:hokuyo_laser>

File: tmc_hsrb_description/urdf/hand_v0/hand.urdf.xacro (robot description, xacro)
@@ -3,5 +3,5 @@
     <xacro:include filename="$(find tmc_hsrb_description)/urdf/hand_v0/hand.transmission.xacro"/>
     <xacro:include filename="$(find tmc_hsrb_description)/urdf/hand_v0/hand.gazebo.xacro"/>
-    <xacro:include filename="$(find tmc_hsrb_description)/urdf/sensors/rgb_camera.urdf.xacro"/>
+    <xacro:include filename="$(find tmc_hsrb_description)/urdf/sensors/wide_camera.urdf.xacro"/>
     <xacro:property name="palm_to_proximal_x" value="-0.01675" />
     <xacro:property name="palm_to_proximal_y" value="-0.0245" />
@@ -75,7 +75,7 @@
         </xacro:hsrb_finger_without_vacuum>
         <!-- camera -->
-        <xacro:rgb_camera prefix="${prefix}" parent="${prefix}_palm_link">
+        <xacro:wide_camera prefix="${prefix}" parent="${prefix}_palm_link" robot_namespace="${robot_name}">
             <origin xyz="0.039 0.0 -0.0045" rpy="${pi} ${-pi/2} 0"/>
-        </xacro:rgb_camera>
+        </xacro:wide_camera>
         <xacro:hsrb_hand_gazebo prefix="${prefix}"/>
         <xacro:hsrb_hand_transmission prefix="${prefix}"/>

File: tmc_hsrb_description/urdf/head_v0/head.urdf.xacro (robot description, xacro)
@@ -5,5 +5,5 @@
     <xacro:include filename="$(find tmc_hsrb_description)/urdf/sensors/depth_camera.urdf.xacro"/>
     <xacro:include filename="$(find tmc_hsrb_description)/urdf/sensors/stereo_camera.urdf.xacro"/>
-    <xacro:include filename="$(find tmc_hsrb_description)/urdf/sensors/rgb_camera.urdf.xacro"/>
+    <xacro:include filename="$(find tmc_hsrb_description)/urdf/sensors/wide_camera.urdf.xacro"/>
     <!-- head -->
     <xacro:macro name="hsrb_head" params="prefix parent *origin">
@@ -14,4 +14,5 @@
             <parent link="${parent}" />
             <child link="${prefix}_pan_link" />
+            <dynamics damping="1.0"/>
         </joint>
         <link name="${prefix}_pan_link">
@@ -41,4 +42,5 @@
             <parent link="${prefix}_pan_link" />
             <child link="${prefix}_tilt_link" />
+            <dynamics damping="10.0"/>
         </joint>
         <link name="${prefix}_tilt_link">
@@ -87,14 +89,14 @@
         </link>
         <!-- cameras -->
-        <xacro:pointgrey_chameleon prefix="${prefix}_left" parent="${prefix}_tilt_link">
+        <xacro:pointgrey_chameleon prefix="${prefix}_left" parent="${prefix}_tilt_link" robot_namespace="${robot_name}">
             <origin xyz="0.02 0.07 0.061" rpy="0 0 0"/>
         </xacro:pointgrey_chameleon>
-        <xacro:pointgrey_chameleon prefix="${prefix}_right" parent="${prefix}_tilt_link">
+        <xacro:pointgrey_chameleon prefix="${prefix}_right" parent="${prefix}_tilt_link" robot_namespace="${robot_name}">
             <origin xyz="0.02 -0.07 0.061" rpy="0 0 0"/>
         </xacro:pointgrey_chameleon>
-        <xacro:rgb_camera prefix="${prefix}_center" parent="${prefix}_tilt_link">
+        <xacro:wide_camera prefix="${prefix}_center" parent="${prefix}_tilt_link" robot_namespace="${robot_name}">
             <origin xyz="0.0195 0.0 0.061" rpy="0 0 0"/>
-        </xacro:rgb_camera>
-        <xacro:depth_camera1 prefix="${prefix}" parent="${prefix}_tilt_link">
+        </xacro:wide_camera>
+        <xacro:depth_camera1 prefix="${prefix}" parent="${prefix}_tilt_link" robot_namespace="${robot_name}">
             <origin xyz="-0.079796 0.022 0.215172" rpy="0 0 0"/>
         </xacro:depth_camera1>

File: tmc_hsrb_description/urdf/sensors/depth_camera.gazebo.xacro (robot description, xacro)
@@ -16,5 +16,5 @@
     <xacro:property name="XtionMaxDistance" value="5"/>
     <xacro:property name="XtionFrameRate" value="30"/>
-    <xacro:macro name="depth_camera_gazebo" params="sensor_name parent_camera_link parent_depth_link">
+    <xacro:macro name="depth_camera_gazebo" params="robot_namespace sensor_name parent_camera_link parent_depth_link">
         <gazebo reference="${parent_camera_link}">
             <sensor type="depth" name="openni_camera_camera">
@@ -35,13 +35,14 @@
                 </camera>
                 <plugin name="camera_controller" filename="libgazebo_ros_openni_kinect.so">
+                    <robotNamespace>${robot_namespace}</robotNamespace>
                     <alwaysOn>true</alwaysOn>
                     <updateRate>10.0</updateRate>
                     <cameraName>${sensor_name}</cameraName>
                     <frameName>${parent_depth_link}</frameName>
-                    <imageTopicName>/${sensor_name}/rgb/image_raw</imageTopicName>
-                    <depthImageTopicName>/${sensor_name}/depth/image_raw</depthImageTopicName>
-                    <pointCloudTopicName>/${sensor_name}/depth/points</pointCloudTopicName>
-                    <cameraInfoTopicName>/${sensor_name}/rgb/camera_info</cameraInfoTopicName>
-                    <depthImageCameraInfoTopicName>/${sensor_name}/depth/camera_info</depthImageCameraInfoTopicName>
+                    <imageTopicName>${sensor_name}/rgb/image_raw</imageTopicName>
+                    <depthImageTopicName>${sensor_name}/depth/image_raw</depthImageTopicName>
+                    <pointCloudTopicName>${sensor_name}/depth/points</pointCloudTopicName>
+                    <cameraInfoTopicName>${sensor_name}/rgb/camera_info</cameraInfoTopicName>
+                    <depthImageCameraInfoTopicName>${sensor_name}/depth/camera_info</depthImageCameraInfoTopicName>
                     <pointCloudCutoff>0.4</pointCloudCutoff>
                     <hackBaseline>0.0</hackBaseline>

File: tmc_hsrb_description/urdf/sensors/depth_camera.urdf.xacro (robot description, xacro)
@@ -3,5 +3,5 @@
     <xacro:include filename="$(find tmc_hsrb_description)/urdf/sensors/depth_camera.gazebo.xacro"/>
     <!-- depth_camera -->
-    <xacro:macro name="depth_camera1" params="prefix parent *origin">
+    <xacro:macro name="depth_camera1" params="prefix parent robot_namespace *origin">
         <joint name="${prefix}_depth_camera_joint" type="fixed">
             <insert_block name="origin" />
@@ -33,4 +33,5 @@
         <link name="${prefix}_depth_camera_pointcloud_frame"></link>
         <xacro:depth_camera_gazebo
+            robot_namespace="${robot_namespace}"
             sensor_name="${prefix}_depth_camera"
             parent_camera_link="${prefix}_depth_camera_link"

File: tmc_hsrb_description/urdf/sensors/stereo_camera.gazebo.xacro (robot description, xacro)
@@ -1,13 +1,13 @@
 <?xml version="1.0" ?>
 <robot name="hsrb" xmlns:xacro="http://www.ros.org/wiki/xacro">
-    <xacro:macro name="pointgrey_chameleon_gazebo" params="sensor_name frame_name">
+    <xacro:macro name="pointgrey_chameleon_gazebo" params="sensor_name frame_name robot_namespace">
         <gazebo reference="${frame_name}">
             <sensor type="camera" name="${sensor_name}">
                 <update_rate>10.0</update_rate>
                 <camera name="${sensor_name}">
-                    <horizontal_fov>1.3962634</horizontal_fov>
+                    <horizontal_fov>1.16762527</horizontal_fov>
                     <image>
-                        <width>320</width>
-                        <height>240</height>
+                        <width>1280</width>
+                        <height>1024</height>
                         <format>R8G8B8</format>
                     </image>
@@ -18,7 +18,4 @@
                     <noise>
                         <type>gaussian</type>
-                        <!-- Noise is sampled independently per pixel on each frame.
-                             That pixel's noise value is added to each of its color
-                             channels, which at that point lie in the range [0,1]. -->
                         <mean>0.0</mean>
                         <stddev>0.007</stddev>
@@ -32,4 +29,5 @@
                     <cameraInfoTopicName>camera_info</cameraInfoTopicName>
                     <frameName>${frame_name}</frameName>
+                    <robotNamespace>${robot_namespace}</robotNamespace>
                     <hackBaseline>0.07</hackBaseline>
                     <distortionK1>0.0</distortionK1>

File: tmc_hsrb_description/urdf/sensors/stereo_camera.urdf.xacro (robot description, xacro)
@@ -2,5 +2,5 @@
 <robot xmlns:xacro="http://ros.org/wiki/xacro">
     <xacro:include filename="$(find tmc_hsrb_description)/urdf/sensors/stereo_camera.gazebo.xacro"/>
-    <xacro:macro name="pointgrey_chameleon" params="prefix parent *origin">
+    <xacro:macro name="pointgrey_chameleon" params="prefix parent robot_namespace *origin">
         <joint name="${prefix}_camera_joint" type="fixed">
             <insert_block name="origin" />
@@ -17,5 +17,8 @@
             </visual>
         </link>
-        <xacro:pointgrey_chameleon_gazebo sensor_name="${prefix}_camera" frame_name="${prefix}_camera_link"/>
+        <xacro:pointgrey_chameleon_gazebo
+            sensor_name="${prefix}_camera"
+            frame_name="${prefix}_camera_link"
+            robot_namespace="${robot_namespace}"/>
     </xacro:macro>
 </robot>

File: tmc_hsrb_description/urdf/sensors/wide_camera.gazebo.xacro (robot description, xacro)
@@ -1,13 +1,13 @@
 <?xml version="1.0" ?>
 <robot name="hsrb" xmlns:xacro="http://www.ros.org/wiki/xacro">
-    <xacro:macro name="rgb_camera_gazebo" params="sensor_name frame_name">
+    <xacro:macro name="wide_camera_gazebo" params="sensor_name frame_name robot_namespace">
         <gazebo reference="${frame_name}">
             <sensor type="camera" name="${sensor_name}">
                 <update_rate>10.0</update_rate>
                 <camera name="${sensor_name}">
-                    <horizontal_fov>1.3962634</horizontal_fov>
+                    <horizontal_fov>1.16762527</horizontal_fov>
                     <image>
-                        <width>320</width>
-                        <height>240</height>
+                        <width>1280</width>
+                        <height>1024</height>
                         <format>R8G8B8</format>
                     </image>
@@ -18,7 +18,4 @@
                     <noise>
                         <type>gaussian</type>
-                        <!-- Noise is sampled independently per pixel on each frame.
-                             That pixel's noise value is added to each of its color
-                             channels, which at that point lie in the range [0,1]. -->
                         <mean>0.0</mean>
                         <stddev>0.007</stddev>
@@ -26,4 +23,5 @@
                 </camera>
                 <plugin name="camera_controller" filename="libgazebo_ros_camera.so">
+                    <robotNamespace>${robot_namespace}</robotNamespace>
                     <alwaysOn>0</alwaysOn>
                     <updateRate>0.0</updateRate>

File: tmc_hsrb_description/urdf/sensors/wide_camera.urdf.xacro (robot description, xacro)
@@ -1,7 +1,7 @@
 <?xml version="1.0"?>
 <robot xmlns:xacro="http://ros.org/wiki/xacro">
-    <xacro:include filename="$(find tmc_hsrb_description)/urdf/sensors/rgb_camera.gazebo.xacro"/>
+    <xacro:include filename="$(find tmc_hsrb_description)/urdf/sensors/wide_camera.gazebo.xacro"/>
     <!-- wide rgb camera -->
-    <xacro:macro name="rgb_camera" params="prefix parent *origin">
+    <xacro:macro name="wide_camera" params="prefix parent robot_namespace *origin">
         <joint name="${prefix}_camera_joint" type="fixed">
             <insert_block name="origin" />
@@ -10,5 +10,9 @@
         </joint>
         <link name="${prefix}_camera_link"></link>
-        <xacro:rgb_camera_gazebo sensor_name="${prefix}_camera" frame_name="${prefix}_camera_link"/>
+        <xacro:wide_camera_gazebo
+            sensor_name="${prefix}_camera"
+            frame_name="${prefix}_camera_link"
+            robot_namespace="${robot_namespace}"
+            />
     </xacro:macro>
 </robot>

File: tmc_hsrb_description/urdf/torso_v0/torso.urdf.xacro (robot description, xacro)
@@ -13,4 +13,5 @@
             <child link="${prefix}_lift_link" />
             <mimic joint="${mimic_joint}" multiplier="0.5" />
+            <dynamics damping="10.0"/>
         </joint>
         <link name="${prefix}_lift_link">

File: tmc_hsrb_description/urdf/wrist_v0/wrist.urdf.xacro (robot description, xacro)
@@ -12,4 +12,5 @@
             <parent link="${parent}" />
             <child link="${prefix}_flex_link" />
+            <dynamics damping="1.0"/>
         </joint>
         <link name="${prefix}_flex_link">
@@ -47,4 +48,5 @@
             <parent link="${prefix}_flex_link" />
             <child link="${prefix}_roll_link" />
+            <dynamics damping="1.0"/>
         </joint>
         <link name="${prefix}_roll_link">
@@ -68,5 +70,9 @@
             </collision>
         </link>
-        <xacro:minebea_ft_sensor prefix="${prefix}" robot_namespace="${robot_namespace}" parent="${prefix}_roll_link" joint_name="${prefix}_roll_joint">
+        <xacro:minebea_ft_sensor
+            prefix="${prefix}"
+            robot_namespace="${robot_namespace}"
+            parent="${prefix}_roll_link"
+            joint_name="${prefix}_roll_joint">
             <origin xyz="0.0 0.0 0.0735" rpy="${pi} 0.0 0.0"/>
         </xacro:minebea_ft_sensor>

Commit message: ロボットモデルの軽量化と肩の色を実機に合わせる

File: tmc_hsrb_description/urdf/arm_v0/arm.urdf.xacro (robot description, xacro)
@@ -28,5 +28,5 @@
             <collision>
                 <geometry>
-                    <mesh filename="package://tmc_hsrb_description/meshes/arm_v0/shoulder.stl" />
+                    <mesh filename="package://tmc_hsrb_description/meshes/arm_v0/shoulder_light.stl" />
                 </geometry>
                 <material name="body_sub" />
@@ -50,5 +50,5 @@
             <visual>
                 <geometry>
-                    <mesh filename="package://tmc_hsrb_description/meshes/arm_v0/arm_flex.dae" />
+                    <mesh filename="package://tmc_hsrb_description/meshes/arm_v0/arm_flex_light.dae" />
                 </geometry>
                 <material name="body_main" />
@@ -56,5 +56,5 @@
             <collision>
                 <geometry>
-                    <mesh filename="package://tmc_hsrb_description/meshes/arm_v0/arm_flex.stl" />
+                    <mesh filename="package://tmc_hsrb_description/meshes/arm_v0/arm_flex_light.stl" />
                 </geometry>
                 <material name="body_main" />
@@ -78,5 +78,5 @@
             <visual>
                 <geometry>
-                    <mesh filename="package://tmc_hsrb_description/meshes/arm_v0/arm_roll.dae" />
+                    <mesh filename="package://tmc_hsrb_description/meshes/arm_v0/arm_roll_light.dae" />
                 </geometry>
                 <material name="body_main" />
@@ -84,5 +84,5 @@
             <collision>
                 <geometry>
-                    <mesh filename="package://tmc_hsrb_description/meshes/arm_v0/arm_roll.stl" />
+                    <mesh filename="package://tmc_hsrb_description/meshes/arm_v0/arm_roll_light.stl" />
                 </geometry>
                 <material name="body_main" />

File: tmc_hsrb_description/urdf/base_v0/base.urdf.xacro (robot description, xacro)
@@ -111,5 +111,5 @@
             <visual>
                 <geometry>
-                    <mesh filename="package://tmc_hsrb_description/meshes/base_v0/base.dae" />
+                    <mesh filename="package://tmc_hsrb_description/meshes/base_v0/base_light.dae" />
                 </geometry>
                 <material name="body_main" />

File: tmc_hsrb_description/urdf/hand_v0/hand.urdf.xacro (robot description, xacro)
@@ -41,5 +41,5 @@
             <visual>
                 <geometry>
-                    <mesh filename="package://tmc_hsrb_description/meshes/hand_v0/palm.dae" />
+                    <mesh filename="package://tmc_hsrb_description/meshes/hand_v0/palm_light.dae" />
                 </geometry>
                 <material name="body_sub" />

File: tmc_hsrb_description/urdf/head_v0/head.urdf.xacro (robot description, xacro)
@@ -77,5 +77,5 @@
             <collision>
                 <geometry>
-                    <mesh filename="package://tmc_hsrb_description/meshes/head_v0/head.stl" />
+                    <mesh filename="package://tmc_hsrb_description/meshes/head_v0/head_light.stl" />
                 </geometry>
                 <material name="body_main" />

File: tmc_hsrb_description/urdf/torso_v0/torso.urdf.xacro (robot description, xacro)
@@ -24,5 +24,5 @@
             <visual>
                 <geometry>
-                    <mesh filename="package://tmc_hsrb_description/meshes/torso_v0/torso.dae" />
+                    <mesh filename="package://tmc_hsrb_description/meshes/torso_v0/torso_light.dae" />
                 </geometry>
                 <material name="body_sub" />

File: tmc_hsrb_description/urdf/wrist_v0/wrist.urdf.xacro (robot description, xacro)
@@ -65,5 +65,5 @@
             <collision>
                 <geometry>
-                    <mesh filename="package://tmc_hsrb_description/meshes/wrist_v0/wrist_roll.stl" />
+                    <mesh filename="package://tmc_hsrb_description/meshes/wrist_v0/wrist_roll_light.stl" />
                 </geometry>
                 <material name="body_main" />

Commit message: collision用mesh修正
裏返っている面を修正、urdfファイルをリダクション前のmesh指定に戻す

File: tmc_hsrb_description/urdf/arm_v0/arm.urdf.xacro (robot description, xacro)
@@ -28,5 +28,5 @@
             <collision>
                 <geometry>
-                    <mesh filename="package://tmc_hsrb_description/meshes/arm_v0/shoulder_light.stl" />
+                    <mesh filename="package://tmc_hsrb_description/meshes/arm_v0/shoulder.stl" />
                 </geometry>
                 <material name="body_sub" />
@@ -56,5 +56,5 @@
             <collision>
                 <geometry>
-                    <mesh filename="package://tmc_hsrb_description/meshes/arm_v0/arm_flex_light.stl" />
+                    <mesh filename="package://tmc_hsrb_description/meshes/arm_v0/arm_flex.stl" />
                 </geometry>
                 <material name="body_main" />
@@ -84,5 +84,5 @@
             <collision>
                 <geometry>
-                    <mesh filename="package://tmc_hsrb_description/meshes/arm_v0/arm_roll_light.stl" />
+                    <mesh filename="package://tmc_hsrb_description/meshes/arm_v0/arm_roll.stl" />
                 </geometry>
                 <material name="body_main" />

File: tmc_hsrb_description/urdf/head_v0/head.urdf.xacro (robot description, xacro)
@@ -77,5 +77,5 @@
             <collision>
                 <geometry>
-                    <mesh filename="package://tmc_hsrb_description/meshes/head_v0/head_light.stl" />
+                    <mesh filename="package://tmc_hsrb_description/meshes/head_v0/head.stl" />
                 </geometry>
                 <material name="body_main" />

File: tmc_hsrb_description/urdf/wrist_v0/wrist.urdf.xacro (robot description, xacro)
@@ -65,5 +65,5 @@
             <collision>
                 <geometry>
-                    <mesh filename="package://tmc_hsrb_description/meshes/wrist_v0/wrist_roll_light.stl" />
+                    <mesh filename="package://tmc_hsrb_description/meshes/wrist_v0/wrist_roll.stl" />
                 </geometry>
                 <material name="body_main" />
