Commit message: Change trajectory-driven transmissions from effort to position

File: tmc_hsrb_description/urdf/arm_v0/arm.transmission.xacro (robot description, xacro)
@@ -2,7 +2,7 @@
 <robot xmlns:xacro="http://ros.org/wiki/xacro">
     <xacro:macro name="hsrb_arm_transmission" params="prefix">
-        <hsrb_effort_joint_transmission joint="${prefix}_lift_joint" reduction="1"/>
-        <hsrb_effort_joint_transmission joint="${prefix}_flex_joint" reduction="1"/>
-        <hsrb_effort_joint_transmission joint="${prefix}_roll_joint" reduction="1"/>
+        <hsrb_position_joint_transmission joint="${prefix}_lift_joint" reduction="1"/>
+        <hsrb_position_joint_transmission joint="${prefix}_flex_joint" reduction="1"/>
+        <hsrb_position_joint_transmission joint="${prefix}_roll_joint" reduction="1"/>
     </xacro:macro>
 </robot>

File: tmc_hsrb_description/urdf/common.xacro (robot description, xacro)
@@ -2,4 +2,16 @@
 <robot xmlns:xacro="http://www.ros.org/wiki.xacro">
   <xacro:property name="pi" value="3.14159265359"/>
+  <macro name="hsrb_position_joint_transmission" params="joint reduction">
+     <transmission name="${joint}_transmission">
+       <type>transmission_interface/SimpleTransmission</type>
+       <joint name="${joint}">
+         <hardwareInterface>PositionJointInterface</hardwareInterface>
+       </joint>
+       <actuator name="${joint}_actuator">
+         <hardwareInterface>PositionJointInterface</hardwareInterface>
+         <mechanicalReduction>${reduction}</mechanicalReduction>
+       </actuator>
+     </transmission>
+  </macro>
   <macro name="hsrb_effort_joint_transmission" params="joint reduction">
      <transmission name="${joint}_transmission">

File: tmc_hsrb_description/urdf/head_v0/head.transmission.xacro (robot description, xacro)
@@ -2,6 +2,6 @@
 <robot xmlns:xacro="http://ros.org/wiki/xacro">
     <xacro:macro name="hsrb_head_transmission" params="prefix">
-        <hsrb_effort_joint_transmission joint="${prefix}_pan_joint" reduction="1"/>
-        <hsrb_effort_joint_transmission joint="${prefix}_tilt_joint" reduction="1"/>
+        <hsrb_position_joint_transmission joint="${prefix}_pan_joint" reduction="1"/>
+        <hsrb_position_joint_transmission joint="${prefix}_tilt_joint" reduction="1"/>
     </xacro:macro>
 </robot>

File: tmc_hsrb_description/urdf/torso_v0/torso.transmission.xacro (robot description, xacro)
@@ -2,5 +2,5 @@
 <robot xmlns:xacro="http://ros.org/wiki/xacro">
     <xacro:macro name="hsrb_torso_transmission" params="prefix">
-        <hsrb_effort_joint_transmission joint="${prefix}_lift_joint" reduction="1"/>
+        <hsrb_position_joint_transmission joint="${prefix}_lift_joint" reduction="1"/>
     </xacro:macro>
 </robot>

File: tmc_hsrb_description/urdf/wrist_v0/wrist.transmission.xacro (robot description, xacro)
@@ -2,6 +2,6 @@
 <robot xmlns:xacro="http://ros.org/wiki/xacro">
     <xacro:macro name="hsrb_wrist_transmission" params="prefix">
-        <hsrb_effort_joint_transmission joint="${prefix}_flex_joint" reduction="1"/>
-        <hsrb_effort_joint_transmission joint="${prefix}_roll_joint" reduction="1"/>
+        <hsrb_position_joint_transmission joint="${prefix}_flex_joint" reduction="1"/>
+        <hsrb_position_joint_transmission joint="${prefix}_roll_joint" reduction="1"/>
     </xacro:macro>
 </robot>
