Commit message: Add hardwareInterface tag for joint transmission.

File: tmc_hsrb_description/urdf/common.xacro (robot description, xacro)
@@ -5,5 +5,7 @@
      <transmission name="${joint}_transmission">
        <type>transmission_interface/SimpleTransmission</type>
-       <joint name="${joint}"/>
+       <joint name="${joint}">
+         <hardwareInterface>EffortJointInterface</hardwareInterface>
+       </joint>
        <actuator name="${joint}_actuator">
          <hardwareInterface>EffortJointInterface</hardwareInterface>
@@ -15,5 +17,7 @@
       <transmission name="${prefix}_transmission">
           <type>transmission_interface/SimpleTransmission</type>
-          <joint name="${joint}"/>
+          <joint name="${joint}">
+            <hardwareInterface>VelocityJointInterface</hardwareInterface>
+          </joint>
           <actuator name="${joint}_actuator">
               <hardwareInterface>VelocityJointInterface</hardwareInterface>
