Commit message: Update passive casters to more realistic model.

File: tmc_hsrb_description/urdf/base_v1/base.gazebo.xacro (robot description, xacro)
@@ -9,4 +9,10 @@
         <gazebo_link_rubber name="${prefix}_right_passive_wheel_z_link"/>
         <gazebo_link_rubber name="${prefix}_left_passive_wheel_z_link"/>
+        <gazebo_link_flat_black name="${prefix}_right_passive_caster_roll_link" gravity="true" collide="false" friction="0.9"/>
+        <gazebo_link_rubber name="${prefix}_right_passive_caster_left_wheel_link"/>
+        <gazebo_link_rubber name="${prefix}_right_passive_caster_right_wheel_link"/>
+        <gazebo_link_flat_black name="${prefix}_left_passive_caster_roll_link" gravity="true" collide="false" friction="0.9"/>
+        <gazebo_link_rubber name="${prefix}_left_passive_caster_left_wheel_link"/>
+        <gazebo_link_rubber name="${prefix}_left_passive_caster_right_wheel_link"/>
         <gazebo_link name="${prefix}_range_sensor_link" gravity="true" collide="false" friction="0.9"/>
         <gazebo_link name="${prefix}_imu_sensor_link" gravity="true" collide="false" friction="0.9"/>

File: tmc_hsrb_description/urdf/base_v1/base.urdf.xacro (robot description, xacro)
@@ -1,6 +1,6 @@
 <?xml version="1.0"?>
 <robot xmlns:xacro="http://ros.org/wiki/xacro">
-    <xacro:include filename="$(find tmc_hsrb_description)/urdf/base_v0/base.transmission.xacro"/>
-    <xacro:include filename="$(find tmc_hsrb_description)/urdf/base_v0/base.gazebo.xacro"/>
+    <xacro:include filename="$(find tmc_hsrb_description)/urdf/base_v1/base.transmission.xacro"/>
+    <xacro:include filename="$(find tmc_hsrb_description)/urdf/base_v1/base.gazebo.xacro"/>
     <xacro:include filename="$(find tmc_hsrb_description)/urdf/sensors/hokuyo_laser.urdf.xacro"/>
     <xacro:include filename="$(find tmc_hsrb_description)/urdf/sensors/imu.urdf.xacro"/>
@@ -10,7 +10,9 @@
     <xacro:property name="drive_wheel_offset_x" value="-0.110" />
     <xacro:property name="drive_wheel_offset_y" value="0.133" />
-    <xacro:property name="passive_wheel_radius" value="0.03" />
-    <xacro:property name="passive_wheel_offset_x" value="0.145" />
-    <xacro:property name="passive_wheel_offset_y" value="0.04" />
+    <xacro:property name="passive_caster_height" value="0.058" />
+    <xacro:property name="passive_caster_radius" value="0.025" />
+    <xacro:property name="passive_caster_width" value="0.014" />
+    <xacro:property name="passive_caster_offset_x" value="0.1495" />
+    <xacro:property name="passive_caster_offset_y" value="0.11" />
     <!-- drive wheel -->
     <xacro:macro name="hsrb_drive_wheel" params="prefix suffix parent *origin">
@@ -46,14 +48,14 @@
     </xacro:macro>
     <!-- passive wheel -->
-    <xacro:macro name="hsrb_passive_wheel" params="prefix suffix parent *origin">
-        <joint name="${prefix}_${suffix}_passive_wheel_x_joint" type="continuous">
+    <xacro:macro name="hsrb_passive_caster" params="prefix suffix parent *origin">
+        <joint name="${prefix}_${suffix}_passive_caster_roll_joint" type="continuous">
             <insert_block name="origin" />
-            <axis xyz="1.0 0.0 0.0" />
+            <axis xyz="0.0 0.0 1.0" />
             <limit effort="1000.0" velocity="100.0" />
             <parent link="${parent}" />
-            <child link="${prefix}_${suffix}_passive_wheel_x_frame" />
-            <dynamics damping="1.0"/>
-        </joint>
-        <link name="${prefix}_${suffix}_passive_wheel_x_frame">
+            <child link="${prefix}_${suffix}_passive_caster_roll_link" />
+            <dynamics damping="0.7"/>
+        </joint>
+        <link name="${prefix}_${suffix}_passive_caster_roll_link">
             <inertial>
                 <mass value="0.3"/>
@@ -61,12 +63,41 @@
                 <inertia ixx="0.001" ixy="0" ixz="0" iyy="0.001" iyz="0" izz="0.001"/>
             </inertial>
-        </link>
-        <joint name="${prefix}_${suffix}_passive_wheel_y_joint" type="continuous">
+            <visual>
+                <origin xyz="0.0 0 -0.0165"/>
+                <geometry>
+                    <cylinder radius="0.0085" length="0.033"/>
+                </geometry>
+                <material name="wheel" />
+            </visual>
+            <visual>
+                <origin xyz="0.017 0.0 -0.033" rpy="1.57 0.0 0.0"/>
+                <geometry>
+                    <cylinder radius="0.02" length="0.021"/>
+                </geometry>
+                <material name="wheel" />
+            </visual>
+        </link>
+        <joint name="${prefix}_${suffix}_passive_caster_left_wheel_joint" type="continuous">
+            <origin xyz="0.017 0.0175 -0.033"/>
             <axis xyz="0.0 1.0 0.0" />
             <limit effort="1000.0" velocity="100.0" />
-            <parent link="${prefix}_${suffix}_passive_wheel_x_frame" />
-            <child link="${prefix}_${suffix}_passive_wheel_y_frame" />
-        </joint>
-        <link name="${prefix}_${suffix}_passive_wheel_y_frame">
+            <parent link="${prefix}_${suffix}_passive_caster_roll_link" />
+            <child link="${prefix}_${suffix}_passive_caster_left_wheel_link" />
+            <dynamics damping="1.0"/>
+        </joint>
+        <link name="${prefix}_${suffix}_passive_caster_left_wheel_link">
+            <visual>
+                <origin rpy="1.57 0.0 0.0"/>
+                <geometry>
+                    <cylinder radius="${passive_caster_radius}" length="${passive_caster_width}"/>
+                </geometry>
+                <material name="wheel" />
+            </visual>
+            <collision>
+                <origin rpy="1.57 0.0 0.0"/>
+                <geometry>
+                    <cylinder radius="${passive_caster_radius}" length="${passive_caster_width}"/>
+                </geometry>
+            </collision>
             <inertial>
                 <mass value="0.3"/>
@@ -75,20 +106,24 @@
             </inertial>
         </link>
-        <joint name="${prefix}_${suffix}_passive_wheel_z_joint" type="continuous">
-            <axis xyz="0.0 0.0 1.0" />
+        <joint name="${prefix}_${suffix}_passive_caster_right_wheel_joint" type="continuous">
+            <origin xyz="0.017 -0.0175 -0.033"/>
+            <axis xyz="0.0 1.0 0.0" />
             <limit effort="1000.0" velocity="100.0" />
-            <parent link="${prefix}_${suffix}_passive_wheel_y_frame" />
-            <child link="${prefix}_${suffix}_passive_wheel_z_link" />
-        </joint>
-        <link name="${prefix}_${suffix}_passive_wheel_z_link">
-            <visual>
-                <geometry>
-                    <sphere radius="${passive_wheel_radius}" />
-                </geometry>
-                <material name="wheel" />
-            </visual>
-            <collision>
-                <geometry>
-                    <sphere radius="${passive_wheel_radius}" />
+            <parent link="${prefix}_${suffix}_passive_caster_roll_link" />
+            <child link="${prefix}_${suffix}_passive_caster_right_wheel_link" />
+            <dynamics damping="1.0"/>
+        </joint>
+        <link name="${prefix}_${suffix}_passive_caster_right_wheel_link">
+            <visual>
+                <origin rpy="1.57 0.0 0.0"/>
+                <geometry>
+                    <cylinder radius="${passive_caster_radius}" length="${passive_caster_width}"/>
+                </geometry>
+                <material name="wheel" />
+            </visual>
+            <collision>
+                <origin rpy="1.57 0.0 0.0"/>
+                <geometry>
+                    <cylinder radius="${passive_caster_radius}" length="${passive_caster_width}"/>
                 </geometry>
                 <material name="wheel" />
@@ -131,5 +166,4 @@
                     <mesh filename="package://tmc_hsrb_description/meshes/base_v1/base.stl" />
                 </geometry>
-                <material name="body_sub" />
             </collision>
         </link>
@@ -158,5 +192,6 @@
                 <origin xyz="-0.01948200 0.00219100 0.07101300" />
                 <mass value="10.239419"/>
-                <inertia ixx="0.07671000"  ixy="-0.01005000"  ixz="0.00174900"
+                <inertia
+                    ixx="0.07671000"  ixy="-0.01005000"  ixz="0.00174900"
                     iyy="0.09057000" iyz="0.00154900" izz="0.14500000" />
             </inertial>
@@ -164,27 +199,23 @@
         <!-- wheels -->
         <xacro:hsrb_drive_wheel prefix="${prefix}" suffix="right" parent="${prefix}_roll_link">
-            <origin xyz="${drive_wheel_offset_x}
-                ${-drive_wheel_offset_y}
-                ${drive_wheel_radius}"
+            <origin
+                xyz="${drive_wheel_offset_x} ${-drive_wheel_offset_y} ${drive_wheel_radius}"
                 rpy="0.0 0.0 0.0" />
         </xacro:hsrb_drive_wheel>
         <xacro:hsrb_drive_wheel prefix="${prefix}" suffix="left" parent="${prefix}_roll_link">
-            <origin xyz="${drive_wheel_offset_x}
-                ${drive_wheel_offset_y}
-                ${drive_wheel_radius}"
+            <origin
+                xyz="${drive_wheel_offset_x} ${drive_wheel_offset_y} ${drive_wheel_radius}"
                 rpy="0.0 0.0 0.0" />
         </xacro:hsrb_drive_wheel>
-        <xacro:hsrb_passive_wheel prefix="${prefix}" suffix="right" parent="${prefix}_roll_link">
-            <origin xyz="${passive_wheel_offset_x}
-                ${-passive_wheel_offset_y}
-                ${passive_wheel_radius}"
-                rpy="0.0 0.0 0.0" />
-        </xacro:hsrb_passive_wheel>
-        <xacro:hsrb_passive_wheel prefix="${prefix}" suffix="left" parent="${prefix}_roll_link">
-            <origin xyz="${passive_wheel_offset_x}
-                ${passive_wheel_offset_y}
-                ${passive_wheel_radius}"
-                rpy="0.0 0.0 0.0" />
-        </xacro:hsrb_passive_wheel>
+        <xacro:hsrb_passive_caster prefix="${prefix}" suffix="right" parent="${prefix}_roll_link">
+            <origin
+                xyz="${passive_caster_offset_x} ${-passive_caster_offset_y} ${passive_caster_height}"
+                rpy="0.0 0.0 0.0" />
+        </xacro:hsrb_passive_caster>
+        <xacro:hsrb_passive_caster prefix="${prefix}" suffix="left" parent="${prefix}_roll_link">
+            <origin
+                xyz="${passive_caster_offset_x} ${passive_caster_offset_y} ${passive_caster_height}"
+                rpy="0.0 0.0 0.0" />
+        </xacro:hsrb_passive_caster>
         <!-- sensors -->
         <xacro:hokuyo_laser

File: tmc_hsrb_description/urdf/common.xacro (robot description, xacro)
@@ -30,4 +30,13 @@
     </gazebo>
   </macro>
+  <macro name="gazebo_link_flat_black" params="name gravity collide friction">
+    <gazebo reference="${name}">
+      <selfCollide>${collide}</selfCollide>
+      <gravity>${gravity}</gravity>
+      <mu1>${friction}</mu1>
+      <mu2>${friction}</mu2>
+      <material value="Gazebo/FlatBlack"/>
+    </gazebo>
+  </macro>
   <macro name="gazebo_link_rubber" params="name">
     <gazebo reference="${name}">

Commit message: 受動輪をキャスターから球に変更

File: tmc_hsrb_description/urdf/base_v1/base.gazebo.xacro (robot description, xacro)
@@ -9,10 +9,4 @@
         <gazebo_link_rubber name="${prefix}_right_passive_wheel_z_link"/>
         <gazebo_link_rubber name="${prefix}_left_passive_wheel_z_link"/>
-        <gazebo_link_flat_black name="${prefix}_right_passive_caster_roll_link" gravity="true" collide="false" friction="0.9"/>
-        <gazebo_link_rubber name="${prefix}_right_passive_caster_left_wheel_link"/>
-        <gazebo_link_rubber name="${prefix}_right_passive_caster_right_wheel_link"/>
-        <gazebo_link_flat_black name="${prefix}_left_passive_caster_roll_link" gravity="true" collide="false" friction="0.9"/>
-        <gazebo_link_rubber name="${prefix}_left_passive_caster_left_wheel_link"/>
-        <gazebo_link_rubber name="${prefix}_left_passive_caster_right_wheel_link"/>
         <gazebo_link name="${prefix}_range_sensor_link" gravity="true" collide="false" friction="0.9"/>
         <gazebo_link name="${prefix}_imu_sensor_link" gravity="true" collide="false" friction="0.9"/>

File: tmc_hsrb_description/urdf/base_v1/base.urdf.xacro (robot description, xacro)
@@ -10,9 +10,7 @@
     <xacro:property name="drive_wheel_offset_x" value="0.110" />
     <xacro:property name="drive_wheel_offset_y" value="0.133" />
-    <xacro:property name="passive_caster_height" value="0.058" />
-    <xacro:property name="passive_caster_radius" value="0.025" />
-    <xacro:property name="passive_caster_width" value="0.014" />
-    <xacro:property name="passive_caster_offset_x" value="0.1495" />
-    <xacro:property name="passive_caster_offset_y" value="0.055" />
+    <xacro:property name="passive_wheel_radius" value="0.03" />
+    <xacro:property name="passive_wheel_offset_x" value="0.1495" />
+    <xacro:property name="passive_wheel_offset_y" value="0.055" />
     <!-- drive wheel -->
     <xacro:macro name="hsrb_drive_wheel" params="prefix suffix parent *origin">
@@ -48,56 +46,14 @@
     </xacro:macro>
     <!-- passive wheel -->
-    <xacro:macro name="hsrb_passive_caster" params="prefix suffix parent *origin">
-        <joint name="${prefix}_${suffix}_passive_caster_roll_joint" type="continuous">
+    <xacro:macro name="hsrb_passive_wheel" params="prefix suffix parent *origin">
+        <joint name="${prefix}_${suffix}_passive_wheel_x_joint" type="continuous">
             <insert_block name="origin" />
-            <axis xyz="0.0 0.0 1.0" />
+            <axis xyz="1.0 0.0 0.0" />
             <limit effort="1000.0" velocity="100.0" />
             <parent link="${parent}" />
-            <child link="${prefix}_${suffix}_passive_caster_roll_link" />
-            <dynamics damping="0.7"/>
-        </joint>
-        <link name="${prefix}_${suffix}_passive_caster_roll_link">
-            <inertial>
-                <mass value="0.3"/>
-                <origin xyz="0 0 0"/>
-                <inertia ixx="0.001" ixy="0" ixz="0" iyy="0.001" iyz="0" izz="0.001"/>
-            </inertial>
-            <visual>
-                <origin xyz="0.0 0 -0.0165"/>
-                <geometry>
-                    <cylinder radius="0.0085" length="0.033"/>
-                </geometry>
-                <material name="wheel" />
-            </visual>
-            <visual>
-                <origin xyz="0.017 0.0 -0.033" rpy="1.57 0.0 0.0"/>
-                <geometry>
-                    <cylinder radius="0.02" length="0.021"/>
-                </geometry>
-                <material name="wheel" />
-            </visual>
-        </link>
-        <joint name="${prefix}_${suffix}_passive_caster_left_wheel_joint" type="continuous">
-            <origin xyz="0.017 0.0175 -0.033"/>
-            <axis xyz="0.0 1.0 0.0" />
-            <limit effort="1000.0" velocity="100.0" />
-            <parent link="${prefix}_${suffix}_passive_caster_roll_link" />
-            <child link="${prefix}_${suffix}_passive_caster_left_wheel_link" />
+            <child link="${prefix}_${suffix}_passive_wheel_x_frame" />
             <dynamics damping="1.0"/>
         </joint>
-        <link name="${prefix}_${suffix}_passive_caster_left_wheel_link">
-            <visual>
-                <origin rpy="1.57 0.0 0.0"/>
-                <geometry>
-                    <cylinder radius="${passive_caster_radius}" length="${passive_caster_width}"/>
-                </geometry>
-                <material name="wheel" />
-            </visual>
-            <collision>
-                <origin rpy="1.57 0.0 0.0"/>
-                <geometry>
-                    <cylinder radius="${passive_caster_radius}" length="${passive_caster_width}"/>
-                </geometry>
-            </collision>
+        <link name="${prefix}_${suffix}_passive_wheel_x_frame">
             <inertial>
                 <mass value="0.3"/>
@@ -106,24 +62,33 @@
             </inertial>
         </link>
-        <joint name="${prefix}_${suffix}_passive_caster_right_wheel_joint" type="continuous">
-            <origin xyz="0.017 -0.0175 -0.033"/>
+        <joint name="${prefix}_${suffix}_passive_wheel_y_joint" type="continuous">
             <axis xyz="0.0 1.0 0.0" />
             <limit effort="1000.0" velocity="100.0" />
-            <parent link="${prefix}_${suffix}_passive_caster_roll_link" />
-            <child link="${prefix}_${suffix}_passive_caster_right_wheel_link" />
-            <dynamics damping="1.0"/>
+            <parent link="${prefix}_${suffix}_passive_wheel_x_frame" />
+            <child link="${prefix}_${suffix}_passive_wheel_y_frame" />
         </joint>
-        <link name="${prefix}_${suffix}_passive_caster_right_wheel_link">
+        <link name="${prefix}_${suffix}_passive_wheel_y_frame">
+            <inertial>
+                <mass value="0.3"/>
+                <origin xyz="0 0 0"/>
+                <inertia ixx="0.001" ixy="0" ixz="0" iyy="0.001" iyz="0" izz="0.001"/>
+            </inertial>
+        </link>
+        <joint name="${prefix}_${suffix}_passive_wheel_z_joint" type="continuous">
+            <axis xyz="0.0 0.0 1.0" />
+            <limit effort="1000.0" velocity="100.0" />
+            <parent link="${prefix}_${suffix}_passive_wheel_y_frame" />
+            <child link="${prefix}_${suffix}_passive_wheel_z_link" />
+        </joint>
+        <link name="${prefix}_${suffix}_passive_wheel_z_link">
             <visual>
-                <origin rpy="1.57 0.0 0.0"/>
                 <geometry>
-                    <cylinder radius="${passive_caster_radius}" length="${passive_caster_width}"/>
+                    <sphere radius="${passive_wheel_radius}" />
                 </geometry>
                 <material name="wheel" />
             </visual>
             <collision>
-                <origin rpy="1.57 0.0 0.0"/>
                 <geometry>
-                    <cylinder radius="${passive_caster_radius}" length="${passive_caster_width}"/>
+                    <sphere radius="${passive_wheel_radius}" />
                 </geometry>
                 <material name="wheel" />
@@ -208,15 +173,16 @@
                 rpy="0.0 0.0 0.0" />
         </xacro:hsrb_drive_wheel>
-        <xacro:hsrb_passive_caster prefix="${prefix}" suffix="right" parent="${prefix}_roll_link">
-            <origin
-                xyz="${passive_caster_offset_x} ${-passive_caster_offset_y} ${passive_caster_height}"
+        <xacro:hsrb_passive_wheel prefix="${prefix}" suffix="right" parent="${prefix}_roll_link">
+            <origin xyz="${passive_wheel_offset_x}
+                ${-passive_wheel_offset_y}
+                ${passive_wheel_radius}"
                 rpy="0.0 0.0 0.0" />
-        </xacro:hsrb_passive_caster>
-        <xacro:hsrb_passive_caster prefix="${prefix}" suffix="left" parent="${prefix}_roll_link">
-            <origin
-                xyz="${passive_caster_offset_x} ${passive_caster_offset_y} ${passive_caster_height}"
+        </xacro:hsrb_passive_wheel>
+        <xacro:hsrb_passive_wheel prefix="${prefix}" suffix="left" parent="${prefix}_roll_link">
+            <origin xyz="${passive_wheel_offset_x}
+                ${passive_wheel_offset_y}
+                ${passive_wheel_radius}"
                 rpy="0.0 0.0 0.0" />
-        </xacro:hsrb_passive_caster>
-        <!-- sensors -->
+        </xacro:hsrb_passive_wheel>
         <xacro:hokuyo_laser
             prefix="${prefix}"
