Commit message: Fix passive caster tread value.

File: tmc_hsrb_description/urdf/base_v1/base.urdf.xacro (robot description, xacro)
@@ -8,5 +8,5 @@
     <xacro:property name="drive_wheel_width" value="0.03" />
     <xacro:property name="drive_wheel_radius" value="0.040" />
-    <xacro:property name="drive_wheel_offset_x" value="-0.110" />
+    <xacro:property name="drive_wheel_offset_x" value="0.110" />
     <xacro:property name="drive_wheel_offset_y" value="0.133" />
     <xacro:property name="passive_caster_height" value="0.058" />
@@ -14,5 +14,5 @@
     <xacro:property name="passive_caster_width" value="0.014" />
     <xacro:property name="passive_caster_offset_x" value="0.1495" />
-    <xacro:property name="passive_caster_offset_y" value="0.11" />
+    <xacro:property name="passive_caster_offset_y" value="0.055" />
     <!-- drive wheel -->
     <xacro:macro name="hsrb_drive_wheel" params="prefix suffix parent *origin">
@@ -200,10 +200,10 @@
         <xacro:hsrb_drive_wheel prefix="${prefix}" suffix="right" parent="${prefix}_roll_link">
             <origin
-                xyz="${drive_wheel_offset_x} ${-drive_wheel_offset_y} ${drive_wheel_radius}"
+                xyz="${-drive_wheel_offset_x} ${-drive_wheel_offset_y} ${drive_wheel_radius}"
                 rpy="0.0 0.0 0.0" />
         </xacro:hsrb_drive_wheel>
         <xacro:hsrb_drive_wheel prefix="${prefix}" suffix="left" parent="${prefix}_roll_link">
             <origin
-                xyz="${drive_wheel_offset_x} ${drive_wheel_offset_y} ${drive_wheel_radius}"
+                xyz="${-drive_wheel_offset_x} ${drive_wheel_offset_y} ${drive_wheel_radius}"
                 rpy="0.0 0.0 0.0" />
         </xacro:hsrb_drive_wheel>

Commit message: beetle3号機用にモデルファイルを修正
base,body,laserモデルを新規作成
すべてのvisualモデルをシェーディング

File: tmc_hsrb_description/urdf/base_v1/base.urdf.xacro (robot description, xacro)
@@ -152,5 +152,5 @@
             <visual>
                 <geometry>
-                    <mesh filename="package://tmc_hsrb_description/meshes/base_v1/body.dae" />
+                    <mesh filename="package://tmc_hsrb_description/meshes/base_v1/body_light.dae" />
                 </geometry>
                 <material name="body_main" />

Commit message: Decrease base wheel torque limit

File: tmc_hsrb_description/urdf/base_v1/base.urdf.xacro (robot description, xacro)
@@ -18,5 +18,5 @@
             <insert_block name="origin" />
             <axis xyz="0.0 1.0 0.0" />
-            <limit effort="1000.0" velocity="10.0" />
+            <limit effort="10.0" velocity="10.0" />
             <parent link="${parent}" />
             <child link="${prefix}_${suffix}_drive_wheel_link" />
@@ -50,5 +50,5 @@
             <insert_block name="origin" />
             <axis xyz="1.0 0.0 0.0" />
-            <limit effort="1000.0" velocity="100.0" />
+            <limit effort="100.0" velocity="100.0" />
             <parent link="${parent}" />
             <child link="${prefix}_${suffix}_passive_wheel_x_frame" />
@@ -64,5 +64,5 @@
         <joint name="${prefix}_${suffix}_passive_wheel_y_joint" type="continuous">
             <axis xyz="0.0 1.0 0.0" />
-            <limit effort="1000.0" velocity="100.0" />
+            <limit effort="100.0" velocity="20.0" />
             <parent link="${prefix}_${suffix}_passive_wheel_x_frame" />
             <child link="${prefix}_${suffix}_passive_wheel_y_frame" />
@@ -77,5 +77,5 @@
         <joint name="${prefix}_${suffix}_passive_wheel_z_joint" type="continuous">
             <axis xyz="0.0 0.0 1.0" />
-            <limit effort="1000.0" velocity="100.0" />
+            <limit effort="1000.0" velocity="20.0" />
             <parent link="${prefix}_${suffix}_passive_wheel_y_frame" />
             <child link="${prefix}_${suffix}_passive_wheel_z_link" />
@@ -142,5 +142,5 @@
             <origin xyz="0.0 0.0 0.0" rpy="0.0 0.0 0.0" />
             <axis xyz="0.0 0.0 1.0" />
-            <limit effort="1000.0" velocity="1.0" />
+            <limit effort="100.0" velocity="10.0" />
             <parent link="${prefix}_link" />
             <child link="${prefix}_roll_link" />
