Commit message: Update hand joint name

File: tmc_hsrb_description/urdf/hand_v0/hand.gazebo.xacro (robot description, xacro)
@@ -4,5 +4,5 @@
         <gazebo_link name="${prefix}_palm_link" gravity="true" collide="false" friction="0.9"/>
         <gazebo_link name="${prefix}_camera_link" gravity="true" collide="false" friction="0.9"/>
-        <gazebo_link name="${prefix}_l_actuated_proximal_link" gravity="true" collide="false" friction="1.0"/>
+        <gazebo_link name="${prefix}_l_proximal_link" gravity="true" collide="false" friction="1.0"/>
         <gazebo_link name="${prefix}_l_spring_proximal_link" gravity="true" collide="false" friction="1.0"/>
         <gazebo_link name="${prefix}_l_mimic_link" gravity="true" collide="false" friction="1.0"/>
@@ -10,5 +10,5 @@
         <gazebo_link name="${prefix}_l_finger_tip_frame" gravity="true" collide="false" friction="1.0"/>
         <gazebo_link name="${prefix}_l_finger_vacuum_frame" gravity="true" collide="false" friction="1.0"/>
-        <gazebo_link name="${prefix}_r_actuated_proximal_link" gravity="true" collide="false" friction="1.0"/>
+        <gazebo_link name="${prefix}_r_proximal_link" gravity="true" collide="false" friction="1.0"/>
         <gazebo_link name="${prefix}_r_spring_proximal_link" gravity="true" collide="false" friction="1.0"/>
         <gazebo_link name="${prefix}_r_mimic_link" gravity="true" collide="false" friction="1.0"/>
@@ -18,9 +18,9 @@
         <gazebo_joint name="${prefix}_palm_joint"/>
         <gazebo_joint name="${prefix}_motor_joint"/>
-        <gazebo_joint name="${prefix}_l_actuated_proximal_joint"/>
+        <gazebo_joint name="${prefix}_l_proximal_joint"/>
         <gazebo_joint name="${prefix}_l_spring_proximal_joint"/>
         <gazebo_joint name="${prefix}_l_mimic_distal_joint"/>
         <gazebo_joint name="${prefix}_l_distal_joint"/>
-        <gazebo_joint name="${prefix}_r_actuated_proximal_joint"/>
+        <gazebo_joint name="${prefix}_r_proximal_joint"/>
         <gazebo_joint name="${prefix}_r_spring_proximal_joint"/>
         <gazebo_joint name="${prefix}_r_mimic_distal_joint"/>

File: tmc_hsrb_description/urdf/hand_v0/hand.transmission.xacro (robot description, xacro)
@@ -3,9 +3,9 @@
     <xacro:macro name="hsrb_hand_transmission" params="prefix">
         <hsrb_effort_joint_transmission joint="${prefix}_motor_joint" reduction="1"/>
-        <hsrb_effort_joint_transmission joint="${prefix}_l_actuated_proximal_joint" reduction="1"/>
+        <hsrb_effort_joint_transmission joint="${prefix}_l_proximal_joint" reduction="1"/>
         <hsrb_effort_joint_transmission joint="${prefix}_l_spring_proximal_joint" reduction="1"/>
         <hsrb_effort_joint_transmission joint="${prefix}_l_mimic_distal_joint" reduction="1"/>
         <hsrb_effort_joint_transmission joint="${prefix}_l_distal_joint" reduction="1"/>
-        <hsrb_effort_joint_transmission joint="${prefix}_r_actuated_proximal_joint" reduction="1"/>
+        <hsrb_effort_joint_transmission joint="${prefix}_r_proximal_joint" reduction="1"/>
         <hsrb_effort_joint_transmission joint="${prefix}_r_spring_proximal_joint" reduction="1"/>
         <hsrb_effort_joint_transmission joint="${prefix}_r_mimic_distal_joint" reduction="1"/>

File: tmc_hsrb_description/urdf/hand_v0/hand.urdf.xacro (robot description, xacro)
@@ -9,6 +9,6 @@
     <xacro:property name="base_joint_angle_range_min" value="-0.1" />
     <xacro:property name="base_joint_angle_range_max" value="1.24" />
-    <xacro:property name="actuated_proximal_joint_angle_range_min" value="-0.1" />
-    <xacro:property name="actuated_proximal_joint_angle_range_max" value="1.24" />
+    <xacro:property name="proximal_joint_angle_range_min" value="-0.1" />
+    <xacro:property name="proximal_joint_angle_range_max" value="1.24" />
     <xacro:property name="spring_proximal_joint_angle_range_min" value="0.0" />
     <xacro:property name="spring_proximal_joint_angle_range_max" value="0.698" />
@@ -55,6 +55,6 @@
             <axis xyz="1.0 0.0 0.0" />
             <limit effort="100.0" velocity="1.0"
-                lower="${actuated_proximal_joint_angle_range_min}"
-                upper="${actuated_proximal_joint_angle_range_max}" />
+                lower="${proximal_joint_angle_range_min}"
+                upper="${proximal_joint_angle_range_max}" />
             <parent link="${prefix}_palm_link" />
             <child link="${prefix}_motor_frame" />
@@ -85,17 +85,17 @@
     <!-- gripper finger proximal base -->
     <xacro:macro name="hsrb_finger_proximal_base" params="prefix suffix parent *origin *axis">
-        <joint name="${prefix}_${suffix}_actuated_proximal_joint" type="revolute">
-            <insert_block name="origin" />
-            <insert_block name="axis" />
-            <limit effort="100.0" velocity="1.0"
-                lower="${actuated_proximal_joint_angle_range_min}"
-                upper="${actuated_proximal_joint_angle_range_max}" />
+        <joint name="${prefix}_${suffix}_proximal_joint" type="revolute">
+            <insert_block name="origin" />
+            <insert_block name="axis" />
+            <limit effort="100.0" velocity="1.0"
+                lower="${proximal_joint_angle_range_min}"
+                upper="${proximal_joint_angle_range_max}" />
             <parent link="${parent}" />
-            <child link="${prefix}_${suffix}_actuated_proximal_link" />
+            <child link="${prefix}_${suffix}_proximal_link" />
             <mimic joint="${prefix}_motor_joint" />
             <dynamics damping="1.0"/>
         </joint>
         <!-- dummy link -->
-        <xacro:hsrb_gripper_dummy_link name="${prefix}_${suffix}_actuated_proximal_link" />
+        <xacro:hsrb_gripper_dummy_link name="${prefix}_${suffix}_proximal_link" />
         <joint name="${prefix}_${suffix}_spring_proximal_joint" type="revolute">
             <insert_block name="axis" />
@@ -103,5 +103,5 @@
                 lower="${spring_proximal_joint_angle_range_min}"
                 upper="${spring_proximal_joint_angle_range_max}" />
-            <parent link="${prefix}_${suffix}_actuated_proximal_link" />
+            <parent link="${prefix}_${suffix}_proximal_link" />
             <child link="${prefix}_${suffix}_spring_proximal_link" />
             <dynamics damping="1.0"/>
@@ -126,6 +126,6 @@
             <insert_block name="axis" />
             <limit effort="100.0" velocity="1.0"
-                lower="${-actuated_proximal_joint_angle_range_max}"
-                upper="${-actuated_proximal_joint_angle_range_min}" />
+                lower="${-proximal_joint_angle_range_max}"
+                upper="${-proximal_joint_angle_range_min}" />
             <parent link="${prefix}_${suffix}_mimic_distal_link" />
             <child link="${prefix}_${suffix}_distal_link" />
