Commit message: Replace invalid inertia tensor with correct parameters.

File: tmc_hsrb_description/urdf/hand_v0/hand.urdf.xacro (robot description, xacro)
@@ -180,6 +180,7 @@
                 <mass value="0.020927"/>
                 <origin xyz="0.014256 -0.008321 0.015591"/>
-                <inertia ixx="0.00000307518" ixy="0.000004176168" ixz="0.000002877537"
-                    iyy="-0.000000049953" iyz="0.000000010237" izz="0.000000866222"/>
+                <inertia ixx="0.00000307518" ixy="-0.00000004954" ixz="0.000000009481"
+                                             iyy="0.000004074079" iyz="0.000000843648"
+                                                                  izz="0.000002807795"/>
             </inertial>
             <visual>

Commit message: Fix review points

File: tmc_hsrb_description/urdf/hand_v0/hand.urdf.xacro (robot description, xacro)
@@ -21,5 +21,5 @@
                 <inertia
                     ixx="0.01" ixy="0.0" ixz="0.0"
-                        iyy="0.01" iyz="0.0" izz="0.01"/>
+                    iyy="0.01" iyz="0.0" izz="0.01"/>
             </inertial>
         </link>
@@ -35,6 +35,7 @@
             <inertial>
                 <mass value="0.1"/>
-                <inertia ixx="0.01" ixy="0.0" ixz="0.0"
-                         iyy="0.01" iyz="0.0" izz="0.01"/>
+                <inertia
+                    ixx="0.01" ixy="0.0" ixz="0.0"
+                    iyy="0.01" iyz="0.0" izz="0.01"/>
             </inertial>
             <visual>
@@ -138,5 +139,6 @@
                 <mass value="0.043589"/>
                 <origin xyz="0.021418 0.00248 0.022688"/>
-                <inertia ixx="0.000026033886" ixy="-0.000000144078" ixz="-0.00000198241"
+                <inertia
+                    ixx="0.000026033886" ixy="-0.000000144078" ixz="-0.00000198241"
                     iyy="0.000028824811" iyz="-0.000001268421" izz="0.000005135919"/>
             </inertial>
@@ -162,5 +164,6 @@
                 <mass value="0.027731"/>
                 <origin xyz="0.011116 0.005679 0.017532"/>
-                <inertia ixx="0.000004451952" ixy="-0.000000617574" ixz="0.000000503765"
+                <inertia
+                    ixx="0.000004451952" ixy="-0.000000617574" ixz="0.000000503765"
                     iyy="0.000000503765" iyz="-0.000000435048" izz="0.000004456764"/>
             </inertial>
@@ -194,5 +197,5 @@
                 <inertia
                     ixx="0.01" ixy="0.0" ixz="0.0"
-                        iyy="0.01" iyz="0.0" izz="0.01"/>
+                    iyy="0.01" iyz="0.0" izz="0.01"/>
             </inertial>
             <visual>
@@ -242,6 +245,5 @@
                 <inertia
                     ixx="0.00000307518" ixy="-0.00000004954" ixz="0.000000009481"
-                    iyy="0.000004074079" iyz="0.000000843648"
-                    izz="0.000002807795"/>
+                    iyy="0.000004074079" iyz="0.000000843648" izz="0.000002807795"/>
             </inertial>
             <visual>

Commit message: Add damping parameter to hand joints.

File: tmc_hsrb_description/urdf/hand_v0/hand.urdf.xacro (robot description, xacro)
@@ -59,4 +59,5 @@
             <parent link="${prefix}_palm_link" />
             <child link="${prefix}_motor_link" />
+            <dynamics damping="1.0"/>
         </joint>
         <!-- dummy link -->
@@ -93,4 +94,5 @@
             <child link="${prefix}_${suffix}_actuated_proximal_link" />
             <mimic joint="${prefix}_motor_joint" />
+            <dynamics damping="1.0"/>
         </joint>
         <!-- dummy link -->
@@ -103,4 +105,5 @@
             <parent link="${prefix}_${suffix}_actuated_proximal_link" />
             <child link="${prefix}_${suffix}_spring_proximal_link" />
+            <dynamics damping="1.0"/>
         </joint>
     </xacro:macro>
@@ -116,4 +119,5 @@
             <child link="${prefix}_${suffix}_mimic_distal_link" />
             <mimic joint="${prefix}_${suffix}_spring_proximal_joint" multiplier="-1.0" />
+            <dynamics damping="1.0"/>
         </joint>
         <!-- dummy link -->
@@ -127,4 +131,5 @@
             <child link="${prefix}_${suffix}_distal_link" />
             <mimic joint="${prefix}_motor_joint" multiplier="-1.0" offset="${-distal_joint_angle_offset}"/>
+            <dynamics damping="1.0"/>
         </joint>
     </xacro:macro>

Commit message: ハンドの可動域変更

File: tmc_hsrb_description/urdf/hand_v0/hand.urdf.xacro (robot description, xacro)
@@ -7,7 +7,5 @@
     <xacro:property name="palm_to_proximal_y" value="-0.0245" />
     <xacro:property name="palm_to_proximal_z" value="-0.0175" />
-    <xacro:property name="base_joint_angle_range_min" value="-0.1" />
-    <xacro:property name="base_joint_angle_range_max" value="1.24" />
-    <xacro:property name="proximal_joint_angle_range_min" value="-0.1" />
+    <xacro:property name="proximal_joint_angle_range_min" value="-0.798" />
     <xacro:property name="proximal_joint_angle_range_max" value="1.24" />
     <xacro:property name="spring_proximal_joint_angle_range_min" value="0.0" />
