Commit message: Rollback hand motor joint
hand_motor_frame_joint -> hand_motor_joint

File: tmc_hsrb_description/urdf/hand_v0/hand.transmission.xacro (robot description, xacro)
@@ -2,5 +2,5 @@
 <robot xmlns:xacro="http://www.ros.org/wiki.xacro">
     <xacro:macro name="hsrb_hand_transmission" params="prefix">
-        <hsrb_effort_joint_transmission joint="${prefix}_motor_frame_joint" reduction="1"/>
+        <hsrb_effort_joint_transmission joint="${prefix}_motor_joint" reduction="1"/>
         <hsrb_effort_joint_transmission joint="${prefix}_l_proximal_joint" reduction="1"/>
         <hsrb_effort_joint_transmission joint="${prefix}_l_spring_proximal_joint" reduction="1"/>

File: tmc_hsrb_description/urdf/hand_v0/hand.urdf.xacro (robot description, xacro)
@@ -50,5 +50,5 @@
             </collision>
         </link>
-        <joint name="${prefix}_motor_frame_joint" type="revolute">
+        <joint name="${prefix}_motor_joint" type="revolute">
             <axis xyz="1.0 0.0 0.0" />
             <limit effort="100.0" velocity="1.0"
@@ -56,9 +56,9 @@
                 upper="${proximal_joint_angle_range_max}" />
             <parent link="${prefix}_palm_link" />
-            <child link="${prefix}_motor_frame" />
+            <child link="${prefix}_motor_dummy_link" />
             <dynamics damping="1.0"/>
         </joint>
         <!-- dummy link -->
-        <xacro:hsrb_gripper_dummy_link name="${prefix}_motor_frame" />
+        <xacro:hsrb_gripper_dummy_link name="${prefix}_motor_dummy_link" />
     </xacro:macro>
     <xacro:macro name="hsrb_hand" params="prefix parent *origin">
@@ -91,5 +91,5 @@
             <parent link="${parent}" />
             <child link="${prefix}_${suffix}_proximal_link" />
-            <mimic joint="${prefix}_motor_frame_joint" />
+            <mimic joint="${prefix}_motor_joint" />
             <dynamics damping="1.0"/>
         </joint>
@@ -128,5 +128,5 @@
             <parent link="${prefix}_${suffix}_mimic_distal_link" />
             <child link="${prefix}_${suffix}_distal_link" />
-            <mimic joint="${prefix}_motor_frame_joint" multiplier="-1.0" offset="${-distal_joint_angle_offset}"/>
+            <mimic joint="${prefix}_motor_joint" multiplier="-1.0" offset="${-distal_joint_angle_offset}"/>
             <dynamics damping="1.0"/>
         </joint>
@@ -189,5 +189,5 @@
             <child link="${prefix}_${suffix}_finger_tip_frame" />
         </joint>
-        <xacro:hsrb_gripper_dummy_link name="${prefix}_${suffix}_finger_tip_frame" />
+        <link name="${prefix}_${suffix}_finger_tip_frame" />
         <joint name="${prefix}_${suffix}_finger_vacuum_frame_joint" type="fixed">
             <origin xyz="0.00475 -0.011539 0.03322" rpy="${pi/4.0} 0.0 0.0" />
@@ -268,5 +268,5 @@
             <child link="${prefix}_${suffix}_finger_tip_frame" />
         </joint>
-        <xacro:hsrb_gripper_dummy_link name="${prefix}_${suffix}_finger_tip_frame" />
+        <link name="${prefix}_${suffix}_finger_tip_frame" />
     </xacro:macro>
 </robot>
