Commit message: Update topic/service/tf names

File: tmc_hsrb_description/urdf/head_v0/head.urdf.xacro (robot description, xacro)
@@ -98,5 +98,5 @@
             <origin xyz="0.0195 0.0 0.061" rpy="0 0 0"/>
         </xacro:wide_camera>
-        <xacro:asus_xtion prefix="${prefix}" parent="${prefix}_tilt_link" robot_namespace="${robot_name}">
+        <xacro:asus_xtion prefix="${prefix}_" parent="${prefix}_tilt_link" robot_namespace="${robot_name}" sensor_name="rgbd_sensor">
             <origin xyz="-0.079796 0.022 0.215172" rpy="0 0 0"/>
         </xacro:asus_xtion>

File: tmc_hsrb_description/urdf/sensors/asus_xtion.gazebo.xacro (robot description, xacro)
@@ -16,5 +16,5 @@
     <xacro:property name="XtionMaxDistance" value="5"/>
     <xacro:property name="XtionFrameRate" value="30"/>
-    <xacro:macro name="depth_camera_gazebo" params="robot_namespace sensor_name parent_camera_link parent_depth_link">
+    <xacro:macro name="asus_xtion_gazebo" params="robot_namespace sensor_name parent_camera_link parent_depth_link">
         <gazebo reference="${parent_camera_link}">
             <sensor type="depth" name="openni_camera_camera">
@@ -35,16 +35,16 @@
                 </camera>
                 <plugin name="camera_controller" filename="libgazebo_ros_openni_kinect.so">
-                    <robotNamespace>${robot_namespace}</robotNamespace>
                     <alwaysOn>true</alwaysOn>
-                    <updateRate>10.0</updateRate>
+                    <baseline>0.2</baseline>
+                    <updateRate>1.0</updateRate>
                     <cameraName>${sensor_name}</cameraName>
                     <frameName>${parent_depth_link}</frameName>
-                    <imageTopicName>rgb/image_raw</imageTopicName>
-                    <depthImageTopicName>depth/image_raw</depthImageTopicName>
-                    <pointCloudTopicName>depth/points</pointCloudTopicName>
-                    <cameraInfoTopicName>rgb/camera_info</cameraInfoTopicName>
-                    <depthImageCameraInfoTopicName>depth/camera_info</depthImageCameraInfoTopicName>
-                    <pointCloudCutoff>0.4</pointCloudCutoff>
-                    <hackBaseline>0.0</hackBaseline>
+                    <imageTopicName>/${robot_namespace}/${sensor_name}/rgb/image_raw</imageTopicName>
+                    <cameraInfoTopicName>/${robot_namespace}/${sensor_name}/rgb/camera_info</cameraInfoTopicName>
+                    <depthImageTopicName>/${robot_namespace}/${sensor_name}/depth/image_raw</depthImageTopicName>
+                    <pointCloudTopicName>/${robot_namespace}/${sensor_name}/depth/points</pointCloudTopicName>
+                    <depthImageCameraInfoTopicName>/${robot_namespace}/${sensor_name}/depth/camera_info</depthImageCameraInfoTopicName>
+                    <pointCloudCutoff>0.5</pointCloudCutoff>
+                    <pointCloudCutoffMax>9.2</pointCloudCutoffMax>
                     <distortionK1>0.0</distortionK1>
                     <distortionK2>0.0</distortionK2>
@@ -56,4 +56,5 @@
                     <Cy>0.0</Cy>
                     <focalLength>0.0</focalLength>
+                    <hackBaseline>0</hackBaseline>
                 </plugin>
             </sensor>

File: tmc_hsrb_description/urdf/sensors/asus_xtion.urdf.xacro (robot description, xacro)
@@ -3,11 +3,11 @@
     <xacro:include filename="$(find tmc_hsrb_description)/urdf/sensors/asus_xtion.gazebo.xacro"/>
     <!-- rgbd_sensor -->
-    <xacro:macro name="asus_xtion" params="prefix parent robot_namespace *origin">
-        <joint name="${prefix}_rgbd_sensor_joint" type="fixed">
+    <xacro:macro name="asus_xtion" params="prefix parent robot_namespace sensor_name *origin">
+        <joint name="${prefix}${sensor_name}_joint" type="fixed">
             <insert_block name="origin" />
             <parent link="${parent}"/>
-            <child link="${prefix}_rgbd_sensor_link"/>
+            <child link="${prefix}${sensor_name}_link"/>
         </joint>
-        <link name="${prefix}_rgbd_sensor_link">
+        <link name="${prefix}${sensor_name}_link">
             <visual>
                 <origin xyz="0 0 0" rpy="${-pi/2.0} 0.0 ${-pi/2.0}"/>
@@ -25,16 +25,16 @@
             </collision>
         </link>
-        <joint name="${prefix}_rgbd_sensor_pointcloud_frame_joint" type="fixed">
+        <joint name="${prefix}${sensor_name}_pointcloud_frame_joint" type="fixed">
             <origin xyz="0 0 0" rpy="${-pi/2.0} 0.0 ${-pi/2.0}"/>
-            <parent link="${prefix}_rgbd_sensor_link"/>
-            <child link="${prefix}_rgbd_sensor_pointcloud_frame"/>
+            <parent link="${prefix}${sensor_name}_link"/>
+            <child link="${prefix}${sensor_name}_pointcloud_frame"/>
         </joint>
         `
-        <link name="${prefix}_rgbd_sensor_pointcloud_frame"></link>
-        <xacro:rgbd_sensor_gazebo
+        <link name="${prefix}${sensor_name}_pointcloud_frame"></link>
+        <xacro:asus_xtion_gazebo
             robot_namespace="${robot_namespace}"
-            sensor_name="${prefix}_rgbd_sensor"
-            parent_camera_link="${prefix}_rgbd_sensor_link"
-            parent_depth_link="${prefix}_rgbd_sensor_pointcloud_frame"/>
+            sensor_name="${sensor_name}"
+            parent_camera_link="${prefix}${sensor_name}_link"
+            parent_depth_link="${prefix}${sensor_name}_pointcloud_frame"/>
     </xacro:macro>
 </robot>

File: tmc_hsrb_description/urdf/sensors/hokuyo_laser.gazebo.xacro (robot description, xacro)
@@ -23,6 +23,5 @@
                 </ray>
                 <plugin name="hokuyo_laser" filename="libgazebo_ros_gpu_laser.so">
-                    <robotNamespace>${robot_namespace}</robotNamespace>
-                    <topicName>${ros_topic}</topicName>
+                    <topicName>${robot_namespace}/${ros_topic}</topicName>
                     <frameName>${frame_name}</frameName>
                 </plugin>

File: tmc_hsrb_description/urdf/sensors/imu.gazebo.xacro (robot description, xacro)
@@ -27,6 +27,6 @@
             <plugin name="imu_plugin" filename="libgazebo_ros_imu.so">
                 <imuName>${sensor_name}</imuName>
-                <topicName>${sensor_name}</topicName>
-                <serviceName>${sensor_name}</serviceName>
+                <topicName>${sensor_name}/data</topicName>
+                <serviceName>${sensor_name}/calibrate</serviceName>
                 <frameName>${frame_name}</frameName>
                 <bodyName>base_link</bodyName>

Commit message: change robot model.
- comply with proposal3001.

File: tmc_hsrb_description/urdf/head_v0/head.urdf.xacro (robot description, xacro)
@@ -90,14 +90,14 @@
         <!-- cameras -->
         <xacro:pointgrey_chameleon prefix="${prefix}_l_stereo" parent="${prefix}_tilt_link" robot_namespace="${robot_name}">
-            <origin xyz="0.02 0.07 0.061" rpy="0 0 0"/>
+            <origin xyz="0.02 0.07 0.061" rpy="${-pi/2.0} 0.0 ${-pi/2.0}"/>
         </xacro:pointgrey_chameleon>
         <xacro:pointgrey_chameleon prefix="${prefix}_r_stereo" parent="${prefix}_tilt_link" robot_namespace="${robot_name}">
-            <origin xyz="0.02 -0.07 0.061" rpy="0 0 0"/>
+            <origin xyz="0.02 -0.07 0.061" rpy="${-pi/2.0} 0.0 ${-pi/2.0}"/>
         </xacro:pointgrey_chameleon>
         <xacro:wide_camera prefix="${prefix}_center" parent="${prefix}_tilt_link" robot_namespace="${robot_name}">
-            <origin xyz="0.0195 0.0 0.061" rpy="0 0 0"/>
+            <origin xyz="0.0195 0.0 0.061" rpy="${-pi/2.0} 0.0 ${-pi/2.0}"/>
         </xacro:wide_camera>
-        <xacro:asus_xtion prefix="${prefix}_" parent="${prefix}_tilt_link" robot_namespace="${robot_name}" sensor_name="rgbd_sensor">
-            <origin xyz="-0.079796 0.022 0.215172" rpy="0 0 0"/>
+        <xacro:asus_xtion prefix="${prefix}" parent="${prefix}_tilt_link" robot_namespace="${robot_name}">
+            <origin xyz="-0.079796 0.022 0.215172" rpy="${-pi/2.0} 0.0 ${-pi/2.0}"/>
         </xacro:asus_xtion>
         <xacro:hsrb_head_gazebo prefix="${prefix}"/>

File: tmc_hsrb_description/urdf/sensors/asus_xtion.urdf.xacro (robot description, xacro)
@@ -11,5 +11,5 @@
         <link name="${prefix}${sensor_name}_link">
             <visual>
-                <origin xyz="0 0 0" rpy="${-pi/2.0} 0.0 ${-pi/2.0}"/>
+                <origin xyz="0 0 0" rpy="0.0 0.0 0.0"/>
                 <geometry>
                     <mesh filename="package://tmc_hsrb_description/meshes/sensors/xtion.dae" />
@@ -18,5 +18,5 @@
             </visual>
             <collision>
-                <origin xyz="0 0 0" rpy="${-pi/2.0} 0.0 ${-pi/2.0}"/>
+                <origin xyz="0 0 0" rpy="0.0 0.0 0.0"/>
                 <geometry>
                     <mesh filename="package://tmc_hsrb_description/meshes/sensors/xtion.stl" />
@@ -25,8 +25,8 @@
             </collision>
         </link>
-        <joint name="${prefix}${sensor_name}_pointcloud_frame_joint" type="fixed">
-            <origin xyz="0 0 0" rpy="${-pi/2.0} 0.0 ${-pi/2.0}"/>
-            <parent link="${prefix}${sensor_name}_link"/>
-            <child link="${prefix}${sensor_name}_pointcloud_frame"/>
+        <joint name="${prefix}_rgbd_sensor_pointcloud_frame_joint" type="fixed">
+            <origin xyz="0 0 0" rpy="0.0 0.0 0.0"/>
+            <parent link="${prefix}_rgbd_sensor_link"/>
+            <child link="${prefix}_rgbd_sensor_pointcloud_frame"/>
         </joint>
         `

File: tmc_hsrb_description/urdf/sensors/pointgrey_chameleon.urdf.xacro (robot description, xacro)
@@ -10,5 +10,5 @@
         <link name="${prefix}_camera_link">
             <visual>
-                <origin xyz="0 0 0" rpy="${-pi/2.0} 0.0 ${-pi/2.0}"/>
+                <origin xyz="0 0 0" rpy="0.0 0.0 0.0"/>
                 <geometry>
                     <mesh filename="package://tmc_hsrb_description/meshes/sensors/head_camera.dae" />
