Commit message: fixed bad parameter of asus_xtion.urdf.xacro

File: tmc_hsrb_description/urdf/sensors/asus_xtion.urdf.xacro (robot description, xacro)
@@ -4,10 +4,10 @@
     <!-- rgbd_sensor -->
     <xacro:macro name="asus_xtion" params="prefix parent robot_namespace sensor_name *origin">
-        <joint name="${prefix}${sensor_name}_joint" type="fixed">
+        <joint name="${prefix}_${sensor_name}_joint" type="fixed">
             <insert_block name="origin" />
             <parent link="${parent}"/>
-            <child link="${prefix}${sensor_name}_link"/>
+            <child link="${prefix}_${sensor_name}_link"/>
         </joint>
-        <link name="${prefix}${sensor_name}_link">
+        <link name="${prefix}_${sensor_name}_link">
             <visual>
                 <origin xyz="0 0 0" rpy="0.0 0.0 0.0"/>
@@ -31,10 +31,10 @@
         </joint>
         `
-        <link name="${prefix}${sensor_name}_pointcloud_frame"></link>
+        <link name="${prefix}_${sensor_name}_pointcloud_frame"></link>
         <xacro:asus_xtion_gazebo
             robot_namespace="${robot_namespace}"
             sensor_name="${sensor_name}"
-            parent_camera_link="${prefix}${sensor_name}_link"
-            parent_depth_link="${prefix}${sensor_name}_pointcloud_frame"/>
+            parent_camera_link="${prefix}_${sensor_name}_link"
+            parent_depth_link="${prefix}_${sensor_name}_pointcloud_frame"/>
     </xacro:macro>
 </robot>
