Commit message: modified limits of wrist roll joint

File: tmc_hsrb_description/urdf/wrist_v0/wrist.urdf.xacro (robot description, xacro)
@@ -45,5 +45,5 @@
             <origin xyz="0.0 0.0 0.0" rpy="0.0 0.0 0.0" />
             <axis xyz="0.0 0.0 1.0" />
-            <limit effort="100.0" velocity="1.5" lower="-3.84" upper="2.09" />
+            <limit effort="100.0" velocity="1.5" lower="-1.92" upper="3.67" />
             <parent link="${prefix}_flex_link" />
             <child link="${prefix}_roll_link" />
