Commit message: change collision pair file name.

File: tmc_hsrb_description/urdf/base_v0/base.urdf.xacro (robot description, xacro)
@@ -18,5 +18,5 @@
             <insert_block name="origin" />
             <axis xyz="0.0 1.0 0.0" />
-            <limit effort="1000.0" velocity="10.0" />
+            <limit effort="1.5" velocity="18.0" />
             <parent link="${parent}" />
             <child link="${prefix}_${suffix}_drive_wheel_link" />
@@ -50,5 +50,5 @@
             <insert_block name="origin" />
             <axis xyz="1.0 0.0 0.0" />
-            <limit effort="1000.0" velocity="100.0" />
+            <limit effort="1.0" velocity="3.0" />
             <parent link="${parent}" />
             <child link="${prefix}_${suffix}_passive_wheel_x_frame" />

File: tmc_hsrb_description/urdf/base_v1/base.urdf.xacro (robot description, xacro)
@@ -18,5 +18,5 @@
             <insert_block name="origin" />
             <axis xyz="0.0 1.0 0.0" />
-            <limit effort="10.0" velocity="10.0" />
+            <limit effort="1.5" velocity="18.0" />
             <parent link="${parent}" />
             <child link="${prefix}_${suffix}_drive_wheel_link" />
@@ -50,5 +50,5 @@
             <insert_block name="origin" />
             <axis xyz="1.0 0.0 0.0" />
-            <limit effort="100.0" velocity="100.0" />
+            <limit effort="1.0" velocity="3.0" />
             <parent link="${parent}" />
             <child link="${prefix}_${suffix}_passive_wheel_x_frame" />

Commit message: correct effort limit and velocity limit.

File: tmc_hsrb_description/urdf/base_v0/base.urdf.xacro (robot description, xacro)
@@ -13,4 +13,8 @@
     <xacro:property name="passive_wheel_offset_x" value="0.145" />
     <xacro:property name="passive_wheel_offset_y" value="0.04" />
+    <xacro:property name="drive_wheel_max_effort" value="3.76" />
+    <xacro:property name="drive_wheel_max_velocity" value="20.8" />
+    <xacro:property name="roll_joint_max_effort" value="23.0" />
+    <xacro:property name="roll_joint_max_velocity" value="2.5" />
     <!-- drive wheel -->
     <xacro:macro name="hsrb_drive_wheel" params="prefix suffix parent *origin">
@@ -18,5 +22,5 @@
             <insert_block name="origin" />
             <axis xyz="0.0 1.0 0.0" />
-            <limit effort="1.5" velocity="18.0" />
+            <limit effort="${drive_wheel_max_effort}" velocity="${drive_wheel_max_velocity}" />
             <parent link="${parent}" />
             <child link="${prefix}_${suffix}_drive_wheel_link" />
@@ -50,5 +54,5 @@
             <insert_block name="origin" />
             <axis xyz="1.0 0.0 0.0" />
-            <limit effort="1.0" velocity="3.0" />
+            <limit effort="1000.0" velocity="100.0" />
             <parent link="${parent}" />
             <child link="${prefix}_${suffix}_passive_wheel_x_frame" />
@@ -143,5 +147,5 @@
             <origin xyz="0.0 0.0 0.0" rpy="0.0 0.0 0.0" />
             <axis xyz="0.0 0.0 1.0" />
-            <limit effort="1000.0" velocity="1.0" />
+            <limit effort="${roll_joint_max_effort}" velocity="${roll_joint_max_velocity}" />
             <parent link="${prefix}_link" />
             <child link="${prefix}_roll_link" />

File: tmc_hsrb_description/urdf/base_v1/base.urdf.xacro (robot description, xacro)
@@ -13,4 +13,8 @@
     <xacro:property name="passive_wheel_offset_x" value="0.1495" />
     <xacro:property name="passive_wheel_offset_y" value="0.055" />
+    <xacro:property name="drive_wheel_max_effort" value="11.067" />
+    <xacro:property name="drive_wheel_max_velocity" value="20.8" />
+    <xacro:property name="roll_joint_max_effort" value="34.46" />
+    <xacro:property name="roll_joint_max_velocity" value="2.5" />
     <!-- drive wheel -->
     <xacro:macro name="hsrb_drive_wheel" params="prefix suffix parent *origin">
@@ -18,5 +22,5 @@
             <insert_block name="origin" />
             <axis xyz="0.0 1.0 0.0" />
-            <limit effort="1.5" velocity="18.0" />
+            <limit effort="${drive_wheel_max_effort}" velocity="${drive_wheel_max_velocity}" />
             <parent link="${parent}" />
             <child link="${prefix}_${suffix}_drive_wheel_link" />
@@ -142,5 +146,5 @@
             <origin xyz="0.0 0.0 0.0" rpy="0.0 0.0 0.0" />
             <axis xyz="0.0 0.0 1.0" />
-            <limit effort="100.0" velocity="10.0" />
+            <limit effort="${roll_joint_max_effort}" velocity="${roll_joint_max_velocity}" />
             <parent link="${prefix}_link" />
             <child link="${prefix}_roll_link" />

Commit message: Update frame joints and gazebo frame

File: tmc_hsrb_description/urdf/base_v0/base.urdf.xacro (robot description, xacro)
@@ -51,5 +51,5 @@
     <!-- passive wheel -->
     <xacro:macro name="hsrb_passive_wheel" params="prefix suffix parent *origin">
-        <joint name="${prefix}_${suffix}_passive_wheel_x_joint" type="continuous">
+        <joint name="${prefix}_${suffix}_passive_wheel_x_frame_joint" type="continuous">
             <insert_block name="origin" />
             <axis xyz="1.0 0.0 0.0" />
@@ -66,5 +66,5 @@
             </inertial>
         </link>
-        <joint name="${prefix}_${suffix}_passive_wheel_y_joint" type="continuous">
+        <joint name="${prefix}_${suffix}_passive_wheel_y_frame_joint" type="continuous">
             <axis xyz="0.0 1.0 0.0" />
             <limit effort="1000.0" velocity="100.0" />
@@ -108,5 +108,5 @@
     <xacro:macro name="hsrb_base" params="prefix robot_namespace">
         <link name="base_footprint"/>
-        <joint name="${prefix}_joint" type="fixed">
+        <joint name="${prefix}_footprint_joint" type="fixed">
             <parent link="base_footprint" />
             <child link="${prefix}_link" />

File: tmc_hsrb_description/urdf/base_v1/base.urdf.xacro (robot description, xacro)
@@ -51,5 +51,5 @@
     <!-- passive wheel -->
     <xacro:macro name="hsrb_passive_wheel" params="prefix suffix parent *origin">
-        <joint name="${prefix}_${suffix}_passive_wheel_x_joint" type="continuous">
+        <joint name="${prefix}_${suffix}_passive_wheel_x_frame_joint" type="continuous">
             <insert_block name="origin" />
             <axis xyz="1.0 0.0 0.0" />
@@ -66,5 +66,5 @@
             </inertial>
         </link>
-        <joint name="${prefix}_${suffix}_passive_wheel_y_joint" type="continuous">
+        <joint name="${prefix}_${suffix}_passive_wheel_y_frame_joint" type="continuous">
             <axis xyz="0.0 1.0 0.0" />
             <limit effort="100.0" velocity="20.0" />
@@ -108,5 +108,5 @@
     <xacro:macro name="hsrb_base" params="prefix robot_namespace">
         <link name="base_footprint"/>
-        <joint name="${prefix}_joint" type="fixed">
+        <joint name="${prefix}_footprint_joint" type="fixed">
             <parent link="base_footprint" />
             <child link="${prefix}_link" />

File: tmc_hsrb_description/urdf/hand_v0/hand.transmission.xacro (robot description, xacro)
@@ -2,5 +2,5 @@
 <robot xmlns:xacro="http://www.ros.org/wiki.xacro">
     <xacro:macro name="hsrb_hand_transmission" params="prefix">
-        <hsrb_effort_joint_transmission joint="${prefix}_motor_joint" reduction="1"/>
+        <hsrb_effort_joint_transmission joint="${prefix}_motor_frame_joint" reduction="1"/>
         <hsrb_effort_joint_transmission joint="${prefix}_l_proximal_joint" reduction="1"/>
         <hsrb_effort_joint_transmission joint="${prefix}_l_spring_proximal_joint" reduction="1"/>

File: tmc_hsrb_description/urdf/hand_v0/hand.urdf.xacro (robot description, xacro)
@@ -52,5 +52,5 @@
             </collision>
         </link>
-        <joint name="${prefix}_motor_joint" type="revolute">
+        <joint name="${prefix}_motor_frame_joint" type="revolute">
             <axis xyz="1.0 0.0 0.0" />
             <limit effort="100.0" velocity="1.0"
@@ -93,5 +93,5 @@
             <parent link="${parent}" />
             <child link="${prefix}_${suffix}_proximal_link" />
-            <mimic joint="${prefix}_motor_joint" />
+            <mimic joint="${prefix}_motor_frame_joint" />
             <dynamics damping="1.0"/>
         </joint>
@@ -130,5 +130,5 @@
             <parent link="${prefix}_${suffix}_mimic_distal_link" />
             <child link="${prefix}_${suffix}_distal_link" />
-            <mimic joint="${prefix}_motor_joint" multiplier="-1.0" offset="${-distal_joint_angle_offset}"/>
+            <mimic joint="${prefix}_motor_frame_joint" multiplier="-1.0" offset="${-distal_joint_angle_offset}"/>
             <dynamics damping="1.0"/>
         </joint>
@@ -186,5 +186,5 @@
             </collision>
         </link>
-        <joint name="${prefix}_${suffix}_finger_tip_joint" type="fixed">
+        <joint name="${prefix}_${suffix}_finger_tip_frame_joint" type="fixed">
             <origin xyz="0.01675 0.0193 0.0379" rpy="${-pi/2.0} 0.0 0.0" />
             <parent link="${prefix}_${suffix}_distal_link" />
@@ -192,5 +192,5 @@
         </joint>
         <xacro:hsrb_gripper_dummy_link name="${prefix}_${suffix}_finger_tip_frame" />
-        <joint name="${prefix}_${suffix}_finger_vacuum_joint" type="fixed">
+        <joint name="${prefix}_${suffix}_finger_vacuum_frame_joint" type="fixed">
             <origin xyz="0.00475 -0.011539 0.03322" rpy="${pi/4.0} 0.0 0.0" />
             <parent link="${prefix}_${suffix}_distal_link" />
@@ -265,5 +265,5 @@
             </collision>
         </link>
-        <joint name="${prefix}_${suffix}_finger_tip_joint" type="fixed">
+        <joint name="${prefix}_${suffix}_finger_tip_frame_joint" type="fixed">
             <origin xyz="0.01675 -0.0193 0.0379" rpy="${pi/2.0} 0.0 0.0" />
             <parent link="${prefix}_${suffix}_distal_link" />

File: tmc_hsrb_description/urdf/sensors/asus_xtion.gazebo.xacro (robot description, xacro)
@@ -16,6 +16,6 @@
     <xacro:property name="XtionMaxDistance" value="5"/>
     <xacro:property name="XtionFrameRate" value="30"/>
-    <xacro:macro name="asus_xtion_gazebo" params="robot_namespace sensor_name parent_camera_link parent_depth_link">
-        <gazebo reference="${parent_camera_link}">
+    <xacro:macro name="asus_xtion_gazebo" params="robot_namespace sensor_name parent_frame topic_frame_id">
+        <gazebo reference="${parent_frame}">
             <sensor type="depth" name="openni_camera_camera">
                 <always_on>0</always_on>
@@ -28,5 +28,6 @@
                         <format>R8G8B8</format>
                     </image>
-                    <depth_camera> </depth_camera>
+                    <depth_camera>
+                    </depth_camera>
                     <clip>
                         <near>0.1</near>
@@ -34,10 +35,10 @@
                     </clip>
                 </camera>
-                <plugin name="camera_controller" filename="libgazebo_ros_openni_kinect.so">
+                <plugin name="${sensor_name}_controller" filename="libgazebo_ros_openni_kinect.so">
                     <alwaysOn>true</alwaysOn>
                     <baseline>0.2</baseline>
                     <updateRate>1.0</updateRate>
                     <cameraName>${sensor_name}</cameraName>
-                    <frameName>${parent_depth_link}</frameName>
+                    <frameName>${topic_frame_id}</frameName>
                     <imageTopicName>/${robot_namespace}/${sensor_name}/rgb/image_raw</imageTopicName>
                     <cameraInfoTopicName>/${robot_namespace}/${sensor_name}/rgb/camera_info</cameraInfoTopicName>

File: tmc_hsrb_description/urdf/sensors/asus_xtion.urdf.xacro (robot description, xacro)
@@ -6,6 +6,5 @@
         <joint name="${prefix}_${sensor_name}_joint" type="fixed">
             <insert_block name="origin" />
-            <parent link="${parent}"/>
-            <child link="${prefix}_${sensor_name}_link"/>
+            <parent link="${parent}"/> <child link="${prefix}_${sensor_name}_link"/>
         </joint>
         <link name="${prefix}_${sensor_name}_link">
@@ -25,16 +24,16 @@
             </collision>
         </link>
-        <joint name="${prefix}_rgbd_sensor_pointcloud_frame_joint" type="fixed">
-            <origin xyz="0 0 0" rpy="0.0 0.0 0.0"/>
-            <parent link="${prefix}_rgbd_sensor_link"/>
-            <child link="${prefix}_rgbd_sensor_pointcloud_frame"/>
+        <joint name="${prefix}_rgbd_sensor_gazebo_frame_joint" type="fixed">
+            <origin xyz="0 0 0" rpy="${pi/2.0} ${-pi/2.0} 0.0"/>
+            <parent link="${prefix}_${sensor_name}_link"/>
+            <child link="${prefix}_${sensor_name}_gazebo_frame"/>
         </joint>
         `
-        <link name="${prefix}_${sensor_name}_pointcloud_frame"></link>
+        <link name="${prefix}_${sensor_name}_gazebo_frame"></link>
         <xacro:asus_xtion_gazebo
             robot_namespace="${robot_namespace}"
             sensor_name="${sensor_name}"
-            parent_camera_link="${prefix}_${sensor_name}_link"
-            parent_depth_link="${prefix}_${sensor_name}_pointcloud_frame"/>
+            parent_frame="${prefix}_${sensor_name}_gazebo_frame"
+            topic_frame_id="${prefix}_${sensor_name}_rgb_frame" />
     </xacro:macro>
 </robot>

File: tmc_hsrb_description/urdf/sensors/imu.urdf.xacro (robot description, xacro)
@@ -4,5 +4,5 @@
     <!-- imu sensor -->
     <xacro:macro name="imu_sensor" params="prefix parent robot_namespace *origin">
-        <joint name="${prefix}_imu_joint" type="fixed">
+        <joint name="${prefix}_imu_frame_joint" type="fixed">
             <insert_block name="origin" />
             <parent link="${parent}" />

File: tmc_hsrb_description/urdf/sensors/minebea_ft_sensor.urdf.xacro (robot description, xacro)
@@ -3,5 +3,5 @@
     <xacro:include filename="$(find tmc_hsrb_description)/urdf/sensors/minebea_ft_sensor.gazebo.xacro"/>
     <xacro:macro name="minebea_ft_sensor" params="prefix robot_namespace parent joint_name *origin">
-        <joint name="${prefix}_ft_sensor_joint" type="fixed">
+        <joint name="${prefix}_ft_sensor_frame_joint" type="fixed">
             <insert_block name="origin"/>
             <parent link="${parent}"/>
@@ -9,5 +9,7 @@
         </joint>
         <link name="${prefix}_ft_sensor_frame"/>
-        <xacro:minebea_ft_sensor_gazebo sensor_name="${prefix}_ft_sensor" robot_namespace="${robot_namespace}" joint_name="${joint_name}" ros_topic="${prefix}_wrench" />
+        <xacro:minebea_ft_sensor_gazebo
+            sensor_name="${prefix}_ft_sensor" robot_namespace="${robot_namespace}"
+            joint_name="${joint_name}" ros_topic="${prefix}_wrench" />
     </xacro:macro>
 </robot>

File: tmc_hsrb_description/urdf/sensors/pointgrey_chameleon.gazebo.xacro (robot description, xacro)
@@ -1,6 +1,6 @@
 <?xml version="1.0" ?>
 <robot name="hsrb" xmlns:xacro="http://www.ros.org/wiki/xacro">
-    <xacro:macro name="pointgrey_chameleon_gazebo" params="sensor_name frame_name robot_namespace">
-        <gazebo reference="${frame_name}">
+    <xacro:macro name="pointgrey_chameleon_gazebo" params="sensor_name parent_frame topic_frame_id robot_namespace">
+        <gazebo reference="${parent_frame}">
             <sensor type="camera" name="${sensor_name}">
                 <update_rate>10.0</update_rate>
@@ -28,5 +28,5 @@
                     <imageTopicName>image_raw</imageTopicName>
                     <cameraInfoTopicName>camera_info</cameraInfoTopicName>
-                    <frameName>${frame_name}</frameName>
+                    <frameName>${topic_frame_id}</frameName>
                     <robotNamespace>${robot_namespace}</robotNamespace>
                     <hackBaseline>0.07</hackBaseline>

File: tmc_hsrb_description/urdf/sensors/pointgrey_chameleon.urdf.xacro (robot description, xacro)
@@ -17,7 +17,14 @@
             </visual>
         </link>
+        <joint name="${prefix}_camera_gazebo_frame_joint" type="fixed">
+            <origin xyz="0 0 0" rpy="${pi/2.0} ${-pi/2.0} 0.0"/>
+            <parent link="${prefix}_camera_link" />
+            <child link="${prefix}_camera_gazebo_frame" />
+        </joint>
+        <link name="${prefix}_camera_gazebo_frame"></link>
         <xacro:pointgrey_chameleon_gazebo
             sensor_name="${prefix}_camera"
-            frame_name="${prefix}_camera_link"
+            parent_frame="${prefix}_camera_gazebo_frame"
+            topic_frame_id="${prefix}_camera_frame"
             robot_namespace="${robot_namespace}"/>
     </xacro:macro>

File: tmc_hsrb_description/urdf/sensors/wide_camera.urdf.xacro (robot description, xacro)
@@ -4,5 +4,5 @@
     <!-- wide rgb camera -->
     <xacro:macro name="wide_camera" params="prefix parent robot_namespace *origin">
-        <joint name="${prefix}_camera_joint" type="fixed">
+        <joint name="${prefix}_camera_frame_joint" type="fixed">
             <insert_block name="origin" />
             <parent link="${parent}" />
