Commit message: update inertial and camera size

File: hsrb_description/urdf/base_v0/base.urdf.xacro (robot description, xacro)
@@ -21,5 +21,5 @@
         <joint name="${prefix}_${suffix}_drive_wheel_joint" type="continuous">
             <insert_block name="origin" />
-            <axis xyz="0.0 1.0 0.0" />
+            <axis xyz="0.0 0.0 1.0" />
             <limit effort="${drive_wheel_max_effort}" velocity="${drive_wheel_max_velocity}" />
             <parent link="${parent}" />
@@ -54,5 +54,5 @@
             <insert_block name="origin" />
             <axis xyz="1.0 0.0 0.0" />
-            <limit effort="1000.0" velocity="100.0" />
+            <limit effort="8.85" velocity="35.0" />
             <parent link="${parent}" />
             <child link="${prefix}_${suffix}_passive_wheel_x_frame" />
@@ -68,5 +68,5 @@
         <joint name="${prefix}_${suffix}_passive_wheel_y_frame_joint" type="continuous">
             <axis xyz="0.0 1.0 0.0" />
-            <limit effort="1000.0" velocity="100.0" />
+            <limit effort="8.85" velocity="100.0" />
             <parent link="${prefix}_${suffix}_passive_wheel_x_frame" />
             <child link="${prefix}_${suffix}_passive_wheel_y_frame" />
@@ -146,5 +146,5 @@
         <joint name="${prefix}_roll_joint" type="continuous">
             <origin xyz="0.0 0.0 0.0" rpy="0.0 0.0 0.0" />
-            <axis xyz="0.0 0.0 1.0" />
+            <axis xyz="0.0 0.0 -1.0" />
             <limit effort="${roll_joint_max_effort}" velocity="${roll_joint_max_velocity}" />
             <parent link="${prefix}_link" />

File: hsrb_description/urdf/base_v1/base.urdf.xacro (robot description, xacro)
@@ -43,7 +43,7 @@
             </collision>
             <inertial>
-                <mass value="0.1"/>
+                <mass value="0.15"/>
                 <origin xyz="0 0 0"/>
-                <inertia ixx="0.001" ixy="0" ixz="0" iyy="0.001" iyz="0" izz="0.001"/>
+                <inertia ixx="0.015" ixy="0" ixz="0" iyy="0.015" iyz="0" izz="0.015"/>
             </inertial>
         </link>
@@ -63,10 +63,10 @@
                 <mass value="0.3"/>
                 <origin xyz="0 0 0"/>
-                <inertia ixx="0.001" ixy="0" ixz="0" iyy="0.001" iyz="0" izz="0.001"/>
+                <inertia ixx="0.015" ixy="0" ixz="0" iyy="0.015" iyz="0" izz="0.015"/>
             </inertial>
         </link>
         <joint name="${prefix}_${suffix}_passive_wheel_y_frame_joint" type="continuous">
             <axis xyz="0.0 1.0 0.0" />
-            <limit effort="100.0" velocity="20.0" />
+            <limit effort="8.85" velocity="20.0" />
             <parent link="${prefix}_${suffix}_passive_wheel_x_frame" />
             <child link="${prefix}_${suffix}_passive_wheel_y_frame" />
@@ -76,10 +76,10 @@
                 <mass value="0.3"/>
                 <origin xyz="0 0 0"/>
-                <inertia ixx="0.001" ixy="0" ixz="0" iyy="0.001" iyz="0" izz="0.001"/>
+                <inertia ixx="0.015" ixy="0" ixz="0" iyy="0.015" iyz="0" izz="0.015"/>
             </inertial>
         </link>
         <joint name="${prefix}_${suffix}_passive_wheel_z_joint" type="continuous">
             <axis xyz="0.0 0.0 1.0" />
-            <limit effort="1000.0" velocity="20.0" />
+            <limit effort="8.85" velocity="20.0" />
             <parent link="${prefix}_${suffix}_passive_wheel_y_frame" />
             <child link="${prefix}_${suffix}_passive_wheel_z_link" />
@@ -101,5 +101,5 @@
                 <mass value="0.3"/>
                 <origin xyz="0 0 0"/>
-                <inertia ixx="0.001" ixy="0" ixz="0" iyy="0.001" iyz="0" izz="0.001"/>
+                <inertia ixx="0.015" ixy="0" ixz="0" iyy="0.015" iyz="0" izz="0.015"/>
             </inertial>
         </link>

File: hsrb_description/urdf/common.xacro (robot description, xacro)
@@ -46,4 +46,17 @@
     </gazebo>
   </macro>
+  <macro name="gazebo_base_link" params="name gravity collide">
+    <gazebo reference="${name}">
+      <kp>100000000.0</kp>
+      <kd>10.0</kd>
+      <mu1>0.1</mu1>
+      <mu2>0.1</mu2>
+      <fdir1>1 0 0</fdir1>
+      <maxVel>1.0</maxVel>
+      <minDepth>0.0005</minDepth>
+      <selfCollide>${collide}</selfCollide>
+      <gravity>${gravity}</gravity>
+    </gazebo>
+  </macro>
   <macro name="gazebo_link_flat_black" params="name gravity collide friction">
     <gazebo reference="${name}">
@@ -60,11 +73,11 @@
       <gravity>true</gravity>
       <turnGravityOff>false</turnGravityOff>
-      <kp>1000000.0</kp>
+      <kp>500000.0</kp>
       <kd>10.0</kd>
-      <mu1>1.0</mu1>
-      <mu2>1.0</mu2>
+      <mu1>10</mu1>
+      <mu2>10</mu2>
       <fdir1>1 0 0</fdir1>
       <maxVel>1.0</maxVel>
-      <minDepth>0.00</minDepth>
+      <minDepth>0.003</minDepth>
       <material value="Gazebo/FlatBlack"/>
     </gazebo>

File: hsrb_description/urdf/sensors/pointgrey_chameleon.gazebo.xacro (robot description, xacro)
@@ -9,5 +9,5 @@
                     <image>
                         <width>1280</width>
-                        <height>1024</height>
+                        <height>960</height>
                         <format>R8G8B8</format>
                     </image>

Commit message: use valid namespace and change sensor config

File: hsrb_description/urdf/base_v0/base.urdf.xacro (robot description, xacro)
@@ -21,5 +21,5 @@
         <joint name="${prefix}_${suffix}_drive_wheel_joint" type="continuous">
             <insert_block name="origin" />
-            <axis xyz="0.0 0.0 1.0" />
+            <axis xyz="0.0 1.0 0.0" />
             <limit effort="${drive_wheel_max_effort}" velocity="${drive_wheel_max_velocity}" />
             <parent link="${parent}" />
@@ -54,5 +54,5 @@
             <insert_block name="origin" />
             <axis xyz="1.0 0.0 0.0" />
-            <limit effort="8.85" velocity="35.0" />
+            <limit effort="8.85" velocity="10.0" />
             <parent link="${parent}" />
             <child link="${prefix}_${suffix}_passive_wheel_x_frame" />
@@ -68,5 +68,5 @@
         <joint name="${prefix}_${suffix}_passive_wheel_y_frame_joint" type="continuous">
             <axis xyz="0.0 1.0 0.0" />
-            <limit effort="8.85" velocity="100.0" />
+            <limit effort="8.85" velocity="10.0" />
             <parent link="${prefix}_${suffix}_passive_wheel_x_frame" />
             <child link="${prefix}_${suffix}_passive_wheel_y_frame" />
@@ -146,5 +146,5 @@
         <joint name="${prefix}_roll_joint" type="continuous">
             <origin xyz="0.0 0.0 0.0" rpy="0.0 0.0 0.0" />
-            <axis xyz="0.0 0.0 -1.0" />
+            <axis xyz="0.0 0.0 1.0" />
             <limit effort="${roll_joint_max_effort}" velocity="${roll_joint_max_velocity}" />
             <parent link="${prefix}_link" />

File: hsrb_description/urdf/base_v1/base.urdf.xacro (robot description, xacro)
@@ -43,5 +43,5 @@
             </collision>
             <inertial>
-                <mass value="0.15"/>
+                <mass value="0.2"/>
                 <origin xyz="0 0 0"/>
                 <inertia ixx="0.015" ixy="0" ixz="0" iyy="0.015" iyz="0" izz="0.015"/>
@@ -61,5 +61,5 @@
         <link name="${prefix}_${suffix}_passive_wheel_x_frame">
             <inertial>
-                <mass value="0.3"/>
+                <mass value="0.2"/>
                 <origin xyz="0 0 0"/>
                 <inertia ixx="0.015" ixy="0" ixz="0" iyy="0.015" iyz="0" izz="0.015"/>
@@ -68,5 +68,5 @@
         <joint name="${prefix}_${suffix}_passive_wheel_y_frame_joint" type="continuous">
             <axis xyz="0.0 1.0 0.0" />
-            <limit effort="8.85" velocity="20.0" />
+            <limit effort="8.85" velocity="10.0" />
             <parent link="${prefix}_${suffix}_passive_wheel_x_frame" />
             <child link="${prefix}_${suffix}_passive_wheel_y_frame" />
@@ -74,5 +74,5 @@
         <link name="${prefix}_${suffix}_passive_wheel_y_frame">
             <inertial>
-                <mass value="0.3"/>
+                <mass value="0.2"/>
                 <origin xyz="0 0 0"/>
                 <inertia ixx="0.015" ixy="0" ixz="0" iyy="0.015" iyz="0" izz="0.015"/>
@@ -81,5 +81,5 @@
         <joint name="${prefix}_${suffix}_passive_wheel_z_joint" type="continuous">
             <axis xyz="0.0 0.0 1.0" />
-            <limit effort="8.85" velocity="20.0" />
+            <limit effort="8.85" velocity="10.0" />
             <parent link="${prefix}_${suffix}_passive_wheel_y_frame" />
             <child link="${prefix}_${suffix}_passive_wheel_z_link" />
@@ -99,5 +99,5 @@
             </collision>
             <inertial>
-                <mass value="0.3"/>
+                <mass value="0.2"/>
                 <origin xyz="0 0 0"/>
                 <inertia ixx="0.015" ixy="0" ixz="0" iyy="0.015" iyz="0" izz="0.015"/>

File: hsrb_description/urdf/common.xacro (robot description, xacro)
@@ -46,17 +46,4 @@
     </gazebo>
   </macro>
-  <macro name="gazebo_base_link" params="name gravity collide">
-    <gazebo reference="${name}">
-      <kp>100000000.0</kp>
-      <kd>10.0</kd>
-      <mu1>0.1</mu1>
-      <mu2>0.1</mu2>
-      <fdir1>1 0 0</fdir1>
-      <maxVel>1.0</maxVel>
-      <minDepth>0.0005</minDepth>
-      <selfCollide>${collide}</selfCollide>
-      <gravity>${gravity}</gravity>
-    </gazebo>
-  </macro>
   <macro name="gazebo_link_flat_black" params="name gravity collide friction">
     <gazebo reference="${name}">
@@ -73,11 +60,11 @@
       <gravity>true</gravity>
       <turnGravityOff>false</turnGravityOff>
-      <kp>500000.0</kp>
+      <kp>1000000.0</kp>
       <kd>10.0</kd>
-      <mu1>10</mu1>
-      <mu2>10</mu2>
+      <mu1>1.0</mu1>
+      <mu2>1.0</mu2>
       <fdir1>1 0 0</fdir1>
       <maxVel>1.0</maxVel>
-      <minDepth>0.003</minDepth>
+      <minDepth>0.00</minDepth>
       <material value="Gazebo/FlatBlack"/>
     </gazebo>

File: hsrb_description/urdf/sensors/asus_xtion.urdf.xacro (robot description, xacro)
@@ -33,5 +33,5 @@
         <xacro:asus_xtion_gazebo
             robot_namespace="${robot_namespace}"
-            sensor_name="${sensor_name}"
+            sensor_name="${prefix}_${sensor_name}"
             parent_frame="${prefix}_${sensor_name}_gazebo_frame"
             topic_frame_id="${prefix}_${sensor_name}_rgb_frame" />
