Commit message: change only frction parameters in base passive link

File: hsrb_description/urdf/base_v0/base.gazebo.xacro (robot description, xacro)
@@ -4,8 +4,8 @@
         <gazebo_link name="${prefix}_link" gravity="true" collide="false" friction="0.9"/>
         <gazebo_link name="${prefix}_roll_link" gravity="true" collide="false" friction="0.9"/>
-        <gazebo_link_rubber name="${prefix}_r_drive_wheel_link"/>
-        <gazebo_link_rubber name="${prefix}_l_drive_wheel_link"/>
-        <gazebo_link_rubber name="${prefix}_r_passive_wheel_z_link"/>
-        <gazebo_link_rubber name="${prefix}_l_passive_wheel_z_link"/>
+        <gazebo_link_rubber name="${prefix}_r_drive_wheel_link" />
+        <gazebo_link_rubber name="${prefix}_l_drive_wheel_link" />
+        <gazebo_link_caster name="${prefix}_r_passive_wheel_z_link" />
+        <gazebo_link_caster name="${prefix}_l_passive_wheel_z_link" />
         <gazebo_link name="${prefix}_range_sensor_link" gravity="true" collide="false" friction="0.9"/>
         <gazebo_link name="${prefix}_imu_frame" gravity="false" collide="false" friction="0.9"/>

File: hsrb_description/urdf/base_v1/base.gazebo.xacro (robot description, xacro)
@@ -4,12 +4,8 @@
         <gazebo_link name="${prefix}_link" gravity="true" collide="false" friction="0.9"/>
         <gazebo_link name="${prefix}_roll_link" gravity="true" collide="false" friction="0.9"/>
-        <gazebo_link_rubber name="${prefix}_r_drive_wheel_link"/>
-        <gazebo_link_rubber name="${prefix}_l_drive_wheel_link"/>
-        <gazebo_link_flat_black
-            name="${prefix}_r_passive_wheel_z_link" gravity="true" collide="false"
-            friction="0.1"/>
-        <gazebo_link_flat_black
-            name="${prefix}_l_passive_wheel_z_link" gravity="true" collide="false"
-            friction="0.1"/>
+        <gazebo_link_rubber name="${prefix}_r_drive_wheel_link" />
+        <gazebo_link_rubber name="${prefix}_l_drive_wheel_link" />
+        <gazebo_link_caster name="${prefix}_r_passive_wheel_z_link" />
+        <gazebo_link_caster name="${prefix}_l_passive_wheel_z_link" />
         <gazebo_link name="${prefix}_range_sensor_link" gravity="true" collide="false" friction="0.9"/>
         <gazebo_link name="${prefix}_imu_frame" gravity="true" collide="false" friction="0.9"/>

File: hsrb_description/urdf/common.xacro (robot description, xacro)
@@ -55,4 +55,14 @@
     </gazebo>
   </macro>
+  <macro name="gazebo_link_caster" params="name">
+    <gazebo reference="${name}">
+      <selfCollide>false</selfCollide>
+      <gravity>true</gravity>
+      <mu1>0.1</mu1>
+      <mu2>0.1</mu2>
+      <maxVel>1.0</maxVel>
+      <material value="Gazebo/FlatBlack"/>
+    </gazebo>
+  </macro>
   <macro name="gazebo_link_rubber" params="name">
     <gazebo reference="${name}">
