Commit message: use heavier base weight to stabilize move base in gazebo

File: hsrb_description/urdf/base_v1/base.urdf.xacro (robot description, xacro)
@@ -114,5 +114,5 @@
         <link name="${prefix}_link">
             <inertial>
-                <mass value="11.017971"/>
+                <mass value="50.00"/>  <!-- use dummy weight to stabilize gazebo move base (real value: 11.017971)-->
                 <origin xyz="-0.025978 -0.005498 0.17633"/>
                 <inertia ixx="0.3742" ixy="0.000434172172" ixz="0.03088"
