Commit message: added head_center_gazebo_frame

File: hsrb_description/urdf/sensors/wide_camera.gazebo.xacro (robot description, xacro)
@@ -1,6 +1,6 @@
 <?xml version="1.0" ?>
 <robot name="hsrb" xmlns:xacro="http://www.ros.org/wiki/xacro">
-    <xacro:macro name="wide_camera_gazebo" params="sensor_name frame_name robot_namespace">
-        <gazebo reference="${frame_name}">
+    <xacro:macro name="wide_camera_gazebo" params="robot_namespace sensor_name parent_frame topic_frame_id">
+        <gazebo reference="${parent_frame}">
             <sensor type="camera" name="${sensor_name}">
                 <update_rate>10.0</update_rate>
@@ -29,5 +29,5 @@
                     <imageTopicName>image_raw</imageTopicName>
                     <cameraInfoTopicName>camera_info</cameraInfoTopicName>
-                    <frameName>${frame_name}</frameName>
+                    <frameName>${topic_frame_id}</frameName>
                     <hackBaseline>0.07</hackBaseline>
                     <distortionK1>0.0</distortionK1>

File: hsrb_description/urdf/sensors/wide_camera.urdf.xacro (robot description, xacro)
@@ -10,8 +10,15 @@
         </joint>
         <link name="${prefix}_camera_frame"></link>
+        <joint name="${prefix}_camera_gazebo_frame_joint" type="fixed">
+            <origin xyz="0 0 0" rpy="${pi/2.0} ${-pi/2.0} 0.0"/>
+            <parent link="${prefix}_camera_frame" />
+            <child link="${prefix}_camera_gazebo_frame" />
+        </joint>
+        <link name="${prefix}_camera_gazebo_frame"></link>
         <xacro:wide_camera_gazebo
+            robot_namespace="${robot_namespace}"
             sensor_name="${prefix}_camera"
-            frame_name="${prefix}_camera_frame"
-            robot_namespace="${robot_namespace}"
+            parent_frame="${prefix}_camera_gazebo_frame"
+            topic_frame_id="${prefix}_camera_frame"
             />
     </xacro:macro>
