Commit message: reduction mesh

File: hsrb_description/urdf/sensors/asus_xtion.urdf.xacro (robot description, xacro)
@@ -12,5 +12,5 @@
                 <origin xyz="0 0 0" rpy="0.0 0.0 0.0"/>
                 <geometry>
-                    <mesh filename="package://hsrb_description/meshes/sensors/xtion.dae" />
+                    <mesh filename="package://hsrb_description/meshes/sensors/xtion_light.dae" />
                 </geometry>
                 <material name="black" />
