Commit message: change torso damping param to solve torso vibration problem

File: hsrb_description/urdf/torso_v0/torso.urdf.xacro (robot description, xacro)
@@ -12,5 +12,5 @@
             <child link="${prefix}_lift_link" />
             <mimic joint="${mimic_joint}" multiplier="0.5" />
-            <dynamics damping="10.0"/>
+            <dynamics damping="500.0"/>
         </joint>
         <link name="${prefix}_lift_link">
