Commit message: add microphone

File: hsrb_description/urdf/head_v2/head.urdf.xacro (robot description, xacro)
@@ -68,10 +68,4 @@
                 <material name="body_sub" />
             </visual>
-            <visual>
-                <geometry>
-                    <mesh filename="package://hsrb_description/meshes/head_v1/tablet.dae" />
-                </geometry>
-                <material name="tablet" />
-            </visual>
             <collision>
                 <geometry>
