Commit message: unable control period.

File: hsrb_description/robots/hsrb3s.urdf.xacro (robot description, xacro)
@@ -17,5 +17,4 @@
     <!-- constant -->
     <xacro:property name="robot_name" value="hsrb"/>
-    <xacro:property name="control_period" value="0.01"/>
     <!-- create robot -->
     <xacro:hsrb_base prefix="base" robot_namespace="${robot_name}"/>
@@ -38,5 +37,4 @@
         <plugin name="${robot_name}_ros_control" filename="lib${robot_name}_gazebo_ros_control.so">
             <robotNamespace>${robot_name}</robotNamespace>
-            <controlPeriod>${control_period}</controlPeriod>
         </plugin>
         <plugin name="${robot_name}_p3d_ground_truth" filename="libgazebo_ros_p3d.so">

File: hsrb_description/robots/hsrb4s.urdf.xacro (robot description, xacro)
@@ -17,5 +17,4 @@
     <!-- constant -->
     <xacro:property name="robot_name" value="hsrb"/>
-    <xacro:property name="control_period" value="0.01"/>
     <!-- create robot -->
     <xacro:hsrb_base prefix="base" robot_namespace="${robot_name}"/>
@@ -38,5 +37,4 @@
         <plugin name="${robot_name}_ros_control" filename="lib${robot_name}_gazebo_ros_control.so">
             <robotNamespace>${robot_name}</robotNamespace>
-            <controlPeriod>${control_period}</controlPeriod>
         </plugin>
         <plugin name="${robot_name}_p3d_ground_truth" filename="libgazebo_ros_p3d.so">
