Commit message: Update internal reference to old package names

File: hsrb_description/robots/hsrb1s.urdf.xacro (robot description, xacro)
@@ -6,13 +6,13 @@
        xmlns:xacro="http://www.ros.org/wiki.xacro">
     <!-- common xacro -->
-    <xacro:include filename="$(find tmc_hsrb_description)/urdf/common.xacro" />
-    <xacro:include filename="$(find tmc_hsrb_description)/urdf/materials.urdf.xacro" />
+    <xacro:include filename="$(find hsrb_description)/urdf/common.xacro" />
+    <xacro:include filename="$(find hsrb_description)/urdf/materials.urdf.xacro" />
     <!-- links and joints -->
-    <xacro:include filename="$(find tmc_hsrb_description)/urdf/base_v0/base.urdf.xacro" />
-    <xacro:include filename="$(find tmc_hsrb_description)/urdf/torso_v0/torso.urdf.xacro" />
-    <xacro:include filename="$(find tmc_hsrb_description)/urdf/head_v0/head.urdf.xacro" />
-    <xacro:include filename="$(find tmc_hsrb_description)/urdf/arm_v0/arm.urdf.xacro" />
-    <xacro:include filename="$(find tmc_hsrb_description)/urdf/wrist_v0/wrist.urdf.xacro" />
-    <xacro:include filename="$(find tmc_hsrb_description)/urdf/hand_v0/hand.urdf.xacro" />
+    <xacro:include filename="$(find hsrb_description)/urdf/base_v0/base.urdf.xacro" />
+    <xacro:include filename="$(find hsrb_description)/urdf/torso_v0/torso.urdf.xacro" />
+    <xacro:include filename="$(find hsrb_description)/urdf/head_v0/head.urdf.xacro" />
+    <xacro:include filename="$(find hsrb_description)/urdf/arm_v0/arm.urdf.xacro" />
+    <xacro:include filename="$(find hsrb_description)/urdf/wrist_v0/wrist.urdf.xacro" />
+    <xacro:include filename="$(find hsrb_description)/urdf/hand_v0/hand.urdf.xacro" />
     <!-- constant -->
     <xacro:property name="robot_name" value="hsrb"/>

File: hsrb_description/robots/hsrb2s.urdf.xacro (robot description, xacro)
@@ -6,13 +6,13 @@
        xmlns:xacro="http://www.ros.org/wiki.xacro">
     <!-- common xacro -->
-    <xacro:include filename="$(find tmc_hsrb_description)/urdf/common.xacro" />
-    <xacro:include filename="$(find tmc_hsrb_description)/urdf/materials.urdf.xacro" />
+    <xacro:include filename="$(find hsrb_description)/urdf/common.xacro" />
+    <xacro:include filename="$(find hsrb_description)/urdf/materials.urdf.xacro" />
     <!-- links and joints -->
-    <xacro:include filename="$(find tmc_hsrb_description)/urdf/base_v1/base.urdf.xacro" />
-    <xacro:include filename="$(find tmc_hsrb_description)/urdf/torso_v0/torso.urdf.xacro" />
-    <xacro:include filename="$(find tmc_hsrb_description)/urdf/head_v0/head.urdf.xacro" />
-    <xacro:include filename="$(find tmc_hsrb_description)/urdf/arm_v0/arm.urdf.xacro" />
-    <xacro:include filename="$(find tmc_hsrb_description)/urdf/wrist_v0/wrist.urdf.xacro" />
-    <xacro:include filename="$(find tmc_hsrb_description)/urdf/hand_v0/hand.urdf.xacro" />
+    <xacro:include filename="$(find hsrb_description)/urdf/base_v1/base.urdf.xacro" />
+    <xacro:include filename="$(find hsrb_description)/urdf/torso_v0/torso.urdf.xacro" />
+    <xacro:include filename="$(find hsrb_description)/urdf/head_v0/head.urdf.xacro" />
+    <xacro:include filename="$(find hsrb_description)/urdf/arm_v0/arm.urdf.xacro" />
+    <xacro:include filename="$(find hsrb_description)/urdf/wrist_v0/wrist.urdf.xacro" />
+    <xacro:include filename="$(find hsrb_description)/urdf/hand_v0/hand.urdf.xacro" />
     <!-- constant -->
     <xacro:property name="robot_name" value="hsrb"/>

File: hsrb_description/urdf/arm_v0/arm.urdf.xacro (robot description, xacro)
@@ -1,6 +1,6 @@
 <?xml version="1.0"?>
 <robot xmlns:xacro="http://ros.org/wiki/xacro">
-    <xacro:include filename="$(find tmc_hsrb_description)/urdf/arm_v0/arm.transmission.xacro"/>
-    <xacro:include filename="$(find tmc_hsrb_description)/urdf/arm_v0/arm.gazebo.xacro"/>
+    <xacro:include filename="$(find hsrb_description)/urdf/arm_v0/arm.transmission.xacro"/>
+    <xacro:include filename="$(find hsrb_description)/urdf/arm_v0/arm.gazebo.xacro"/>
     <!-- arm -->
     <xacro:macro name="hsrb_arm" params="prefix parent *origin">
@@ -22,5 +22,5 @@
             <visual>
                 <geometry>
-                    <mesh filename="package://tmc_hsrb_description/meshes/arm_v0/shoulder.dae" />
+                    <mesh filename="package://hsrb_description/meshes/arm_v0/shoulder.dae" />
                 </geometry>
                 <material name="body_sub" />
@@ -28,5 +28,5 @@
             <collision>
                 <geometry>
-                    <mesh filename="package://tmc_hsrb_description/meshes/arm_v0/shoulder.stl" />
+                    <mesh filename="package://hsrb_description/meshes/arm_v0/shoulder.stl" />
                 </geometry>
                 <material name="body_sub" />
@@ -50,5 +50,5 @@
             <visual>
                 <geometry>
-                    <mesh filename="package://tmc_hsrb_description/meshes/arm_v0/arm_flex_light.dae" />
+                    <mesh filename="package://hsrb_description/meshes/arm_v0/arm_flex_light.dae" />
                 </geometry>
                 <material name="body_main" />
@@ -56,5 +56,5 @@
             <collision>
                 <geometry>
-                    <mesh filename="package://tmc_hsrb_description/meshes/arm_v0/arm_flex.stl" />
+                    <mesh filename="package://hsrb_description/meshes/arm_v0/arm_flex.stl" />
                 </geometry>
                 <material name="body_main" />
@@ -78,5 +78,5 @@
             <visual>
                 <geometry>
-                    <mesh filename="package://tmc_hsrb_description/meshes/arm_v0/arm_roll_light.dae" />
+                    <mesh filename="package://hsrb_description/meshes/arm_v0/arm_roll_light.dae" />
                 </geometry>
                 <material name="body_main" />
@@ -84,5 +84,5 @@
             <collision>
                 <geometry>
-                    <mesh filename="package://tmc_hsrb_description/meshes/arm_v0/arm_roll.stl" />
+                    <mesh filename="package://hsrb_description/meshes/arm_v0/arm_roll.stl" />
                 </geometry>
                 <material name="body_main" />

File: hsrb_description/urdf/base_v0/base.urdf.xacro (robot description, xacro)
@@ -1,8 +1,8 @@
 <?xml version="1.0"?>
 <robot xmlns:xacro="http://ros.org/wiki/xacro">
-    <xacro:include filename="$(find tmc_hsrb_description)/urdf/base_v0/base.transmission.xacro"/>
-    <xacro:include filename="$(find tmc_hsrb_description)/urdf/base_v0/base.gazebo.xacro"/>
-    <xacro:include filename="$(find tmc_hsrb_description)/urdf/sensors/hokuyo_laser.urdf.xacro"/>
-    <xacro:include filename="$(find tmc_hsrb_description)/urdf/sensors/imu.urdf.xacro"/>
+    <xacro:include filename="$(find hsrb_description)/urdf/base_v0/base.transmission.xacro"/>
+    <xacro:include filename="$(find hsrb_description)/urdf/base_v0/base.gazebo.xacro"/>
+    <xacro:include filename="$(find hsrb_description)/urdf/sensors/hokuyo_laser.urdf.xacro"/>
+    <xacro:include filename="$(find hsrb_description)/urdf/sensors/imu.urdf.xacro"/>
     <!-- constant -->
     <xacro:property name="drive_wheel_width" value="0.03" />
@@ -121,5 +121,5 @@
             <visual>
                 <geometry>
-                    <mesh filename="package://tmc_hsrb_description/meshes/base_v0/base_light.dae" />
+                    <mesh filename="package://hsrb_description/meshes/base_v0/base_light.dae" />
                 </geometry>
                 <material name="body_main" />
@@ -127,5 +127,5 @@
             <visual>
                 <geometry>
-                    <mesh filename="package://tmc_hsrb_description/meshes/base_v0/body.dae" />
+                    <mesh filename="package://hsrb_description/meshes/base_v0/body.dae" />
                 </geometry>
                 <material name="body_main" />
@@ -133,5 +133,5 @@
             <visual>
                 <geometry>
-                    <mesh filename="package://tmc_hsrb_description/meshes/base_v0/torso_base.dae" />
+                    <mesh filename="package://hsrb_description/meshes/base_v0/torso_base.dae" />
                 </geometry>
                 <material name="body_sub" />
@@ -139,5 +139,5 @@
             <collision>
                 <geometry>
-                    <mesh filename="package://tmc_hsrb_description/meshes/base_v0/base.stl" />
+                    <mesh filename="package://hsrb_description/meshes/base_v0/base.stl" />
                 </geometry>
                 <material name="body_sub" />

File: hsrb_description/urdf/base_v1/base.urdf.xacro (robot description, xacro)
@@ -1,8 +1,8 @@
 <?xml version="1.0"?>
 <robot xmlns:xacro="http://ros.org/wiki/xacro">
-    <xacro:include filename="$(find tmc_hsrb_description)/urdf/base_v1/base.transmission.xacro"/>
-    <xacro:include filename="$(find tmc_hsrb_description)/urdf/base_v1/base.gazebo.xacro"/>
-    <xacro:include filename="$(find tmc_hsrb_description)/urdf/sensors/hokuyo_laser.urdf.xacro"/>
-    <xacro:include filename="$(find tmc_hsrb_description)/urdf/sensors/imu.urdf.xacro"/>
+    <xacro:include filename="$(find hsrb_description)/urdf/base_v1/base.transmission.xacro"/>
+    <xacro:include filename="$(find hsrb_description)/urdf/base_v1/base.gazebo.xacro"/>
+    <xacro:include filename="$(find hsrb_description)/urdf/sensors/hokuyo_laser.urdf.xacro"/>
+    <xacro:include filename="$(find hsrb_description)/urdf/sensors/imu.urdf.xacro"/>
     <!-- constant -->
     <xacro:property name="drive_wheel_width" value="0.03" />
@@ -121,5 +121,5 @@
             <visual>
                 <geometry>
-                    <mesh filename="package://tmc_hsrb_description/meshes/base_v1/base_light.dae" />
+                    <mesh filename="package://hsrb_description/meshes/base_v1/base_light.dae" />
                 </geometry>
                 <material name="body_main" />
@@ -127,5 +127,5 @@
             <visual>
                 <geometry>
-                    <mesh filename="package://tmc_hsrb_description/meshes/base_v1/body_light.dae" />
+                    <mesh filename="package://hsrb_description/meshes/base_v1/body_light.dae" />
                 </geometry>
                 <material name="body_main" />
@@ -133,5 +133,5 @@
             <visual>
                 <geometry>
-                    <mesh filename="package://tmc_hsrb_description/meshes/base_v1/torso_base.dae" />
+                    <mesh filename="package://hsrb_description/meshes/base_v1/torso_base.dae" />
                 </geometry>
                 <material name="body_sub" />
@@ -139,5 +139,5 @@
             <collision>
                 <geometry>
-                    <mesh filename="package://tmc_hsrb_description/meshes/base_v1/base.stl" />
+                    <mesh filename="package://hsrb_description/meshes/base_v1/base.stl" />
                 </geometry>
             </collision>

File: hsrb_description/urdf/hand_v0/hand.urdf.xacro (robot description, xacro)
@@ -1,7 +1,7 @@
 <?xml version="1.0"?>
 <robot xmlns:xacro="http://ros.org/wiki/xacro">
-    <xacro:include filename="$(find tmc_hsrb_description)/urdf/hand_v0/hand.transmission.xacro"/>
-    <xacro:include filename="$(find tmc_hsrb_description)/urdf/hand_v0/hand.gazebo.xacro"/>
-    <xacro:include filename="$(find tmc_hsrb_description)/urdf/sensors/wide_camera.urdf.xacro"/>
+    <xacro:include filename="$(find hsrb_description)/urdf/hand_v0/hand.transmission.xacro"/>
+    <xacro:include filename="$(find hsrb_description)/urdf/hand_v0/hand.gazebo.xacro"/>
+    <xacro:include filename="$(find hsrb_description)/urdf/sensors/wide_camera.urdf.xacro"/>
     <xacro:property name="palm_to_proximal_x" value="-0.01675" />
     <xacro:property name="palm_to_proximal_y" value="-0.0245" />
@@ -39,11 +39,11 @@
             <visual>
                 <geometry>
-                    <mesh filename="package://tmc_hsrb_description/meshes/hand_v0/palm_light.dae" />
-                </geometry>
-                <material name="body_sub" />
-            </visual>
-            <collision>
-                <geometry>
-                    <mesh filename="package://tmc_hsrb_description/meshes/hand_v0/palm.stl" />
+                    <mesh filename="package://hsrb_description/meshes/hand_v0/palm_light.dae" />
+                </geometry>
+                <material name="body_sub" />
+            </visual>
+            <collision>
+                <geometry>
+                    <mesh filename="package://hsrb_description/meshes/hand_v0/palm.stl" />
                 </geometry>
                 <material name="body_sub" />
@@ -148,11 +148,11 @@
             <visual>
                 <geometry>
-                    <mesh filename="package://tmc_hsrb_description/meshes/hand_v0/l_proximal.dae" />
-                </geometry>
-                <material name="body_sub" />
-            </visual>
-            <collision>
-                <geometry>
-                    <mesh filename="package://tmc_hsrb_description/meshes/hand_v0/l_proximal.stl" />
+                    <mesh filename="package://hsrb_description/meshes/hand_v0/l_proximal.dae" />
+                </geometry>
+                <material name="body_sub" />
+            </visual>
+            <collision>
+                <geometry>
+                    <mesh filename="package://hsrb_description/meshes/hand_v0/l_proximal.stl" />
                 </geometry>
                 <material name="body_sub" />
@@ -173,11 +173,11 @@
             <visual>
                 <geometry>
-                    <mesh filename="package://tmc_hsrb_description/meshes/hand_v0/l_distal.dae" />
-                </geometry>
-                <material name="body_sub" />
-            </visual>
-            <collision>
-                <geometry>
-                    <mesh filename="package://tmc_hsrb_description/meshes/hand_v0/l_distal.stl" />
+                    <mesh filename="package://hsrb_description/meshes/hand_v0/l_distal.dae" />
+                </geometry>
+                <material name="body_sub" />
+            </visual>
+            <collision>
+                <geometry>
+                    <mesh filename="package://hsrb_description/meshes/hand_v0/l_distal.stl" />
                 </geometry>
                 <material name="body_sub" />
@@ -227,11 +227,11 @@
             <visual>
                 <geometry>
-                    <mesh filename="package://tmc_hsrb_description/meshes/hand_v0/r_proximal.dae" />
-                </geometry>
-                <material name="body_sub" />
-            </visual>
-            <collision>
-                <geometry>
-                    <mesh filename="package://tmc_hsrb_description/meshes/hand_v0/r_proximal.stl" />
+                    <mesh filename="package://hsrb_description/meshes/hand_v0/r_proximal.dae" />
+                </geometry>
+                <material name="body_sub" />
+            </visual>
+            <collision>
+                <geometry>
+                    <mesh filename="package://hsrb_description/meshes/hand_v0/r_proximal.stl" />
                 </geometry>
                 <material name="body_sub" />
@@ -252,11 +252,11 @@
             <visual>
                 <geometry>
-                    <mesh filename="package://tmc_hsrb_description/meshes/hand_v0/r_distal.dae" />
-                </geometry>
-                <material name="body_sub" />
-            </visual>
-            <collision>
-                <geometry>
-                    <mesh filename="package://tmc_hsrb_description/meshes/hand_v0/r_distal.stl" />
+                    <mesh filename="package://hsrb_description/meshes/hand_v0/r_distal.dae" />
+                </geometry>
+                <material name="body_sub" />
+            </visual>
+            <collision>
+                <geometry>
+                    <mesh filename="package://hsrb_description/meshes/hand_v0/r_distal.stl" />
                 </geometry>
                 <material name="body_sub" />

File: hsrb_description/urdf/head_v0/head.urdf.xacro (robot description, xacro)
@@ -1,9 +1,9 @@
 <?xml version="1.0"?>
 <robot xmlns:xacro="http://ros.org/wiki/xacro">
-    <xacro:include filename="$(find tmc_hsrb_description)/urdf/head_v0/head.transmission.xacro"/>
-    <xacro:include filename="$(find tmc_hsrb_description)/urdf/head_v0/head.gazebo.xacro"/>
-    <xacro:include filename="$(find tmc_hsrb_description)/urdf/sensors/asus_xtion.urdf.xacro"/>
-    <xacro:include filename="$(find tmc_hsrb_description)/urdf/sensors/pointgrey_chameleon.urdf.xacro"/>
-    <xacro:include filename="$(find tmc_hsrb_description)/urdf/sensors/wide_camera.urdf.xacro"/>
+    <xacro:include filename="$(find hsrb_description)/urdf/head_v0/head.transmission.xacro"/>
+    <xacro:include filename="$(find hsrb_description)/urdf/head_v0/head.gazebo.xacro"/>
+    <xacro:include filename="$(find hsrb_description)/urdf/sensors/asus_xtion.urdf.xacro"/>
+    <xacro:include filename="$(find hsrb_description)/urdf/sensors/pointgrey_chameleon.urdf.xacro"/>
+    <xacro:include filename="$(find hsrb_description)/urdf/sensors/wide_camera.urdf.xacro"/>
     <!-- head -->
     <xacro:macro name="hsrb_head" params="prefix parent *origin">
@@ -25,5 +25,5 @@
             <visual>
                 <geometry>
-                    <mesh filename="package://tmc_hsrb_description/meshes/head_v0/head_pan.dae" />
+                    <mesh filename="package://hsrb_description/meshes/head_v0/head_pan.dae" />
                 </geometry>
                 <material name="body_main" />
@@ -31,5 +31,5 @@
             <collision>
                 <geometry>
-                    <mesh filename="package://tmc_hsrb_description/meshes/head_v0/head_pan.stl" />
+                    <mesh filename="package://hsrb_description/meshes/head_v0/head_pan.stl" />
                 </geometry>
                 <material name="body_main" />
@@ -53,5 +53,5 @@
             <visual>
                 <geometry>
-                    <mesh filename="package://tmc_hsrb_description/meshes/head_v0/head_upper.dae" />
+                    <mesh filename="package://hsrb_description/meshes/head_v0/head_upper.dae" />
                 </geometry>
                 <material name="body_sub" />
@@ -59,5 +59,5 @@
             <visual>
                 <geometry>
-                    <mesh filename="package://tmc_hsrb_description/meshes/head_v0/head_tilt.dae" />
+                    <mesh filename="package://hsrb_description/meshes/head_v0/head_tilt.dae" />
                 </geometry>
                 <material name="body_main" />
@@ -65,5 +65,5 @@
             <visual>
                 <geometry>
-                    <mesh filename="package://tmc_hsrb_description/meshes/head_v0/tablet_base.dae" />
+                    <mesh filename="package://hsrb_description/meshes/head_v0/tablet_base.dae" />
                 </geometry>
                 <material name="body_sub" />
@@ -71,5 +71,5 @@
             <visual>
                 <geometry>
-                    <mesh filename="package://tmc_hsrb_description/meshes/head_v0/tablet.dae" />
+                    <mesh filename="package://hsrb_description/meshes/head_v0/tablet.dae" />
                 </geometry>
                 <material name="tablet" />
@@ -77,5 +77,5 @@
             <collision>
                 <geometry>
-                    <mesh filename="package://tmc_hsrb_description/meshes/head_v0/head.stl" />
+                    <mesh filename="package://hsrb_description/meshes/head_v0/head.stl" />
                 </geometry>
                 <material name="body_main" />
@@ -83,5 +83,5 @@
             <collision>
                 <geometry>
-                    <mesh filename="package://tmc_hsrb_description/meshes/head_v0/tablet.stl" />
+                    <mesh filename="package://hsrb_description/meshes/head_v0/tablet.stl" />
                 </geometry>
                 <material name="tablet" />

File: hsrb_description/urdf/sensors/asus_xtion.urdf.xacro (robot description, xacro)
@@ -1,5 +1,5 @@
 <?xml version="1.0" ?>
 <robot name="hsrb" xmlns:xacro="http://www.ros.org/wiki/xacro">
-    <xacro:include filename="$(find tmc_hsrb_description)/urdf/sensors/asus_xtion.gazebo.xacro"/>
+    <xacro:include filename="$(find hsrb_description)/urdf/sensors/asus_xtion.gazebo.xacro"/>
     <!-- rgbd_sensor -->
     <xacro:macro name="asus_xtion" params="prefix parent robot_namespace sensor_name *origin">
@@ -12,5 +12,5 @@
                 <origin xyz="0 0 0" rpy="0.0 0.0 0.0"/>
                 <geometry>
-                    <mesh filename="package://tmc_hsrb_description/meshes/sensors/xtion.dae" />
+                    <mesh filename="package://hsrb_description/meshes/sensors/xtion.dae" />
                 </geometry>
                 <material name="black" />
@@ -19,5 +19,5 @@
                 <origin xyz="0 0 0" rpy="0.0 0.0 0.0"/>
                 <geometry>
-                    <mesh filename="package://tmc_hsrb_description/meshes/sensors/xtion.stl" />
+                    <mesh filename="package://hsrb_description/meshes/sensors/xtion.stl" />
                 </geometry>
                 <material name="black" />

File: hsrb_description/urdf/sensors/hokuyo_laser.urdf.xacro (robot description, xacro)
@@ -1,4 +1,4 @@
 <robot xmlns:xacro="http://ros.org/wiki/xacro">
-    <xacro:include filename="$(find tmc_hsrb_description)/urdf/sensors/hokuyo_laser.gazebo.xacro"/>
+    <xacro:include filename="$(find hsrb_description)/urdf/sensors/hokuyo_laser.gazebo.xacro"/>
     <!-- range sensor -->
     <xacro:macro name="hokuyo_laser" params="prefix robot_namespace parent *origin">
@@ -11,5 +11,5 @@
             <visual>
                 <geometry>
-                    <mesh filename="package://tmc_hsrb_description/meshes/sensors/laser.dae" />
+                    <mesh filename="package://hsrb_description/meshes/sensors/laser.dae" />
                 </geometry>
                 <material name="black" />
@@ -17,5 +17,5 @@
             <collision>
                 <geometry>
-                    <mesh filename="package://tmc_hsrb_description/meshes/sensors/laser.stl" />
+                    <mesh filename="package://hsrb_description/meshes/sensors/laser.stl" />
                 </geometry>
                 <material name="black" />

File: hsrb_description/urdf/sensors/imu.urdf.xacro (robot description, xacro)
@@ -1,5 +1,5 @@
 <?xml version="1.0" ?>
 <robot xmlns:xacro="http://www.ros.org/wiki/xacro" name="hsrb">
-    <xacro:include filename="$(find tmc_hsrb_description)/urdf/sensors/imu.gazebo.xacro"/>
+    <xacro:include filename="$(find hsrb_description)/urdf/sensors/imu.gazebo.xacro"/>
     <!-- imu sensor -->
     <xacro:macro name="imu_sensor" params="prefix parent robot_namespace *origin">
