Commit message: Update internal reference to old package names

File: hsrb_description/urdf/sensors/minebea_ft_sensor.urdf.xacro (robot description, xacro)
@@ -1,5 +1,5 @@
 <?xml version="1.0" ?>
 <robot name="hsrb" xmlns:xacro="http://www.ros.org/wiki/xacro">
-    <xacro:include filename="$(find tmc_hsrb_description)/urdf/sensors/minebea_ft_sensor.gazebo.xacro"/>
+    <xacro:include filename="$(find hsrb_description)/urdf/sensors/minebea_ft_sensor.gazebo.xacro"/>
     <xacro:macro name="minebea_ft_sensor" params="prefix robot_namespace parent joint_name *origin">
         <joint name="${prefix}_ft_sensor_frame_joint" type="fixed">

File: hsrb_description/urdf/sensors/pointgrey_chameleon.urdf.xacro (robot description, xacro)
@@ -1,5 +1,5 @@
 <?xml version="1.0"?>
 <robot xmlns:xacro="http://ros.org/wiki/xacro">
-    <xacro:include filename="$(find tmc_hsrb_description)/urdf/sensors/pointgrey_chameleon.gazebo.xacro"/>
+    <xacro:include filename="$(find hsrb_description)/urdf/sensors/pointgrey_chameleon.gazebo.xacro"/>
     <xacro:macro name="pointgrey_chameleon" params="prefix parent robot_namespace *origin">
         <joint name="${prefix}_camera_joint" type="fixed">
@@ -12,5 +12,5 @@
                 <origin xyz="0 0 0" rpy="0.0 0.0 0.0"/>
                 <geometry>
-                    <mesh filename="package://tmc_hsrb_description/meshes/sensors/head_camera.dae" />
+                    <mesh filename="package://hsrb_description/meshes/sensors/head_camera.dae" />
                 </geometry>
                 <material name="black" />

File: hsrb_description/urdf/sensors/wide_camera.urdf.xacro (robot description, xacro)
@@ -1,5 +1,5 @@
 <?xml version="1.0"?>
 <robot xmlns:xacro="http://ros.org/wiki/xacro">
-    <xacro:include filename="$(find tmc_hsrb_description)/urdf/sensors/wide_camera.gazebo.xacro"/>
+    <xacro:include filename="$(find hsrb_description)/urdf/sensors/wide_camera.gazebo.xacro"/>
     <!-- wide rgb camera -->
     <xacro:macro name="wide_camera" params="prefix parent robot_namespace *origin">

File: hsrb_description/urdf/torso_v0/torso.urdf.xacro (robot description, xacro)
@@ -1,5 +1,5 @@
 <?xml version="1.0"?>
 <robot xmlns:xacro="http://ros.org/wiki/xacro">
-    <xacro:include filename="$(find tmc_hsrb_description)/urdf/torso_v0/torso.gazebo.xacro"/>
+    <xacro:include filename="$(find hsrb_description)/urdf/torso_v0/torso.gazebo.xacro"/>
     <!-- torso -->
     <xacro:macro name="hsrb_torso" params="prefix parent mimic_joint *origin">
@@ -23,5 +23,5 @@
             <visual>
                 <geometry>
-                    <mesh filename="package://tmc_hsrb_description/meshes/torso_v0/torso_light.dae" />
+                    <mesh filename="package://hsrb_description/meshes/torso_v0/torso_light.dae" />
                 </geometry>
                 <material name="body_sub" />
@@ -29,5 +29,5 @@
             <collision>
                 <geometry>
-                    <mesh filename="package://tmc_hsrb_description/meshes/torso_v0/torso.stl" />
+                    <mesh filename="package://hsrb_description/meshes/torso_v0/torso.stl" />
                 </geometry>
                 <material name="body_sub" />

File: hsrb_description/urdf/wrist_v0/wrist.urdf.xacro (robot description, xacro)
@@ -1,7 +1,7 @@
 <?xml version="1.0"?>
 <robot xmlns:xacro="http://ros.org/wiki/xacro">
-    <xacro:include filename="$(find tmc_hsrb_description)/urdf/wrist_v0/wrist.transmission.xacro"/>
-    <xacro:include filename="$(find tmc_hsrb_description)/urdf/wrist_v0/wrist.gazebo.xacro"/>
-    <xacro:include filename="$(find tmc_hsrb_description)/urdf/sensors/minebea_ft_sensor.urdf.xacro"/>
+    <xacro:include filename="$(find hsrb_description)/urdf/wrist_v0/wrist.transmission.xacro"/>
+    <xacro:include filename="$(find hsrb_description)/urdf/wrist_v0/wrist.gazebo.xacro"/>
+    <xacro:include filename="$(find hsrb_description)/urdf/sensors/minebea_ft_sensor.urdf.xacro"/>
     <!-- wrist -->
     <xacro:macro name="hsrb_wrist" params="prefix robot_namespace parent *origin">
@@ -23,5 +23,5 @@
             <visual>
                 <geometry>
-                    <mesh filename="package://tmc_hsrb_description/meshes/wrist_v0/wrist_flex.dae" />
+                    <mesh filename="package://hsrb_description/meshes/wrist_v0/wrist_flex.dae" />
                 </geometry>
                 <material name="body_sub" />
@@ -59,5 +59,5 @@
             <visual>
                 <geometry>
-                    <mesh filename="package://tmc_hsrb_description/meshes/wrist_v0/wrist_roll.dae" />
+                    <mesh filename="package://hsrb_description/meshes/wrist_v0/wrist_roll.dae" />
                 </geometry>
                 <material name="body_main" />
@@ -65,5 +65,5 @@
             <collision>
                 <geometry>
-                    <mesh filename="package://tmc_hsrb_description/meshes/wrist_v0/wrist_roll.stl" />
+                    <mesh filename="package://hsrb_description/meshes/wrist_v0/wrist_roll.stl" />
                 </geometry>
                 <material name="body_main" />

Commit message: fixed control period / add implicit damping to deal with high cfm

File: hsrb_description/robots/hsrb1s.urdf.xacro (robot description, xacro)
@@ -35,5 +35,5 @@
     </xacro:hsrb_hand>
     <gazebo>
-        <plugin name="${robot_name}_ros_control" filename="libgazebo_ros_control.so">
+        <plugin name="${robot_name}_ros_control" filename="lib${robot_name}_gazebo_ros_control.so">
             <robotNamespace>${robot_name}</robotNamespace>
         </plugin>

File: hsrb_description/robots/hsrb2s.urdf.xacro (robot description, xacro)
@@ -35,5 +35,5 @@
     </xacro:hsrb_hand>
     <gazebo>
-        <plugin name="${robot_name}_ros_control" filename="libgazebo_ros_control.so">
+        <plugin name="${robot_name}_ros_control" filename="lib${robot_name}_gazebo_ros_control.so">
             <robotNamespace>${robot_name}</robotNamespace>
         </plugin>

File: hsrb_description/robots/hsrb3s.urdf.xacro (robot description, xacro)
@@ -17,4 +17,5 @@
     <!-- constant -->
     <xacro:property name="robot_name" value="hsrb"/>
+    <xacro:property name="control_period" value="0.01"/>
     <!-- create robot -->
     <xacro:hsrb_base prefix="base" robot_namespace="${robot_name}"/>
@@ -35,6 +36,7 @@
     </xacro:hsrb_hand>
     <gazebo>
-        <plugin name="${robot_name}_ros_control" filename="libgazebo_ros_control.so">
+        <plugin name="${robot_name}_ros_control" filename="lib${robot_name}_gazebo_ros_control.so">
             <robotNamespace>${robot_name}</robotNamespace>
+            <controlPeriod>${control_period}</controlPeriod>
         </plugin>
         <plugin name="${robot_name}_p3d_ground_truth" filename="libgazebo_ros_p3d.so">

File: hsrb_description/urdf/common.xacro (robot description, xacro)
@@ -1,4 +1,5 @@
 <?xml version="1.0"?>
 <robot xmlns:xacro="http://www.ros.org/wiki.xacro">
+  <xacro:arg name="implicit_damping" default="false" />
   <xacro:property name="pi" value="3.14159265359"/>
   <macro name="hsrb_position_joint_transmission" params="joint reduction">
@@ -81,5 +82,13 @@
   </macro>
   <macro name="gazebo_joint" params="name">
-      <gazebo reference="${name}"></gazebo>
+    <gazebo reference="${name}">
+      <xacro:if value="$(arg implicit_damping)">
+        <implicitSpringDamper>1</implicitSpringDamper>
+      </xacro:if>
+    </gazebo>
+  </macro>
+  <macro name="gazebo_joint_mimic" params="name">
+    <gazebo reference="${name}">
+    </gazebo>
   </macro>
 </robot>

File: hsrb_description/urdf/torso_v0/torso.gazebo.xacro (robot description, xacro)
@@ -3,5 +3,5 @@
     <xacro:macro name="hsrb_torso_gazebo" params="prefix mimic_joint">
         <gazebo_link name="${prefix}_lift_link" gravity="true" collide="false" friction="0.9"/>
-        <gazebo_joint name="${prefix}_lift_joint"/>
+        <gazebo_joint_mimic name="${prefix}_lift_joint"/>
         <gazebo>
             <plugin name="torso_mimic_plugin" filename="libtmc_gazebo_mimic_plugin.so">
