Commit message: Add multi robot simulation function

File: hsrb_description/robots/hsrb1s.urdf.xacro (robot description, xacro)
@@ -15,6 +15,9 @@
     <xacro:include filename="$(find hsrb_description)/urdf/wrist_v0/wrist.urdf.xacro" />
     <xacro:include filename="$(find hsrb_description)/urdf/hand_v0/hand.urdf.xacro" />
+    <xacro:arg name="personal_name" default="hsrb"/>
     <!-- constant -->
+    <xacro:property name="personal_name" value="$(arg personal_name)"/>
     <xacro:property name="robot_name" value="hsrb"/>
+    <xacro:property name="robot_type" value="hsrb"/>
     <!-- create robot -->
     <xacro:hsrb_base prefix="base" robot_namespace="${robot_name}"/>
@@ -37,7 +40,8 @@
         <plugin name="${robot_name}_ros_control" filename="lib${robot_name}_gazebo_ros_control.so">
             <robotNamespace>${robot_name}</robotNamespace>
+            <legacyModeNS>false</legacyModeNS>
         </plugin>
         <plugin name="${robot_name}_p3d_ground_truth" filename="libgazebo_ros_p3d.so">
-            <robotNamespace>${robot_name}</robotNamespace>
+            <robotNamespace>${personal_name}/${robot_type}</robotNamespace>
             <bodyName>base_footprint</bodyName>
             <topicName>odom_ground_truth</topicName>

File: hsrb_description/robots/hsrb2s.urdf.xacro (robot description, xacro)
@@ -15,6 +15,9 @@
     <xacro:include filename="$(find hsrb_description)/urdf/wrist_v0/wrist.urdf.xacro" />
     <xacro:include filename="$(find hsrb_description)/urdf/hand_v0/hand.urdf.xacro" />
+    <xacro:arg name="personal_name" default="hsrb"/>
     <!-- constant -->
+    <xacro:property name="personal_name" value="$(arg personal_name)"/>
     <xacro:property name="robot_name" value="hsrb"/>
+    <xacro:property name="robot_type" value="hsrb"/>
     <!-- create robot -->
     <xacro:hsrb_base prefix="base" robot_namespace="${robot_name}"/>
@@ -36,8 +39,9 @@
     <gazebo>
         <plugin name="${robot_name}_ros_control" filename="lib${robot_name}_gazebo_ros_control.so">
-            <robotNamespace>${robot_name}</robotNamespace>
+            <robotNamespace>${personal_name}/${robot_type}</robotNamespace>
+            <legacyModeNS>false</legacyModeNS>
         </plugin>
         <plugin name="${robot_name}_p3d_ground_truth" filename="libgazebo_ros_p3d.so">
-            <robotNamespace>${robot_name}</robotNamespace>
+            <robotNamespace>${personal_name}/${robot_type}</robotNamespace>
             <bodyName>base_footprint</bodyName>
             <topicName>odom_ground_truth</topicName>

File: hsrb_description/robots/hsrb3s.urdf.xacro (robot description, xacro)
@@ -15,6 +15,9 @@
     <xacro:include filename="$(find hsrb_description)/urdf/wrist_v0/wrist.urdf.xacro" />
     <xacro:include filename="$(find hsrb_description)/urdf/hand_v0/hand.urdf.xacro" />
+    <xacro:arg name="personal_name" default="hsrb"/>
     <!-- constant -->
+    <xacro:property name="personal_name" value="$(arg personal_name)"/>
     <xacro:property name="robot_name" value="hsrb"/>
+    <xacro:property name="robot_type" value="hsrb"/>
     <!-- create robot -->
     <xacro:hsrb_base prefix="base" robot_namespace="${robot_name}"/>
@@ -36,8 +39,9 @@
     <gazebo>
         <plugin name="${robot_name}_ros_control" filename="lib${robot_name}_gazebo_ros_control.so">
-            <robotNamespace>${robot_name}</robotNamespace>
+            <robotNamespace>${personal_name}/${robot_type}</robotNamespace>
+            <legacyModeNS>false</legacyModeNS>
         </plugin>
         <plugin name="${robot_name}_p3d_ground_truth" filename="libgazebo_ros_p3d.so">
-            <robotNamespace>${robot_name}</robotNamespace>
+            <robotNamespace>${personal_name}/${robot_type}</robotNamespace>
             <bodyName>base_footprint</bodyName>
             <topicName>odom_ground_truth</topicName>

File: hsrb_description/robots/hsrb4s.urdf.xacro (robot description, xacro)
@@ -15,8 +15,11 @@
     <xacro:include filename="$(find hsrb_description)/urdf/wrist_v0/wrist.urdf.xacro" />
     <xacro:include filename="$(find hsrb_description)/urdf/hand_v0/hand.urdf.xacro" />
+    <xacro:arg name="personal_name" default="hsrb"/>
     <!-- constant -->
+    <xacro:property name="personal_name" value="$(arg personal_name)"/>
     <xacro:property name="robot_name" value="hsrb"/>
+    <xacro:property name="robot_type" value="hsrb"/>
     <!-- create robot -->
-    <xacro:hsrb_base prefix="base" robot_namespace="${robot_name}"/>
+    <xacro:hsrb_base prefix="base" personal_name="${personal_name}" robot_namespace="${robot_name}" robot_type="${robot_type}" />
     <xacro:hsrb_torso prefix="torso" parent="base_link" mimic_joint="arm_lift_joint">
         <origin xyz="0.0 0.0 0.752" rpy="0.0 0.0 0.0"/>
@@ -35,9 +38,10 @@
     </xacro:hsrb_hand>
     <gazebo>
-        <plugin name="${robot_name}_ros_control" filename="lib${robot_name}_gazebo_ros_control.so">
-            <robotNamespace>${robot_name}</robotNamespace>
+        <plugin name="${robot_type}_ros_control" filename="lib${robot_type}_gazebo_ros_control.so">
+            <robotNamespace>${personal_name}/${robot_type}</robotNamespace>
+            <legacyModeNS>false</legacyModeNS>
         </plugin>
-        <plugin name="${robot_name}_p3d_ground_truth" filename="libgazebo_ros_p3d.so">
-            <robotNamespace>${robot_name}</robotNamespace>
+        <plugin name="${robot_type}_p3d_ground_truth" filename="libgazebo_ros_p3d.so">
+            <robotNamespace>${personal_name}/${robot_type}</robotNamespace>
             <bodyName>base_footprint</bodyName>
             <topicName>odom_ground_truth</topicName>

File: hsrb_description/urdf/base_v0/base.urdf.xacro (robot description, xacro)
@@ -183,8 +183,9 @@
             prefix="${prefix}"
             robot_namespace="${robot_namespace}"
-            parent="${prefix}_link">
+            parent="${prefix}_link"
+            min_angle="-2.1" max_angle="2.1">
             <origin xyz="0.1375 0.0 0.1895" rpy="0.0 0.0 0.0" />
         </xacro:hokuyo_laser>
-        <xacro:imu_sensor prefix="${prefix}" robot_namespace="${robot_namespace}" parent="${prefix}_link">
+        <xacro:imu_sensor prefix="${prefix}" robot_namespace="${robot_namespace}" parent="${prefix}_link" topic_name="data">
             <origin xyz="0.0005 0.1296 0.181" rpy="${pi} 0.0 0.0" />
         </xacro:imu_sensor>

File: hsrb_description/urdf/base_v1/base.urdf.xacro (robot description, xacro)
@@ -181,8 +181,9 @@
             prefix="${prefix}"
             robot_namespace="${robot_namespace}"
-            parent="${prefix}_link">
+            parent="${prefix}_link"
+            min_angle="-2.1" max_angle="2.1">
             <origin xyz="0.1675 0.0 0.1844" rpy="0.0 0.0 0.0" />
         </xacro:hokuyo_laser>
-        <xacro:imu_sensor prefix="${prefix}" robot_namespace="${robot_namespace}" parent="${prefix}_link">
+        <xacro:imu_sensor prefix="${prefix}" robot_namespace="${robot_namespace}" parent="${prefix}_link" topic_name="data">
             <origin xyz="0.0005 0.1296 0.181" rpy="${pi} 0.0 0.0" />
         </xacro:imu_sensor>

File: hsrb_description/urdf/base_v2/base.gazebo.xacro (robot description, xacro)
@@ -1,5 +1,5 @@
 <?xml version="1.0"?>
 <robot xmlns:xacro="http://ros.org/wiki/xacro">
-    <xacro:macro name="hsrb_base_gazebo" params="prefix">
+    <xacro:macro name="hsrb_base_gazebo" params="personal_name prefix robot_type">
         <gazebo_link name="${prefix}_link" gravity="true" collide="false" friction="0.9"/>
         <gazebo_link name="${prefix}_roll_link" gravity="true" collide="false" friction="0.9"/>
@@ -10,6 +10,6 @@
         <gazebo_link name="${prefix}_range_sensor_link" gravity="true" collide="false" friction="0.9"/>
         <gazebo_link name="${prefix}_imu_frame" gravity="true" collide="false" friction="0.9"/>
-        <gazebo_link_bumper name="${prefix}_f_bumper" gravity="true" collide="false" friction="0.9"/>
-        <gazebo_link_bumper name="${prefix}_b_bumper" gravity="true" collide="false" friction="0.9"/>
+        <gazebo_link_bumper name="${prefix}_f_bumper" personal_name="${personal_name}" robot_type="${robot_type}" gravity="true" collide="false" friction="0.9"/>
+        <gazebo_link_bumper name="${prefix}_b_bumper" personal_name="${personal_name}" robot_type="${robot_type}" gravity="true" collide="false" friction="0.9"/>
     </xacro:macro>
 </robot>

File: hsrb_description/urdf/base_v2/base.urdf.xacro (robot description, xacro)
@@ -132,5 +132,5 @@
     </xacro:macro>
     <!-- base -->
-    <xacro:macro name="hsrb_base" params="prefix robot_namespace">
+    <xacro:macro name="hsrb_base" params="prefix personal_name robot_namespace robot_type">
         <link name="base_footprint">
         </link>
@@ -210,8 +210,9 @@
             prefix="${prefix}"
             robot_namespace="${robot_namespace}"
-            parent="${prefix}_link">
+            parent="${prefix}_link"
+            min_angle="-2.1" max_angle="2.1">
             <origin xyz="0.1675 0.0 0.1844" rpy="0.0 0.0 0.0" />
         </xacro:hokuyo_laser>
-        <xacro:imu_sensor prefix="${prefix}" robot_namespace="${robot_namespace}" parent="${prefix}_link">
+        <xacro:imu_sensor prefix="${prefix}" robot_namespace="${robot_namespace}" parent="${prefix}_link" topic_name="data">
             <origin xyz="0.0005 0.1296 0.181" rpy="0.0 0.0 0.0" />
         </xacro:imu_sensor>
@@ -227,5 +228,5 @@
                 rpy="0.0 0.0 ${pi}" />
         </xacro:hsrb_bumper>
-        <xacro:hsrb_base_gazebo prefix="${prefix}"/>
+        <xacro:hsrb_base_gazebo personal_name="${personal_name}" prefix="${prefix}" robot_type="${robot_type}"/>
         <xacro:hsrb_base_transmission prefix="${prefix}"/>
     </xacro:macro>

File: hsrb_description/urdf/common/kinetic/common.xacro (robot description, xacro)
@@ -79,5 +79,5 @@
     </gazebo>
   </xacro:macro>
-  <xacro:macro name="gazebo_link_bumper" params="name gravity collide friction">
+  <xacro:macro name="gazebo_link_bumper" params="name personal_name robot_type gravity collide friction">
     <gazebo reference="${name}_link">
       <selfCollide>${collide}</selfCollide>
@@ -92,5 +92,5 @@
         </contact>
         <plugin name="hsrb_gazebo_ros_bumper_controller" filename="libhsrb_gazebo_ros_bumper.so">
-          <robotNamespace>hsrb</robotNamespace>
+          <robotNamespace>${personal_name}/${robot_type}</robotNamespace>
           <bumperTopicName>${name}_sensor</bumperTopicName>
           <frameName>${name}_link</frameName>

File: hsrb_description/urdf/hand_v0/hand.gazebo.xacro (robot description, xacro)
@@ -33,4 +33,5 @@
             <error_tolerance>0.0872</error_tolerance>
             <stall_timeout>2.0</stall_timeout>
+            <robot_namespace>${personal_name}/${robot_name}</robot_namespace>
           </plugin>
           <plugin name="hsrb_grasp_hack_plugin" filename="libhsrb_grasp_hack.so">
@@ -47,4 +48,5 @@
 	    <!-- hand_palm_link is merged with wrist_ft_sensor_frame by fixed joint  -->
             <palm_link>wrist_ft_sensor_frame</palm_link>
+            <robot_namespace>${personal_name}/${robot_name}</robot_namespace>
           </plugin>
         </gazebo>

File: hsrb_description/urdf/hand_v0/hand.urdf.xacro (robot description, xacro)
@@ -74,5 +74,5 @@
         </xacro:hsrb_finger_without_vacuum>
         <!-- camera -->
-        <xacro:wide_camera prefix="${prefix}" parent="${prefix}_palm_link" robot_namespace="${robot_name}" rpy="${pi/2.0} ${-pi/2.0} 0" >
+        <xacro:wide_camera prefix="${prefix}" parent="${prefix}_palm_link" robot_namespace="${personal_name}/${robot_name}" rpy="${pi/2.0} ${-pi/2.0} 0" >
             <origin xyz="0.039 0.0 -0.0045" rpy="0.0 0.0 0.0"/>
         </xacro:wide_camera>

File: hsrb_description/urdf/head_v2/head.urdf.xacro (robot description, xacro)
@@ -76,14 +76,14 @@
         </link>
         <!-- cameras -->
-        <xacro:pointgrey_chameleon prefix="${prefix}_l_stereo" parent="${prefix}_tilt_link" robot_namespace="${robot_name}" baseline="0.00">
+        <xacro:pointgrey_chameleon prefix="${prefix}_l_stereo" parent="${prefix}_tilt_link" robot_namespace="${personal_name}/${robot_name}" baseline="0.00">
             <origin xyz="0.02 0.07 0.061" rpy="${-pi/2.0} 0.0 ${-pi/2.0}"/>
         </xacro:pointgrey_chameleon>
-        <xacro:pointgrey_chameleon prefix="${prefix}_r_stereo" parent="${prefix}_tilt_link" robot_namespace="${robot_name}" baseline="0.14">
+        <xacro:pointgrey_chameleon prefix="${prefix}_r_stereo" parent="${prefix}_tilt_link" robot_namespace="${personal_name}/${robot_name}" baseline="0.14">
             <origin xyz="0.02 -0.07 0.061" rpy="${-pi/2.0} 0.0 ${-pi/2.0}"/>
         </xacro:pointgrey_chameleon>
-        <xacro:wide_camera prefix="${prefix}_center" parent="${prefix}_tilt_link" robot_namespace="${robot_name}" rpy="${pi/2.0} ${-pi/2.0} 0.0" >
+        <xacro:wide_camera prefix="${prefix}_center" parent="${prefix}_tilt_link" robot_namespace="${personal_name}/${robot_name}" rpy="${pi/2.0} ${-pi/2.0} 0.0" >
             <origin xyz="0.0195 0.0 0.061" rpy="${-pi/2.0} 0.0 ${-pi/2.0}"/>
         </xacro:wide_camera>
-        <xacro:asus_xtion prefix="${prefix}" parent="${prefix}_tilt_link" robot_namespace="${robot_name}" sensor_name="rgbd_sensor">
+        <xacro:asus_xtion prefix="${prefix}" parent="${prefix}_tilt_link" robot_namespace="${personal_name}/${robot_name}" sensor_name="rgbd_sensor">
             <origin xyz="-0.079796 0.022 0.215172" rpy="${-pi/2.0} 0.0 ${-pi/2.0}"/>
         </xacro:asus_xtion>

File: hsrb_description/urdf/wrist_v0/wrist.urdf.xacro (robot description, xacro)
@@ -83,5 +83,5 @@
         <xacro:minebea_ft_sensor
             prefix="${prefix}"
-            robot_namespace="${robot_namespace}"
+            robot_namespace="${personal_name}/${robot_namespace}"
             parent="${prefix}_ft_sensor_mount_link">
             <origin xyz="0.0 0.0 0.0735" rpy="${pi} 0.0 0.0"/>

File: hsrb_parts_description/urdf/sensors/hokuyo_laser.gazebo.xacro (robot description, xacro)
@@ -13,6 +13,6 @@
                             <samples>721</samples>
                             <resolution>1</resolution>
-                            <min_angle>-2.1</min_angle>
-                            <max_angle>2.1</max_angle>
+                            <min_angle>${min_angle}</min_angle>
+                            <max_angle>${max_angle}</max_angle>
                         </horizontal>
                     </scan>

File: hsrb_parts_description/urdf/sensors/hokuyo_laser.urdf.xacro (robot description, xacro)
@@ -3,5 +3,5 @@
     <xacro:include filename="$(find hsrb_parts_description)/urdf/sensors/hokuyo_laser.gazebo.xacro"/>
     <!-- range sensor -->
-    <xacro:macro name="hokuyo_laser" params="prefix robot_namespace parent *origin">
+    <xacro:macro name="hokuyo_laser" params="prefix robot_namespace parent min_angle max_angle *origin">
         <joint name="${prefix}_range_sensor_joint" type="fixed">
             <xacro:insert_block name="origin" />
@@ -31,5 +31,5 @@
             ros_topic="${prefix}_scan"
             frame_name="${prefix}_range_sensor_link"
-            min_angle="-2.3562" max_angle="2.3562" />
+            min_angle="${min_angle}" max_angle="${max_angle}" />
     </xacro:macro>
 </robot>

File: hsrb_parts_description/urdf/sensors/imu.urdf.xacro (robot description, xacro)
@@ -3,5 +3,5 @@
     <xacro:include filename="$(find hsrb_parts_description)/urdf/sensors/$(env ROS_DISTRO)/imu.gazebo.xacro"/>
     <!-- imu sensor -->
-    <xacro:macro name="imu_sensor" params="prefix parent robot_namespace *origin">
+    <xacro:macro name="imu_sensor" params="prefix parent topic_name robot_namespace *origin">
         <joint name="${prefix}_imu_frame_joint" type="fixed">
             <xacro:insert_block name="origin" />
@@ -18,6 +18,7 @@
         <xacro:imu_gazebo
             sensor_name="${prefix}_imu"
-            robot_namespace="${robot_namespace}"
-            frame_name="${prefix}_imu_frame"/>
+            frame_name="${prefix}_imu_frame"
+            topic_name="${topic_name}"
+            robot_namespace="${robot_namespace}"/>
     </xacro:macro>
 </robot>

File: hsrb_parts_description/urdf/sensors/kinetic/mynteye_imu.gazebo.xacro (robot description, xacro)
@@ -1,13 +1,13 @@
 <?xml version="1.0" ?>
 <robot name="hsrb" xmlns:xacro="http://ros.org/wiki/xacro">
-    <xacro:macro name="imu_gazebo" params="sensor_name frame_name topic_name robot_namespace">
+    <xacro:macro name="mynteye_imu_gazebo" params="sensor_name frame_name topic_name robot_namespace">
         <gazebo reference="${frame_name}">
             <sensor type="imu" name="${sensor_name}">
                 <update_rate>10.0</update_rate>
 	        <plugin name="${sensor_name}_plugin" filename="libgazebo_ros_imu_sensor.so">
-		    <updateRateHZ>50.0</updateRateHZ>
+		    <updateRateHZ>100.0</updateRateHZ>
 		    <bodyName>base_link</bodyName>
-                    <topicName>${robot_namespace}/${sensor_name}/data</topicName>
-                    <frameName>${personal_name}/${frame_name}</frameName>
+		    <topicName>${sensor_name}/${topic_name}</topicName>
+		    <frameName>${personal_name}/${frame_name}</frameName>
 		    <gaussianNoise>0.0</gaussianNoise>
 		    <xyzOffset>0.0 0.0 0.0</xyzOffset>

File: hsrc_description/robots/hsrc1s.urdf.xacro (robot description, xacro)
@@ -15,8 +15,11 @@
     <xacro:include filename="$(find hsrc_description)/urdf/wrist_v0/wrist.urdf.xacro" />
     <xacro:include filename="$(find hsrc_description)/urdf/hand_v0/hand.urdf.xacro" />
+    <xacro:arg name="personal_name" default="hsrb"/>
     <!-- constant -->
+    <xacro:property name="personal_name" value="$(arg personal_name)"/>
     <xacro:property name="robot_name" value="hsrb"/>
+    <xacro:property name="robot_type" value="hsrb"/>
     <!-- create robot -->
-    <xacro:hsrb_base prefix="base" robot_namespace="${robot_name}"/>
+    <xacro:hsrb_base prefix="base" personal_name="${personal_name}" robot_namespace="${robot_name}" robot_type="${robot_type}"/>
     <xacro:hsrb_torso prefix="torso" parent="base_link" mimic_joint="arm_lift_joint">
         <origin xyz="0.0 0.0 0.762" rpy="0.0 0.0 0.0"/>
@@ -36,8 +39,9 @@
     <gazebo>
         <plugin name="${robot_name}_ros_control" filename="lib${robot_name}_gazebo_ros_control.so">
-            <robotNamespace>${robot_name}</robotNamespace>
+            <robotNamespace>${personal_name}/${robot_name}</robotNamespace>
+            <legacyModeNS>false</legacyModeNS>
         </plugin>
         <plugin name="${robot_name}_p3d_ground_truth" filename="libgazebo_ros_p3d.so">
-            <robotNamespace>${robot_name}</robotNamespace>
+            <robotNamespace>${personal_name}/${robot_name}</robotNamespace>
             <bodyName>base_footprint</bodyName>
             <topicName>odom_ground_truth</topicName>

File: hsrc_description/urdf/base_v0/base.urdf.xacro (robot description, xacro)
@@ -132,5 +132,5 @@
     </xacro:macro>
     <!-- base -->
-    <xacro:macro name="hsrb_base" params="prefix robot_namespace">
+    <xacro:macro name="hsrb_base" params="prefix personal_name robot_namespace robot_type">
         <link name="base_footprint">
         </link>
@@ -210,5 +210,6 @@
             prefix="${prefix}"
             robot_namespace="${robot_namespace}"
-            parent="${prefix}_link">
+            parent="${prefix}_link"
+            min_angle="-2.1" max_angle="2.1">
             <origin xyz="0.167 0.0 0.1904" rpy="0.0 0.0 0.0" />
         </xacro:hokuyo_laser>
@@ -224,8 +225,8 @@
                 rpy="0.0 0.0 ${pi}" />
         </xacro:hsrb_bumper>
-        <xacro:imu_sensor prefix="${prefix}" robot_namespace="${robot_namespace}" parent="${prefix}_link">
+        <xacro:imu_sensor prefix="${prefix}" robot_namespace="${robot_namespace}" parent="${prefix}_link" topic_name="data">
             <origin xyz="0.003 -0.08594 0.203" rpy="0.0 0.0 0.0" />
         </xacro:imu_sensor>
-        <xacro:hsrb_base_gazebo prefix="${prefix}"/>
+        <xacro:hsrb_base_gazebo personal_name="${personal_name}" prefix="${prefix}" robot_type="${robot_type}"/>
         <xacro:hsrb_base_transmission prefix="${prefix}"/>
     </xacro:macro>

File: hsrc_description/urdf/hand_v0/hand.gazebo.xacro (robot description, xacro)
@@ -33,4 +33,5 @@
                 <error_tolerance>0.0872</error_tolerance>
                 <stall_timeout>2.0</stall_timeout>
+                <robot_namespace>${personal_name}/${robot_name}</robot_namespace>
             </plugin>
             <plugin name="hsrb_grasp_hack_plugin" filename="libhsrb_grasp_hack.so">
@@ -47,4 +48,5 @@
 		<!-- hand_palm_link is merged with wrist_ft_sensor_frame by fixed joint  -->
 		<palm_link>wrist_ft_sensor_frame</palm_link>
+                <robot_namespace>${personal_name}/${robot_name}</robot_namespace>
             </plugin>
         </gazebo>
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