Commit message: Fix namespace handling

File: hsrb_description/robots/hsrb1s.urdf.xacro (robot description, xacro)
@@ -19,5 +19,4 @@
     <xacro:property name="personal_name" value="$(arg personal_name)"/>
     <xacro:property name="robot_name" value="hsrb"/>
-    <xacro:property name="robot_type" value="hsrb"/>
     <!-- create robot -->
     <xacro:hsrb_base prefix="base" robot_namespace="${robot_name}"/>
@@ -43,5 +42,5 @@
         </plugin>
         <plugin name="${robot_name}_p3d_ground_truth" filename="libgazebo_ros_p3d.so">
-            <robotNamespace>${personal_name}/${robot_type}</robotNamespace>
+            <robotNamespace>${personal_name}/${robot_name}</robotNamespace>
             <bodyName>base_footprint</bodyName>
             <topicName>odom_ground_truth</topicName>

File: hsrb_description/robots/hsrb2s.urdf.xacro (robot description, xacro)
@@ -19,5 +19,4 @@
     <xacro:property name="personal_name" value="$(arg personal_name)"/>
     <xacro:property name="robot_name" value="hsrb"/>
-    <xacro:property name="robot_type" value="hsrb"/>
     <!-- create robot -->
     <xacro:hsrb_base prefix="base" robot_namespace="${robot_name}"/>
@@ -39,9 +38,9 @@
     <gazebo>
         <plugin name="${robot_name}_ros_control" filename="lib${robot_name}_gazebo_ros_control.so">
-            <robotNamespace>${personal_name}/${robot_type}</robotNamespace>
+            <robotNamespace>${personal_name}/${robot_name}</robotNamespace>
             <legacyModeNS>false</legacyModeNS>
         </plugin>
         <plugin name="${robot_name}_p3d_ground_truth" filename="libgazebo_ros_p3d.so">
-            <robotNamespace>${personal_name}/${robot_type}</robotNamespace>
+            <robotNamespace>${personal_name}/${robot_name}</robotNamespace>
             <bodyName>base_footprint</bodyName>
             <topicName>odom_ground_truth</topicName>

File: hsrb_description/robots/hsrb3s.urdf.xacro (robot description, xacro)
@@ -19,5 +19,4 @@
     <xacro:property name="personal_name" value="$(arg personal_name)"/>
     <xacro:property name="robot_name" value="hsrb"/>
-    <xacro:property name="robot_type" value="hsrb"/>
     <!-- create robot -->
     <xacro:hsrb_base prefix="base" robot_namespace="${robot_name}"/>
@@ -39,9 +38,9 @@
     <gazebo>
         <plugin name="${robot_name}_ros_control" filename="lib${robot_name}_gazebo_ros_control.so">
-            <robotNamespace>${personal_name}/${robot_type}</robotNamespace>
+            <robotNamespace>${personal_name}/${robot_name}</robotNamespace>
             <legacyModeNS>false</legacyModeNS>
         </plugin>
         <plugin name="${robot_name}_p3d_ground_truth" filename="libgazebo_ros_p3d.so">
-            <robotNamespace>${personal_name}/${robot_type}</robotNamespace>
+            <robotNamespace>${personal_name}/${robot_name}</robotNamespace>
             <bodyName>base_footprint</bodyName>
             <topicName>odom_ground_truth</topicName>

File: hsrb_description/robots/hsrb4s.urdf.xacro (robot description, xacro)
@@ -19,7 +19,6 @@
     <xacro:property name="personal_name" value="$(arg personal_name)"/>
     <xacro:property name="robot_name" value="hsrb"/>
-    <xacro:property name="robot_type" value="hsrb"/>
     <!-- create robot -->
-    <xacro:hsrb_base prefix="base" personal_name="${personal_name}" robot_namespace="${robot_name}" robot_type="${robot_type}" />
+    <xacro:hsrb_base prefix="base" personal_name="${personal_name}" robot_namespace="${robot_name}" robot_name="${robot_name}"/>
     <xacro:hsrb_torso prefix="torso" parent="base_link" mimic_joint="arm_lift_joint">
         <origin xyz="0.0 0.0 0.752" rpy="0.0 0.0 0.0"/>
@@ -39,9 +38,9 @@
     <gazebo>
         <plugin name="${robot_name}_ros_control" filename="lib${robot_name}_gazebo_ros_control.so">
-            <robotNamespace>${robot_name}</robotNamespace>
-            <legacyModeNS>true</legacyModeNS>
+            <robotNamespace>${personal_name}/${robot_name}</robotNamespace>
+            <legacyModeNS>false</legacyModeNS>
         </plugin>
-        <plugin name="${robot_type}_p3d_ground_truth" filename="libgazebo_ros_p3d.so">
-            <robotNamespace>${personal_name}/${robot_type}</robotNamespace>
+        <plugin name="${robot_name}_p3d_ground_truth" filename="libgazebo_ros_p3d.so">
+            <robotNamespace>${personal_name}/${robot_name}</robotNamespace>
             <bodyName>base_footprint</bodyName>
             <topicName>odom_ground_truth</topicName>

File: hsrb_description/urdf/base_v2/base.gazebo.xacro (robot description, xacro)
@@ -1,5 +1,5 @@
 <?xml version="1.0"?>
 <robot xmlns:xacro="http://ros.org/wiki/xacro">
-    <xacro:macro name="hsrb_base_gazebo" params="personal_name prefix robot_type">
+    <xacro:macro name="hsrb_base_gazebo" params="personal_name prefix robot_name">
         <gazebo_link name="${prefix}_link" gravity="true" collide="false" friction="0.9"/>
         <gazebo_link name="${prefix}_roll_link" gravity="true" collide="false" friction="0.9"/>
@@ -10,6 +10,6 @@
         <gazebo_link name="${prefix}_range_sensor_link" gravity="true" collide="false" friction="0.9"/>
         <gazebo_link name="${prefix}_imu_frame" gravity="true" collide="false" friction="0.9"/>
-        <gazebo_link_bumper name="${prefix}_f_bumper" personal_name="${personal_name}" robot_type="${robot_type}" gravity="true" collide="false" friction="0.9"/>
-        <gazebo_link_bumper name="${prefix}_b_bumper" personal_name="${personal_name}" robot_type="${robot_type}" gravity="true" collide="false" friction="0.9"/>
+        <gazebo_link_bumper name="${prefix}_f_bumper" personal_name="${personal_name}" robot_name="${robot_name}" gravity="true" collide="false" friction="0.9"/>
+        <gazebo_link_bumper name="${prefix}_b_bumper" personal_name="${personal_name}" robot_name="${robot_name}" gravity="true" collide="false" friction="0.9"/>
     </xacro:macro>
 </robot>

File: hsrb_description/urdf/base_v2/base.urdf.xacro (robot description, xacro)
@@ -132,5 +132,5 @@
     </xacro:macro>
     <!-- base -->
-    <xacro:macro name="hsrb_base" params="prefix personal_name robot_namespace robot_type">
+    <xacro:macro name="hsrb_base" params="prefix personal_name robot_namespace robot_name">
         <link name="base_footprint">
         </link>
@@ -228,5 +228,5 @@
                 rpy="0.0 0.0 ${pi}" />
         </xacro:hsrb_bumper>
-        <xacro:hsrb_base_gazebo personal_name="${personal_name}" prefix="${prefix}" robot_type="${robot_type}"/>
+        <xacro:hsrb_base_gazebo personal_name="${personal_name}" prefix="${prefix}" robot_name="${robot_name}"/>
         <xacro:hsrb_base_transmission prefix="${prefix}"/>
     </xacro:macro>

File: hsrb_description/urdf/common.xacro (robot description, xacro)
@@ -79,5 +79,5 @@
     </gazebo>
   </xacro:macro>
-  <xacro:macro name="gazebo_link_bumper" params="name personal_name robot_type gravity collide friction">
+  <xacro:macro name="gazebo_link_bumper" params="name personal_name robot_name gravity collide friction">
     <gazebo reference="${name}_link">
       <selfCollide>${collide}</selfCollide>
@@ -92,5 +92,5 @@
         </contact>
         <plugin name="hsrb_gazebo_ros_bumper_controller" filename="libhsrb_gazebo_ros_bumper.so">
-          <robotNamespace>${personal_name}/${robot_type}</robotNamespace>
+          <robotNamespace>${personal_name}/${robot_name}</robotNamespace>
           <bumperTopicName>${name}_sensor</bumperTopicName>
           <frameName>${name}_link</frameName>

File: hsrb_description/urdf/wrist_v0/wrist.urdf.xacro (robot description, xacro)
@@ -83,5 +83,5 @@
         <xacro:minebea_ft_sensor
             prefix="${prefix}"
-            robot_namespace="${personal_name}/${robot_namespace}"
+            robot_namespace="${personal_name}"
             parent="${prefix}_ft_sensor_mount_link">
             <origin xyz="0.0 0.0 0.0735" rpy="${pi} 0.0 0.0"/>

File: hsrb_parts_description/urdf/sensors/asus_xtion.gazebo.xacro (robot description, xacro)
@@ -42,4 +42,5 @@
                     <cameraName>${sensor_name}</cameraName>
                     <frameName>${topic_frame_id}</frameName>
+                    <robotNamespace>${robot_namespace}</robotNamespace>
                     <imageTopicName>/${robot_namespace}/${sensor_name}/rgb/image_rect_color</imageTopicName>
                     <cameraInfoTopicName>/${robot_namespace}/${sensor_name}/rgb/camera_info</cameraInfoTopicName>

File: hsrb_parts_description/urdf/sensors/minebea_ft_sensor.urdf.xacro (robot description, xacro)
@@ -18,5 +18,6 @@
         <xacro:minebea_ft_sensor_gazebo
             robot_namespace="${robot_namespace}"
-            joint_name="${prefix}_ft_sensor_frame_joint" ros_topic="${prefix}_wrench/raw" />
+            joint_name="${prefix}_ft_sensor_frame_joint"
+            ros_topic="${robot_name}/${prefix}_wrench/raw" />
     </xacro:macro>
 </robot>

File: hsrc_description/robots/hsrc1s.urdf.xacro (robot description, xacro)
@@ -19,7 +19,6 @@
     <xacro:property name="personal_name" value="$(arg personal_name)"/>
     <xacro:property name="robot_name" value="hsrb"/>
-    <xacro:property name="robot_type" value="hsrb"/>
     <!-- create robot -->
-    <xacro:hsrb_base prefix="base" personal_name="${personal_name}" robot_namespace="${robot_name}" robot_type="${robot_type}"/>
+    <xacro:hsrb_base prefix="base" personal_name="${personal_name}" robot_namespace="${robot_name}" robot_name="${robot_name}"/>
     <xacro:hsrb_torso prefix="torso" parent="base_link" mimic_joint="arm_lift_joint">
         <origin xyz="0.0 0.0 0.762" rpy="0.0 0.0 0.0"/>
@@ -39,6 +38,6 @@
     <gazebo>
         <plugin name="${robot_name}_ros_control" filename="lib${robot_name}_gazebo_ros_control.so">
-            <robotNamespace>${robot_name}</robotNamespace>
-            <legacyModeNS>true</legacyModeNS>
+            <robotNamespace>${personal_name}/${robot_name}</robotNamespace>
+            <legacyModeNS>false</legacyModeNS>
         </plugin>
         <plugin name="${robot_name}_p3d_ground_truth" filename="libgazebo_ros_p3d.so">

File: hsrc_description/urdf/base_v0/base.urdf.xacro (robot description, xacro)
@@ -132,5 +132,5 @@
     </xacro:macro>
     <!-- base -->
-    <xacro:macro name="hsrb_base" params="prefix personal_name robot_namespace robot_type">
+    <xacro:macro name="hsrb_base" params="prefix personal_name robot_namespace robot_name">
         <link name="base_footprint">
         </link>
@@ -228,5 +228,5 @@
             <origin xyz="0.003 -0.08594 0.203" rpy="0.0 0.0 0.0" />
         </xacro:imu_sensor>
-        <xacro:hsrb_base_gazebo personal_name="${personal_name}" prefix="${prefix}" robot_type="${robot_type}"/>
+        <xacro:hsrb_base_gazebo personal_name="${personal_name}" prefix="${prefix}" robot_name="${robot_name}"/>
         <xacro:hsrb_base_transmission prefix="${prefix}"/>
     </xacro:macro>

File: hsrc_description/urdf/wrist_v0/wrist.urdf.xacro (robot description, xacro)
@@ -83,5 +83,5 @@
         <xacro:minebea_ft_sensor
             prefix="${prefix}"
-            robot_namespace="${personal_name}/${robot_namespace}"
+            robot_namespace="${personal_name}"
 	    parent="${prefix}_ft_sensor_mount_link">
 	  <origin xyz="0.0 0.0 0.1" rpy="${pi} 0.0 0.0"/>
