Commit message: add control_period to hsrb4s.urdf.xacro

File: hsrb_description/robots/hsrb4s.urdf.xacro (robot description, xacro)
@@ -17,4 +17,5 @@
     <!-- constant -->
     <xacro:property name="robot_name" value="hsrb"/>
+    <xacro:property name="control_period" value="0.01"/>
     <!-- create robot -->
     <xacro:hsrb_base prefix="base" robot_namespace="${robot_name}"/>
@@ -35,6 +36,7 @@
     </xacro:hsrb_hand>
     <gazebo>
-        <plugin name="${robot_name}_ros_control" filename="libgazebo_ros_control.so">
+        <plugin name="${robot_name}_ros_control" filename="lib${robot_name}_gazebo_ros_control.so">
             <robotNamespace>${robot_name}</robotNamespace>
+            <controlPeriod>${control_period}</controlPeriod>
         </plugin>
         <plugin name="${robot_name}_p3d_ground_truth" filename="libgazebo_ros_p3d.so">

Commit message: Migrate hsrb_description to ROS2

File: hsrb_description/robots/hsrb4s.urdf.xacro (robot description, xacro)
@@ -1,8 +1,4 @@
 <?xml version="1.0"?>
-<robot name="hsrb"
-       xmlns:controller="http://playerstage.sourceforge.net/gazebo/xmlschema/#controller"
-       xmlns:interface="http://playerstage.sourceforge.net/gazebo/xmlschema/#interface"
-       xmlns:sensor="http://playerstage.sourceforge.net/gazebo/xmlschema/#sensor"
-       xmlns:xacro="http://ros.org/wiki/xacro">
+<robot name="hsrb" xmlns:xacro="http://ros.org/wiki/xacro">
     <!-- common xacro -->
     <xacro:include filename="$(find hsrb_description)/urdf/common.xacro" />
@@ -15,4 +11,6 @@
     <xacro:include filename="$(find hsrb_description)/urdf/wrist_v0/wrist.urdf.xacro" />
     <xacro:include filename="$(find hsrb_description)/urdf/hand_v0/hand.urdf.xacro" />
+    <xacro:arg name="gazebo_sim" default="False"/>
+    <xacro:arg name="rviz_sim" default="False"/>
     <xacro:arg name="personal_name" default=""/>
     <xacro:arg name="ground_truth_xyz_offset" default="0.0\ 0.0\ 0.0"/>
@@ -38,18 +36,12 @@
         <origin xyz="0.012 0.0 0.1405" rpy="0.0 0.0 ${pi}"/>
     </xacro:hsrb_hand>
-    <gazebo>
-        <plugin name="${robot_name}_ros_control" filename="lib${robot_name}_gazebo_ros_control.so">
-            <robotNamespace>${personal_name}/${robot_name}</robotNamespace>
-            <legacyModeNS>false</legacyModeNS>
-        </plugin>
-        <plugin name="${robot_name}_p3d_ground_truth" filename="lib${robot_name}_gazebo_ros_p3d.so">
-            <robotNamespace>${personal_name}/${robot_name}</robotNamespace>
-            <bodyName>base_footprint</bodyName>
-            <topicName>odom_ground_truth</topicName>
-            <frameName>map</frameName>
-            <updateRate>30</updateRate>
-	    <xyzOffset>$(arg ground_truth_xyz_offset)</xyzOffset>
-	    <rpyOffset>$(arg ground_truth_rpy_offset)</rpyOffset>
-        </plugin>
-    </gazebo>
+    <!-- Import ros2_control description -->
+    <xacro:if value="${not $(arg gazebo_sim) and not $(arg rviz_sim)}">
+      <xacro:include filename="$(find hsrb_description)/urdf/ros2_control.robot.xacro" />
+      <xacro:ros2_contorl_robot/>
+    </xacro:if>
+    <xacro:if value="$(arg gazebo_sim)">
+      <xacro:include filename="$(find hsrb_description)/urdf/ros2_control.gazebo.xacro" />
+      <xacro:ros2_contorl_gazebo/>
+    </xacro:if>
 </robot>

File: hsrb_description/urdf/arm_v0/arm.urdf.xacro (robot description, xacro)
@@ -1,5 +1,4 @@
 <?xml version="1.0"?>
 <robot name="arm" xmlns:xacro="http://ros.org/wiki/xacro">
-    <xacro:include filename="$(find hsrb_description)/urdf/arm_v0/arm.transmission.xacro"/>
     <xacro:include filename="$(find hsrb_description)/urdf/arm_v0/arm.gazebo.xacro"/>
     <!-- arm -->
@@ -84,5 +83,4 @@
         </link>
         <xacro:hsrb_arm_gazebo prefix="${prefix}"/>
-        <xacro:hsrb_arm_transmission prefix="${prefix}"/>
     </xacro:macro>
 </robot>

File: hsrb_description/urdf/base_v2/base.urdf.xacro (robot description, xacro)
@@ -1,5 +1,4 @@
 <?xml version="1.0"?>
 <robot name="base" xmlns:xacro="http://ros.org/wiki/xacro">
-    <xacro:include filename="$(find hsrb_description)/urdf/base_v2/base.transmission.xacro"/>
     <xacro:include filename="$(find hsrb_description)/urdf/base_v2/base.gazebo.xacro"/>
     <xacro:include filename="$(find hsrb_parts_description)/urdf/sensors/hokuyo_laser.urdf.xacro"/>
@@ -141,12 +140,12 @@
         <link name="${prefix}_link">
             <inertial>
-                <mass value="50.00"/>  <!-- use dummy weight to stabilize gazebo move base (real value: 11.017971)-->
+                <mass value="50.0"/>
                 <origin xyz="-0.025978 -0.005498 0.17633"/>
                 <inertia ixx="0.3742" ixy="0.000434172172" ixz="0.03088"
-                    iyy="0.3436" iyz="0.01775" izz="0.1509"/>
-            </inertial>
-            <visual>
-                <geometry>
-                    <mesh filename="package://hsrb_description/meshes/base_v2/base_light.dae" />
+                         iyy="0.3436" iyz="0.01775" izz="0.1509"/>
+            </inertial>
+            <visual>
+                <geometry>
+                    <mesh filename="package://hsrb_description/meshes/base_v2/base_light.dae"/>
                 </geometry>
             </visual>
@@ -229,5 +228,4 @@
         </xacro:hsrb_bumper>
         <xacro:hsrb_base_gazebo personal_name="${personal_name}" prefix="${prefix}" robot_name="${robot_name}"/>
-        <xacro:hsrb_base_transmission prefix="${prefix}"/>
     </xacro:macro>
 </robot>

File: hsrb_description/urdf/common.xacro (robot description, xacro)
@@ -2,40 +2,4 @@
 <robot xmlns:xacro="http://ros.org/wiki/xacro">
   <xacro:arg name="implicit_damping" default="false" />
-  <xacro:macro name="hsrb_position_joint_transmission" params="joint reduction">
-     <transmission name="${joint}_transmission">
-       <type>transmission_interface/SimpleTransmission</type>
-       <joint name="${joint}">
-         <hardwareInterface>hardware_interface/PositionJointInterface</hardwareInterface>
-       </joint>
-       <actuator name="${joint}_actuator">
-         <hardwareInterface>hardware_interface/PositionJointInterface</hardwareInterface>
-         <mechanicalReduction>${reduction}</mechanicalReduction>
-       </actuator>
-     </transmission>
-  </xacro:macro>
-  <xacro:macro name="hsrb_effort_joint_transmission" params="joint reduction">
-     <transmission name="${joint}_transmission">
-       <type>transmission_interface/SimpleTransmission</type>
-       <joint name="${joint}">
-         <hardwareInterface>hardware_interface/EffortJointInterface</hardwareInterface>
-       </joint>
-       <actuator name="${joint}_actuator">
-         <hardwareInterface>hardware_interface/EffortJointInterface</hardwareInterface>
-         <mechanicalReduction>${reduction}</mechanicalReduction>
-       </actuator>
-     </transmission>
-  </xacro:macro>
-  <xacro:macro name="hsrb_velocity_joint_transmission" params="joint reduction">
-      <transmission name="${prefix}_transmission">
-          <type>transmission_interface/SimpleTransmission</type>
-          <joint name="${joint}">
-            <hardwareInterface>hardware_interface/VelocityJointInterface</hardwareInterface>
-          </joint>
-          <actuator name="${joint}_actuator">
-              <hardwareInterface>hardware_interface/VelocityJointInterface</hardwareInterface>
-              <mechanicalReduction>${reduction}</mechanicalReduction>
-          </actuator>
-      </transmission>
-  </xacro:macro>
   <xacro:macro name="gazebo_link" params="name gravity collide friction">
     <gazebo reference="${name}">

File: hsrb_description/urdf/hand_v0/hand.gazebo.xacro (robot description, xacro)
@@ -26,14 +26,13 @@
         <xacro:gazebo_joint name="${prefix}_r_distal_joint"/>
         <gazebo>
-          <plugin name="hsrb_hrh_gripper_plugin" filename="libtmc_gazebo_hrh_gripper.so">
+          <plugin name="hsrb_hrh_gripper_plugin" filename="libtmc_gazebo_ros_hrh_gripper.so">
             <sensitiveness>0.05</sensitiveness>
             <update_rate>1000.0</update_rate>
             <max_torque>8.0</max_torque>
-            <!-- 5[deg] -->
             <error_tolerance>0.0872</error_tolerance>
             <stall_timeout>2.0</stall_timeout>
             <robot_namespace>${personal_name}/${robot_name}</robot_namespace>
           </plugin>
-          <plugin name="hsrb_grasp_hack_plugin" filename="libhsrb_grasp_hack.so">
+          <!-- <plugin name="hsrb_grasp_hack_plugin" filename="libhsrb_grasp_hack.so">
             <grasp_check>
               <attach_steps>1</attach_steps>
@@ -45,9 +44,9 @@
             <gripper_link>${prefix}_l_distal_link</gripper_link>
             <gripper_link>${prefix}_r_spring_proximal_link</gripper_link>
-            <gripper_link>${prefix}_l_spring_proximal_link</gripper_link>
+            <gripper_link>${prefix}_l_spring_proximal_link</gripper_link> -->
 	    <!-- hand_palm_link is merged with wrist_ft_sensor_frame by fixed joint  -->
-            <palm_link>wrist_ft_sensor_frame</palm_link>
+            <!-- <palm_link>wrist_ft_sensor_frame</palm_link>
             <robot_namespace>${personal_name}/${robot_name}</robot_namespace>
-          </plugin>
+          </plugin> -->
         </gazebo>
     </xacro:macro>

File: hsrb_description/urdf/hand_v0/hand.urdf.xacro (robot description, xacro)
@@ -1,5 +1,4 @@
 <?xml version="1.0"?>
 <robot name="hand" xmlns:xacro="http://ros.org/wiki/xacro">
-    <xacro:include filename="$(find hsrb_description)/urdf/hand_v0/hand.transmission.xacro"/>
     <xacro:include filename="$(find hsrb_description)/urdf/hand_v0/hand.gazebo.xacro"/>
     <xacro:include filename="$(find hsrb_parts_description)/urdf/sensors/wide_camera.urdf.xacro"/>
@@ -78,5 +77,4 @@
         </xacro:wide_camera>
         <xacro:hsrb_hand_gazebo prefix="${prefix}"/>
-        <xacro:hsrb_hand_transmission prefix="${prefix}"/>
     </xacro:macro>
     <!-- gripper finger proximal base -->

File: hsrb_description/urdf/head_v2/head.urdf.xacro (robot description, xacro)
@@ -1,5 +1,4 @@
 <?xml version="1.0"?>
 <robot name="head" xmlns:xacro="http://ros.org/wiki/xacro">
-    <xacro:include filename="$(find hsrb_description)/urdf/head_v2/head.transmission.xacro"/>
     <xacro:include filename="$(find hsrb_description)/urdf/head_v2/head.gazebo.xacro"/>
     <xacro:include filename="$(find hsrb_parts_description)/urdf/sensors/asus_xtion.urdf.xacro"/>
@@ -89,5 +88,4 @@
         </xacro:asus_xtion>
         <xacro:hsrb_head_gazebo prefix="${prefix}"/>
-        <xacro:hsrb_head_transmission prefix="${prefix}"/>
     </xacro:macro>
 </robot>

File: hsrb_description/urdf/torso_v0/torso.gazebo.xacro (robot description, xacro)
@@ -5,7 +5,7 @@
         <xacro:gazebo_joint_mimic name="${prefix}_lift_joint"/>
         <gazebo>
-            <plugin name="torso_mimic_plugin" filename="libtmc_gazebo_mimic_plugin.so">
+            <plugin name="torso_mimic_plugin" filename="libtmc_gazebo_ros_mimic_joint.so">
                 <joint>${prefix}_lift_joint</joint>
-                <mimicJoint>${mimic_joint}</mimicJoint>
+                <mimic_joint>${mimic_joint}</mimic_joint>
                 <multiplier>0.5</multiplier>
             </plugin>

File: hsrb_description/urdf/wrist_v0/wrist.urdf.xacro (robot description, xacro)
@@ -1,5 +1,4 @@
 <?xml version="1.0"?>
 <robot name="wrist" xmlns:xacro="http://ros.org/wiki/xacro">
-    <xacro:include filename="$(find hsrb_description)/urdf/wrist_v0/wrist.transmission.xacro"/>
     <xacro:include filename="$(find hsrb_description)/urdf/wrist_v0/wrist.gazebo.xacro"/>
     <xacro:include filename="$(find hsrb_parts_description)/urdf/sensors/minebea_ft_sensor.urdf.xacro"/>
@@ -88,5 +87,4 @@
         </xacro:minebea_ft_sensor>
         <xacro:hsrb_wrist_gazebo prefix="${prefix}"/>
-        <xacro:hsrb_wrist_transmission prefix="${prefix}"/>
     </xacro:macro>
 </robot>
