Commit message: Release/2.1.0

File: hsrb_description/robots/hsrb4s.urdf.xacro (robot description, xacro)
@@ -12,4 +12,5 @@
     <xacro:include filename="$(find hsrb_description)/urdf/hand_v0/hand.urdf.xacro" />
     <xacro:arg name="gazebo_sim" default="False"/>
+    <xacro:arg name="ignition_gazebo_sim" default="False"/>
     <xacro:arg name="rviz_sim" default="False"/>
     <xacro:arg name="personal_name" default=""/>
@@ -37,5 +38,5 @@
     </xacro:hsrb_hand>
     <!-- Import ros2_control description -->
-    <xacro:if value="${not $(arg gazebo_sim) and not $(arg rviz_sim)}">
+    <xacro:if value="${not $(arg gazebo_sim) and not $(arg ignition_gazebo_sim) and not $(arg rviz_sim)}">
       <xacro:include filename="$(find hsrb_description)/urdf/ros2_control.robot.xacro" />
       <xacro:ros2_contorl_robot/>
@@ -45,4 +46,8 @@
       <xacro:ros2_contorl_gazebo/>
     </xacro:if>
+    <xacro:if value="$(arg ignition_gazebo_sim)">
+      <xacro:include filename="$(find hsrb_description)/urdf/ros2_control.ignition_gazebo.xacro" />
+      <xacro:ros2_contorl_gazebo/>
+    </xacro:if>
     <xacro:if value="$(arg rviz_sim)">
       <xacro:include filename="$(find hsrb_description)/urdf/ros2_control.rviz.xacro" />

File: hsrb_description/urdf/arm_v0/arm.urdf.xacro (robot description, xacro)
@@ -42,5 +42,5 @@
                 <mass value="1.339295"/>
                 <origin xyz="0.000632 0.006404 0.118529"/>
-                <inertia ixx="7.528" ixy="-0.000020284207" ixz="-0.000022947194"
+                <inertia ixx="0.007528" ixy="-0.000020284207" ixz="-0.000022947194"
                     iyy="0.007102" iyz="-0.000091796075" izz="0.001552"/>
             </inertial>

File: hsrb_description/urdf/base_v2/base.gazebo.xacro (robot description, xacro)
@@ -14,17 +14,4 @@
         <xacro:gazebo_link_bumper name="${prefix}_f_bumper" robot_namespace="${robot_namespace}" gravity="true" collide="false" friction="0.9"/>
         <xacro:gazebo_link_bumper name="${prefix}_b_bumper" robot_namespace="${robot_namespace}" gravity="true" collide="false" friction="0.9"/>
-        <gazebo>
-            <plugin name="odom_ground_truth" filename="libtmc_gazebo_ros_p3d.so">
-                <body_name>${prefix}_footprint</body_name>
-                <frame_name>map</frame_name>
-                <update_rate>30</update_rate>
-                <xyz_offset>$(arg ground_truth_xyz_offset)</xyz_offset>
-                <rpy_offset>$(arg ground_truth_rpy_offset)</rpy_offset>
-                <ros>
-                    <namespace>${robot_namespace}</namespace>
-                    <remapping>odom:=odom_ground_truth</remapping>
-                </ros>
-            </plugin>
-        </gazebo>
     </xacro:macro>
 </robot>

File: hsrb_description/urdf/base_v2/base.urdf.xacro (robot description, xacro)
@@ -115,6 +115,6 @@
                 <mass value="0.06"/>
                 <inertia
-                    ixx="0.001437"  ixy="0.0"  ixz="0.0"
-                    iyy="0.001437" iyz="0.0" izz="0.002875" />
+                    ixx="0.001537"  ixy="0.0"  ixz="0.0"
+                    iyy="0.001537" iyz="0.0" izz="0.002875" />
             </inertial>
             <visual>

File: hsrb_description/urdf/common.xacro (robot description, xacro)
@@ -1,4 +1,5 @@
 <?xml version="1.0"?>
 <robot xmlns:xacro="http://ros.org/wiki/xacro">
+  <xacro:arg name="ignition_gazebo_sim" default="False" />
   <xacro:arg name="implicit_damping" default="false" />
   <xacro:macro name="gazebo_link" params="name gravity collide friction">
@@ -49,17 +50,28 @@
       <mu1>${friction}</mu1>
       <mu2>${friction}</mu2>
-      <sensor name="${name}_contact" type="contact">
-        <always_on>true</always_on>
-        <update_rate>10</update_rate>
-        <contact>
-          <collision>${name}_link_collision</collision>
-        </contact>
-        <plugin name="${name}_bumper_controller" filename="libtmc_gazebo_ros_bumper.so">
-          <ros>
-            <namespace>${robot_namespace}</namespace>
-            <remapping>bumper_states:=${name}_sensor</remapping>
-          </ros>
-        </plugin>
-      </sensor>
+      <xacro:if value="$(arg ignition_gazebo_sim)">
+        <sensor name="${name}_contact" type="contact">
+          <always_on>true</always_on>
+          <update_rate>10</update_rate>
+          <contact>
+            <collision>${name}_link_collision</collision>
+          </contact>
+        </sensor>
+      </xacro:if>
+      <xacro:unless value="$(arg ignition_gazebo_sim)">
+        <sensor name="${name}_contact" type="contact">
+          <always_on>true</always_on>
+          <update_rate>10</update_rate>
+          <contact>
+            <collision>${name}_link_collision</collision>
+          </contact>
+          <plugin name="${name}_bumper_controller" filename="libtmc_gazebo_ros_bumper.so">
+            <ros>
+              <namespace>${robot_namespace}</namespace>
+              <remapping>bumper_states:=${name}_sensor</remapping>
+            </ros>
+          </plugin>
+        </sensor>
+      </xacro:unless>
     </gazebo>
   </xacro:macro>

File: hsrb_description/urdf/hand_v0/hand.urdf.xacro (robot description, xacro)
@@ -21,6 +21,6 @@
                 <mass value="0.001"/>
                 <inertia
-                    ixx="0.0" ixy="0.0" ixz="0.0"
-                    iyy="0.0" iyz="0.0" izz="0.0"/>
+                    ixx="0.001" ixy="0.0" ixz="0.0"
+                    iyy="0.001" iyz="0.0" izz="0.001"/>
             </inertial>
         </link>
@@ -143,6 +143,6 @@
                 <origin xyz="0.021418 0.00248 0.022688"/>
                 <inertia
-                    ixx="0.00" ixy="-0.00000" ixz="-0.0000"
-                    iyy="0.00" iyz="-0.00000" izz="0.00000"/>
+                    ixx="0.001" ixy="-0.00000" ixz="-0.0000"
+                    iyy="0.001" iyz="-0.00000" izz="0.001"/>
             </inertial>
             <visual>
@@ -152,6 +152,7 @@
             </visual>
             <collision>
-                <geometry>
-                    <mesh filename="package://hsrb_description/meshes/hand_v0/l_proximal.stl" />
+                <origin xyz="0.0169 -0.004125 0.035" rpy="0.0 0.0 0.0" />
+                <geometry>
+                    <box size="0.0362 0.01575 0.04"/>
                 </geometry>
             </collision>
@@ -166,6 +167,6 @@
                 <origin xyz="0.011116 0.005679 0.017532"/>
                 <inertia
-                    ixx="0.0" ixy="-0.00" ixz="0.0"
-                    iyy="0.0" iyz="-0.000" izz="0.0"/>
+                    ixx="0.001" ixy="-0.00" ixz="0.0"
+                    iyy="0.001" iyz="-0.000" izz="0.001"/>
             </inertial>
             <visual>
@@ -175,6 +176,13 @@
             </visual>
             <collision>
-                <geometry>
-                    <mesh filename="package://hsrb_description/meshes/hand_v0/l_distal.stl" />
+                <origin xyz="0.02 0.014 0.025" rpy="0.0 0.0 0.0" />
+                <geometry>
+                    <box size="0.04 0.01 0.032"/>
+                </geometry>
+            </collision>
+            <collision>
+                <origin xyz="0.02 0.0015 0.02" rpy="0.0 0.0 0.0" />
+                <geometry>
+                    <box size="0.04 0.023 0.04"/>
                 </geometry>
             </collision>
@@ -197,6 +205,6 @@
                 <mass value="0.001"/>
                 <inertia
-                    ixx="0.0" ixy="0.0" ixz="0.0"
-                    iyy="0.0" iyz="0.0" izz="0.0"/>
+                    ixx="0.001" ixy="0.0" ixz="0.0"
+                    iyy="0.001" iyz="0.0" izz="0.001"/>
             </inertial>
             <visual>
@@ -220,6 +228,6 @@
                 <origin xyz="0.013203 0.002096 0.023311"/>
                 <inertia
-                    ixx="0.0" ixy="0.0" ixz="0.0"
-                    iyy="0.0" iyz="0.0" izz="0.0"/>
+                    ixx="0.001" ixy="0.0" ixz="0.0"
+                    iyy="0.001" iyz="0.0" izz="0.001"/>
             </inertial>
             <visual>
@@ -229,6 +237,7 @@
             </visual>
             <collision>
-                <geometry>
-                    <mesh filename="package://hsrb_description/meshes/hand_v0/r_proximal.stl" />
+                <origin xyz="0.0169 0.004125 0.035" rpy="0.0 0.0 0.0" />
+                <geometry>
+                    <box size="0.0362 0.01575 0.04"/>
                 </geometry>
             </collision>
@@ -243,6 +252,6 @@
                 <origin xyz="0.014256 -0.008321 0.015591"/>
                 <inertia
-                    ixx="0.0" ixy="0.0" ixz="0.0"
-                    iyy="0.0" iyz="0.0" izz="0.0"/>
+                    ixx="0.001" ixy="0.0" ixz="0.0"
+                    iyy="0.001" iyz="0.0" izz="0.001"/>
             </inertial>
             <visual>
@@ -252,6 +261,13 @@
             </visual>
             <collision>
-                <geometry>
-                    <mesh filename="package://hsrb_description/meshes/hand_v0/r_distal.stl" />
+                <origin xyz="0.02 -0.014 0.025" rpy="0.0 0.0 0.0" />
+                <geometry>
+                    <box size="0.04 0.01 0.032"/>
+                </geometry>
+            </collision>
+            <collision>
+                <origin xyz="0.02 -0.0015 0.02" rpy="0.0 0.0 0.0" />
+                <geometry>
+                    <box size="0.04 0.023 0.04"/>
                 </geometry>
             </collision>

File: hsrb_description/urdf/torso_v0/torso.gazebo.xacro (robot description, xacro)
@@ -4,11 +4,4 @@
         <xacro:gazebo_link name="${prefix}_lift_link" gravity="true" collide="false" friction="0.9"/>
         <xacro:gazebo_joint_mimic name="${prefix}_lift_joint"/>
-        <gazebo>
-            <plugin name="torso_mimic_plugin" filename="libtmc_gazebo_ros_mimic_joint.so">
-                <joint>${prefix}_lift_joint</joint>
-                <mimic_joint>${mimic_joint}</mimic_joint>
-                <multiplier>0.5</multiplier>
-            </plugin>
-        </gazebo>
     </xacro:macro>
 </robot>

File: hsrb_description/urdf/wrist_v0/wrist.urdf.xacro (robot description, xacro)
@@ -34,5 +34,5 @@
             </visual>
             <collision>
-                <origin xyz="0.0 0.0 0.03" rpy="0.0 0.0 0.0"/>
+                <origin xyz="0.0 0.0 0.025" rpy="0.0 0.0 0.0"/>
                 <geometry>
                     <cylinder radius="0.017" length="0.04" />
@@ -75,6 +75,13 @@
             </visual>
             <collision>
+                <origin xyz="-0.027 0.000 0.0945" rpy="0.0 0.0 0.0" />
                 <geometry>
-                    <mesh filename="package://hsrb_description/meshes/wrist_v0/wrist_roll.stl" />
+                    <box size="0.040 0.102 0.093"/>
+                </geometry>
+            </collision>
+            <collision>
+                <origin xyz="-0.0080 0.00 0.0805" rpy="0.0 0.0 0.0" />
+                <geometry>
+                    <box size="0.079 0.102 0.065"/>
                 </geometry>
             </collision>

File: hsrb_parts_description/urdf/sensors/asus_xtion.gazebo.xacro (robot description, xacro)
@@ -37,11 +37,13 @@
                     <min_depth>0.5</min_depth>
                     <max_depth>9.2</max_depth>
+                    <cx>0.0</cx>
+                    <cy>0.0</cy>
                     <ros>
-                      <namespace>${robot_namespace}</namespace>
-                      <remapping>${sensor_name}/image_raw:=${sensor_name}/rgb/image_rect_color</remapping>
-                      <remapping>${sensor_name}/camera_info:=${sensor_name}/rgb/camera_info</remapping>
-                      <remapping>${sensor_name}/depth/image_raw:=${sensor_name}/depth_registered/image_rect_raw</remapping>
-                      <remapping>${sensor_name}/depth/camera_info:=${sensor_name}/depth_registered/camera_info</remapping>
-                      <remapping>${sensor_name}/points:=${sensor_name}/depth_registered/rectified_points</remapping>
+                        <namespace>${robot_namespace}</namespace>
+                        <remapping>${sensor_name}/image_raw:=${sensor_name}/rgb/image_rect_color</remapping>
+                        <remapping>${sensor_name}/camera_info:=${sensor_name}/rgb/camera_info</remapping>
+                        <remapping>${sensor_name}/depth/image_raw:=${sensor_name}/depth_registered/image_rect_raw</remapping>
+                        <remapping>${sensor_name}/depth/camera_info:=${sensor_name}/depth_registered/camera_info</remapping>
+                        <remapping>${sensor_name}/points:=${sensor_name}/depth_registered/rectified_points</remapping>
                     </ros>
                 </plugin>
@@ -49,3 +51,46 @@
         </gazebo>
     </xacro:macro>
+    <xacro:macro name="asus_xtion_gazebo_ignition" params="robot_namespace sensor_name parent_frame topic_frame_id">
+        <gazebo reference="${parent_frame}">
+            <sensor type="camera" name="openni_camera_camera_rgb">
+                <always_on>0</always_on>
+                <update_rate>30</update_rate>
+                <visualize>true</visualize>
+                <camera>
+                    <horizontal_fov>1.047</horizontal_fov>
+                    <image>
+                        <width>640</width>
+                        <height>480</height>
+                        <format>B8G8R8</format>
+                    </image>
+                    <clip>
+                        <near>0.1</near>
+                        <far>100</far>
+                    </clip>
+                </camera>
+                <gz_frame_id>${topic_frame_id}</gz_frame_id>
+                <topic>${robot_namespace}/${sensor_name}/rgb/image_rect_color</topic>
+            </sensor>
+            <sensor type="depth_camera" name="openni_camera_camera_depth">
+                <always_on>0</always_on>
+                <update_rate>30</update_rate>
+                <visualize>true</visualize>
+                <camera>
+                    <horizontal_fov>1.047</horizontal_fov>
+                    <image>
+                        <width>640</width>
+                        <height>480</height>
+                        <!-- Not working. Float only -->
+                        <format>L_INT16</format>
+                    </image>
+                    <clip>
+                        <near>0.1</near>
+                        <far>100</far>
+                    </clip>
+                </camera>
+                <gz_frame_id>${topic_frame_id}</gz_frame_id>
+                <topic>${robot_namespace}/${sensor_name}/depth_registered/image</topic>
+            </sensor>
+        </gazebo>
+    </xacro:macro>
 </robot>

File: hsrb_parts_description/urdf/sensors/asus_xtion.urdf.xacro (robot description, xacro)
@@ -2,4 +2,5 @@
 <robot name="hsrb" xmlns:xacro="http://ros.org/wiki/xacro">
     <xacro:include filename="$(find hsrb_parts_description)/urdf/sensors/asus_xtion.gazebo.xacro"/>
+    <xacro:arg name="ignition_gazebo_sim" default="false" />
     <!-- rgbd_sensor -->
     <xacro:macro name="asus_xtion" params="prefix parent robot_namespace sensor_name *origin">
@@ -40,9 +41,18 @@
             </inertial>
         </link>
-        <xacro:asus_xtion_gazebo
-            robot_namespace="${robot_namespace}"
-            sensor_name="${prefix}_${sensor_name}"
-            parent_frame="${prefix}_${sensor_name}_gazebo_frame"
-            topic_frame_id="${prefix}_${sensor_name}_rgb_frame" />
+        <xacro:if value="$(arg ignition_gazebo_sim)">
+            <xacro:asus_xtion_gazebo_ignition
+                robot_namespace="${robot_namespace}"
+                sensor_name="${prefix}_${sensor_name}"
+                parent_frame="${prefix}_${sensor_name}_gazebo_frame"
+                topic_frame_id="${prefix}_${sensor_name}_rgb_frame" />
+        </xacro:if>
+        <xacro:unless value="$(arg ignition_gazebo_sim)">
+            <xacro:asus_xtion_gazebo
+                robot_namespace="${robot_namespace}"
+                sensor_name="${prefix}_${sensor_name}"
+                parent_frame="${prefix}_${sensor_name}_gazebo_frame"
+                topic_frame_id="${prefix}_${sensor_name}_rgb_frame" />
+        </xacro:unless>
     </xacro:macro>
 </robot>

File: hsrb_parts_description/urdf/sensors/hokuyo_laser.gazebo.xacro (robot description, xacro)
@@ -23,8 +23,9 @@
                     </range>
                 </ray>
-                <plugin name="${sensor_name}" filename="libgazebo_ros_ray_sensor.so">
+                <plugin name="hokuyo_laser" filename="libgazebo_ros_ray_sensor.so">
                     <output_type>sensor_msgs/LaserScan</output_type>
                     <frame_name>${frame_name}</frame_name>
                     <ros>
+                        <namespace>${robot_namespace}</namespace>
                         <remapping>~/out:=${ros_topic}</remapping>
                     </ros>
@@ -36,30 +37,30 @@
         <gazebo reference="${frame_name}">
             <sensor name="${sensor_name}" type="gpu_lidar">
-            <pose>0 0 0 0 0 0</pose>
-            <topic>${robot_namespace}/${sensor_name}/${ros_topic}</topic>
-            <gz_frame_id>${frame_name}</gz_frame_id>
-            <update_rate>30.0</update_rate>
-            <visualize>$(arg gazebo_visualization_enabled)</visualize>
-            <lidar>
-                <scan>
-                <horizontal>
-                    <samples>721</samples>
-                    <resolution>1</resolution>
-                    <min_angle>${min_angle}</min_angle>
-                    <max_angle>${max_angle}</max_angle>
-                </horizontal>
-                <vertical>
-                    <samples>1</samples>
-                    <resolution>1</resolution>
-                    <min_angle>0.0</min_angle>
-                    <max_angle>0.0</max_angle>
-                </vertical>
-                </scan>
-                <range>
-                <min>0.05</min>
-                <max>60.0</max>
-                <resolution>0.001</resolution>
-                </range>
-            </lidar>
+                <pose>0 0 0 0 0 0</pose>
+                <topic>${robot_namespace}/${sensor_name}/${ros_topic}</topic>
+                <gz_frame_id>${frame_name}</gz_frame_id>
+                <update_rate>30.0</update_rate>
+                <visualize>$(arg gazebo_visualization_enabled)</visualize>
+                <lidar>
+                    <scan>
+                        <horizontal>
+                            <samples>721</samples>
+                            <resolution>1</resolution>
+                            <min_angle>${min_angle}</min_angle>
+                            <max_angle>${max_angle}</max_angle>
+                        </horizontal>
+                        <vertical>
+                            <samples>1</samples>
+                            <resolution>1</resolution>
+                            <min_angle>0.0</min_angle>
+                            <max_angle>0.0</max_angle>
+                        </vertical>
+                    </scan>
+                    <range>
+                        <min>0.05</min>
+                        <max>60.0</max>
+                        <resolution>0.001</resolution>
+                    </range>
+                </lidar>
             </sensor>
         </gazebo>

File: hsrb_parts_description/urdf/sensors/minebea_ft_sensor.gazebo.xacro (robot description, xacro)
@@ -17,3 +17,16 @@
         </gazebo>
     </xacro:macro>
+    <xacro:macro name="minebea_ft_sensor_gazebo_ignition" params="robot_namespace joint_name ros_topic">
+        <gazebo reference="${joint_name}">
+            <sensor type="force_torque" name="${joint_name}_force_torque_sensor">
+                <update_rate>30.0</update_rate>
+                <topic>${robot_namespace}/${ros_topic}</topic>
+                <gz_frame_id>${personal_name}/wrist_ft_sensor_frame</gz_frame_id>
+                <force_torque>
+                    <frame>sensor</frame>
+                    <measure_direction>parent_to_child</measure_direction>
+                </force_torque>
+            </sensor>
+        </gazebo>
+    </xacro:macro>
 </robot>

File: hsrb_parts_description/urdf/sensors/minebea_ft_sensor.urdf.xacro (robot description, xacro)
@@ -2,4 +2,5 @@
 <robot name="hsrb" xmlns:xacro="http://ros.org/wiki/xacro">
     <xacro:include filename="$(find hsrb_parts_description)/urdf/sensors/minebea_ft_sensor.gazebo.xacro"/>
+    <xacro:arg name="ignition_gazebo_sim" default="false" />
     <xacro:macro name="minebea_ft_sensor" params="prefix robot_namespace parent *origin">
         <joint name="${prefix}_ft_sensor_frame_joint" type="revolute">
@@ -16,8 +17,16 @@
             </inertial>
         </link>
-        <xacro:minebea_ft_sensor_gazebo
-            robot_namespace="${robot_namespace}"
-            joint_name="${prefix}_ft_sensor_frame_joint"
-            ros_topic="${prefix}_wrench/raw" />
+        <xacro:if value="$(arg ignition_gazebo_sim)">
+            <xacro:minebea_ft_sensor_gazebo_ignition
+                robot_namespace="${robot_namespace}"
+                joint_name="${prefix}_ft_sensor_frame_joint"
+                ros_topic="${prefix}_wrench/raw"/>
+        </xacro:if>
+        <xacro:unless value="$(arg ignition_gazebo_sim)">
+            <xacro:minebea_ft_sensor_gazebo
+                robot_namespace="${robot_namespace}"
+                joint_name="${prefix}_ft_sensor_frame_joint"
+                ros_topic="${prefix}_wrench/raw"/>
+        </xacro:unless>
     </xacro:macro>
 </robot>

File: hsrb_parts_description/urdf/sensors/mynteye_imu.urdf.xacro (robot description, xacro)
@@ -6,13 +6,13 @@
             <sensor type="imu" name="${sensor_name}">
                 <update_rate>10.0</update_rate>
-	        <plugin name="${sensor_name}_plugin" filename="libgazebo_ros_imu_sensor.so">
-		    <updateRateHZ>100.0</updateRateHZ>
-		    <bodyName>base_link</bodyName>
-		    <topicName>${sensor_name}/${topic_name}</topicName>
-		    <frameName>${personal_name}/${frame_name}</frameName>
-		    <gaussianNoise>0.0</gaussianNoise>
-		    <xyzOffset>0.0 0.0 0.0</xyzOffset>
-		    <rpyOffset>0.0 -0.0 0.0</rpyOffset>
-		</plugin>
+                <plugin name="${sensor_name}_plugin" filename="libgazebo_ros_imu_sensor.so">
+                    <updateRateHZ>100.0</updateRateHZ>
+                    <bodyName>base_link</bodyName>
+                    <topicName>${sensor_name}/${topic_name}</topicName>
+                    <frameName>${personal_name}/${frame_name}</frameName>
+                    <gaussianNoise>0.0</gaussianNoise>
+                    <xyzOffset>0.0 0.0 0.0</xyzOffset>
+                    <rpyOffset>0.0 -0.0 0.0</rpyOffset>
+                </plugin>
                 <imu>
                     <noise>
