Commit message: Release/2.1.0

File: hsrb_parts_description/urdf/sensors/pointgrey_chameleon.gazebo.xacro (robot description, xacro)
@@ -41,3 +41,36 @@
         </gazebo>
     </xacro:macro>
+    <xacro:macro name="pointgrey_chameleon_gazebo_ignition" params="sensor_name parent_frame topic_frame_id robot_namespace baseline">
+        <gazebo reference="${parent_frame}">
+            <sensor type="camera" name="${sensor_name}">
+                <update_rate>4.0</update_rate>
+                <camera name="${sensor_name}">
+                    <horizontal_fov>1.16762527</horizontal_fov>
+                    <image>
+                        <width>1280</width>
+                        <height>960</height>
+                        <format>R8G8B8</format>
+                    </image>
+                    <clip>
+                        <near>0.05</near>
+                        <far>100</far>
+                    </clip>
+                    <noise>
+                        <type>gaussian</type>
+                        <mean>0.0</mean>
+                        <stddev>0.007</stddev>
+                    </noise>
+                    <distortion>
+                        <k1>0.0</k1>
+                        <k2>0.0</k2>
+                        <k3>0.0</k3>
+                        <p1>0.0</p1>
+                        <p2>0.0</p2>
+                    </distortion>
+                </camera>
+                <gz_frame_id>${topic_frame_id}</gz_frame_id>
+                <topic>${robot_namespace}/${sensor_name}/image_rect_color</topic>
+            </sensor>
+        </gazebo>
+    </xacro:macro>
 </robot>

File: hsrb_parts_description/urdf/sensors/pointgrey_chameleon.urdf.xacro (robot description, xacro)
@@ -2,4 +2,5 @@
 <robot xmlns:xacro="http://ros.org/wiki/xacro">
     <xacro:include filename="$(find hsrb_parts_description)/urdf/sensors/pointgrey_chameleon.gazebo.xacro"/>
+    <xacro:arg name="ignition_gazebo_sim" default="false" />
     <xacro:macro name="pointgrey_chameleon" params="prefix parent robot_namespace *origin baseline">
         <joint name="${prefix}_camera_joint" type="fixed">
@@ -33,10 +34,20 @@
             </inertial>
         </link>
-        <xacro:pointgrey_chameleon_gazebo
-            sensor_name="${prefix}_camera"
-            parent_frame="${prefix}_camera_gazebo_frame"
-            topic_frame_id="${prefix}_camera_frame"
-            robot_namespace="${robot_namespace}"
-            baseline="${baseline}" />
+        <xacro:if value="$(arg ignition_gazebo_sim)">
+            <xacro:pointgrey_chameleon_gazebo_ignition
+                sensor_name="${prefix}_camera"
+                parent_frame="${prefix}_camera_gazebo_frame"
+                topic_frame_id="${prefix}_camera_frame"
+                robot_namespace="${robot_namespace}"
+                baseline="${baseline}" />
+        </xacro:if>
+        <xacro:unless value="$(arg ignition_gazebo_sim)">
+            <xacro:pointgrey_chameleon_gazebo
+                sensor_name="${prefix}_camera"
+                parent_frame="${prefix}_camera_gazebo_frame"
+                topic_frame_id="${prefix}_camera_frame"
+                robot_namespace="${robot_namespace}"
+                baseline="${baseline}" />
+        </xacro:unless>
     </xacro:macro>
 </robot>

File: hsrb_parts_description/urdf/sensors/wide_camera.gazebo.xacro (robot description, xacro)
@@ -1,3 +1,3 @@
-<?xml version="1.0" ?>
+<?xml version="1.0"?>
 <robot name="hsrb" xmlns:xacro="http://ros.org/wiki/xacro">
     <xacro:macro name="wide_camera_gazebo" params="robot_namespace sensor_name parent_frame topic_frame_id">
@@ -29,5 +29,6 @@
                     </distortion>
                 </camera>
-                <plugin name="${sensor_name}_camera_controller" filename="libgazebo_ros_camera.so">
+                <plugin name="${sensor_name}_camera_controller"
+                    filename="libgazebo_ros_camera.so">
                     <camera_name>${sensor_name}</camera_name>
                     <frame_name>${topic_frame_id}</frame_name>
@@ -40,3 +41,36 @@
         </gazebo>
     </xacro:macro>
+    <xacro:macro name="wide_camera_gazebo_ignition" params="robot_namespace sensor_name parent_frame topic_frame_id">
+        <gazebo reference="${parent_frame}">
+            <sensor type="camera" name="${sensor_name}">
+                <update_rate>10.0</update_rate>
+                <camera name="${sensor_name}">
+                    <horizontal_fov>2.00</horizontal_fov>
+                    <image>
+                        <width>640</width>
+                        <height>480</height>
+                        <format>R8G8B8</format>
+                    </image>
+                    <clip>
+                        <near>0.01</near>
+                        <far>100</far>
+                    </clip>
+                    <noise>
+                        <type>gaussian</type>
+                        <mean>0.0</mean>
+                        <stddev>0.007</stddev>
+                    </noise>
+                    <distortion>
+                        <k1>0.0</k1>
+                        <k2>0.0</k2>
+                        <k3>0.0</k3>
+                        <p1>0.0</p1>
+                        <p2>0.0</p2>
+                    </distortion>
+                </camera>
+                <gz_frame_id>${topic_frame_id}</gz_frame_id>
+                <topic>${robot_namespace}/${sensor_name}/image_rect_color</topic>
+            </sensor>
+        </gazebo>
+    </xacro:macro>
 </robot>

File: hsrb_parts_description/urdf/sensors/wide_camera.urdf.xacro (robot description, xacro)
@@ -2,4 +2,5 @@
 <robot xmlns:xacro="http://ros.org/wiki/xacro">
     <xacro:include filename="$(find hsrb_parts_description)/urdf/sensors/wide_camera.gazebo.xacro"/>
+    <xacro:arg name="ignition_gazebo_sim" default="false" />
     <!-- wide rgb camera -->
     <xacro:macro name="wide_camera" params="prefix parent robot_namespace rpy *origin">
@@ -28,10 +29,18 @@
             </inertial>
         </link>
-        <xacro:wide_camera_gazebo
-            robot_namespace="${robot_namespace}"
-            sensor_name="${prefix}_camera"
-            parent_frame="${prefix}_camera_gazebo_frame"
-            topic_frame_id="${prefix}_camera_frame"
-            />
+        <xacro:if value="$(arg ignition_gazebo_sim)">
+            <xacro:wide_camera_gazebo_ignition
+                robot_namespace="${robot_namespace}"
+                sensor_name="${prefix}_camera"
+                parent_frame="${prefix}_camera_gazebo_frame"
+                topic_frame_id="${prefix}_camera_frame" />
+        </xacro:if>
+        <xacro:unless value="$(arg ignition_gazebo_sim)">
+            <xacro:wide_camera_gazebo
+                robot_namespace="${robot_namespace}"
+                sensor_name="${prefix}_camera"
+                parent_frame="${prefix}_camera_gazebo_frame"
+                topic_frame_id="${prefix}_camera_frame" />
+        </xacro:unless>
     </xacro:macro>
 </robot>

File: hsrc_description/robots/hsrc1s.urdf.xacro (robot description, xacro)
@@ -16,4 +16,5 @@
     <xacro:include filename="$(find hsrc_description)/urdf/hand_v0/hand.urdf.xacro" />
     <xacro:arg name="gazebo_sim" default="False"/>
+    <xacro:arg name="ignition_gazebo_sim" default="False"/>
     <xacro:arg name="rviz_sim" default="False"/>
     <xacro:arg name="personal_name" default=""/>
@@ -41,5 +42,5 @@
     </xacro:hsrb_hand>
     <!-- Import ros2_control description -->
-    <xacro:if value="${not $(arg gazebo_sim) and not $(arg rviz_sim)}">
+    <xacro:if value="${not $(arg gazebo_sim) and not $(arg ignition_gazebo_sim) and not $(arg rviz_sim)}">
       <xacro:include filename="$(find hsrc_description)/urdf/ros2_control.robot.xacro" />
       <xacro:ros2_contorl_robot/>
@@ -49,4 +50,8 @@
       <xacro:ros2_contorl_gazebo/>
     </xacro:if>
+    <xacro:if value="$(arg ignition_gazebo_sim)">
+      <xacro:include filename="$(find hsrb_description)/urdf/ros2_control.ignition_gazebo.xacro" />
+      <xacro:ros2_contorl_gazebo/>
+    </xacro:if>
     <xacro:if value="$(arg rviz_sim)">
       <xacro:include filename="$(find hsrb_description)/urdf/ros2_control.rviz.xacro" />

File: hsrc_description/urdf/arm_v0/arm.urdf.xacro (robot description, xacro)
@@ -42,5 +42,5 @@
                 <mass value="1.339295"/>
                 <origin xyz="0.000632 0.006404 0.118529"/>
-                <inertia ixx="7.528" ixy="-0.000020284207" ixz="-0.000022947194"
+                <inertia ixx="0.007528" ixy="-0.000020284207" ixz="-0.000022947194"
                     iyy="0.007102" iyz="-0.000091796075" izz="0.001552"/>
             </inertial>

Commit message: Release/2.2.0

File: hsrb_description/robots/hsrb4s.urdf.xacro (robot description, xacro)
@@ -40,5 +40,5 @@
     <xacro:if value="${not $(arg gazebo_sim) and not $(arg ignition_gazebo_sim) and not $(arg rviz_sim)}">
       <xacro:include filename="$(find hsrb_description)/urdf/ros2_control.robot.xacro" />
-      <xacro:ros2_contorl_robot/>
+      <xacro:ros2_control_robot/>
     </xacro:if>
     <xacro:if value="$(arg gazebo_sim)">
@@ -48,9 +48,9 @@
     <xacro:if value="$(arg ignition_gazebo_sim)">
       <xacro:include filename="$(find hsrb_description)/urdf/ros2_control.ignition_gazebo.xacro" />
-      <xacro:ros2_contorl_gazebo/>
+      <xacro:ros2_control_gazebo robot_name="hsrb"/>
     </xacro:if>
     <xacro:if value="$(arg rviz_sim)">
       <xacro:include filename="$(find hsrb_description)/urdf/ros2_control.rviz.xacro" />
-      <xacro:ros2_contorl_rviz/>
+      <xacro:ros2_control_rviz/>
     </xacro:if>
 </robot>

File: hsrb_description/urdf/ros2_control.gazebo.xacro (robot description, xacro)
@@ -17,5 +17,5 @@
         <stall_timeout>2.0</stall_timeout>
         <robot_namespace>${personal_name}/${robot_name}</robot_namespace>
-        <pid_params>
+        <parameters>
           <hand_motor_joint p="50.0" d="20.0"/>
           <hand_l_proximal_joint p="50.0" d="20.0"/>
@@ -27,5 +27,5 @@
           <hand_r_mimic_distal_joint p="20.0" d="8.0"/>
           <hand_r_distal_joint p="20.0" d="8.0"/>
-        </pid_params>
+        </parameters>
       </plugin>
       <plugin name="grasp_hack_plugin" filename="libtmc_gazebo_grasp_hack_hrh_gripper.so">

File: hsrb_description/urdf/ros2_control.ignition_gazebo.xacro (robot description, xacro)
@@ -3,5 +3,5 @@
   <xacro:arg name="ground_truth_xyz_offset" default="0.0 0.0 0.0"/>
   <xacro:arg name="ground_truth_rpy_offset" default="0.0 0.0 0.0"/>
-  <xacro:macro name="ros2_contorl_gazebo">
+  <xacro:macro name="ros2_control_gazebo" params="robot_name">
     <gazebo>
       <self_collide>1</self_collide>
@@ -10,4 +10,6 @@
       <plugin name="gz_ros2_control::GazeboSimROS2ControlPlugin" filename="gz_ros2_control-system">
         <parameters>$(find hsrb_gazebo_bringup)/config/gazebo_ros2_control.yaml</parameters>
+        <!-- Parameters specified later override the earlier ones -->
+        <parameters>$(find hsrb_gazebo_bringup)/config/gazebo_ros2_control_${robot_name}.yaml</parameters>
         <robot_param_node>/whole_body/robot_state_publisher</robot_param_node>
       </plugin>

File: hsrb_description/urdf/ros2_control.robot.xacro (robot description, xacro)
@@ -1,32 +1,31 @@
 <?xml version="1.0"?>
 <robot xmlns:xacro="http://www.ros.org/wiki/xacro">
-  <xacro:macro name="ros2_contorl_robot">
+  <xacro:macro name="hsrb_joint" params="name min_angle max_angle motor_id reduction drive_mode velocity_limit gear_ratio torque_constant control_type:=ActiveJoint">
+    <joint name="${name}">
+      <command_interface name="position">
+        <param name="min">${min_angle}</param>
+        <param name="max">${max_angle}</param>
+      </command_interface>
+      <command_interface name="velocity">
+        <param name="min">${-velocity_limit}</param>
+        <param name="max">${velocity_limit}</param>
+      </command_interface>
+      <state_interface name="position"/>
+      <state_interface name="velocity"/>
+      <state_interface name="effort"/>
+      <param name="control_type">${control_type}</param>
+      <param name="motor_id">${motor_id}</param>
+      <param name="reduction">${reduction}</param>
+      <param name="drive_mode">${drive_mode}</param>
+      <param name="velocity_limit">${velocity_limit}</param>
+      <param name="gear_ratio">${gear_ratio}</param>
+      <param name="torque_constant">${torque_constant}</param>
+    </joint>
+  </xacro:macro>
+  <xacro:macro name="ros2_control_robot">
     <ros2_control name="hsrb" type="system">
       <hardware>
         <plugin>hsrb_robot_hardware/HsrbHW</plugin>
       </hardware>
-      <xacro:macro name="hsrb_joint" params="name min_angle max_angle motor_id reduction drive_mode velocity_limit gear_ratio torque_constant control_type:=ActiveJoint acceleration_limit:=1000.0">
-        <joint name="${name}">
-          <command_interface name="position">
-            <param name="min">${min_angle}</param>
-            <param name="max">${max_angle}</param>
-          </command_interface>
-          <command_interface name="velocity">
-            <param name="min">${-velocity_limit}</param>
-            <param name="max">${velocity_limit}</param>
-          </command_interface>
-          <state_interface name="position"/>
-          <state_interface name="velocity"/>
-          <state_interface name="effort"/>
-          <param name="control_type">${control_type}</param>
-          <param name="motor_id">${motor_id}</param>
-          <param name="reduction">${reduction}</param>
-          <param name="drive_mode">${drive_mode}</param>
-          <param name="velocity_limit">${velocity_limit}</param>
-          <param name="acceleration_limit">${acceleration_limit}</param>
-          <param name="gear_ratio">${gear_ratio}</param>
-          <param name="torque_constant">${torque_constant}</param>
-        </joint>
-      </xacro:macro>
       <xacro:macro name="gripper_active_joint" params="name min_angle max_angle motor_id reduction drive_mode velocity_limit  gear_ratio torque_constant left_spring_joint right_spring_joint">
         <joint name="${name}">
@@ -43,5 +42,4 @@
           <param name="drive_mode">${drive_mode}</param>
           <param name="velocity_limit">${velocity_limit}</param>
-          <param name="acceleration_limit">1000.0</param>
           <param name="gear_ratio">${gear_ratio}</param>
           <param name="torque_constant">${torque_constant}</param>
@@ -133,6 +131,5 @@
                         gear_ratio="0.006451613"
                         torque_constant="0.0174"
-                        control_type="Wheel"
-                        acceleration_limit="41.7"/>
+                        control_type="Wheel"/>
       <xacro:hsrb_joint name="base_r_drive_wheel_joint"
                         min_angle="-999999"
@@ -144,6 +141,5 @@
                         gear_ratio="0.006451613"
                         torque_constant="0.0174"
-                        control_type="Wheel"
-                        acceleration_limit="41.7"/>
+                        control_type="Wheel"/>
       <xacro:hsrb_joint name="base_roll_joint"
                         min_angle="-999999"
@@ -154,6 +150,5 @@
                         velocity_limit="2.5"
                         gear_ratio="0.003333333"
-                        torque_constant="0.0368"
-                        acceleration_limit="5.0"/>
+                        torque_constant="0.0368"/>
     </ros2_control>
   </xacro:macro>

File: hsrb_description/urdf/ros2_control.rviz.xacro (robot description, xacro)
@@ -1,5 +1,5 @@
 <?xml version="1.0"?>
 <robot xmlns:xacro="http://www.ros.org/wiki/xacro">
-  <xacro:macro name="ros2_contorl_rviz">
+  <xacro:macro name="ros2_control_rviz">
     <ros2_control name="GenericSystem" type="system">
       <hardware>

File: hsrc_description/robots/hsrc1s.urdf.xacro (robot description, xacro)
@@ -44,5 +44,5 @@
     <xacro:if value="${not $(arg gazebo_sim) and not $(arg ignition_gazebo_sim) and not $(arg rviz_sim)}">
       <xacro:include filename="$(find hsrc_description)/urdf/ros2_control.robot.xacro" />
-      <xacro:ros2_contorl_robot/>
+      <xacro:ros2_control_robot/>
     </xacro:if>
     <xacro:if value="$(arg gazebo_sim)">
@@ -52,9 +52,9 @@
     <xacro:if value="$(arg ignition_gazebo_sim)">
       <xacro:include filename="$(find hsrb_description)/urdf/ros2_control.ignition_gazebo.xacro" />
-      <xacro:ros2_contorl_gazebo/>
+      <xacro:ros2_control_gazebo robot_name="hsrc"/>
     </xacro:if>
     <xacro:if value="$(arg rviz_sim)">
       <xacro:include filename="$(find hsrb_description)/urdf/ros2_control.rviz.xacro" />
-      <xacro:ros2_contorl_rviz/>
+      <xacro:ros2_control_rviz/>
     </xacro:if>
 </robot>

File: hsrc_description/urdf/base_v0/base.urdf.xacro (robot description, xacro)
@@ -213,4 +213,7 @@
             <origin xyz="0.167 0.0 0.1904" rpy="0.0 0.0 0.0" />
         </xacro:hokuyo_laser>
+        <xacro:imu_sensor prefix="${prefix}" robot_namespace="${robot_namespace}" parent="${prefix}_link" topic_name="data">
+            <origin xyz="0.0005 0.1296 0.181" rpy="0.0 0.0 0.0" />
+        </xacro:imu_sensor>
         <!-- bumper -->
         <xacro:hsrb_bumper prefix="${prefix}" suffix="f" parent="${prefix}_link">

File: hsrc_description/urdf/ros2_control.gazebo.xacro (robot description, xacro)
@@ -17,5 +17,5 @@
         <stall_timeout>2.0</stall_timeout>
         <robot_namespace>${personal_name}/${robot_name}</robot_namespace>
-        <pid_params>
+        <parameters>
           <hand_l_proximal_joint p="50.0" d="20.0"/>
           <hand_l_spring_proximal_joint p="50.0" d="20.0"/>
@@ -26,5 +26,5 @@
           <hand_r_mimic_distal_joint p="20.0" d="8.0"/>
           <hand_r_distal_joint p="20.0" d="8.0"/>
-        </pid_params>
+        </parameters>
       </plugin>
       <plugin name="grasp_hack_plugin" filename="libtmc_gazebo_grasp_hack_hrh_gripper.so">

File: hsrc_description/urdf/ros2_control.robot.xacro (robot description, xacro)
@@ -1,32 +1,31 @@
 <?xml version="1.0"?>
 <robot xmlns:xacro="http://www.ros.org/wiki/xacro">
-  <xacro:macro name="ros2_contorl_robot">
+  <xacro:macro name="hsrb_joint" params="name min_angle max_angle motor_id reduction drive_mode velocity_limit gear_ratio torque_constant control_type:=ActiveJoint">
+    <joint name="${name}">
+      <command_interface name="position">
+        <param name="min">${min_angle}</param>
+        <param name="max">${max_angle}</param>
+      </command_interface>
+      <command_interface name="velocity">
+        <param name="min">${-velocity_limit}</param>
+        <param name="max">${velocity_limit}</param>
+      </command_interface>
+      <state_interface name="position"/>
+      <state_interface name="velocity"/>
+      <state_interface name="effort"/>
+      <param name="control_type">${control_type}</param>
+      <param name="motor_id">${motor_id}</param>
+      <param name="reduction">${reduction}</param>
+      <param name="drive_mode">${drive_mode}</param>
+      <param name="velocity_limit">${velocity_limit}</param>
+      <param name="gear_ratio">${gear_ratio}</param>
+      <param name="torque_constant">${torque_constant}</param>
+    </joint>
+  </xacro:macro>
+  <xacro:macro name="ros2_control_robot">
     <ros2_control name="hsrb" type="system">
       <hardware>
         <plugin>hsrb_robot_hardware/HsrbHW</plugin>
       </hardware>
-      <xacro:macro name="hsrb_joint" params="name min_angle max_angle motor_id reduction drive_mode velocity_limit gear_ratio torque_constant control_type:=ActiveJoint acceleration_limit:=1000.0">
-        <joint name="${name}">
-          <command_interface name="position">
-            <param name="min">${min_angle}</param>
-            <param name="max">${max_angle}</param>
-          </command_interface>
-          <command_interface name="velocity">
-            <param name="min">${-velocity_limit}</param>
-            <param name="max">${velocity_limit}</param>
-          </command_interface>
-          <state_interface name="position"/>
-          <state_interface name="velocity"/>
-          <state_interface name="effort"/>
-          <param name="control_type">${control_type}</param>
-          <param name="motor_id">${motor_id}</param>
-          <param name="reduction">${reduction}</param>
-          <param name="drive_mode">${drive_mode}</param>
-          <param name="velocity_limit">${velocity_limit}</param>
-          <param name="acceleration_limit">${acceleration_limit}</param>
-          <param name="gear_ratio">${gear_ratio}</param>
-          <param name="torque_constant">${torque_constant}</param>
-        </joint>
-      </xacro:macro>
       <xacro:macro name="gripper_active_joint" params="name min_angle max_angle motor_id reduction drive_mode velocity_limit  gear_ratio torque_constant left_spring_joint right_spring_joint">
         <joint name="${name}">
@@ -43,5 +42,4 @@
           <param name="drive_mode">${drive_mode}</param>
           <param name="velocity_limit">${velocity_limit}</param>
-          <param name="acceleration_limit">1000.0</param>
           <param name="gear_ratio">${gear_ratio}</param>
           <param name="torque_constant">${torque_constant}</param>
@@ -133,6 +131,5 @@
                         gear_ratio="0.006451613"
                         torque_constant="0.0174"
-                        control_type="Wheel"
-                        acceleration_limit="41.7"/>
+                        control_type="Wheel"/>
       <xacro:hsrb_joint name="base_r_drive_wheel_joint"
                         min_angle="-999999"
@@ -144,6 +141,5 @@
                         gear_ratio="0.006451613"
                         torque_constant="0.0174"
-                        control_type="Wheel"
-                        acceleration_limit="41.7"/>
+                        control_type="Wheel"/>
       <xacro:hsrb_joint name="base_roll_joint"
                         min_angle="-999999"
@@ -154,6 +150,5 @@
                         velocity_limit="2.5"
                         gear_ratio="0.003333333"
-                        torque_constant="0.0368"
-                        acceleration_limit="5.0"/>
+                        torque_constant="0.0368"/>
     </ros2_control>
     <ros2_control name="hsrb_gpio" type="system">
