Commit message: Remove material tag from collision element

File: hsrb_description/urdf/arm_v0/arm.urdf.xacro (robot description, xacro)
@@ -30,5 +30,4 @@
                     <mesh filename="package://hsrb_description/meshes/arm_v0/shoulder.stl" />
                 </geometry>
-                <material name="body_sub" />
             </collision>
         </link>
@@ -58,5 +57,4 @@
                     <mesh filename="package://hsrb_description/meshes/arm_v0/arm_flex.stl" />
                 </geometry>
-                <material name="body_main" />
             </collision>
         </link>
@@ -86,5 +84,4 @@
                     <mesh filename="package://hsrb_description/meshes/arm_v0/arm_roll.stl" />
                 </geometry>
-                <material name="body_main" />
             </collision>
         </link>

File: hsrb_description/urdf/base_v0/base.urdf.xacro (robot description, xacro)
@@ -40,5 +40,4 @@
                     <cylinder radius="${drive_wheel_radius}" length="${drive_wheel_width}" />
                 </geometry>
-                <material name="wheel" />
             </collision>
             <inertial>
@@ -96,5 +95,4 @@
                     <sphere radius="${passive_wheel_radius}" />
                 </geometry>
-                <material name="wheel" />
             </collision>
             <inertial>
@@ -141,5 +139,4 @@
                     <mesh filename="package://hsrb_description/meshes/base_v0/base.stl" />
                 </geometry>
-                <material name="body_sub" />
             </collision>
         </link>

File: hsrb_description/urdf/base_v1/base.urdf.xacro (robot description, xacro)
@@ -40,5 +40,4 @@
                     <cylinder radius="${drive_wheel_radius}" length="${drive_wheel_width}" />
                 </geometry>
-                <material name="wheel" />
             </collision>
             <inertial>
@@ -96,5 +95,4 @@
                     <sphere radius="${passive_wheel_radius}" />
                 </geometry>
-                <material name="wheel" />
             </collision>
             <inertial>

File: hsrb_description/urdf/hand_v0/hand.urdf.xacro (robot description, xacro)
@@ -47,5 +47,4 @@
                     <mesh filename="package://hsrb_description/meshes/hand_v0/palm.stl" />
                 </geometry>
-                <material name="body_sub" />
             </collision>
         </link>
@@ -156,5 +155,4 @@
                     <mesh filename="package://hsrb_description/meshes/hand_v0/l_proximal.stl" />
                 </geometry>
-                <material name="body_sub" />
             </collision>
         </link>
@@ -181,5 +179,4 @@
                     <mesh filename="package://hsrb_description/meshes/hand_v0/l_distal.stl" />
                 </geometry>
-                <material name="body_sub" />
             </collision>
         </link>
@@ -236,5 +233,4 @@
                     <mesh filename="package://hsrb_description/meshes/hand_v0/r_proximal.stl" />
                 </geometry>
-                <material name="body_sub" />
             </collision>
         </link>
@@ -261,5 +257,4 @@
                     <mesh filename="package://hsrb_description/meshes/hand_v0/r_distal.stl" />
                 </geometry>
-                <material name="body_sub" />
             </collision>
         </link>

File: hsrb_description/urdf/head_v0/head.urdf.xacro (robot description, xacro)
@@ -33,5 +33,4 @@
                     <mesh filename="package://hsrb_description/meshes/head_v0/head_pan.stl" />
                 </geometry>
-                <material name="body_main" />
             </collision>
         </link>
@@ -79,5 +78,4 @@
                     <mesh filename="package://hsrb_description/meshes/head_v0/head.stl" />
                 </geometry>
-                <material name="body_main" />
             </collision>
             <collision>
@@ -85,5 +83,4 @@
                     <mesh filename="package://hsrb_description/meshes/head_v0/tablet.stl" />
                 </geometry>
-                <material name="tablet" />
             </collision>
         </link>

File: hsrb_description/urdf/head_v1/head.urdf.xacro (robot description, xacro)
@@ -33,5 +33,4 @@
                     <mesh filename="package://hsrb_description/meshes/head_v0/head_pan.stl" />
                 </geometry>
-                <material name="body_main" />
             </collision>
         </link>
@@ -79,5 +78,4 @@
                     <mesh filename="package://hsrb_description/meshes/head_v0/head.stl" />
                 </geometry>
-                <material name="body_main" />
             </collision>
             <collision>
@@ -85,5 +83,4 @@
                     <mesh filename="package://hsrb_description/meshes/head_v0/tablet.stl" />
                 </geometry>
-                <material name="tablet" />
             </collision>
         </link>

File: hsrb_description/urdf/sensors/asus_xtion.urdf.xacro (robot description, xacro)
@@ -21,5 +21,4 @@
                     <mesh filename="package://hsrb_description/meshes/sensors/xtion.stl" />
                 </geometry>
-                <material name="black" />
             </collision>
         </link>

File: hsrb_description/urdf/sensors/hokuyo_laser.urdf.xacro (robot description, xacro)
@@ -1,2 +1,3 @@
+<?xml version="1.0" ?>
 <robot xmlns:xacro="http://ros.org/wiki/xacro">
     <xacro:include filename="$(find hsrb_description)/urdf/sensors/hokuyo_laser.gazebo.xacro"/>
@@ -19,5 +20,4 @@
                     <mesh filename="package://hsrb_description/meshes/sensors/laser.stl" />
                 </geometry>
-                <material name="black" />
             </collision>
         </link>

File: hsrb_description/urdf/torso_v0/torso.urdf.xacro (robot description, xacro)
@@ -31,5 +31,4 @@
                     <mesh filename="package://hsrb_description/meshes/torso_v0/torso.stl" />
                 </geometry>
-                <material name="body_sub" />
             </collision>
         </link>

File: hsrb_description/urdf/wrist_v0/wrist.urdf.xacro (robot description, xacro)
@@ -39,5 +39,4 @@
                     <cylinder radius="0.017" length="0.04" />
                 </geometry>
-                <material name="body_sub" />
             </collision>
         </link>
@@ -67,5 +66,4 @@
                     <mesh filename="package://hsrb_description/meshes/wrist_v0/wrist_roll.stl" />
                 </geometry>
-                <material name="body_main" />
             </collision>
         </link>

Commit message: delete some material items

File: hsrb_description/urdf/arm_v0/arm.urdf.xacro (robot description, xacro)
@@ -24,5 +24,4 @@
                     <mesh filename="package://hsrb_description/meshes/arm_v0/shoulder.dae" />
                 </geometry>
-                <material name="body_sub" />
             </visual>
             <collision>
@@ -51,5 +50,4 @@
                     <mesh filename="package://hsrb_description/meshes/arm_v0/arm_flex_light.dae" />
                 </geometry>
-                <material name="body_main" />
             </visual>
             <collision>
@@ -78,5 +76,4 @@
                     <mesh filename="package://hsrb_description/meshes/arm_v0/arm_roll_light.dae" />
                 </geometry>
-                <material name="body_main" />
             </visual>
             <collision>

File: hsrb_description/urdf/base_v0/base.urdf.xacro (robot description, xacro)
@@ -121,5 +121,4 @@
                     <mesh filename="package://hsrb_description/meshes/base_v0/base_light.dae" />
                 </geometry>
-                <material name="body_main" />
             </visual>
             <visual>
@@ -127,5 +126,4 @@
                     <mesh filename="package://hsrb_description/meshes/base_v0/body.dae" />
                 </geometry>
-                <material name="body_main" />
             </visual>
             <visual>
@@ -133,5 +131,4 @@
                     <mesh filename="package://hsrb_description/meshes/base_v0/torso_base.dae" />
                 </geometry>
-                <material name="body_sub" />
             </visual>
             <collision>

File: hsrb_description/urdf/base_v1/base.urdf.xacro (robot description, xacro)
@@ -121,5 +121,4 @@
                     <mesh filename="package://hsrb_description/meshes/base_v1/base_light.dae" />
                 </geometry>
-                <material name="body_main" />
             </visual>
             <visual>
@@ -127,5 +126,4 @@
                     <mesh filename="package://hsrb_description/meshes/base_v1/body_light.dae" />
                 </geometry>
-                <material name="body_main" />
             </visual>
             <visual>
@@ -133,5 +131,4 @@
                     <mesh filename="package://hsrb_description/meshes/base_v1/torso_base.dae" />
                 </geometry>
-                <material name="body_sub" />
             </visual>
             <collision>

File: hsrb_description/urdf/hand_v0/hand.urdf.xacro (robot description, xacro)
@@ -42,5 +42,4 @@
                     <mesh filename="package://hsrb_description/meshes/hand_v0/palm_light.dae" />
                 </geometry>
-                <material name="body_sub" />
             </visual>
             <collision>
@@ -150,5 +149,4 @@
                     <mesh filename="package://hsrb_description/meshes/hand_v0/l_proximal.dae" />
                 </geometry>
-                <material name="body_sub" />
             </visual>
             <collision>
@@ -174,5 +172,4 @@
                     <mesh filename="package://hsrb_description/meshes/hand_v0/l_distal.dae" />
                 </geometry>
-                <material name="body_sub" />
             </visual>
             <collision>
@@ -228,5 +225,4 @@
                     <mesh filename="package://hsrb_description/meshes/hand_v0/r_proximal.dae" />
                 </geometry>
-                <material name="body_sub" />
             </visual>
             <collision>
@@ -252,5 +248,4 @@
                     <mesh filename="package://hsrb_description/meshes/hand_v0/r_distal.dae" />
                 </geometry>
-                <material name="body_sub" />
             </visual>
             <collision>

File: hsrb_description/urdf/head_v0/head.urdf.xacro (robot description, xacro)
@@ -27,5 +27,4 @@
                     <mesh filename="package://hsrb_description/meshes/head_v0/head_pan.dae" />
                 </geometry>
-                <material name="body_main" />
             </visual>
             <collision>
@@ -54,5 +53,4 @@
                     <mesh filename="package://hsrb_description/meshes/head_v0/head_upper.dae" />
                 </geometry>
-                <material name="body_sub" />
             </visual>
             <visual>
@@ -60,5 +58,4 @@
                     <mesh filename="package://hsrb_description/meshes/head_v0/head_tilt.dae" />
                 </geometry>
-                <material name="body_main" />
             </visual>
             <visual>
@@ -66,5 +63,4 @@
                     <mesh filename="package://hsrb_description/meshes/head_v0/tablet_base.dae" />
                 </geometry>
-                <material name="body_sub" />
             </visual>
             <visual>
@@ -72,5 +68,4 @@
                     <mesh filename="package://hsrb_description/meshes/head_v0/tablet.dae" />
                 </geometry>
-                <material name="tablet" />
             </visual>
             <collision>

File: hsrb_description/urdf/head_v1/head.urdf.xacro (robot description, xacro)
@@ -27,5 +27,4 @@
                     <mesh filename="package://hsrb_description/meshes/head_v0/head_pan.dae" />
                 </geometry>
-                <material name="body_main" />
             </visual>
             <collision>
@@ -54,5 +53,4 @@
                     <mesh filename="package://hsrb_description/meshes/head_v0/head_upper.dae" />
                 </geometry>
-                <material name="body_sub" />
             </visual>
             <visual>
@@ -60,5 +58,4 @@
                     <mesh filename="package://hsrb_description/meshes/head_v0/head_tilt.dae" />
                 </geometry>
-                <material name="body_main" />
             </visual>
             <visual>
@@ -66,5 +63,4 @@
                     <mesh filename="package://hsrb_description/meshes/head_v0/tablet_base.dae" />
                 </geometry>
-                <material name="body_sub" />
             </visual>
             <visual>
@@ -72,5 +68,4 @@
                     <mesh filename="package://hsrb_description/meshes/head_v0/tablet.dae" />
                 </geometry>
-                <material name="tablet" />
             </visual>
             <collision>

File: hsrb_description/urdf/sensors/asus_xtion.urdf.xacro (robot description, xacro)
@@ -14,5 +14,4 @@
                     <mesh filename="package://hsrb_description/meshes/sensors/xtion_light.dae" />
                 </geometry>
-                <material name="black" />
             </visual>
             <collision>

File: hsrb_description/urdf/sensors/hokuyo_laser.urdf.xacro (robot description, xacro)
@@ -14,5 +14,4 @@
                     <mesh filename="package://hsrb_description/meshes/sensors/laser.dae" />
                 </geometry>
-                <material name="black" />
             </visual>
             <collision>

File: hsrb_description/urdf/sensors/pointgrey_chameleon.urdf.xacro (robot description, xacro)
@@ -14,5 +14,4 @@
                     <mesh filename="package://hsrb_description/meshes/sensors/head_camera.dae" />
                 </geometry>
-                <material name="black" />
             </visual>
         </link>

File: hsrb_description/urdf/torso_v0/torso.urdf.xacro (robot description, xacro)
@@ -25,5 +25,4 @@
                     <mesh filename="package://hsrb_description/meshes/torso_v0/torso_light.dae" />
                 </geometry>
-                <material name="body_sub" />
             </visual>
             <collision>

File: hsrb_description/urdf/wrist_v0/wrist.urdf.xacro (robot description, xacro)
@@ -60,5 +60,4 @@
                     <mesh filename="package://hsrb_description/meshes/wrist_v0/wrist_roll.dae" />
                 </geometry>
-                <material name="body_main" />
             </visual>
             <collision>
