Commit message: Add xacro namespace

File: hsrb_description/urdf/arm_v0/arm.urdf.xacro (robot description, xacro)
@@ -6,5 +6,5 @@
     <xacro:macro name="hsrb_arm" params="prefix parent *origin">
         <joint name="${prefix}_lift_joint" type="prismatic">
-            <insert_block name="origin" />
+            <xacro:insert_block name="origin" />
             <axis xyz="0.0 0.0 1.0" />
             <limit effort="100.0" velocity="0.2" lower="0.0" upper="0.69" />

File: hsrb_description/urdf/base_v0/base.urdf.xacro (robot description, xacro)
@@ -20,5 +20,5 @@
     <xacro:macro name="hsrb_drive_wheel" params="prefix suffix parent *origin">
         <joint name="${prefix}_${suffix}_drive_wheel_joint" type="continuous">
-            <insert_block name="origin" />
+            <xacro:insert_block name="origin" />
             <axis xyz="0.0 1.0 0.0" />
             <limit effort="${drive_wheel_max_effort}" velocity="${drive_wheel_max_velocity}" />
@@ -51,5 +51,5 @@
     <xacro:macro name="hsrb_passive_wheel" params="prefix suffix parent *origin">
         <joint name="${prefix}_${suffix}_passive_wheel_x_frame_joint" type="continuous">
-            <insert_block name="origin" />
+            <xacro:insert_block name="origin" />
             <axis xyz="1.0 0.0 0.0" />
             <limit effort="8.85" velocity="10.0" />

File: hsrb_description/urdf/base_v1/base.urdf.xacro (robot description, xacro)
@@ -20,5 +20,5 @@
     <xacro:macro name="hsrb_drive_wheel" params="prefix suffix parent *origin">
         <joint name="${prefix}_${suffix}_drive_wheel_joint" type="continuous">
-            <insert_block name="origin" />
+            <xacro:insert_block name="origin" />
             <axis xyz="0.0 1.0 0.0" />
             <limit effort="${drive_wheel_max_effort}" velocity="${drive_wheel_max_velocity}" />
@@ -51,5 +51,5 @@
     <xacro:macro name="hsrb_passive_wheel" params="prefix suffix parent *origin">
         <joint name="${prefix}_${suffix}_passive_wheel_x_frame_joint" type="continuous">
-            <insert_block name="origin" />
+            <xacro:insert_block name="origin" />
             <axis xyz="1.0 0.0 0.0" />
             <limit effort="1.0" velocity="3.0" />

File: hsrb_description/urdf/base_v2/base.urdf.xacro (robot description, xacro)
@@ -20,5 +20,5 @@
     <xacro:macro name="hsrb_drive_wheel" params="prefix suffix parent *origin">
         <joint name="${prefix}_${suffix}_drive_wheel_joint" type="continuous">
-            <insert_block name="origin" />
+            <xacro:insert_block name="origin" />
             <axis xyz="0.0 1.0 0.0" />
             <limit effort="${drive_wheel_max_effort}" velocity="${drive_wheel_max_velocity}" />
@@ -51,5 +51,5 @@
     <xacro:macro name="hsrb_passive_wheel" params="prefix suffix parent *origin">
         <joint name="${prefix}_${suffix}_passive_wheel_x_frame_joint" type="continuous">
-            <insert_block name="origin" />
+            <xacro:insert_block name="origin" />
             <axis xyz="1.0 0.0 0.0" />
             <limit effort="1.0" velocity="3.0" />

File: hsrb_description/urdf/common.xacro (robot description, xacro)
@@ -3,5 +3,5 @@
   <xacro:arg name="implicit_damping" default="false" />
   <xacro:property name="pi" value="3.14159265359"/>
-  <macro name="hsrb_position_joint_transmission" params="joint reduction">
+  <xacro:macro name="hsrb_position_joint_transmission" params="joint reduction">
      <transmission name="${joint}_transmission">
        <type>transmission_interface/SimpleTransmission</type>
@@ -14,6 +14,6 @@
        </actuator>
      </transmission>
-  </macro>
-  <macro name="hsrb_effort_joint_transmission" params="joint reduction">
+  </xacro:macro>
+  <xacro:macro name="hsrb_effort_joint_transmission" params="joint reduction">
      <transmission name="${joint}_transmission">
        <type>transmission_interface/SimpleTransmission</type>
@@ -26,6 +26,6 @@
        </actuator>
      </transmission>
-  </macro>
-  <macro name="hsrb_velocity_joint_transmission" params="joint reduction">
+  </xacro:macro>
+  <xacro:macro name="hsrb_velocity_joint_transmission" params="joint reduction">
       <transmission name="${prefix}_transmission">
           <type>transmission_interface/SimpleTransmission</type>
@@ -38,6 +38,6 @@
           </actuator>
       </transmission>
-  </macro>
-  <macro name="gazebo_link" params="name gravity collide friction">
+  </xacro:macro>
+  <xacro:macro name="gazebo_link" params="name gravity collide friction">
     <gazebo reference="${name}">
       <selfCollide>${collide}</selfCollide>
@@ -46,6 +46,6 @@
       <mu2>${friction}</mu2>
     </gazebo>
-  </macro>
-  <macro name="gazebo_link_flat_black" params="name gravity collide friction">
+  </xacro:macro>
+  <xacro:macro name="gazebo_link_flat_black" params="name gravity collide friction">
     <gazebo reference="${name}">
       <selfCollide>${collide}</selfCollide>
@@ -55,6 +55,6 @@
       <material value="Gazebo/FlatBlack"/>
     </gazebo>
-  </macro>
-  <macro name="gazebo_link_caster" params="name">
+  </xacro:macro>
+  <xacro:macro name="gazebo_link_caster" params="name">
     <gazebo reference="${name}">
       <selfCollide>false</selfCollide>
@@ -65,6 +65,6 @@
       <material value="Gazebo/FlatBlack"/>
     </gazebo>
-  </macro>
-  <macro name="gazebo_link_rubber" params="name">
+  </xacro:macro>
+  <xacro:macro name="gazebo_link_rubber" params="name">
     <gazebo reference="${name}">
       <selfCollide>false</selfCollide>
@@ -80,6 +80,6 @@
       <material value="Gazebo/FlatBlack"/>
     </gazebo>
-  </macro>
-  <macro name="gazebo_joint" params="name">
+  </xacro:macro>
+  <xacro:macro name="gazebo_joint" params="name">
     <gazebo reference="${name}">
       <xacro:if value="$(arg implicit_damping)">
@@ -87,8 +87,8 @@
       </xacro:if>
     </gazebo>
-  </macro>
-  <macro name="gazebo_joint_mimic" params="name">
+  </xacro:macro>
+  <xacro:macro name="gazebo_joint_mimic" params="name">
     <gazebo reference="${name}">
     </gazebo>
-  </macro>
+  </xacro:macro>
 </robot>

File: hsrb_description/urdf/hand_v0/hand.urdf.xacro (robot description, xacro)
@@ -27,5 +27,5 @@
     <xacro:macro name="hsrb_gripper_base" params="prefix parent *origin">
         <joint name="${prefix}_palm_joint" type="fixed">
-            <insert_block name="origin" />
+            <xacro:insert_block name="origin" />
             <parent link="${parent}" />
             <child link="${prefix}_palm_link" />
@@ -63,5 +63,5 @@
     <xacro:macro name="hsrb_hand" params="prefix parent *origin">
         <xacro:hsrb_gripper_base prefix="${prefix}" parent="${parent}">
-            <insert_block name="origin" />
+            <xacro:insert_block name="origin" />
         </xacro:hsrb_gripper_base>
         <xacro:hsrb_finger_with_vacuum prefix="${prefix}" suffix="l" parent="${prefix}_palm_link">
@@ -83,6 +83,6 @@
     <xacro:macro name="hsrb_finger_proximal_base" params="prefix suffix parent *origin *axis">
         <joint name="${prefix}_${suffix}_proximal_joint" type="revolute">
-            <insert_block name="origin" />
-            <insert_block name="axis" />
+            <xacro:insert_block name="origin" />
+            <xacro:insert_block name="axis" />
             <limit effort="100.0" velocity="1.0"
                 lower="${proximal_joint_angle_range_min}"
@@ -96,5 +96,5 @@
         <xacro:hsrb_gripper_dummy_link name="${prefix}_${suffix}_proximal_link" />
         <joint name="${prefix}_${suffix}_spring_proximal_joint" type="revolute">
-            <insert_block name="axis" />
+            <xacro:insert_block name="axis" />
             <limit effort="100.0" velocity="1.0"
                 lower="${spring_proximal_joint_angle_range_min}"
@@ -108,6 +108,6 @@
     <xacro:macro name="hsrb_finger_distal_base" params="prefix suffix parent *origin *axis">
         <joint name="${prefix}_${suffix}_mimic_distal_joint" type="revolute">
-            <insert_block name="origin" />
-            <insert_block name="axis" />
+            <xacro:insert_block name="origin" />
+            <xacro:insert_block name="axis" />
             <limit effort="100.0" velocity="1.0"
                 lower="${-spring_proximal_joint_angle_range_max}"
@@ -121,5 +121,5 @@
         <xacro:hsrb_gripper_dummy_link name="${prefix}_${suffix}_mimic_distal_link" />
         <joint name="${prefix}_${suffix}_distal_joint" type="revolute">
-            <insert_block name="axis" />
+            <xacro:insert_block name="axis" />
             <limit effort="100.0" velocity="1.0"
                 lower="${-proximal_joint_angle_range_max}"
@@ -134,5 +134,5 @@
     <xacro:macro name="hsrb_finger_with_vacuum" params="prefix suffix parent *origin">
         <xacro:hsrb_finger_proximal_base prefix="${prefix}" suffix="${suffix}" parent="${parent}">
-            <insert_block name="origin" />
+            <xacro:insert_block name="origin" />
             <axis xyz="1.0 0.0 0.0" />
         </xacro:hsrb_finger_proximal_base>
@@ -210,5 +210,5 @@
     <xacro:macro name="hsrb_finger_without_vacuum" params="prefix suffix parent *origin">
         <xacro:hsrb_finger_proximal_base prefix="${prefix}" suffix="${suffix}" parent="${parent}">
-            <insert_block name="origin" />
+            <xacro:insert_block name="origin" />
             <axis xyz="-1.0 0.0 0.0" />
         </xacro:hsrb_finger_proximal_base>

File: hsrb_description/urdf/head_v0/head.urdf.xacro (robot description, xacro)
@@ -9,5 +9,5 @@
     <xacro:macro name="hsrb_head" params="prefix parent *origin">
         <joint name="${prefix}_pan_joint" type="revolute">
-            <insert_block name="origin" />
+            <xacro:insert_block name="origin" />
             <axis xyz="0.0 0.0 1.0" />
             <limit effort="100.0" velocity="1.0" lower="-3.84" upper="2.09" />

File: hsrb_description/urdf/head_v1/head.urdf.xacro (robot description, xacro)
@@ -9,5 +9,5 @@
     <xacro:macro name="hsrb_head" params="prefix parent *origin">
         <joint name="${prefix}_pan_joint" type="revolute">
-            <insert_block name="origin" />
+            <xacro:insert_block name="origin" />
             <axis xyz="0.0 0.0 1.0" />
             <limit effort="100.0" velocity="1.0" lower="-3.84" upper="1.75" />

File: hsrb_description/urdf/head_v2/head.urdf.xacro (robot description, xacro)
@@ -9,5 +9,5 @@
     <xacro:macro name="hsrb_head" params="prefix parent *origin">
         <joint name="${prefix}_pan_joint" type="revolute">
-            <insert_block name="origin" />
+            <xacro:insert_block name="origin" />
             <axis xyz="0.0 0.0 1.0" />
             <limit effort="100.0" velocity="1.0" lower="-3.84" upper="1.75" />

File: hsrb_description/urdf/sensors/asus_xtion.urdf.xacro (robot description, xacro)
@@ -5,5 +5,5 @@
     <xacro:macro name="asus_xtion" params="prefix parent robot_namespace sensor_name *origin">
         <joint name="${prefix}_${sensor_name}_joint" type="fixed">
-            <insert_block name="origin" />
+            <xacro:insert_block name="origin" />
             <parent link="${parent}"/> <child link="${prefix}_${sensor_name}_link"/>
         </joint>

File: hsrb_description/urdf/sensors/hokuyo_laser.urdf.xacro (robot description, xacro)
@@ -5,5 +5,5 @@
     <xacro:macro name="hokuyo_laser" params="prefix robot_namespace parent *origin">
         <joint name="${prefix}_range_sensor_joint" type="fixed">
-            <insert_block name="origin" />
+            <xacro:insert_block name="origin" />
             <parent link="${parent}" />
             <child link="${prefix}_range_sensor_link" />

File: hsrb_description/urdf/sensors/imu.urdf.xacro (robot description, xacro)
@@ -5,5 +5,5 @@
     <xacro:macro name="imu_sensor" params="prefix parent robot_namespace *origin">
         <joint name="${prefix}_imu_frame_joint" type="fixed">
-            <insert_block name="origin" />
+            <xacro:insert_block name="origin" />
             <parent link="${parent}" />
             <child link="${prefix}_imu_frame" />

File: hsrb_description/urdf/sensors/minebea_ft_sensor.urdf.xacro (robot description, xacro)
@@ -4,5 +4,5 @@
     <xacro:macro name="minebea_ft_sensor" params="prefix robot_namespace parent joint_name *origin">
         <joint name="${prefix}_ft_sensor_frame_joint" type="fixed">
-            <insert_block name="origin"/>
+            <xacro:insert_block name="origin"/>
             <parent link="${parent}"/>
             <child link="${prefix}_ft_sensor_frame"/>

File: hsrb_description/urdf/sensors/pointgrey_chameleon.urdf.xacro (robot description, xacro)
@@ -4,5 +4,5 @@
     <xacro:macro name="pointgrey_chameleon" params="prefix parent robot_namespace *origin baseline">
         <joint name="${prefix}_camera_joint" type="fixed">
-            <insert_block name="origin" />
+            <xacro:insert_block name="origin" />
             <parent link="${parent}" />
             <child link="${prefix}_camera_link" />

File: hsrb_description/urdf/sensors/wide_camera.urdf.xacro (robot description, xacro)
@@ -5,5 +5,5 @@
     <xacro:macro name="wide_camera" params="prefix parent robot_namespace rpy *origin">
         <joint name="${prefix}_camera_frame_joint" type="fixed">
-            <insert_block name="origin" />
+            <xacro:insert_block name="origin" />
             <parent link="${parent}" />
             <child link="${prefix}_camera_frame" />

File: hsrb_description/urdf/torso_v0/torso.urdf.xacro (robot description, xacro)
@@ -5,5 +5,5 @@
     <xacro:macro name="hsrb_torso" params="prefix parent mimic_joint *origin">
         <joint name="${prefix}_lift_joint" type="prismatic">
-            <insert_block name="origin" />
+            <xacro:insert_block name="origin" />
             <!-- <origin xyz="0.0 0.0 0.752" rpy="0.0 0.0 0.0" /> -->
             <axis xyz="0.0 0.0 1.0" />

Commit message: increase torso and arm_lift effort maximum.

File: hsrb_description/urdf/arm_v0/arm.urdf.xacro (robot description, xacro)
@@ -8,5 +8,5 @@
             <xacro:insert_block name="origin" />
             <axis xyz="0.0 0.0 1.0" />
-            <limit effort="100.0" velocity="0.2" lower="0.0" upper="0.69" />
+            <limit effort="300.0" velocity="0.2" lower="0.0" upper="0.69" />
             <parent link="${parent}" />
             <child link="${prefix}_lift_link" />

File: hsrb_description/urdf/torso_v0/torso.urdf.xacro (robot description, xacro)
@@ -8,5 +8,5 @@
             <!-- <origin xyz="0.0 0.0 0.752" rpy="0.0 0.0 0.0" /> -->
             <axis xyz="0.0 0.0 1.0" />
-            <limit effort="100.0" velocity="0.1" lower="0.0" upper="0.345" />
+            <limit effort="300.0" velocity="0.1" lower="0.0" upper="0.345" />
             <parent link="${parent}" />
             <child link="${prefix}_lift_link" />
