Commit message: fix deprecated descriptions.

File: hsrb_description/urdf/common/indigo/common.xacro (robot description, xacro)
@@ -2,5 +2,4 @@
 <robot xmlns:xacro="http://ros.org/wiki/xacro">
   <xacro:arg name="implicit_damping" default="false" />
-  <xacro:property name="pi" value="3.14159265359"/>
   <xacro:macro name="hsrb_position_joint_transmission" params="joint reduction">
      <transmission name="${joint}_transmission">

File: hsrb_description/urdf/common/kinetic/common.xacro (robot description, xacro)
@@ -2,5 +2,4 @@
 <robot xmlns:xacro="http://ros.org/wiki/xacro">
   <xacro:arg name="implicit_damping" default="false" />
-  <xacro:property name="pi" value="3.14159265359"/>
   <xacro:macro name="hsrb_position_joint_transmission" params="joint reduction">
      <transmission name="${joint}_transmission">

File: hsrb_description/urdf/sensors/kinetic/imu.gazebo.xacro (robot description, xacro)
@@ -1,4 +1,4 @@
 <?xml version="1.0" ?>
-<robot name="hsrb" xmlns:xacro="http://www.ros.org/wiki/xacro">
+<robot name="hsrb" xmlns:xacro="http://ros.org/wiki/xacro">
     <xacro:macro name="imu_gazebo" params="sensor_name frame_name robot_namespace">
         <gazebo reference="${frame_name}">
