Commit message: use tmc_openni2_kinect_plugin to correct format.

File: hsrb_parts_description/urdf/sensors/asus_xtion.gazebo.xacro (robot description, xacro)
@@ -36,5 +36,5 @@
                     </clip>
                 </camera>
-                <plugin name="${sensor_name}_controller" filename="libgazebo_ros_openni_kinect.so">
+                <plugin name="${sensor_name}_controller" filename="libhsrb_gazebo_ros_openni_kinect.so">
                     <alwaysOn>true</alwaysOn>
                     <baseline>0.2</baseline>

File: hsrb_parts_description/urdf/sensors/asus_xtion.urdf.xacro (robot description, xacro)
@@ -21,4 +21,9 @@
                 </geometry>
             </collision>
+            <inertial>
+                <origin xyz="0 0 0"/>
+                <mass value="0.01"/>
+                <inertia ixx="0.001" ixy="0" ixz="0" iyy="0.001" iyz="0" izz="0.001"/>
+            </inertial>
         </link>
         <joint name="${prefix}_rgbd_sensor_gazebo_frame_joint" type="fixed">
@@ -28,5 +33,11 @@
         </joint>
         `
-        <link name="${prefix}_${sensor_name}_gazebo_frame"></link>
+        <link name="${prefix}_${sensor_name}_gazebo_frame">
+            <inertial>
+                <origin xyz="0 0 0"/>
+                <mass value="0.01"/>
+                <inertia ixx="0.001" ixy="0" ixz="0" iyy="0.001" iyz="0" izz="0.001"/>
+            </inertial>
+        </link>
         <xacro:asus_xtion_gazebo
             robot_namespace="${robot_namespace}"
