Commit message: make wrist_ft_sensor_frame_joint fixed

File: hsrb_parts_description/urdf/sensors/minebea_ft_sensor.urdf.xacro (robot description, xacro)
@@ -3,5 +3,5 @@
     <xacro:include filename="$(find hsrb_parts_description)/urdf/sensors/minebea_ft_sensor.gazebo.xacro"/>
     <xacro:macro name="minebea_ft_sensor" params="prefix robot_namespace parent *origin">
-        <joint name="${prefix}_ft_sensor_frame_joint" type="revolute">
+        <joint name="${prefix}_ft_sensor_frame_joint" type="fixed">
             <xacro:insert_block name="origin"/>
             <parent link="${parent}"/>

Commit message: Revert ft_sensor joint revolute from fixed

File: hsrb_parts_description/urdf/sensors/minebea_ft_sensor.urdf.xacro (robot description, xacro)
@@ -3,5 +3,5 @@
     <xacro:include filename="$(find hsrb_parts_description)/urdf/sensors/minebea_ft_sensor.gazebo.xacro"/>
     <xacro:macro name="minebea_ft_sensor" params="prefix robot_namespace parent *origin">
-        <joint name="${prefix}_ft_sensor_frame_joint" type="fixed">
+        <joint name="${prefix}_ft_sensor_frame_joint" type="revolute">
             <xacro:insert_block name="origin"/>
             <parent link="${parent}"/>
