Commit message: Insert ceiling camera link

File: hsrb_parts_description/urdf/sensors/mynteye.urdf.xacro (robot description, xacro)
@@ -3,10 +3,10 @@
     <xacro:include filename="$(find hsrb_parts_description)/urdf/sensors/mynteye.gazebo.xacro"/>
     <xacro:macro name="mynteye" params="prefix parent sensor_name robot_namespace baseline *origin">
-        <joint name="${prefix}_camera_frame_joint" type="fixed">
+        <joint name="${prefix}_camera_link_joint" type="fixed">
             <xacro:insert_block name="origin" />
             <parent link="${parent}" />
-            <child link="${prefix}_camera_frame" />
+            <child link="${prefix}_camera_link" />
         </joint>
-        <link name="${prefix}_camera_frame">
+        <link name="${prefix}_camera_link">
             <visual>
                 <origin xyz="0 0 0" rpy="0.0 0.0 0.0"/>
@@ -22,10 +22,10 @@
             </inertial>
         </link>
-        <gazebo reference="${prefix}_camera_frame">
+        <gazebo reference="${prefix}_camera_link">
             <material>Gazebo/Black</material>
         </gazebo>
         <joint name="${prefix}_camera_gazebo_frame_joint" type="fixed">
             <origin xyz="0 0 0" rpy="${pi/2.0} ${-pi/2.0} 0.0"/>
-            <parent link="${prefix}_camera_frame" />
+            <parent link="${prefix}_camera_link" />
             <child link="${prefix}_camera_gazebo_frame" />
         </joint>
