Commit message: update d435 model

File: hsrb_parts_description/urdf/sensors/intel_d435.urdf.xacro (robot description, xacro)
@@ -13,5 +13,11 @@
                 <origin xyz="0 0 0" rpy="0.0 0.0 0.0"/>
                 <geometry>
-                    <mesh filename="package://hsrb_parts_description/meshes/sensors/xtion.dae" />
+                    <mesh filename="package://hsrb_parts_description/meshes/sensors/d435_body.dae" />
+                </geometry>
+            </visual>
+            <visual>
+                <origin xyz="0 0 0" rpy="0.0 0.0 0.0"/>
+                <geometry>
+                    <mesh filename="package://hsrb_parts_description/meshes/sensors/d435_front.dae" />
                 </geometry>
             </visual>
@@ -19,5 +25,5 @@
                 <origin xyz="0 0 0" rpy="0.0 0.0 0.0"/>
                 <geometry>
-                    <mesh filename="package://hsrb_parts_description/meshes/sensors/xtion.stl" />
+                    <mesh filename="package://hsrb_parts_description/meshes/sensors/d435.stl" />
                 </geometry>
             </collision>

Commit message: Fix d435 model pose.

File: hsrb_parts_description/urdf/sensors/intel_d435.urdf.xacro (robot description, xacro)
@@ -11,5 +11,5 @@
         <link name="${sensor_name}_link">
             <visual>
-                <origin xyz="0 0 0" rpy="0.0 0.0 0.0"/>
+                <origin xyz="0 -0.029 0" rpy="${-pi/2.0} 0.0 ${-pi/2.0}"/>
                 <geometry>
                     <mesh filename="package://hsrb_parts_description/meshes/sensors/d435_body.dae" />
@@ -17,5 +17,5 @@
             </visual>
             <visual>
-                <origin xyz="0 0 0" rpy="0.0 0.0 0.0"/>
+                <origin xyz="0 -0.029 0" rpy="${-pi/2.0} 0.0 ${-pi/2.0}"/>
                 <geometry>
                     <mesh filename="package://hsrb_parts_description/meshes/sensors/d435_front.dae" />
@@ -23,5 +23,5 @@
             </visual>
             <collision>
-                <origin xyz="0 0 0" rpy="0.0 0.0 0.0"/>
+                <origin xyz="0 -0.029 0" rpy="${-pi/2.0} 0.0 ${-pi/2.0}"/>
                 <geometry>
                     <mesh filename="package://hsrb_parts_description/meshes/sensors/d435.stl" />

Commit message: Fix d435 gazebo frame.

File: hsrb_parts_description/urdf/sensors/intel_d435.urdf.xacro (robot description, xacro)
@@ -35,5 +35,5 @@
         </link>
         <joint name="${sensor_name}_gazebo_frame_joint" type="fixed">
-            <origin xyz="0 0 0" rpy="${pi/2.0} ${-pi/2.0} 0.0"/>
+            <origin xyz="0 0 0" rpy="0 0 0"/>
             <parent link="${sensor_name}_link"/>
             <child link="${sensor_name}_gazebo_frame"/>
