Commit message: Add ir cameras to d435

File: hsrb_parts_description/urdf/sensors/intel_d435.gazebo.xacro (robot description, xacro)
@@ -6,10 +6,61 @@
     https://click.intel.com/intelr-realsensetm-depth-camera-d435.html
     -->
-    <xacro:macro name="d435_gazebo" params="robot_namespace sensor_name parent_frame topic_frame_id">
-        <gazebo reference="${parent_frame}">
+    <xacro:macro name="ir_camera" params="robot_namespace sensor_name gazebo_frame topic_frame_id baseline">
+        <gazebo reference="${gazebo_frame}">
+            <sensor type="camera" name="${sensor_name}">
+                <always_on>0</always_on>
+                <update_rate>30.0</update_rate>
+                <camera name="${sensor_name}">
+                    <horizontal_fov>1.591739947</horizontal_fov>
+                    <image>
+                        <width>1280</width>
+                        <height>720</height>
+                        <format>L8</format>
+                    </image>
+                    <clip>
+                        <near>0.05</near>
+                        <far>100</far>
+                    </clip>
+                    <noise>
+                        <type>gaussian</type>
+                        <mean>0.0</mean>
+                        <stddev>0.0</stddev>
+                    </noise>
+                </camera>
+                <plugin name="camera_controller" filename="libhsrb_gazebo_ros_camera.so">
+                    <alwaysOn>0</alwaysOn>
+                    <updateRate>0.0</updateRate>
+                    <cameraName>${sensor_name}</cameraName>
+                    <imageTopicName>image_rect_raw</imageTopicName>
+                    <cameraInfoTopicName>camera_info</cameraInfoTopicName>
+                    <frameName>${topic_frame_id}</frameName>
+                    <robotNamespace>${robot_namespace}</robotNamespace>
+                    <hackBaseline>${baseline}</hackBaseline>
+                    <distortionK1>0.0</distortionK1>
+                    <distortionK2>0.0</distortionK2>
+                    <distortionK3>0.0</distortionK3>
+                    <distortionT1>0.0</distortionT1>
+                    <distortionT2>0.0</distortionT2>
+                </plugin>
+            </sensor>
+        </gazebo>
+    </xacro:macro>
+    <xacro:macro name="d435_gazebo" params="robot_namespace sensor_name depth_frame depth_topic_frame_id left_ir_frame left_ir_topic_frame right_ir_frame right_ir_topic_frame baseline">
+        <xacro:ir_camera
+            robot_namespace="${robot_namespace}/${sensor_name}"
+            sensor_name="infra1"
+            gazebo_frame="${left_ir_frame}"
+            topic_frame_id="${left_ir_topic_frame}"
+            baseline="0.0" />
+        <xacro:ir_camera
+            robot_namespace="${robot_namespace}/${sensor_name}"
+            sensor_name="infra2"
+            gazebo_frame="${right_ir_frame}"
+            topic_frame_id="${right_ir_topic_frame}"
+            baseline="${baseline}" />
+        <gazebo reference="${depth_frame}">
             <sensor type="depth" name="openni_camera_camera">
                 <always_on>0</always_on>
                 <update_rate>30</update_rate>
-                <visualize>true</visualize>
                 <camera>
                     <horizontal_fov>1.501</horizontal_fov>
@@ -31,5 +82,5 @@
                     <updateRate>1.0</updateRate>
                     <cameraName>${sensor_name}</cameraName>
-                    <frameName>${topic_frame_id}</frameName>
+                    <frameName>${depth_topic_frame_id}</frameName>
                     <imageTopicName>/${robot_namespace}/${sensor_name}/rgb/image_rect_color</imageTopicName>
                     <cameraInfoTopicName>/${robot_namespace}/${sensor_name}/rgb/camera_info</cameraInfoTopicName>

File: hsrb_parts_description/urdf/sensors/intel_d435.urdf.xacro (robot description, xacro)
@@ -4,4 +4,5 @@
     <!-- rgbd_sensor -->
     <xacro:macro name="d435" params="parent robot_namespace sensor_name *origin">
+        <xacro:property name="depth_to_right_ir_offset" value="0.050"/>
         <joint name="${sensor_name}_joint" type="fixed">
             <xacro:insert_block name="origin" />
@@ -34,4 +35,5 @@
             </inertial>
         </link>
+        <!-- For backward compatibility. It may not be necessary-->
         <joint name="${sensor_name}_gazebo_frame_joint" type="fixed">
             <origin xyz="0 0 0" rpy="0 0 0"/>
@@ -46,9 +48,32 @@
             </inertial>
         </link>
+        <joint name="${sensor_name}_gazebo_depth_frame_joint" type="fixed">
+            <origin xyz="0 0 0" rpy="0 0 0"/>
+            <parent link="${sensor_name}_link"/>
+            <child link="${sensor_name}_gazebo_depth_frame"/>
+        </joint>
+        <link name="${sensor_name}_gazebo_depth_frame" />
+        <joint name="${sensor_name}_gazebo_left_ir_frame_joint" type="fixed">
+            <origin xyz="0 0 0" rpy="0 0 0"/>
+            <parent link="${sensor_name}_gazebo_depth_frame"/>
+            <child link="${sensor_name}_gazebo_left_ir_frame"/>
+        </joint>
+        <link name="${sensor_name}_gazebo_left_ir_frame" />
+        <joint name="${sensor_name}_gazebo_right_ir_frame_joint" type="fixed">
+            <origin xyz="0 -${depth_to_right_ir_offset} 0" rpy="0 0 0"/>
+            <parent link="${sensor_name}_gazebo_depth_frame"/>
+            <child link="${sensor_name}_gazebo_right_ir_frame"/>
+        </joint>
+        <link name="${sensor_name}_gazebo_right_ir_frame" />
         <xacro:d435_gazebo
             robot_namespace="${robot_namespace}"
             sensor_name="${sensor_name}"
-            parent_frame="${sensor_name}_gazebo_frame"
-            topic_frame_id="${sensor_name}_rgb_frame" />
+            depth_frame="${sensor_name}_gazebo_frame"
+            depth_topic_frame_id="${sensor_name}_rgb_frame"
+            left_ir_frame="${sensor_name}_gazebo_left_ir_frame"
+            left_ir_topic_frame="${sensor_name}_infra1_optical_frame"
+            right_ir_frame="${sensor_name}_gazebo_right_ir_frame"
+            right_ir_topic_frame="${sensor_name}_infra2_optical_frame"
+            baseline="${depth_to_right_ir_offset}" />
     </xacro:macro>
 </robot>
