Commit message: Fix the issue of sensor name conflict for hokuyo_laser in Gazebo, and use the topic name as an argument

File: hsrb_parts_description/urdf/sensors/hokuyo_laser.gazebo.xacro (robot description, xacro)
@@ -23,9 +23,8 @@
                     </range>
                 </ray>
-                <plugin name="hokuyo_laser" filename="libgazebo_ros_ray_sensor.so">
+                <plugin name="${sensor_name}" filename="libgazebo_ros_ray_sensor.so">
                     <output_type>sensor_msgs/LaserScan</output_type>
                     <frame_name>${frame_name}</frame_name>
                     <ros>
-                        <namespace>${robot_namespace}</namespace>
                         <remapping>~/out:=${ros_topic}</remapping>
                     </ros>

File: hsrb_parts_description/urdf/sensors/hokuyo_laser.urdf.xacro (robot description, xacro)
@@ -3,5 +3,5 @@
     <xacro:include filename="$(find hsrb_parts_description)/urdf/sensors/hokuyo_laser.gazebo.xacro"/>
     <!-- range sensor -->
-    <xacro:macro name="hokuyo_laser" params="prefix robot_namespace parent min_angle max_angle *origin">
+    <xacro:macro name="hokuyo_laser" params="prefix robot_namespace parent min_angle max_angle ros_topic:='scan' *origin">
         <joint name="${prefix}_range_sensor_joint" type="fixed">
             <xacro:insert_block name="origin" />
@@ -29,5 +29,5 @@
             sensor_name="${prefix}_range_sensor"
             robot_namespace="${robot_namespace}"
-            ros_topic="scan"
+            ros_topic="${ros_topic}"
             frame_name="${prefix}_range_sensor_link"
             min_angle="${min_angle}" max_angle="${max_angle}" />

Commit message: Add Ignition-specific settings for IMU and Hokuyo Laser

File: hsrb_parts_description/urdf/sensors/hokuyo_laser.gazebo.xacro (robot description, xacro)
@@ -33,3 +33,35 @@
         </gazebo>
     </xacro:macro>
+    <xacro:macro name="hokuyo_laser_gazebo_ignition" params="sensor_name robot_namespace ros_topic frame_name min_angle max_angle">
+        <gazebo reference="${frame_name}">
+            <sensor name="${sensor_name}" type="gpu_lidar">
+            <pose>0 0 0 0 0 0</pose>
+            <topic>${robot_namespace}/${sensor_name}/${ros_topic}</topic>
+            <gz_frame_id>${frame_name}</gz_frame_id>
+            <update_rate>30.0</update_rate>
+            <visualize>$(arg gazebo_visualization_enabled)</visualize>
+            <lidar>
+                <scan>
+                <horizontal>
+                    <samples>721</samples>
+                    <resolution>1</resolution>
+                    <min_angle>${min_angle}</min_angle>
+                    <max_angle>${max_angle}</max_angle>
+                </horizontal>
+                <vertical>
+                    <samples>1</samples>
+                    <resolution>1</resolution>
+                    <min_angle>0.0</min_angle>
+                    <max_angle>0.0</max_angle>
+                </vertical>
+                </scan>
+                <range>
+                <min>0.05</min>
+                <max>60.0</max>
+                <resolution>0.001</resolution>
+                </range>
+            </lidar>
+            </sensor>
+        </gazebo>
+    </xacro:macro>
 </robot>

File: hsrb_parts_description/urdf/sensors/hokuyo_laser.urdf.xacro (robot description, xacro)
@@ -2,4 +2,5 @@
 <robot xmlns:xacro="http://ros.org/wiki/xacro">
     <xacro:include filename="$(find hsrb_parts_description)/urdf/sensors/hokuyo_laser.gazebo.xacro"/>
+    <xacro:arg name="ignition_gazebo_sim" default="false" />
     <!-- range sensor -->
     <xacro:macro name="hokuyo_laser" params="prefix robot_namespace parent min_angle max_angle ros_topic:='scan' *origin">
@@ -26,10 +27,20 @@
             </inertial>
         </link>
-        <xacro:hokuyo_laser_gazebo
-            sensor_name="${prefix}_range_sensor"
-            robot_namespace="${robot_namespace}"
-            ros_topic="${ros_topic}"
-            frame_name="${prefix}_range_sensor_link"
-            min_angle="${min_angle}" max_angle="${max_angle}" />
+        <xacro:if value="$(arg ignition_gazebo_sim)">
+            <xacro:hokuyo_laser_gazebo_ignition
+                sensor_name="${prefix}_range_sensor"
+                robot_namespace="${robot_namespace}"
+                ros_topic="${ros_topic}"
+                frame_name="${prefix}_range_sensor_link"
+                min_angle="${min_angle}" max_angle="${max_angle}" />
+        </xacro:if>
+        <xacro:unless value="$(arg ignition_gazebo_sim)">
+            <xacro:hokuyo_laser_gazebo
+                sensor_name="${prefix}_range_sensor"
+                robot_namespace="${robot_namespace}"
+                ros_topic="${ros_topic}"
+                frame_name="${prefix}_range_sensor_link"
+                min_angle="${min_angle}" max_angle="${max_angle}" />
+        </xacro:unless>
     </xacro:macro>
 </robot>

File: hsrb_parts_description/urdf/sensors/imu.urdf.xacro (robot description, xacro)
@@ -1,4 +1,5 @@
 <?xml version="1.0" ?>
 <robot xmlns:xacro="http://ros.org/wiki/xacro" name="hsrb">
+    <xacro:arg name="ignition_gazebo_sim" default="false" />
     <!-- imu sensor gazebo -->
     <xacro:macro name="imu_gazebo" params="sensor_name frame_name topic_name robot_namespace">
@@ -33,4 +34,13 @@
         </gazebo>
     </xacro:macro>
+    <xacro:macro name="imu_gazebo_ignition" params="sensor_name frame_name topic_name robot_namespace">
+        <gazebo reference="${frame_name}">
+            <sensor type="imu" name="${sensor_name}">
+                <update_rate>100.0</update_rate>
+                <topic>${robot_namespace}/${sensor_name}/${topic_name}</topic>
+                <gz_frame_id>${personal_name}/${frame_name}</gz_frame_id>
+            </sensor>
+        </gazebo>
+    </xacro:macro>
     <!-- imu sensor -->
     <xacro:macro name="imu_sensor" params="prefix parent topic_name robot_namespace *origin">
@@ -47,9 +57,18 @@
             </inertial>
         </link>
-        <xacro:imu_gazebo
-            sensor_name="${prefix}_imu"
-            frame_name="${prefix}_imu_frame"
-            topic_name="${topic_name}"
-            robot_namespace="${robot_namespace}"/>
+        <xacro:if value="$(arg ignition_gazebo_sim)">
+            <xacro:imu_gazebo_ignition
+                sensor_name="${prefix}_imu"
+                frame_name="${prefix}_imu_frame"
+                topic_name="${topic_name}"
+                robot_namespace="${robot_namespace}"/>
+        </xacro:if>
+        <xacro:unless value="$(arg ignition_gazebo_sim)">
+            <xacro:imu_gazebo
+                sensor_name="${prefix}_imu"
+                frame_name="${prefix}_imu_frame"
+                topic_name="${topic_name}"
+                robot_namespace="${robot_namespace}"/>
+        </xacro:unless>
     </xacro:macro>
 </robot>
