Commit message: change hsrc setting

File: hsrc_description/urdf/hand_v0/hand.gazebo.xacro (robot description, xacro)
@@ -38,6 +38,6 @@
                 <gripper_link>${prefix}_r_spring_proximal_link</gripper_link>
                 <gripper_link>${prefix}_l_spring_proximal_link</gripper_link>
-                <!-- hand_palm_link is merged with wrist_roll_link by fixed joint -->
-                <palm_link>wrist_roll_link</palm_link>
+		<!-- hand_palm_link is merged with wrist_ft_sensor_frame by fixed joint  -->
+		<palm_link>wrist_ft_sensor_frame</palm_link>
             </plugin>
         </gazebo>

File: hsrc_description/urdf/wrist_v0/wrist.urdf.xacro (robot description, xacro)
@@ -46,6 +46,20 @@
             <limit effort="100.0" velocity="1.5" lower="-1.92" upper="3.67" />
             <parent link="${prefix}_flex_link" />
+            <child link="${prefix}_ft_sensor_mount_link" />
+            <dynamics damping="1.0"/>
+        </joint>
+        <!-- each link must have mass in URDF so we apply very small mass (10 gram) for this coupling link -->
+        <link name="${prefix}_ft_sensor_mount_link">
+          <inertial>
+            <mass value="0.01"/>
+            <inertia ixx="0.001" ixy="0.0" ixz="0.0"
+                     iyy="0.001" iyz="0.0"
+                     izz="0.001" />
+          </inertial>
+        </link>
+        <joint name="${prefix}_ft_sensor_frame_inverse_joint" type="fixed">
+            <origin xyz="0.0 0.0 0.0735" rpy="-${pi} 0.0 0.0"/>
+            <parent link="${prefix}_ft_sensor_frame" />
             <child link="${prefix}_roll_link" />
-            <dynamics damping="1.0"/>
         </joint>
         <link name="${prefix}_roll_link">
@@ -70,7 +84,6 @@
             prefix="${prefix}"
             robot_namespace="${robot_namespace}"
-            parent="${prefix}_roll_link"
-            joint_name="${prefix}_roll_joint">
-            <origin xyz="0.0 0.0 0.1" rpy="${pi} 0.0 0.0"/>
+	    parent="${prefix}_ft_sensor_mount_link">
+	  <origin xyz="0.0 0.0 0.1" rpy="${pi} 0.0 0.0"/>
         </xacro:minebea_ft_sensor>
         <xacro:hsrb_wrist_gazebo prefix="${prefix}"/>
