Commit message: add base_footprint inertial and fix gripper_dummy_link mass value for hsrc

File: hsrc_description/urdf/hand_v0/hand.urdf.xacro (robot description, xacro)
@@ -17,5 +17,5 @@
         <link name="${name}">
             <inertial>
-                <mass value="0.15"/>
+                <mass value="0.2"/>
                 <inertia
                     ixx="0.015" ixy="0.0" ixz="0.0"

Commit message: delete hsrc hand_motor_joint xyz

File: hsrc_description/urdf/hand_v0/hand.urdf.xacro (robot description, xacro)
@@ -50,5 +50,4 @@
         </link>
         <joint name="${prefix}_motor_joint" type="revolute">
-            <origin xyz="0.0 0.0 0.155"/>
             <axis xyz="1.0 0.0 0.0" />
             <limit effort="100.0" velocity="1.0"

Commit message: Change HSR-C's hand model mass and gain to the same as HSR-B's for avoid vibration

File: hsrc_description/urdf/hand_v0/hand.urdf.xacro (robot description, xacro)
@@ -12,4 +12,7 @@
     <xacro:property name="spring_proximal_joint_angle_range_max" value="0.698" />
     <xacro:property name="distal_joint_angle_offset" value="0.087" />
+    <!-- The weight of all hand links is set lightly.
+         The reason is to make it easy to adjust the hand control gain in gazebo.
+         TODO Reset the weight parameter to the correct value -->
     <!-- dummy link -->
     <xacro:macro name="hsrb_gripper_dummy_link" params="name">
@@ -18,6 +21,6 @@
                 <mass value="0.01"/>
                 <inertia
-                    ixx="0.0015" ixy="0.0" ixz="0.0"
-                    iyy="0.0015" iyz="0.0" izz="0.0015"/>
+                    ixx="0.0" ixy="0.0" ixz="0.0"
+                    iyy="0.0" iyz="0.0" izz="0.0"/>
             </inertial>
         </link>
@@ -137,9 +140,9 @@
         <link name="${prefix}_${suffix}_spring_proximal_link">
             <inertial>
-                <mass value="0.043589"/>
+                <mass value="0.001"/>
                 <origin xyz="0.021418 0.00248 0.022688"/>
                 <inertia
-                    ixx="0.000026033886" ixy="-0.000000144078" ixz="-0.00000198241"
-                    iyy="0.000028824811" iyz="-0.000001268421" izz="0.000005135919"/>
+                    ixx="0.0" ixy="0.0" ixz="0.0"
+                    iyy="0.0" iyz="0.0" izz="0.0"/>
             </inertial>
             <visual>
@@ -160,9 +163,9 @@
         <link name="${prefix}_${suffix}_distal_link">
             <inertial>
-                <mass value="0.027731"/>
+                <mass value="0.001"/>
                 <origin xyz="0.011116 0.005679 0.017532"/>
                 <inertia
-                    ixx="0.000004451952" ixy="-0.000000617574" ixz="0.000000503765"
-                    iyy="0.000000503765" iyz="-0.000000435048" izz="0.000004456764"/>
+                    ixx="0.0" ixy="0.0" ixz="0.0"
+                    iyy="0.0" iyz="0.0" izz="0.0"/>
             </inertial>
             <visual>
@@ -192,8 +195,8 @@
         <link name="${prefix}_${suffix}_finger_vacuum_frame">
             <inertial>
-                <mass value="0.01"/>
-                <inertia
-                    ixx="0.0015" ixy="0.0" ixz="0.0"
-                    iyy="0.0015" iyz="0.0" izz="0.0015"/>
+                <mass value="0.001"/>
+                <inertia
+                    ixx="0.0" ixy="0.0" ixz="0.0"
+                    iyy="0.0" iyz="0.0" izz="0.0"/>
             </inertial>
             <visual>
@@ -214,9 +217,9 @@
         <link name="${prefix}_${suffix}_spring_proximal_link">
             <inertial>
-                <mass value="0.043956"/>
+                <mass value="0.001"/>
                 <origin xyz="0.013203 0.002096 0.023311"/>
                 <inertia
-                    ixx="0.00002623664" ixy="0.00000001631" ixz="0.000001281845"
-                    iyy="0.000028838232" iyz="-0.000001621709" izz="0.000004957151"/>
+                    ixx="0.0" ixy="0.0" ixz="0.0"
+                    iyy="0.0" iyz="0.0" izz="0.0"/>
             </inertial>
             <visual>
@@ -237,9 +240,9 @@
         <link name="${prefix}_${suffix}_distal_link">
             <inertial>
-                <mass value="0.020927"/>
+                <mass value="0.001"/>
                 <origin xyz="0.014256 -0.008321 0.015591"/>
                 <inertia
-                    ixx="0.00000307518" ixy="-0.00000004954" ixz="0.000000009481"
-                    iyy="0.000004074079" iyz="0.000000843648" izz="0.000002807795"/>
+                    ixx="0.0" ixy="0.0" ixz="0.0"
+                    iyy="0.0" iyz="0.0" izz="0.0"/>
             </inertial>
             <visual>

File: hsrc_description/urdf/ros2_control.gazebo.xacro (robot description, xacro)
@@ -18,13 +18,12 @@
         <robot_namespace>${personal_name}/${robot_name}</robot_namespace>
         <parameters>
-          <hand_motor_joint p="2.0" d="0.1"/>
-          <hand_l_proximal_joint p="2.0" d="0.1"/>
-          <hand_l_spring_proximal_joint p="2.0" d="0.1"/>
-          <hand_l_mimic_distal_joint p="1.0" d="0.1"/>
-          <hand_l_distal_joint p="2.0" d="0.1"/>
-          <hand_r_proximal_joint p="1.0" d="0.1"/>
-          <hand_r_spring_proximal_joint p="1.0" d="0.1"/>
-          <hand_r_mimic_distal_joint p="1.0" d="0.1"/>
-          <hand_r_distal_joint p="1.0" d="0.1"/>
+          <hand_l_proximal_joint p="50.0" d="20.0"/>
+          <hand_l_spring_proximal_joint p="50.0" d="20.0"/>
+          <hand_l_mimic_distal_joint p="20.0" d="8.0"/>
+          <hand_l_distal_joint p="1.0" d="0.0"/>
+          <hand_r_proximal_joint p="50.0" d="20.0"/>
+          <hand_r_spring_proximal_joint p="50.0" d="20.0"/>
+          <hand_r_mimic_distal_joint p="20.0" d="8.0"/>
+          <hand_r_distal_joint p="20.0" d="8.0"/>
         </parameters>
       </plugin>
