Commit message: addjust hsrc_description to hsrb_description

File: hsrc_description/urdf/arm_v0/arm.urdf.xacro (robot description, xacro)
@@ -6,7 +6,7 @@
     <xacro:macro name="hsrb_arm" params="prefix parent *origin">
         <joint name="${prefix}_lift_joint" type="prismatic">
-            <insert_block name="origin" />
+            <xacro:insert_block name="origin" />
             <axis xyz="0.0 0.0 1.0" />
-            <limit effort="100.0" velocity="0.2" lower="0.0" upper="0.69" />
+            <limit effort="300.0" velocity="0.2" lower="0.0" upper="0.69" />
             <parent link="${parent}" />
             <child link="${prefix}_lift_link" />

File: hsrc_description/urdf/base_v0/base.urdf.xacro (robot description, xacro)
@@ -20,5 +20,5 @@
     <xacro:macro name="hsrb_drive_wheel" params="prefix suffix parent *origin">
         <joint name="${prefix}_${suffix}_drive_wheel_joint" type="continuous">
-            <insert_block name="origin" />
+            <xacro:insert_block name="origin" />
             <axis xyz="0.0 1.0 0.0" />
             <limit effort="${drive_wheel_max_effort}" velocity="${drive_wheel_max_velocity}" />
@@ -51,5 +51,5 @@
     <xacro:macro name="hsrb_passive_wheel" params="prefix suffix parent *origin">
         <joint name="${prefix}_${suffix}_passive_wheel_x_frame_joint" type="continuous">
-            <insert_block name="origin" />
+            <xacro:insert_block name="origin" />
             <axis xyz="1.0 0.0 0.0" />
             <limit effort="1.0" velocity="3.0" />
@@ -186,5 +186,5 @@
         </xacro:hokuyo_laser>
         <xacro:imu_sensor prefix="${prefix}" robot_namespace="${robot_namespace}" parent="${prefix}_link">
-            <origin xyz="0.003 -0.08594 0.203" rpy="${pi} 0.0 0.0" />
+            <origin xyz="0.003 -0.08594 0.203" rpy="0.0 0.0 0.0" />
         </xacro:imu_sensor>
         <xacro:hsrb_base_gazebo prefix="${prefix}"/>

File: hsrc_description/urdf/hand_v0/hand.urdf.xacro (robot description, xacro)
@@ -17,8 +17,8 @@
         <link name="${name}">
             <inertial>
-                <mass value="0.2"/>
-                <inertia
-                    ixx="0.015" ixy="0.0" ixz="0.0"
-                    iyy="0.015" iyz="0.0" izz="0.015"/>
+                <mass value="0.01"/>
+                <inertia
+                    ixx="0.0015" ixy="0.0" ixz="0.0"
+                    iyy="0.0015" iyz="0.0" izz="0.0015"/>
             </inertial>
         </link>
@@ -27,5 +27,5 @@
     <xacro:macro name="hsrb_gripper_base" params="prefix parent *origin">
         <joint name="${prefix}_palm_joint" type="fixed">
-            <insert_block name="origin" />
+            <xacro:insert_block name="origin" />
             <parent link="${parent}" />
             <child link="${prefix}_palm_link" />
@@ -57,5 +57,5 @@
             <parent link="${prefix}_palm_link" />
             <child link="${prefix}_motor_dummy_link" />
-            <dynamics damping="1.0"/>
+            <dynamics damping="0.0001"/>
         </joint>
         <!-- dummy link -->
@@ -64,5 +64,5 @@
     <xacro:macro name="hsrb_hand" params="prefix parent *origin">
         <xacro:hsrb_gripper_base prefix="${prefix}" parent="${parent}">
-            <insert_block name="origin" />
+            <xacro:insert_block name="origin" />
         </xacro:hsrb_gripper_base>
         <xacro:hsrb_finger_with_vacuum prefix="${prefix}" suffix="l" parent="${prefix}_palm_link">
@@ -84,6 +84,6 @@
     <xacro:macro name="hsrb_finger_proximal_base" params="prefix suffix parent *origin *axis">
         <joint name="${prefix}_${suffix}_proximal_joint" type="revolute">
-            <insert_block name="origin" />
-            <insert_block name="axis" />
+            <xacro:insert_block name="origin" />
+            <xacro:insert_block name="axis" />
             <limit effort="100.0" velocity="1.0"
                 lower="${proximal_joint_angle_range_min}"
@@ -92,16 +92,16 @@
             <child link="${prefix}_${suffix}_proximal_link" />
             <mimic joint="${prefix}_motor_joint" />
-            <dynamics damping="1.0"/>
+            <dynamics damping="0.0001"/>
         </joint>
         <!-- dummy link -->
         <xacro:hsrb_gripper_dummy_link name="${prefix}_${suffix}_proximal_link" />
         <joint name="${prefix}_${suffix}_spring_proximal_joint" type="revolute">
-            <insert_block name="axis" />
-            <limit effort="100.0" velocity="1.0"
+            <xacro:insert_block name="axis" />
+            <limit effort="10.0" velocity="1.0"
                 lower="${spring_proximal_joint_angle_range_min}"
                 upper="${spring_proximal_joint_angle_range_max}" />
             <parent link="${prefix}_${suffix}_proximal_link" />
             <child link="${prefix}_${suffix}_spring_proximal_link" />
-            <dynamics damping="1.0"/>
+            <dynamics damping="0.0001"/>
         </joint>
     </xacro:macro>
@@ -109,6 +109,6 @@
     <xacro:macro name="hsrb_finger_distal_base" params="prefix suffix parent *origin *axis">
         <joint name="${prefix}_${suffix}_mimic_distal_joint" type="revolute">
-            <insert_block name="origin" />
-            <insert_block name="axis" />
+            <xacro:insert_block name="origin" />
+            <xacro:insert_block name="axis" />
             <limit effort="100.0" velocity="1.0"
                 lower="${-spring_proximal_joint_angle_range_max}"
@@ -117,10 +117,10 @@
             <child link="${prefix}_${suffix}_mimic_distal_link" />
             <mimic joint="${prefix}_${suffix}_spring_proximal_joint" multiplier="-1.0" />
-            <dynamics damping="1.0"/>
+            <dynamics damping="0.0001"/>
         </joint>
         <!-- dummy link -->
         <xacro:hsrb_gripper_dummy_link name="${prefix}_${suffix}_mimic_distal_link" />
         <joint name="${prefix}_${suffix}_distal_joint" type="revolute">
-            <insert_block name="axis" />
+            <xacro:insert_block name="axis" />
             <limit effort="100.0" velocity="1.0"
                 lower="${-proximal_joint_angle_range_max}"
@@ -129,5 +129,5 @@
             <child link="${prefix}_${suffix}_distal_link" />
             <mimic joint="${prefix}_motor_joint" multiplier="-1.0" offset="${-distal_joint_angle_offset}"/>
-            <dynamics damping="1.0"/>
+            <dynamics damping="0.0001"/>
         </joint>
     </xacro:macro>
@@ -135,5 +135,5 @@
     <xacro:macro name="hsrb_finger_with_vacuum" params="prefix suffix parent *origin">
         <xacro:hsrb_finger_proximal_base prefix="${prefix}" suffix="${suffix}" parent="${parent}">
-            <insert_block name="origin" />
+            <xacro:insert_block name="origin" />
             <axis xyz="1.0 0.0 0.0" />
         </xacro:hsrb_finger_proximal_base>
@@ -184,4 +184,5 @@
             <parent link="${prefix}_${suffix}_distal_link" />
             <child link="${prefix}_${suffix}_finger_tip_frame" />
+            <dynamics damping="0.0001"/>
         </joint>
         <!-- TODO: this is the right format: <link name="${prefix}_${suffix}_finger_tip_frame" /> -->
@@ -194,8 +195,8 @@
         <link name="${prefix}_${suffix}_finger_vacuum_frame">
             <inertial>
-                <mass value="0.15"/>
-                <inertia
-                    ixx="0.015" ixy="0.0" ixz="0.0"
-                    iyy="0.015" iyz="0.0" izz="0.015"/>
+                <mass value="0.01"/>
+                <inertia
+                    ixx="0.0015" ixy="0.0" ixz="0.0"
+                    iyy="0.0015" iyz="0.0" izz="0.0015"/>
             </inertial>
             <visual>
@@ -211,5 +212,5 @@
     <xacro:macro name="hsrb_finger_without_vacuum" params="prefix suffix parent *origin">
         <xacro:hsrb_finger_proximal_base prefix="${prefix}" suffix="${suffix}" parent="${parent}">
-            <insert_block name="origin" />
+            <xacro:insert_block name="origin" />
             <axis xyz="-1.0 0.0 0.0" />
         </xacro:hsrb_finger_proximal_base>

File: hsrc_description/urdf/head_v0/head.urdf.xacro (robot description, xacro)
@@ -9,5 +9,5 @@
     <xacro:macro name="hsrb_head" params="prefix parent *origin">
         <joint name="${prefix}_pan_joint" type="revolute">
-            <insert_block name="origin" />
+            <xacro:insert_block name="origin" />
             <axis xyz="0.0 0.0 1.0" />
             <limit effort="100.0" velocity="1.0" lower="-3.84" upper="1.75" />

File: hsrc_description/urdf/torso_v0/torso.urdf.xacro (robot description, xacro)
@@ -5,8 +5,8 @@
     <xacro:macro name="hsrb_torso" params="prefix parent mimic_joint *origin">
         <joint name="${prefix}_lift_joint" type="prismatic">
-            <insert_block name="origin" />
+            <xacro:insert_block name="origin" />
             <!-- <origin xyz="0.0 0.0 0.762" rpy="0.0 0.0 0.0" /> -->
             <axis xyz="0.0 0.0 1.0" />
-            <limit effort="100.0" velocity="0.1" lower="0.0" upper="0.345" />
+            <limit effort="300.0" velocity="0.1" lower="0.0" upper="0.345" />
             <parent link="${parent}" />
             <child link="${prefix}_lift_link" />
