Commit message: modify hsrc_description urdf

File: hsrc_description/urdf/base_v0/base.urdf.xacro (robot description, xacro)
@@ -105,11 +105,5 @@
     <!-- base -->
     <xacro:macro name="hsrb_base" params="prefix robot_namespace">
-        <link name="base_footprint">
-            <inertial>
-                <origin xyz="0 0 0"/>
-                <mass value="0.01"/>
-                <inertia ixx="0.001" ixy="0" ixz="0" iyy="0.001" iyz="0" izz="0.001"/>
-            </inertial>
-        </link>
+        <link name="base_footprint"/>
         <joint name="${prefix}_footprint_joint" type="fixed">
             <parent link="base_footprint" />

File: hsrc_description/urdf/hand_v0/hand.urdf.xacro (robot description, xacro)
@@ -17,5 +17,5 @@
         <link name="${name}">
             <inertial>
-                <mass value="0.01"/>
+                <mass value="0.15"/>
                 <inertia
                     ixx="0.015" ixy="0.0" ixz="0.0"

Commit message: Separate base visuals for interactive markers

File: hsrc_description/urdf/base_v0/base.urdf.xacro (robot description, xacro)
@@ -119,5 +119,10 @@
             <visual>
                 <geometry>
-                    <mesh filename="package://hsrc_description/meshes/base_v0/base.dae" />
+                    <mesh filename="package://hsrc_description/meshes/base_v0/base_light.dae" />
+                </geometry>
+            </visual>
+            <visual>
+                <geometry>
+                    <mesh filename="package://hsrc_description/meshes/base_v0/body_light.dae" />
                 </geometry>
             </visual>
