Commit message: fixed hand_v0 inertial and mass parameters

File: hsrb_description/urdf/hand_v0/hand.urdf.xacro (robot description, xacro)
@@ -16,8 +16,8 @@
         <link name="${name}">
             <inertial>
-                <mass value="0.1"/>
-                <inertia
-                    ixx="0.01" ixy="0.0" ixz="0.0"
-                    iyy="0.01" iyz="0.0" izz="0.01"/>
+                <mass value="0.15"/>
+                <inertia
+                    ixx="0.015" ixy="0.0" ixz="0.0"
+                    iyy="0.015" iyz="0.0" izz="0.015"/>
             </inertial>
         </link>
@@ -32,8 +32,8 @@
         <link name="${prefix}_palm_link">
             <inertial>
-                <mass value="0.1"/>
-                <inertia
-                    ixx="0.01" ixy="0.0" ixz="0.0"
-                    iyy="0.01" iyz="0.0" izz="0.01"/>
+                <mass value="0.15"/>
+                <inertia
+                    ixx="0.015" ixy="0.0" ixz="0.0"
+                    iyy="0.015" iyz="0.0" izz="0.015"/>
             </inertial>
             <visual>
@@ -197,8 +197,8 @@
         <link name="${prefix}_${suffix}_finger_vacuum_frame">
             <inertial>
-                <mass value="0.1"/>
-                <inertia
-                    ixx="0.01" ixy="0.0" ixz="0.0"
-                    iyy="0.01" iyz="0.0" izz="0.01"/>
+                <mass value="0.15"/>
+                <inertia
+                    ixx="0.015" ixy="0.0" ixz="0.0"
+                    iyy="0.015" iyz="0.0" izz="0.015"/>
             </inertial>
             <visual>

Commit message: use inertial to finger tip frame

File: hsrb_description/urdf/hand_v0/hand.urdf.xacro (robot description, xacro)
@@ -189,5 +189,6 @@
             <child link="${prefix}_${suffix}_finger_tip_frame" />
         </joint>
-        <link name="${prefix}_${suffix}_finger_tip_frame" />
+        <!-- TODO: this is the right format: <link name="${prefix}_${suffix}_finger_tip_frame" /> -->
+        <xacro:hsrb_gripper_dummy_link name="${prefix}_${suffix}_finger_tip_frame" />
         <joint name="${prefix}_${suffix}_finger_vacuum_frame_joint" type="fixed">
             <origin xyz="0.00475 -0.011539 0.03322" rpy="${pi/4.0} 0.0 0.0" />
@@ -268,5 +269,6 @@
             <child link="${prefix}_${suffix}_finger_tip_frame" />
         </joint>
-        <link name="${prefix}_${suffix}_finger_tip_frame" />
+        <!-- TODO: this is the right format: <link name="${prefix}_${suffix}_finger_tip_frame" /> -->
+        <xacro:hsrb_gripper_dummy_link name="${prefix}_${suffix}_finger_tip_frame" />
     </xacro:macro>
 </robot>

Commit message: fixed wrong links related to wide camera

File: hsrb_description/urdf/hand_v0/hand.urdf.xacro (robot description, xacro)
@@ -75,6 +75,6 @@
         </xacro:hsrb_finger_without_vacuum>
         <!-- camera -->
-        <xacro:wide_camera prefix="${prefix}" parent="${prefix}_palm_link" robot_namespace="${robot_name}">
-            <origin xyz="0.039 0.0 -0.0045" rpy="${pi} ${-pi/2} 0"/>
+        <xacro:wide_camera prefix="${prefix}" parent="${prefix}_palm_link" robot_namespace="${robot_name}" rpy="${pi/2.0} ${-pi/2.0} 0" >
+            <origin xyz="0.039 0.0 -0.0045" rpy="0.0 0.0 0.0"/>
         </xacro:wide_camera>
         <xacro:hsrb_hand_gazebo prefix="${prefix}"/>

File: hsrb_description/urdf/head_v0/head.urdf.xacro (robot description, xacro)
@@ -95,5 +95,5 @@
             <origin xyz="0.02 -0.07 0.061" rpy="${-pi/2.0} 0.0 ${-pi/2.0}"/>
         </xacro:pointgrey_chameleon>
-        <xacro:wide_camera prefix="${prefix}_center" parent="${prefix}_tilt_link" robot_namespace="${robot_name}">
+        <xacro:wide_camera prefix="${prefix}_center" parent="${prefix}_tilt_link" robot_namespace="${robot_name}" rpy="${pi/2.0} ${-pi/2.0} 0.0" >
             <origin xyz="0.0195 0.0 0.061" rpy="${-pi/2.0} 0.0 ${-pi/2.0}"/>
         </xacro:wide_camera>

File: hsrb_description/urdf/head_v1/head.urdf.xacro (robot description, xacro)
@@ -95,5 +95,5 @@
             <origin xyz="0.02 -0.07 0.061" rpy="${-pi/2.0} 0.0 ${-pi/2.0}"/>
         </xacro:pointgrey_chameleon>
-        <xacro:wide_camera prefix="${prefix}_center" parent="${prefix}_tilt_link" robot_namespace="${robot_name}">
+        <xacro:wide_camera prefix="${prefix}_center" parent="${prefix}_tilt_link" robot_namespace="${robot_name}" rpy="${pi/2.0} ${-pi/2.0} 0.0" >
             <origin xyz="0.0195 0.0 0.061" rpy="${-pi/2.0} 0.0 ${-pi/2.0}"/>
         </xacro:wide_camera>

File: hsrb_description/urdf/sensors/wide_camera.urdf.xacro (robot description, xacro)
@@ -3,5 +3,5 @@
     <xacro:include filename="$(find hsrb_description)/urdf/sensors/wide_camera.gazebo.xacro"/>
     <!-- wide rgb camera -->
-    <xacro:macro name="wide_camera" params="prefix parent robot_namespace *origin">
+    <xacro:macro name="wide_camera" params="prefix parent robot_namespace rpy *origin">
         <joint name="${prefix}_camera_frame_joint" type="fixed">
             <insert_block name="origin" />
@@ -11,5 +11,5 @@
         <link name="${prefix}_camera_frame"></link>
         <joint name="${prefix}_camera_gazebo_frame_joint" type="fixed">
-            <origin xyz="0 0 0" rpy="${pi/2.0} ${-pi/2.0} 0.0"/>
+            <origin xyz="0 0 0" rpy="${rpy}"/>
             <parent link="${prefix}_camera_frame" />
             <child link="${prefix}_camera_gazebo_frame" />

Commit message: fix hand_motor_joint range

File: hsrb_description/urdf/hand_v0/hand.urdf.xacro (robot description, xacro)
@@ -7,5 +7,5 @@
     <xacro:property name="palm_to_proximal_y" value="-0.0245" />
     <xacro:property name="palm_to_proximal_z" value="-0.0175" />
-    <xacro:property name="proximal_joint_angle_range_min" value="-0.798" />
+    <xacro:property name="proximal_joint_angle_range_min" value="-0.105" />
     <xacro:property name="proximal_joint_angle_range_max" value="1.24" />
     <xacro:property name="spring_proximal_joint_angle_range_min" value="0.0" />

Commit message: fix hand min limit / add comment

File: hsrb_description/urdf/hand_v0/hand.urdf.xacro (robot description, xacro)
@@ -7,5 +7,6 @@
     <xacro:property name="palm_to_proximal_y" value="-0.0245" />
     <xacro:property name="palm_to_proximal_z" value="-0.0175" />
-    <xacro:property name="proximal_joint_angle_range_min" value="-0.105" />
+    <!-- soft limit:-0.1 = proximal_joint_angle_range_min + spring_proximal_joint_angle_range_max -->
+    <xacro:property name="proximal_joint_angle_range_min" value="-0.798" />
     <xacro:property name="proximal_joint_angle_range_max" value="1.24" />
     <xacro:property name="spring_proximal_joint_angle_range_min" value="0.0" />

Commit message: modify hand mimic joint

File: hsrb_description/urdf/hand_v0/hand.urdf.xacro (robot description, xacro)
@@ -90,4 +90,5 @@
             <parent link="${parent}" />
             <child link="${prefix}_${suffix}_proximal_link" />
+            <mimic joint="${prefix}_motor_joint" />
 	    <dynamics damping="0.0001"/>
         </joint>
@@ -101,5 +102,4 @@
             <parent link="${prefix}_${suffix}_proximal_link" />
             <child link="${prefix}_${suffix}_spring_proximal_link" />
-	    <mimic joint="${prefix}_motor_joint" />
             <dynamics damping="0.0001"/>
         </joint>

Commit message: fix indent

File: hsrb_description/urdf/hand_v0/hand.urdf.xacro (robot description, xacro)
@@ -91,5 +91,5 @@
             <child link="${prefix}_${suffix}_proximal_link" />
             <mimic joint="${prefix}_motor_joint" />
-	    <dynamics damping="0.0001"/>
+            <dynamics damping="0.0001"/>
         </joint>
         <!-- dummy link -->
@@ -115,6 +115,6 @@
             <parent link="${parent}" />
             <child link="${prefix}_${suffix}_mimic_distal_link" />
-	    <mimic joint="${prefix}_${suffix}_spring_proximal_joint" multiplier="-1.0" />
-	    <dynamics damping="0.0001"/>
+            <mimic joint="${prefix}_${suffix}_spring_proximal_joint" multiplier="-1.0" />
+            <dynamics damping="0.0001"/>
         </joint>
         <!-- dummy link -->
@@ -127,5 +127,5 @@
             <parent link="${prefix}_${suffix}_mimic_distal_link" />
             <child link="${prefix}_${suffix}_distal_link" />
-	    <dynamics damping="0.0001"/>
+            <dynamics damping="0.0001"/>
         </joint>
     </xacro:macro>
@@ -182,5 +182,5 @@
             <parent link="${prefix}_${suffix}_distal_link" />
             <child link="${prefix}_${suffix}_finger_tip_frame" />
-	    <dynamics damping="0.0001"/>
+            <dynamics damping="0.0001"/>
         </joint>
         <!-- TODO: this is the right format: <link name="${prefix}_${suffix}_finger_tip_frame" /> -->

Commit message: fix hand offset

File: hsrb_description/urdf/hand_v0/hand.urdf.xacro (robot description, xacro)
@@ -127,4 +127,5 @@
             <parent link="${prefix}_${suffix}_mimic_distal_link" />
             <child link="${prefix}_${suffix}_distal_link" />
+            <mimic joint="${prefix}_motor_joint" multiplier="-1.0" offset="${-distal_joint_angle_offset}"/>
             <dynamics damping="0.0001"/>
         </joint>

Commit message: fix reviewed points.

File: hsrb_description/urdf/hand_v0/hand.urdf.xacro (robot description, xacro)
@@ -127,5 +127,5 @@
             <parent link="${prefix}_${suffix}_mimic_distal_link" />
             <child link="${prefix}_${suffix}_distal_link" />
-	    <mimic joint="${prefix}_motor_joint" multiplier="-1.0" offset="${-distal_joint_angle_offset}"/>
+            <mimic joint="${prefix}_motor_joint" multiplier="-1.0" offset="${-distal_joint_angle_offset}"/>
             <dynamics damping="0.0001"/>
         </joint>

File: hsrb_parts_description/urdf/sensors/minebea_ft_sensor.urdf.xacro (robot description, xacro)
@@ -18,5 +18,5 @@
         <xacro:minebea_ft_sensor_gazebo
             robot_namespace="${robot_namespace}"
-            joint_name="${prefix}_ft_sensor_frame_joint" ros_topic="${prefix}_wrench" />
+            joint_name="${prefix}_ft_sensor_frame_joint" ros_topic="${prefix}_wrench/raw" />
     </xacro:macro>
 </robot>

File: hsrc_description/urdf/base_v0/base.urdf.xacro (robot description, xacro)
@@ -105,5 +105,11 @@
     <!-- base -->
     <xacro:macro name="hsrb_base" params="prefix robot_namespace">
-        <link name="base_footprint"/>
+        <link name="base_footprint">
+            <inertial>
+                <origin xyz="0 0 0"/>
+                <mass value="0.01"/>
+                <inertia ixx="0.001" ixy="0" ixz="0" iyy="0.001" iyz="0" izz="0.001"/>
+            </inertial>
+        </link>
         <joint name="${prefix}_footprint_joint" type="fixed">
             <parent link="base_footprint" />

File: hsrc_description/urdf/hand_v0/hand.urdf.xacro (robot description, xacro)
@@ -17,5 +17,5 @@
         <link name="${name}">
             <inertial>
-                <mass value="0.15"/>
+                <mass value="0.01"/>
                 <inertia
                     ixx="0.015" ixy="0.0" ixz="0.0"

Commit message: Modify finger_tip_frame

File: hsrb_description/urdf/hand_v0/hand.urdf.xacro (robot description, xacro)
@@ -180,5 +180,5 @@
         </link>
         <joint name="${prefix}_${suffix}_finger_tip_frame_joint" type="fixed">
-            <origin xyz="0.01675 0.0193 0.0379" rpy="${-pi/2.0} 0.0 0.0" />
+            <origin xyz="0.01675 0.018 0.039" rpy="${-pi/2.0} 0.0 0.0" />
             <parent link="${prefix}_${suffix}_distal_link" />
             <child link="${prefix}_${suffix}_finger_tip_frame" />
@@ -257,5 +257,5 @@
         </link>
         <joint name="${prefix}_${suffix}_finger_tip_frame_joint" type="fixed">
-            <origin xyz="0.01675 -0.0193 0.0379" rpy="${pi/2.0} 0.0 0.0" />
+            <origin xyz="0.01675 -0.018 0.039" rpy="${pi/2.0} 0.0 0.0" />
             <parent link="${prefix}_${suffix}_distal_link" />
             <child link="${prefix}_${suffix}_finger_tip_frame" />

Commit message: Adjust to design value

File: hsrb_description/urdf/hand_v0/hand.urdf.xacro (robot description, xacro)
@@ -180,5 +180,5 @@
         </link>
         <joint name="${prefix}_${suffix}_finger_tip_frame_joint" type="fixed">
-            <origin xyz="0.01675 0.018 0.039" rpy="${-pi/2.0} 0.0 0.0" />
+            <origin xyz="0.01675 0.01865 0.04289" rpy="${-pi/2.0} 0.0 0.0" />
             <parent link="${prefix}_${suffix}_distal_link" />
             <child link="${prefix}_${suffix}_finger_tip_frame" />
@@ -257,5 +257,5 @@
         </link>
         <joint name="${prefix}_${suffix}_finger_tip_frame_joint" type="fixed">
-            <origin xyz="0.01675 -0.018 0.039" rpy="${pi/2.0} 0.0 0.0" />
+            <origin xyz="0.01675 -0.01865 0.04289" rpy="${pi/2.0} 0.0 0.0" />
             <parent link="${prefix}_${suffix}_distal_link" />
             <child link="${prefix}_${suffix}_finger_tip_frame" />
