Commit message: changed sensor configuration and grasp hack parameter

File: hsrb_description/urdf/hand_v0/hand.gazebo.xacro (robot description, xacro)
@@ -30,5 +30,5 @@
                 <grasp_check>
                     <attach_steps>1</attach_steps>
-                    <detach_steps>5</detach_steps>
+                    <detach_steps>2</detach_steps>
                     <min_contact_count>1</min_contact_count>
                 </grasp_check>

File: hsrb_description/urdf/head_v0/head.urdf.xacro (robot description, xacro)
@@ -89,8 +89,8 @@
         </link>
         <!-- cameras -->
-        <xacro:pointgrey_chameleon prefix="${prefix}_l_stereo" parent="${prefix}_tilt_link" robot_namespace="${robot_name}">
+        <xacro:pointgrey_chameleon prefix="${prefix}_l_stereo" parent="${prefix}_tilt_link" robot_namespace="${robot_name}" baseline="0.00">
             <origin xyz="0.02 0.07 0.061" rpy="${-pi/2.0} 0.0 ${-pi/2.0}"/>
         </xacro:pointgrey_chameleon>
-        <xacro:pointgrey_chameleon prefix="${prefix}_r_stereo" parent="${prefix}_tilt_link" robot_namespace="${robot_name}">
+        <xacro:pointgrey_chameleon prefix="${prefix}_r_stereo" parent="${prefix}_tilt_link" robot_namespace="${robot_name}" baseline="0.14">
             <origin xyz="0.02 -0.07 0.061" rpy="${-pi/2.0} 0.0 ${-pi/2.0}"/>
         </xacro:pointgrey_chameleon>

File: hsrb_description/urdf/sensors/pointgrey_chameleon.gazebo.xacro (robot description, xacro)
@@ -1,13 +1,13 @@
 <?xml version="1.0" ?>
 <robot name="hsrb" xmlns:xacro="http://www.ros.org/wiki/xacro">
-    <xacro:macro name="pointgrey_chameleon_gazebo" params="sensor_name parent_frame topic_frame_id robot_namespace">
+    <xacro:macro name="pointgrey_chameleon_gazebo" params="sensor_name parent_frame topic_frame_id robot_namespace baseline">
         <gazebo reference="${parent_frame}">
-            <sensor type="multicamera" name="stereo_camera">
+            <sensor type="camera" name="${sensor_name}">
                 <update_rate>10.0</update_rate>
-                <camera name="left">
+                <camera name="${sensor_name}">
                     <horizontal_fov>1.16762527</horizontal_fov>
                     <image>
                         <width>1280</width>
-                        <height>960</height>
+                        <height>1024</height>
                         <format>R8G8B8</format>
                     </image>
@@ -22,23 +22,5 @@
                     </noise>
                 </camera>
-                <camera name="right">
-                  <pose>0 -0.07 0 0 0 0</pose>
-                    <horizontal_fov>1.16762527</horizontal_fov>
-                    <image>
-                        <width>1280</width>
-                        <height>960</height>
-                        <format>R8G8B8</format>
-                    </image>
-                    <clip>
-                        <near>0.05</near>
-                        <far>100</far>
-                    </clip>
-                    <noise>
-                        <type>gaussian</type>
-                        <mean>0.0</mean>
-                        <stddev>0.007</stddev>
-                    </noise>
-                </camera>
-                <plugin name="camera_controller" filename="libgazebo_ros_multicamera.so">
+                <plugin name="camera_controller" filename="libgazebo_ros_camera.so">
                     <alwaysOn>0</alwaysOn>
                     <updateRate>0.0</updateRate>
@@ -48,5 +30,5 @@
                     <frameName>${topic_frame_id}</frameName>
                     <robotNamespace>${robot_namespace}</robotNamespace>
-                    <hackBaseline>0.07</hackBaseline>
+                    <hackBaseline>${baseline}</hackBaseline>
                     <distortionK1>0.0</distortionK1>
                     <distortionK2>0.0</distortionK2>

File: hsrb_description/urdf/sensors/pointgrey_chameleon.urdf.xacro (robot description, xacro)
@@ -2,5 +2,5 @@
 <robot xmlns:xacro="http://ros.org/wiki/xacro">
     <xacro:include filename="$(find hsrb_description)/urdf/sensors/pointgrey_chameleon.gazebo.xacro"/>
-    <xacro:macro name="pointgrey_chameleon" params="prefix parent robot_namespace *origin">
+    <xacro:macro name="pointgrey_chameleon" params="prefix parent robot_namespace *origin baseline">
         <joint name="${prefix}_camera_joint" type="fixed">
             <insert_block name="origin" />
@@ -27,5 +27,6 @@
             parent_frame="${prefix}_camera_gazebo_frame"
             topic_frame_id="${prefix}_camera_frame"
-            robot_namespace="${robot_namespace}"/>
+            robot_namespace="${robot_namespace}"
+            baseline="${baseline}" />
     </xacro:macro>
 </robot>

Commit message: Stabilize gripper control.
- light weight dummy mass.
- fasten control period.
- update dumping factor(for sim only)
- set max_torque

File: hsrb_description/urdf/hand_v0/hand.gazebo.xacro (robot description, xacro)
@@ -26,5 +26,9 @@
         <gazebo_joint name="${prefix}_r_distal_joint"/>
         <gazebo>
-            <plugin name="hsrb_hrh_gripper_plugin" filename="libtmc_gazebo_hrh_gripper.so"></plugin>
+          <plugin name="hsrb_hrh_gripper_plugin" filename="libtmc_gazebo_hrh_gripper.so">
+	    <sensitiveness>0.05</sensitiveness>
+	    <update_rate>1000.0</update_rate>
+	    <max_torque>8.0</max_torque>
+	  </plugin>
             <plugin name="hsrb_grasp_hack_plugin" filename="libhsrb_grasp_hack.so">
                 <grasp_check>
@@ -38,5 +42,5 @@
                 <gripper_link>${prefix}_r_spring_proximal_link</gripper_link>
                 <gripper_link>${prefix}_l_spring_proximal_link</gripper_link>
-                <!-- hand_palm_link is merged with wrist_roll_link by fixed joint -->
+		<!-- hand_palm_link is merged with wrist_roll_link by fixed joint  -->
                 <palm_link>wrist_roll_link</palm_link>
             </plugin>

File: hsrb_description/urdf/hand_v0/hand.urdf.xacro (robot description, xacro)
@@ -17,8 +17,8 @@
         <link name="${name}">
             <inertial>
-                <mass value="0.15"/>
-                <inertia
-                    ixx="0.015" ixy="0.0" ixz="0.0"
-                    iyy="0.015" iyz="0.0" izz="0.015"/>
+                <mass value="0.001"/>
+                <inertia
+                    ixx="0.00015" ixy="0.0" ixz="0.0"
+                    iyy="0.00015" iyz="0.0" izz="0.00015"/>
             </inertial>
         </link>
@@ -56,5 +56,5 @@
             <parent link="${prefix}_palm_link" />
             <child link="${prefix}_motor_dummy_link" />
-            <dynamics damping="1.0"/>
+            <dynamics damping="0.0001"/>
         </joint>
         <!-- dummy link -->
@@ -90,6 +90,5 @@
             <parent link="${parent}" />
             <child link="${prefix}_${suffix}_proximal_link" />
-            <mimic joint="${prefix}_motor_joint" />
-            <dynamics damping="1.0"/>
+	    <dynamics damping="0.0001"/>
         </joint>
         <!-- dummy link -->
@@ -97,10 +96,11 @@
         <joint name="${prefix}_${suffix}_spring_proximal_joint" type="revolute">
             <xacro:insert_block name="axis" />
-            <limit effort="100.0" velocity="1.0"
+            <limit effort="10.0" velocity="1.0"
                 lower="${spring_proximal_joint_angle_range_min}"
                 upper="${spring_proximal_joint_angle_range_max}" />
             <parent link="${prefix}_${suffix}_proximal_link" />
             <child link="${prefix}_${suffix}_spring_proximal_link" />
-            <dynamics damping="1.0"/>
+	    <mimic joint="${prefix}_motor_joint" />
+            <dynamics damping="0.0001"/>
         </joint>
     </xacro:macro>
@@ -115,6 +115,6 @@
             <parent link="${parent}" />
             <child link="${prefix}_${suffix}_mimic_distal_link" />
-            <mimic joint="${prefix}_${suffix}_spring_proximal_joint" multiplier="-1.0" />
-            <dynamics damping="1.0"/>
+	    <mimic joint="${prefix}_${suffix}_spring_proximal_joint" multiplier="-1.0" />
+	    <dynamics damping="0.0001"/>
         </joint>
         <!-- dummy link -->
@@ -127,6 +127,5 @@
             <parent link="${prefix}_${suffix}_mimic_distal_link" />
             <child link="${prefix}_${suffix}_distal_link" />
-            <mimic joint="${prefix}_motor_joint" multiplier="-1.0" offset="${-distal_joint_angle_offset}"/>
-            <dynamics damping="1.0"/>
+	    <dynamics damping="0.0001"/>
         </joint>
     </xacro:macro>
@@ -183,4 +182,5 @@
             <parent link="${prefix}_${suffix}_distal_link" />
             <child link="${prefix}_${suffix}_finger_tip_frame" />
+	    <dynamics damping="0.0001"/>
         </joint>
         <!-- TODO: this is the right format: <link name="${prefix}_${suffix}_finger_tip_frame" /> -->
@@ -193,8 +193,8 @@
         <link name="${prefix}_${suffix}_finger_vacuum_frame">
             <inertial>
-                <mass value="0.15"/>
-                <inertia
-                    ixx="0.015" ixy="0.0" ixz="0.0"
-                    iyy="0.015" iyz="0.0" izz="0.015"/>
+                <mass value="0.001"/>
+                <inertia
+                    ixx="0.00015" ixy="0.0" ixz="0.0"
+                    iyy="0.00015" iyz="0.0" izz="0.00015"/>
             </inertial>
             <visual>

Commit message: add sensor frame to collect force sensor direction.

File: hsrb_description/urdf/hand_v0/hand.gazebo.xacro (robot description, xacro)
@@ -42,6 +42,6 @@
             <gripper_link>${prefix}_r_spring_proximal_link</gripper_link>
             <gripper_link>${prefix}_l_spring_proximal_link</gripper_link>
-	    <!-- hand_palm_link is merged with wrist_roll_link by fixed joint  -->
-            <palm_link>wrist_roll_link</palm_link>
+	    <!-- hand_palm_link is merged with wrist_ft_sensor_frame by fixed joint  -->
+            <palm_link>wrist_ft_sensor_frame</palm_link>
           </plugin>
         </gazebo>

File: hsrb_description/urdf/wrist_v0/wrist.urdf.xacro (robot description, xacro)
@@ -46,6 +46,20 @@
             <limit effort="100.0" velocity="1.5" lower="-1.92" upper="3.67" />
             <parent link="${prefix}_flex_link" />
+            <child link="${prefix}_ft_sensor_mount_link" />
+            <dynamics damping="1.0"/>
+        </joint>
+        <!-- each link must have mass in URDF so we apply very small mass (10 gram) for this coupling link -->
+        <link name="${prefix}_ft_sensor_mount_link">
+          <inertial>
+            <mass value="0.01"/>
+            <inertia ixx="0.001" ixy="0.0" ixz="0.0"
+                     iyy="0.001" iyz="0.0"
+                     izz="0.001" />
+          </inertial>
+        </link>
+        <joint name="${prefix}_ft_sensor_frame_inverse_joint" type="fixed">
+            <origin xyz="0.0 0.0 0.0735" rpy="-${pi} 0.0 0.0"/>
+            <parent link="${prefix}_ft_sensor_frame" />
             <child link="${prefix}_roll_link" />
-            <dynamics damping="1.0"/>
         </joint>
         <link name="${prefix}_roll_link">
@@ -70,6 +84,5 @@
             prefix="${prefix}"
             robot_namespace="${robot_namespace}"
-            parent="${prefix}_roll_link"
-            joint_name="${prefix}_roll_joint">
+            parent="${prefix}_ft_sensor_mount_link">
             <origin xyz="0.0 0.0 0.0735" rpy="${pi} 0.0 0.0"/>
         </xacro:minebea_ft_sensor>

File: hsrb_parts_description/urdf/sensors/minebea_ft_sensor.gazebo.xacro (robot description, xacro)
@@ -1,14 +1,13 @@
 <?xml version="1.0" ?>
 <robot name="hsrb" xmlns:xacro="http://ros.org/wiki/xacro">
-    <xacro:macro name="minebea_ft_sensor_gazebo" params="sensor_name robot_namespace joint_name ros_topic">
+    <xacro:macro name="minebea_ft_sensor_gazebo" params="robot_namespace joint_name ros_topic">
         <gazebo reference="${joint_name}">
             <provideFeedback>true</provideFeedback>
         </gazebo>
         <gazebo>
-            <plugin name="ft_sensor" filename="libgazebo_ros_force.so">
+            <plugin name="ft_sensor" filename="libgazebo_ros_ft_sensor.so">
                 <updateRate>30.0</updateRate>
                 <topicName>${ros_topic}</topicName>
                 <jointName>${joint_name}</jointName>
-                <bodyName>wrist_roll_link</bodyName>
                 <robotNamespace>${robot_namespace}</robotNamespace>
             </plugin>

File: hsrb_parts_description/urdf/sensors/minebea_ft_sensor.urdf.xacro (robot description, xacro)
@@ -2,14 +2,21 @@
 <robot name="hsrb" xmlns:xacro="http://ros.org/wiki/xacro">
     <xacro:include filename="$(find hsrb_parts_description)/urdf/sensors/minebea_ft_sensor.gazebo.xacro"/>
-    <xacro:macro name="minebea_ft_sensor" params="prefix robot_namespace parent joint_name *origin">
-        <joint name="${prefix}_ft_sensor_frame_joint" type="fixed">
+    <xacro:macro name="minebea_ft_sensor" params="prefix robot_namespace parent *origin">
+        <joint name="${prefix}_ft_sensor_frame_joint" type="revolute">
             <xacro:insert_block name="origin"/>
             <parent link="${parent}"/>
             <child link="${prefix}_ft_sensor_frame"/>
+            <limit effort="100.0" velocity="1.5" lower="0" upper="0" />
         </joint>
-        <link name="${prefix}_ft_sensor_frame"/>
+        <link name="${prefix}_ft_sensor_frame">
+            <inertial>
+                <origin xyz="0 0 0"/>
+                <mass value="0.01"/>
+                <inertia ixx="0.001" ixy="0" ixz="0" iyy="0.001" iyz="0" izz="0.001"/>
+            </inertial>
+        </link>
         <xacro:minebea_ft_sensor_gazebo
-            sensor_name="${prefix}_ft_sensor" robot_namespace="${robot_namespace}"
-            joint_name="${joint_name}" ros_topic="${prefix}_wrench" />
+            robot_namespace="${robot_namespace}"
+            joint_name="${prefix}_ft_sensor_frame_joint" ros_topic="${prefix}_wrench/raw" />
     </xacro:macro>
 </robot>

Commit message: Add gain parameters for gazebo gripper plugin

File: hsrb_description/urdf/hand_v0/hand.gazebo.xacro (robot description, xacro)
@@ -25,29 +25,4 @@
         <xacro:gazebo_joint name="${prefix}_r_mimic_distal_joint"/>
         <xacro:gazebo_joint name="${prefix}_r_distal_joint"/>
-        <gazebo>
-          <plugin name="hsrb_hrh_gripper_plugin" filename="libtmc_gazebo_ros_hrh_gripper.so">
-            <sensitiveness>0.05</sensitiveness>
-            <update_rate>1000.0</update_rate>
-            <max_torque>8.0</max_torque>
-            <error_tolerance>0.0872</error_tolerance>
-            <stall_timeout>2.0</stall_timeout>
-            <robot_namespace>${personal_name}/${robot_name}</robot_namespace>
-          </plugin>
-          <!-- <plugin name="hsrb_grasp_hack_plugin" filename="libhsrb_grasp_hack.so">
-            <grasp_check>
-              <attach_steps>1</attach_steps>
-              <detach_steps>2</detach_steps>
-              <min_contact_count>1</min_contact_count>
-              <max_attach_weight>1.2</max_attach_weight>
-            </grasp_check>
-            <gripper_link>${prefix}_r_distal_link</gripper_link>
-            <gripper_link>${prefix}_l_distal_link</gripper_link>
-            <gripper_link>${prefix}_r_spring_proximal_link</gripper_link>
-            <gripper_link>${prefix}_l_spring_proximal_link</gripper_link> -->
-	    <!-- hand_palm_link is merged with wrist_ft_sensor_frame by fixed joint  -->
-            <!-- <palm_link>wrist_ft_sensor_frame</palm_link>
-            <robot_namespace>${personal_name}/${robot_name}</robot_namespace>
-          </plugin> -->
-        </gazebo>
     </xacro:macro>
 </robot>

File: hsrb_description/urdf/hand_v0/hand.urdf.xacro (robot description, xacro)
@@ -16,8 +16,8 @@
         <link name="${name}">
             <inertial>
-                <mass value="0.01"/>
-                <inertia
-                    ixx="0.0015" ixy="0.0" ixz="0.0"
-                    iyy="0.0015" iyz="0.0" izz="0.0015"/>
+                <mass value="0.001"/>
+                <inertia
+                    ixx="0.0" ixy="0.0" ixz="0.0"
+                    iyy="0.0" iyz="0.0" izz="0.0"/>
             </inertial>
         </link>
@@ -137,9 +137,9 @@
         <link name="${prefix}_${suffix}_spring_proximal_link">
             <inertial>
-                <mass value="0.043589"/>
+                <mass value="0.001"/>
                 <origin xyz="0.021418 0.00248 0.022688"/>
                 <inertia
-                    ixx="0.000026033886" ixy="-0.000000144078" ixz="-0.00000198241"
-                    iyy="0.000028824811" iyz="-0.000001268421" izz="0.000005135919"/>
+                    ixx="0.00" ixy="-0.00000" ixz="-0.0000"
+                    iyy="0.00" iyz="-0.00000" izz="0.00000"/>
             </inertial>
             <visual>
@@ -160,9 +160,9 @@
         <link name="${prefix}_${suffix}_distal_link">
             <inertial>
-                <mass value="0.027731"/>
+                <mass value="0.001"/>
                 <origin xyz="0.011116 0.005679 0.017532"/>
                 <inertia
-                    ixx="0.000004451952" ixy="-0.000000617574" ixz="0.000000503765"
-                    iyy="0.000000503765" iyz="-0.000000435048" izz="0.000004456764"/>
+                    ixx="0.0" ixy="-0.00" ixz="0.0"
+                    iyy="0.0" iyz="-0.000" izz="0.0"/>
             </inertial>
             <visual>
@@ -192,8 +192,8 @@
         <link name="${prefix}_${suffix}_finger_vacuum_frame">
             <inertial>
-                <mass value="0.01"/>
-                <inertia
-                    ixx="0.0015" ixy="0.0" ixz="0.0"
-                    iyy="0.0015" iyz="0.0" izz="0.0015"/>
+                <mass value="0.001"/>
+                <inertia
+                    ixx="0.0" ixy="0.0" ixz="0.0"
+                    iyy="0.0" iyz="0.0" izz="0.0"/>
             </inertial>
             <visual>
@@ -214,9 +214,9 @@
         <link name="${prefix}_${suffix}_spring_proximal_link">
             <inertial>
-                <mass value="0.043956"/>
+                <mass value="0.001"/>
                 <origin xyz="0.013203 0.002096 0.023311"/>
                 <inertia
-                    ixx="0.00002623664" ixy="0.00000001631" ixz="0.000001281845"
-                    iyy="0.000028838232" iyz="-0.000001621709" izz="0.000004957151"/>
+                    ixx="0.0" ixy="0.0" ixz="0.0"
+                    iyy="0.0" iyz="0.0" izz="0.0"/>
             </inertial>
             <visual>
@@ -237,9 +237,9 @@
         <link name="${prefix}_${suffix}_distal_link">
             <inertial>
-                <mass value="0.020927"/>
+                <mass value="0.001"/>
                 <origin xyz="0.014256 -0.008321 0.015591"/>
                 <inertia
-                    ixx="0.00000307518" ixy="-0.00000004954" ixz="0.000000009481"
-                    iyy="0.000004074079" iyz="0.000000843648" izz="0.000002807795"/>
+                    ixx="0.0" ixy="0.0" ixz="0.0"
+                    iyy="0.0" iyz="0.0" izz="0.0"/>
             </inertial>
             <visual>

File: hsrb_description/urdf/ros2_control.gazebo.xacro (robot description, xacro)
@@ -3,9 +3,28 @@
   <xacro:macro name="ros2_contorl_gazebo">
     <gazebo>
-      <plugin filename="libgazebo_ros2_control.so" name="gazebo_ros2_control">
+      <plugin name="gazebo_ros2_control" filename="libgazebo_ros2_control.so">
         <robot_sim_type>gazebo_ros2_control/GazeboSystem</robot_sim_type>
         <parameters>$(find hsrb_gazebo_bringup)/config/gazebo_ros2_control.yaml</parameters>
         <ros>
         </ros>
+      </plugin>
+      <plugin name="hrh_gripper_plugin" filename="libtmc_gazebo_ros_hrh_gripper.so">
+        <sensitiveness>0.05</sensitiveness>
+        <update_rate>1000.0</update_rate>
+        <max_torque>20.0</max_torque>
+        <error_tolerance>0.0872</error_tolerance>
+        <stall_timeout>2.0</stall_timeout>
+        <robot_namespace>${personal_name}/${robot_name}</robot_namespace>
+        <parameters>
+          <hand_motor_joint p="50.0" d="20.0"/>
+          <hand_l_proximal_joint p="50.0" d="20.0"/>
+          <hand_l_spring_proximal_joint p="50.0" d="20.0"/>
+          <hand_l_mimic_distal_joint p="20.0" d="8.0"/>
+          <hand_l_distal_joint p="1.0" d="0.0"/>
+          <hand_r_proximal_joint p="50.0" d="20.0"/>
+          <hand_r_spring_proximal_joint p="50.0" d="20.0"/>
+          <hand_r_mimic_distal_joint p="20.0" d="8.0"/>
+          <hand_r_distal_joint p="20.0" d="8.0"/>
+        </parameters>
       </plugin>
     </gazebo>
