Commit message: Parameterize IMU topic name

File: hsrb_parts_description/urdf/sensors/kinetic/imu.gazebo.xacro (robot description, xacro)
@@ -1,5 +1,5 @@
 <?xml version="1.0" ?>
 <robot name="hsrb" xmlns:xacro="http://ros.org/wiki/xacro">
-    <xacro:macro name="imu_gazebo" params="sensor_name frame_name robot_namespace">
+    <xacro:macro name="imu_gazebo" params="sensor_name frame_name topic_name robot_namespace">
         <gazebo reference="${frame_name}">
             <sensor type="imu" name="${sensor_name}">
