Commit message: fix

File: hsrb_description/urdf/common/melodic/common.xacro (robot description, xacro)
@@ -79,5 +79,5 @@
     </gazebo>
   </xacro:macro>
-  <xacro:macro name="gazebo_link_bumper" params="name personal_name robot_type gravity collide friction">
+  <xacro:macro name="gazebo_link_bumper" params="name gravity collide friction">
     <gazebo reference="${name}_link">
       <selfCollide>${collide}</selfCollide>
@@ -92,5 +92,5 @@
         </contact>
         <plugin name="hsrb_gazebo_ros_bumper_controller" filename="libhsrb_gazebo_ros_bumper.so">
-          <robotNamespace>${personal_name}/${robot_type}</robotNamespace>
+          <robotNamespace>hsrb</robotNamespace>
           <bumperTopicName>${name}_sensor</bumperTopicName>
           <frameName>${name}_link</frameName>

File: hsrb_parts_description/urdf/sensors/melodic/imu.gazebo.xacro (robot description, xacro)
@@ -8,6 +8,6 @@
 		    <updateRateHZ>50.0</updateRateHZ>
 		    <bodyName>base_link</bodyName>
-                    <topicName>${robot_namespace}/${sensor_name}/data</topicName>
-                    <frameName>${personal_name}/${frame_name}</frameName>
+		    <topicName>${robot_namespace}/${sensor_name}/data</topicName>
+		    <frameName>${frame_name}</frameName>
 		    <gaussianNoise>0.0</gaussianNoise>
 		    <xyzOffset>0.0 0.0 0.0</xyzOffset>

File: hsrb_parts_description/urdf/sensors/melodic/mynteye_imu.gazebo.xacro (robot description, xacro)
@@ -8,6 +8,6 @@
 		    <updateRateHZ>100.0</updateRateHZ>
 		    <bodyName>base_link</bodyName>
-		    <topicName>${sensor_name}/${topic_name}</topicName>
-		    <frameName>${personal_name}/${frame_name}</frameName>
+		    <topicName>${robot_namespace}/${sensor_name}/data</topicName>
+		    <frameName>${frame_name}</frameName>
 		    <gaussianNoise>0.0</gaussianNoise>
 		    <xyzOffset>0.0 0.0 0.0</xyzOffset>
