Commit message: change common.xacro depends on ros distributions.

File: hsrb_description/urdf/common.xacro (robot description, xacro)
@@ -1,94 +1,4 @@
 <?xml version="1.0"?>
 <robot xmlns:xacro="http://ros.org/wiki/xacro">
-  <xacro:arg name="implicit_damping" default="false" />
-  <xacro:property name="pi" value="3.14159265359"/>
-  <xacro:macro name="hsrb_position_joint_transmission" params="joint reduction">
-     <transmission name="${joint}_transmission">
-       <type>transmission_interface/SimpleTransmission</type>
-       <joint name="${joint}">
-         <hardwareInterface>hardware_interface/PositionJointInterface</hardwareInterface>
-       </joint>
-       <actuator name="${joint}_actuator">
-         <hardwareInterface>hardware_interface/PositionJointInterface</hardwareInterface>
-         <mechanicalReduction>${reduction}</mechanicalReduction>
-       </actuator>
-     </transmission>
-  </xacro:macro>
-  <xacro:macro name="hsrb_effort_joint_transmission" params="joint reduction">
-     <transmission name="${joint}_transmission">
-       <type>transmission_interface/SimpleTransmission</type>
-       <joint name="${joint}">
-         <hardwareInterface>hardware_interface/EffortJointInterface</hardwareInterface>
-       </joint>
-       <actuator name="${joint}_actuator">
-         <hardwareInterface>hardware_interface/EffortJointInterface</hardwareInterface>
-         <mechanicalReduction>${reduction}</mechanicalReduction>
-       </actuator>
-     </transmission>
-  </xacro:macro>
-  <xacro:macro name="hsrb_velocity_joint_transmission" params="joint reduction">
-      <transmission name="${prefix}_transmission">
-          <type>transmission_interface/SimpleTransmission</type>
-          <joint name="${joint}">
-            <hardwareInterface>hardware_interface/VelocityJointInterface</hardwareInterface>
-          </joint>
-          <actuator name="${joint}_actuator">
-              <hardwareInterface>hardware_interface/VelocityJointInterface</hardwareInterface>
-              <mechanicalReduction>${reduction}</mechanicalReduction>
-          </actuator>
-      </transmission>
-  </xacro:macro>
-  <xacro:macro name="gazebo_link" params="name gravity collide friction">
-    <gazebo reference="${name}">
-      <selfCollide>${collide}</selfCollide>
-      <gravity>${gravity}</gravity>
-      <mu1>${friction}</mu1>
-      <mu2>${friction}</mu2>
-    </gazebo>
-  </xacro:macro>
-  <xacro:macro name="gazebo_link_flat_black" params="name gravity collide friction">
-    <gazebo reference="${name}">
-      <selfCollide>${collide}</selfCollide>
-      <gravity>${gravity}</gravity>
-      <mu1>${friction}</mu1>
-      <mu2>${friction}</mu2>
-      <material value="Gazebo/FlatBlack"/>
-    </gazebo>
-  </xacro:macro>
-  <xacro:macro name="gazebo_link_caster" params="name">
-    <gazebo reference="${name}">
-      <selfCollide>false</selfCollide>
-      <gravity>true</gravity>
-      <mu1>0.1</mu1>
-      <mu2>0.1</mu2>
-      <maxVel>1.0</maxVel>
-      <material value="Gazebo/FlatBlack"/>
-    </gazebo>
-  </xacro:macro>
-  <xacro:macro name="gazebo_link_rubber" params="name">
-    <gazebo reference="${name}">
-      <selfCollide>false</selfCollide>
-      <gravity>true</gravity>
-      <turnGravityOff>false</turnGravityOff>
-      <kp>1000000.0</kp>
-      <kd>10.0</kd>
-      <mu1>1.0</mu1>
-      <mu2>1.0</mu2>
-      <fdir1>1 0 0</fdir1>
-      <maxVel>1.0</maxVel>
-      <minDepth>0.00</minDepth>
-      <material value="Gazebo/FlatBlack"/>
-    </gazebo>
-  </xacro:macro>
-  <xacro:macro name="gazebo_joint" params="name">
-    <gazebo reference="${name}">
-      <xacro:if value="$(arg implicit_damping)">
-        <implicitSpringDamper>1</implicitSpringDamper>
-      </xacro:if>
-    </gazebo>
-  </xacro:macro>
-  <xacro:macro name="gazebo_joint_mimic" params="name">
-    <gazebo reference="${name}">
-    </gazebo>
-  </xacro:macro>
+    <xacro:include filename="$(find hsrb_description)/urdf/common/$(env ROS_DISTRO)/common.xacro"/>
 </robot>

Commit message: Update common.xacro and imu.gazebo.xacro for melodic

File: hsrb_description/urdf/common.xacro (robot description, xacro)
@@ -1,4 +1,112 @@
 <?xml version="1.0"?>
 <robot xmlns:xacro="http://ros.org/wiki/xacro">
-    <xacro:include filename="$(find hsrb_description)/urdf/common/$(env ROS_DISTRO)/common.xacro"/>
+  <xacro:arg name="implicit_damping" default="false" />
+  <xacro:macro name="hsrb_position_joint_transmission" params="joint reduction">
+     <transmission name="${joint}_transmission">
+       <type>transmission_interface/SimpleTransmission</type>
+       <joint name="${joint}">
+         <hardwareInterface>hardware_interface/PositionJointInterface</hardwareInterface>
+       </joint>
+       <actuator name="${joint}_actuator">
+         <hardwareInterface>hardware_interface/PositionJointInterface</hardwareInterface>
+         <mechanicalReduction>${reduction}</mechanicalReduction>
+       </actuator>
+     </transmission>
+  </xacro:macro>
+  <xacro:macro name="hsrb_effort_joint_transmission" params="joint reduction">
+     <transmission name="${joint}_transmission">
+       <type>transmission_interface/SimpleTransmission</type>
+       <joint name="${joint}">
+         <hardwareInterface>hardware_interface/EffortJointInterface</hardwareInterface>
+       </joint>
+       <actuator name="${joint}_actuator">
+         <hardwareInterface>hardware_interface/EffortJointInterface</hardwareInterface>
+         <mechanicalReduction>${reduction}</mechanicalReduction>
+       </actuator>
+     </transmission>
+  </xacro:macro>
+  <xacro:macro name="hsrb_velocity_joint_transmission" params="joint reduction">
+      <transmission name="${prefix}_transmission">
+          <type>transmission_interface/SimpleTransmission</type>
+          <joint name="${joint}">
+            <hardwareInterface>hardware_interface/VelocityJointInterface</hardwareInterface>
+          </joint>
+          <actuator name="${joint}_actuator">
+              <hardwareInterface>hardware_interface/VelocityJointInterface</hardwareInterface>
+              <mechanicalReduction>${reduction}</mechanicalReduction>
+          </actuator>
+      </transmission>
+  </xacro:macro>
+  <xacro:macro name="gazebo_link" params="name gravity collide friction">
+    <gazebo reference="${name}">
+      <selfCollide>${collide}</selfCollide>
+      <gravity>${gravity}</gravity>
+      <mu1>${friction}</mu1>
+      <mu2>${friction}</mu2>
+    </gazebo>
+  </xacro:macro>
+  <xacro:macro name="gazebo_link_flat_black" params="name gravity collide friction">
+    <gazebo reference="${name}">
+      <selfCollide>${collide}</selfCollide>
+      <gravity>${gravity}</gravity>
+      <mu1>${friction}</mu1>
+      <mu2>${friction}</mu2>
+      <material value="Gazebo/FlatBlack"/>
+    </gazebo>
+  </xacro:macro>
+  <xacro:macro name="gazebo_link_caster" params="name">
+    <gazebo reference="${name}">
+      <selfCollide>false</selfCollide>
+      <gravity>true</gravity>
+      <mu1>0.1</mu1>
+      <mu2>0.1</mu2>
+      <maxVel>1.0</maxVel>
+      <material value="Gazebo/FlatBlack"/>
+    </gazebo>
+  </xacro:macro>
+  <xacro:macro name="gazebo_link_rubber" params="name">
+    <gazebo reference="${name}">
+      <selfCollide>false</selfCollide>
+      <gravity>true</gravity>
+      <turnGravityOff>false</turnGravityOff>
+      <kp>1000000.0</kp>
+      <kd>10.0</kd>
+      <mu1>1.0</mu1>
+      <mu2>1.0</mu2>
+      <maxVel>1.0</maxVel>
+      <minDepth>0.00</minDepth>
+      <material value="Gazebo/FlatBlack"/>
+    </gazebo>
+  </xacro:macro>
+  <xacro:macro name="gazebo_link_bumper" params="name personal_name robot_type gravity collide friction">
+    <gazebo reference="${name}_link">
+      <selfCollide>${collide}</selfCollide>
+      <gravity>${gravity}</gravity>
+      <mu1>${friction}</mu1>
+      <mu2>${friction}</mu2>
+      <sensor name="${name}_contact" type="contact">
+        <always_on>true</always_on>
+        <update_rate>10</update_rate>
+        <contact>
+          <collision>${name}_link_collision</collision>
+        </contact>
+        <plugin name="hsrb_gazebo_ros_bumper_controller" filename="libhsrb_gazebo_ros_bumper.so">
+          <robotNamespace>${personal_name}/${robot_type}</robotNamespace>
+          <bumperTopicName>${name}_sensor</bumperTopicName>
+          <frameName>${name}_link</frameName>
+        </plugin>
+      </sensor>
+    </gazebo>
+  </xacro:macro>
+  <xacro:macro name="gazebo_joint" params="name">
+    <gazebo reference="${name}">
+      <xacro:if value="$(arg implicit_damping)">
+        <implicitSpringDamper>1</implicitSpringDamper>
+      </xacro:if>
+    </gazebo>
+  </xacro:macro>
+  <xacro:macro name="gazebo_joint_mimic" params="name">
+    <gazebo reference="${name}">
+    </gazebo>
+  </xacro:macro>
 </robot>

File: hsrb_parts_description/urdf/sensors/imu.urdf.xacro (robot description, xacro)
@@ -1,5 +1,38 @@
 <?xml version="1.0" ?>
 <robot xmlns:xacro="http://ros.org/wiki/xacro" name="hsrb">
-    <xacro:include filename="$(find hsrb_parts_description)/urdf/sensors/$(env ROS_DISTRO)/imu.gazebo.xacro"/>
+    <!-- imu sensor gazebo -->
+    <xacro:macro name="imu_gazebo" params="sensor_name frame_name topic_name robot_namespace">
+        <gazebo reference="${frame_name}">
+            <sensor type="imu" name="${sensor_name}">
+                <update_rate>10.0</update_rate>
+	        <plugin name="${sensor_name}_plugin" filename="libgazebo_ros_imu_sensor.so">
+		    <updateRateHZ>50.0</updateRateHZ>
+		    <bodyName>base_link</bodyName>
+                    <topicName>${robot_namespace}/${sensor_name}/data</topicName>
+                    <frameName>${personal_name}/${frame_name}</frameName>
+		    <gaussianNoise>0.0</gaussianNoise>
+		    <xyzOffset>0.0 0.0 0.0</xyzOffset>
+		    <rpyOffset>0.0 -0.0 0.0</rpyOffset>
+		</plugin>
+                <imu>
+                    <noise>
+                        <type>gaussian</type>
+                        <rate>
+                            <mean>0.0</mean>
+                            <stddev>2e-4</stddev>
+                            <bias_mean>0.0000075</bias_mean>
+                            <bias_stddev>0.0000008</bias_stddev>
+                        </rate>
+                        <accel>
+                            <mean>0.0</mean>
+                            <stddev>1.7e-2</stddev>
+                            <bias_mean>0.1</bias_mean>
+                            <bias_stddev>0.001</bias_stddev>
+                        </accel>
+                    </noise>
+                </imu>
+            </sensor>
+        </gazebo>
+    </xacro:macro>
     <!-- imu sensor -->
     <xacro:macro name="imu_sensor" params="prefix parent topic_name robot_namespace *origin">

File: hsrb_parts_description/urdf/sensors/mynteye_imu.urdf.xacro (robot description, xacro)
@@ -1,5 +1,38 @@
 <?xml version="1.0" ?>
 <robot xmlns:xacro="http://ros.org/wiki/xacro" name="hsrb">
-    <xacro:include filename="$(find hsrb_parts_description)/urdf/sensors/$(env ROS_DISTRO)/mynteye_imu.gazebo.xacro"/>
+    <!-- imu sensor gazebo -->
+    <xacro:macro name="mynteye_imu_gazebo" params="sensor_name frame_name topic_name robot_namespace">
+        <gazebo reference="${frame_name}">
+            <sensor type="imu" name="${sensor_name}">
+                <update_rate>10.0</update_rate>
+	        <plugin name="${sensor_name}_plugin" filename="libgazebo_ros_imu_sensor.so">
+		    <updateRateHZ>100.0</updateRateHZ>
+		    <bodyName>base_link</bodyName>
+		    <topicName>${sensor_name}/${topic_name}</topicName>
+		    <frameName>${personal_name}/${frame_name}</frameName>
+		    <gaussianNoise>0.0</gaussianNoise>
+		    <xyzOffset>0.0 0.0 0.0</xyzOffset>
+		    <rpyOffset>0.0 -0.0 0.0</rpyOffset>
+		</plugin>
+                <imu>
+                    <noise>
+                        <type>gaussian</type>
+                        <rate>
+                            <mean>0.0</mean>
+                            <stddev>2e-4</stddev>
+                            <bias_mean>0.0000075</bias_mean>
+                            <bias_stddev>0.0000008</bias_stddev>
+                        </rate>
+                        <accel>
+                            <mean>0.0</mean>
+                            <stddev>1.7e-2</stddev>
+                            <bias_mean>0.1</bias_mean>
+                            <bias_stddev>0.001</bias_stddev>
+                        </accel>
+                    </noise>
+                </imu>
+            </sensor>
+        </gazebo>
+    </xacro:macro>
     <!-- imu sensor -->
     <xacro:macro name="mynteye_imu" params="prefix parent sensor_name topic_name robot_namespace *origin">

File: hsrc_description/urdf/common.xacro (robot description, xacro)
@@ -1,4 +1,112 @@
 <?xml version="1.0"?>
 <robot xmlns:xacro="http://ros.org/wiki/xacro">
-    <xacro:include filename="$(find hsrc_description)/urdf/common/$(env ROS_DISTRO)/common.xacro"/>
+  <xacro:arg name="implicit_damping" default="false" />
+  <xacro:macro name="hsrb_position_joint_transmission" params="joint reduction">
+     <transmission name="${joint}_transmission">
+       <type>transmission_interface/SimpleTransmission</type>
+       <joint name="${joint}">
+         <hardwareInterface>hardware_interface/PositionJointInterface</hardwareInterface>
+       </joint>
+       <actuator name="${joint}_actuator">
+         <hardwareInterface>hardware_interface/PositionJointInterface</hardwareInterface>
+         <mechanicalReduction>${reduction}</mechanicalReduction>
+       </actuator>
+     </transmission>
+  </xacro:macro>
+  <xacro:macro name="hsrb_effort_joint_transmission" params="joint reduction">
+     <transmission name="${joint}_transmission">
+       <type>transmission_interface/SimpleTransmission</type>
+       <joint name="${joint}">
+         <hardwareInterface>hardware_interface/EffortJointInterface</hardwareInterface>
+       </joint>
+       <actuator name="${joint}_actuator">
+         <hardwareInterface>hardware_interface/EffortJointInterface</hardwareInterface>
+         <mechanicalReduction>${reduction}</mechanicalReduction>
+       </actuator>
+     </transmission>
+  </xacro:macro>
+  <xacro:macro name="hsrb_velocity_joint_transmission" params="joint reduction">
+      <transmission name="${prefix}_transmission">
+          <type>transmission_interface/SimpleTransmission</type>
+          <joint name="${joint}">
+            <hardwareInterface>hardware_interface/VelocityJointInterface</hardwareInterface>
+          </joint>
+          <actuator name="${joint}_actuator">
+              <hardwareInterface>hardware_interface/VelocityJointInterface</hardwareInterface>
+              <mechanicalReduction>${reduction}</mechanicalReduction>
+          </actuator>
+      </transmission>
+  </xacro:macro>
+  <xacro:macro name="gazebo_link" params="name gravity collide friction">
+    <gazebo reference="${name}">
+      <selfCollide>${collide}</selfCollide>
+      <gravity>${gravity}</gravity>
+      <mu1>${friction}</mu1>
+      <mu2>${friction}</mu2>
+    </gazebo>
+  </xacro:macro>
+  <xacro:macro name="gazebo_link_flat_black" params="name gravity collide friction">
+    <gazebo reference="${name}">
+      <selfCollide>${collide}</selfCollide>
+      <gravity>${gravity}</gravity>
+      <mu1>${friction}</mu1>
+      <mu2>${friction}</mu2>
+      <material value="Gazebo/FlatBlack"/>
+    </gazebo>
+  </xacro:macro>
+  <xacro:macro name="gazebo_link_caster" params="name">
+    <gazebo reference="${name}">
+      <selfCollide>false</selfCollide>
+      <gravity>true</gravity>
+      <mu1>0.1</mu1>
+      <mu2>0.1</mu2>
+      <maxVel>1.0</maxVel>
+      <material value="Gazebo/FlatBlack"/>
+    </gazebo>
+  </xacro:macro>
+  <xacro:macro name="gazebo_link_rubber" params="name">
+    <gazebo reference="${name}">
+      <selfCollide>false</selfCollide>
+      <gravity>true</gravity>
+      <turnGravityOff>false</turnGravityOff>
+      <kp>1000000.0</kp>
+      <kd>10.0</kd>
+      <mu1>1.0</mu1>
+      <mu2>1.0</mu2>
+      <maxVel>1.0</maxVel>
+      <minDepth>0.00</minDepth>
+      <material value="Gazebo/FlatBlack"/>
+    </gazebo>
+  </xacro:macro>
+  <xacro:macro name="gazebo_link_bumper" params="name personal_name robot_type gravity collide friction">
+    <gazebo reference="${name}_link">
+      <selfCollide>${collide}</selfCollide>
+      <gravity>${gravity}</gravity>
+      <mu1>${friction}</mu1>
+      <mu2>${friction}</mu2>
+      <sensor name="${name}_contact" type="contact">
+        <always_on>true</always_on>
+        <update_rate>10</update_rate>
+        <contact>
+          <collision>${name}_link_collision</collision>
+        </contact>
+        <plugin name="hsrb_gazebo_ros_bumper_controller" filename="libhsrb_gazebo_ros_bumper.so">
+          <robotNamespace>${personal_name}/${robot_type}</robotNamespace>
+          <bumperTopicName>${name}_sensor</bumperTopicName>
+          <frameName>${name}_link</frameName>
+        </plugin>
+      </sensor>
+    </gazebo>
+  </xacro:macro>
+  <xacro:macro name="gazebo_joint" params="name">
+    <gazebo reference="${name}">
+      <xacro:if value="$(arg implicit_damping)">
+        <implicitSpringDamper>1</implicitSpringDamper>
+      </xacro:if>
+    </gazebo>
+  </xacro:macro>
+  <xacro:macro name="gazebo_joint_mimic" params="name">
+    <gazebo reference="${name}">
+    </gazebo>
+  </xacro:macro>
 </robot>
