Commit message: Add support for publishing hand joint state by joint_state_broadcaster at gazebo simulation

File: hsrb_description/urdf/ros2_control.gazebo.xacro (robot description, xacro)
@@ -30,4 +30,11 @@
         </joint>
       </xacro:macro>
+      <xacro:macro name="gazebo_read_only_joint" params="name">
+        <joint name="${name}">
+          <state_interface name="position" />
+          <state_interface name="velocity" />
+          <state_interface name="effort" />
+        </joint>
+      </xacro:macro>
       <xacro:gazebo_position_joint name="head_tilt_joint" />
       <xacro:gazebo_position_joint name="head_pan_joint" />
@@ -40,4 +47,7 @@
       <xacro:gazebo_velocity_joint name="base_r_drive_wheel_joint" />
       <xacro:gazebo_velocity_joint name="base_l_drive_wheel_joint" />
+      <xacro:gazebo_read_only_joint name="hand_motor_joint" />
+      <xacro:gazebo_read_only_joint name="hand_l_spring_proximal_joint" />
+      <xacro:gazebo_read_only_joint name="hand_r_spring_proximal_joint" />
     </ros2_control>
   </xacro:macro>

Commit message: Add pid gain parameters for gazebo simulation

File: hsrb_description/urdf/ros2_control.gazebo.xacro (robot description, xacro)
@@ -42,5 +42,5 @@
         </joint>
       </xacro:macro>
-      <xacro:macro name="gazebo_position_joint" params="name">
+      <xacro:macro name="gazebo_position_joint" params="name p_gain i_gain d_gain">
         <joint name="${name}">
           <command_interface name="position" />
@@ -48,4 +48,8 @@
           <state_interface name="velocity" />
           <state_interface name="effort" />
+          <param name="p_gain">${p_gain}</param>
+          <param name="i_gain">${i_gain}</param>
+          <param name="d_gain">${d_gain}</param>
+          <param name="i_max">200.0</param>
         </joint>
       </xacro:macro>
@@ -57,12 +61,12 @@
         </joint>
       </xacro:macro>
-      <xacro:gazebo_position_joint name="head_tilt_joint" />
-      <xacro:gazebo_position_joint name="head_pan_joint" />
-      <xacro:gazebo_position_joint name="arm_lift_joint" />
-      <xacro:gazebo_position_joint name="arm_flex_joint" />
-      <xacro:gazebo_position_joint name="arm_roll_joint" />
-      <xacro:gazebo_position_joint name="wrist_flex_joint" />
-      <xacro:gazebo_position_joint name="wrist_roll_joint" />
-      <xacro:gazebo_position_joint name="base_roll_joint" />
+      <xacro:gazebo_position_joint name="head_tilt_joint" p_gain="1200.0" i_gain="0.0" d_gain="10.0"/>
+      <xacro:gazebo_position_joint name="head_pan_joint" p_gain="1200.0" i_gain="0.0" d_gain="10.0"/>
+      <xacro:gazebo_position_joint name="arm_lift_joint" p_gain="900.0" i_gain="200.0" d_gain="100.0"/>
+      <xacro:gazebo_position_joint name="arm_flex_joint" p_gain="2000.0" i_gain="10.0" d_gain="20.0"/>
+      <xacro:gazebo_position_joint name="arm_roll_joint" p_gain="1000.0" i_gain="10.0" d_gain="1.0"/>
+      <xacro:gazebo_position_joint name="wrist_flex_joint" p_gain="900.0" i_gain="1.0" d_gain="30.0"/>
+      <xacro:gazebo_position_joint name="wrist_roll_joint" p_gain="900.0" i_gain="1.0" d_gain="10.0"/>
+      <xacro:gazebo_position_joint name="base_roll_joint" p_gain="900.0" i_gain="200.0" d_gain="100.0"/>
       <xacro:gazebo_velocity_joint name="base_r_drive_wheel_joint" />
       <xacro:gazebo_velocity_joint name="base_l_drive_wheel_joint" />

Commit message: Add PID parameter to wheel joint for gazebo ros2 control

File: hsrb_description/urdf/ros2_control.gazebo.xacro (robot description, xacro)
@@ -34,5 +34,5 @@
          <plugin>gazebo_ros2_control/GazeboSystem</plugin>
       </hardware>
-      <xacro:macro name="gazebo_velocity_joint" params="name">
+      <xacro:macro name="gazebo_velocity_joint" params="name p_gain i_gain d_gain">
         <joint name="${name}">
           <command_interface name="velocity" />
@@ -40,4 +40,8 @@
           <state_interface name="velocity" />
           <state_interface name="effort" />
+          <param name="p_gain">${p_gain}</param>
+          <param name="i_gain">${i_gain}</param>
+          <param name="d_gain">${d_gain}</param>
+          <param name="i_max">3.0</param>
         </joint>
       </xacro:macro>
@@ -69,6 +73,6 @@
       <xacro:gazebo_position_joint name="wrist_roll_joint" p_gain="900.0" i_gain="1.0" d_gain="10.0"/>
       <xacro:gazebo_position_joint name="base_roll_joint" p_gain="1000.0" i_gain="1.0" d_gain="10.0"/>
-      <xacro:gazebo_velocity_joint name="base_r_drive_wheel_joint" />
-      <xacro:gazebo_velocity_joint name="base_l_drive_wheel_joint" />
+      <xacro:gazebo_velocity_joint name="base_r_drive_wheel_joint" p_gain="35.0" i_gain="0.5" d_gain="0.0"/>
+      <xacro:gazebo_velocity_joint name="base_l_drive_wheel_joint" p_gain="35.0" i_gain="0.5" d_gain="0.0"/>
       <xacro:gazebo_read_only_joint name="hand_motor_joint" />
       <xacro:gazebo_read_only_joint name="hand_l_spring_proximal_joint" />

File: hsrc_description/urdf/ros2_control.gazebo.xacro (robot description, xacro)
@@ -33,10 +33,14 @@
          <plugin>gazebo_ros2_control/GazeboSystem</plugin>
       </hardware>
-      <xacro:macro name="gazebo_velocity_joint" params="name">
+      <xacro:macro name="gazebo_position_joint" params="name p_gain i_gain d_gain">
         <joint name="${name}">
-          <command_interface name="velocity" />
+          <command_interface name="position" />
           <state_interface name="position" />
           <state_interface name="velocity" />
           <state_interface name="effort" />
+          <param name="p_gain">${p_gain}</param>
+          <param name="i_gain">${i_gain}</param>
+          <param name="d_gain">${d_gain}</param>
+          <param name="i_max">200.0</param>
         </joint>
       </xacro:macro>
@@ -68,6 +72,6 @@
       <xacro:gazebo_position_joint name="wrist_roll_joint" p_gain="900.0" i_gain="0.0" d_gain="0.0"/>
       <xacro:gazebo_position_joint name="base_roll_joint" p_gain="1000.0" i_gain="1.0" d_gain="10.0"/>
-      <xacro:gazebo_velocity_joint name="base_r_drive_wheel_joint" />
-      <xacro:gazebo_velocity_joint name="base_l_drive_wheel_joint" />
+      <xacro:gazebo_velocity_joint name="base_r_drive_wheel_joint" p_gain="35.0" i_gain="0.5" d_gain="0.0"/>
+      <xacro:gazebo_velocity_joint name="base_l_drive_wheel_joint" p_gain="35.0" i_gain="0.5" d_gain="0.0"/>
       <xacro:gazebo_read_only_joint name="hand_motor_joint" />
       <xacro:gazebo_read_only_joint name="hand_l_spring_proximal_joint" />

Commit message: Enable grasp hack plugin

File: hsrb_description/urdf/ros2_control.gazebo.xacro (robot description, xacro)
@@ -28,4 +28,17 @@
           <hand_r_distal_joint p="20.0" d="8.0"/>
         </parameters>
+      </plugin>
+      <plugin name="grasp_hack_plugin" filename="libtmc_gazebo_grasp_hack_hrh_gripper.so">
+        <grasp_check>
+          <attach_steps>1</attach_steps>
+          <detach_steps>2</detach_steps>
+          <min_contact_count>1</min_contact_count>
+          <max_attach_weight>1.2</max_attach_weight>
+        </grasp_check>
+        <gripper_link>hand_r_distal_link</gripper_link>
+        <gripper_link>hand_l_distal_link</gripper_link>
+        <gripper_link>hand_r_spring_proximal_link</gripper_link>
+        <gripper_link>hand_l_spring_proximal_link</gripper_link>
+        <palm_link>wrist_ft_sensor_frame</palm_link>
       </plugin>
     </gazebo>

File: hsrc_description/urdf/ros2_control.gazebo.xacro (robot description, xacro)
@@ -28,4 +28,17 @@
         </parameters>
       </plugin>
+      <plugin name="grasp_hack_plugin" filename="libtmc_gazebo_grasp_hack_hrh_gripper.so">
+        <grasp_check>
+          <attach_steps>1</attach_steps>
+          <detach_steps>2</detach_steps>
+          <min_contact_count>1</min_contact_count>
+          <max_attach_weight>1.2</max_attach_weight>
+        </grasp_check>
+        <gripper_link>hand_r_distal_link</gripper_link>
+        <gripper_link>hand_l_distal_link</gripper_link>
+        <gripper_link>hand_r_spring_proximal_link</gripper_link>
+        <gripper_link>hand_l_spring_proximal_link</gripper_link>
+        <palm_link>wrist_ft_sensor_frame</palm_link>
+      </plugin>
     </gazebo>
     <ros2_control name="GazeboSystem" type="system">
@@ -45,7 +58,7 @@
         </joint>
       </xacro:macro>
-      <xacro:macro name="gazebo_position_joint" params="name p_gain i_gain d_gain">
+      <xacro:macro name="gazebo_velocity_joint" params="name p_gain i_gain d_gain">
         <joint name="${name}">
-          <command_interface name="position" />
+          <command_interface name="velocity" />
           <state_interface name="position" />
           <state_interface name="velocity" />
@@ -54,5 +67,5 @@
           <param name="i_gain">${i_gain}</param>
           <param name="d_gain">${d_gain}</param>
-          <param name="i_max">200.0</param>
+          <param name="i_max">3.0</param>
         </joint>
       </xacro:macro>
