Commit message: Update ros2_control.rviz.xacro

File: hsrb_description/urdf/ros2_control.rviz.xacro (robot description, xacro)
@@ -2,5 +2,5 @@
 <robot xmlns:xacro="http://www.ros.org/wiki/xacro">
   <xacro:macro name="ros2_contorl_rviz">
-    <ros2_control name="hsrb" type="system">
+    <ros2_control name="GenericSystem" type="system">
       <hardware>
         <plugin>fake_components/GenericSystem</plugin>
@@ -8,84 +8,24 @@
         <param name="state_following_offset">0.0</param>
       </hardware>
-      <xacro:macro name="hsrb_joint" params="name min_angle max_angle velocity_limit control_type:=ActiveJoint">
+      <xacro:macro name="rviz_joint" params="name">
         <joint name="${name}">
-          <command_interface name="position">
-            <param name="min">"${min_angle}"</param>
-            <param name="max">"${max_angle}"</param>
-          </command_interface>
-          <command_interface name="velocity">
-            <param name="min">>${-velocity_limit}</param>
-            <param name="max">>${velocity_limit}</param>
-          </command_interface>
+          <command_interface name="velocity"/>
+          <command_interface name="position"/>
           <state_interface name="position"/>
           <state_interface name="velocity"/>
           <state_interface name="effort"/>
-          <param name="control_type">${control_type}</param>
-          <param name="velocity_limit">${velocity_limit}</param>
         </joint>
       </xacro:macro>
-      <xacro:macro name="gripper_active_joint" params="name min_angle max_angle velocity_limit left_spring_joint right_spring_joint">
-        <joint name="${name}">
-          <command_interface name="position">
-            <param name="min">"${min_angle}"</param>
-            <param name="max">"${max_angle}"</param>
-          </command_interface>
-          <state_interface name="position"/>
-          <state_interface name="velocity"/>
-          <state_interface name="effort"/>
-          <param name="control_type">Gripper</param>
-          <param name="velocity_limit">${velocity_limit}</param>
-          <param name="left_spring_joint">${left_spring_joint}</param>
-          <param name="right_spring_joint">${right_spring_joint}</param>
-        </joint>
-      </xacro:macro>
-      <xacro:hsrb_joint name="arm_lift_joint"
-                        min_angle="0.0"
-                        max_angle="0.69"
-                        velocity_limit="1.0"/>
-      <xacro:hsrb_joint name="arm_flex_joint"
-                        min_angle="-2.62"
-                        max_angle="0.0"
-                        velocity_limit="1.0"/>
-      <xacro:hsrb_joint name="arm_roll_joint"
-                        min_angle="-2.09"
-                        max_angle="3.84"
-                        velocity_limit="1.0"/>
-      <xacro:hsrb_joint name="wrist_flex_joint"
-                        min_angle="-1.92"
-                        max_angle="1.22"
-                        velocity_limit="1.0"/>
-      <xacro:hsrb_joint name="wrist_roll_joint"
-                        min_angle="-1.92"
-                        max_angle="3.67"
-                        velocity_limit="1.0"/>
-      <xacro:hsrb_joint name="head_pan_joint"
-                        min_angle="-3.84"
-                        max_angle="1.75"
-                        velocity_limit="1.0"/>
-      <xacro:hsrb_joint name="head_tilt_joint"
-                        min_angle="-1.57"
-                        max_angle="0.52"
-                        velocity_limit="1.0"/>
-      <xacro:gripper_active_joint name="hand_motor_joint"
-                                  min_angle="-0.798"
-                                  max_angle="1.24"
-                                  velocity_limit="1.0"
-                                  left_spring_joint="hand_l_spring_proximal_joint"
-                                  right_spring_joint="hand_r_spring_proximal_joint"/>
-      <xacro:hsrb_joint name="base_l_drive_wheel_joint"
-                        min_angle="-999999"
-                        max_angle="999999"
-                        velocity_limit="20.8"
-                        control_type="Wheel"/>
-      <xacro:hsrb_joint name="base_r_drive_wheel_joint"
-                        min_angle="-999999"
-                        max_angle="999999"
-                        velocity_limit="20.8"
-                        control_type="Wheel"/>
-      <xacro:hsrb_joint name="base_roll_joint"
-                        min_angle="-999999"
-                        max_angle="999999"
-                        velocity_limit="2.5"/>
+      <xacro:rviz_joint name="arm_lift_joint"/>
+      <xacro:rviz_joint name="arm_flex_joint"/>
+      <xacro:rviz_joint name="arm_roll_joint"/>
+      <xacro:rviz_joint name="wrist_flex_joint"/>
+      <xacro:rviz_joint name="wrist_roll_joint"/>
+      <xacro:rviz_joint name="head_pan_joint"/>
+      <xacro:rviz_joint name="head_tilt_joint"/>
+      <xacro:rviz_joint name="hand_motor_joint"/>
+      <xacro:rviz_joint name="base_l_drive_wheel_joint"/>
+      <xacro:rviz_joint name="base_r_drive_wheel_joint"/>
+      <xacro:rviz_joint name="base_roll_joint"/>
     </ros2_control>
   </xacro:macro>

Commit message: add gripper bridge for simulator

File: hsrb_description/urdf/ros2_control.rviz.xacro (robot description, xacro)
@@ -11,9 +11,19 @@
       <xacro:macro name="rviz_joint" params="name">
         <joint name="${name}">
+          <command_interface name="position"/>
           <command_interface name="velocity"/>
-          <command_interface name="position"/>
+          <command_interface name="command_drive_mode"/>
+          <state_interface name="command_drive_mode"/>
+          <state_interface name="command_position"/>
+          <state_interface name="command_velocity"/>
           <state_interface name="position"/>
           <state_interface name="velocity"/>
           <state_interface name="effort"/>
+          <state_interface name="current"/>
+          <state_interface name="temperature"/>
+          <state_interface name="MrPos"/>
+          <state_interface name="AvagoPos"/>
+          <state_interface name="current_drive_mode"/>
+          <state_interface name="error_status"/>
         </joint>
       </xacro:macro>
@@ -29,4 +39,16 @@
       <xacro:rviz_joint name="base_r_drive_wheel_joint"/>
       <xacro:rviz_joint name="base_roll_joint"/>
+      <xacro:rviz_joint name="hand_l_spring_proximal_joint"/>
+      <xacro:rviz_joint name="hand_r_spring_proximal_joint"/>
+    </ros2_control>
+    <ros2_control name="HsrbSIMGripper" type="system">
+      <hardware>
+        <plugin>hsrb_gripper_bridge/HsrbSIMGripperBridge</plugin>
+      </hardware>
+      <xacro:macro name="rviz_joint" params="name">
+        <joint name="${name}">
+        </joint>
+      </xacro:macro>
+      <xacro:rviz_joint name="hand_motor_joint_bridge"/>
     </ros2_control>
   </xacro:macro>

Commit message: rename controller, use joint

File: hsrb_description/urdf/ros2_control.rviz.xacro (robot description, xacro)
@@ -7,5 +7,4 @@
         <param name="fake_sensor_commands">False</param>
         <param name="state_following_offset">0.0</param>
-        <param name="calculate_dynamics">True</param>
       </hardware>
       <xacro:macro name="rviz_joint" params="name">
@@ -31,13 +30,12 @@
       <xacro:rviz_joint name="hand_r_spring_proximal_joint"/>
     </ros2_control>
-    <ros2_control name="ForwardCommandController" type="system">
+    <ros2_control name="HsrbGripperFakeInterface" type="system">
       <hardware>
-        <plugin>forward_command_controller/ForwardCommandController</plugin>
+        <plugin>hsrb_gripper_fake_interface/HsrbGripperFakeInterface</plugin>
+        <!-- effortの閾値 -->
+        <param name="effort_min">0.011</param>
       </hardware>
-      <xacro:macro name="rviz_joint" params="name">
-        <joint name="${name}">
-        </joint>
-      </xacro:macro>
-      <xacro:rviz_joint name="hand_motor_joint"/>
+      <joint name="hand_motor_joint">
+      </joint>
     </ros2_control>
   </xacro:macro>
