Commit message: Remove depends of gazebo_ros

File: hsrb_description/urdf/ros2_control.robot.xacro (robot description, xacro)
@@ -6,5 +6,5 @@
         <plugin>hsrb_robot_hardware/HsrbHW</plugin>
       </hardware>
-      <xacro:macro name="hsrb_joint" params="name min_angle max_angle motor_id reduction drive_mode velocity_limit">
+      <xacro:macro name="hsrb_joint" params="name min_angle max_angle motor_id reduction drive_mode velocity_limit gear_ratio torque_constant control_type:=ActiveJoint">
         <joint name="${name}">
           <command_interface name="position">
@@ -19,12 +19,14 @@
           <state_interface name="velocity"/>
           <state_interface name="effort"/>
-          <param name="control_type">ActiveJoint</param>
+          <param name="control_type">${control_type}</param>
           <param name="motor_id">${motor_id}</param>
           <param name="reduction">${reduction}</param>
           <param name="drive_mode">${drive_mode}</param>
           <param name="velocity_limit">${velocity_limit}</param>
+          <param name="gear_ratio">${gear_ratio}</param>
+          <param name="torque_constant">${torque_constant}</param>
         </joint>
       </xacro:macro>
-      <xacro:macro name="gripper_active_joint" params="name min_angle max_angle motor_id reduction drive_mode velocity_limit left_spring_joint right_spring_joint">
+      <xacro:macro name="gripper_active_joint" params="name min_angle max_angle motor_id reduction drive_mode velocity_limit  gear_ratio torque_constant left_spring_joint right_spring_joint">
         <joint name="${name}">
           <command_interface name="position">
@@ -40,4 +42,6 @@
           <param name="drive_mode">${drive_mode}</param>
           <param name="velocity_limit">${velocity_limit}</param>
+          <param name="gear_ratio">${gear_ratio}</param>
+          <param name="torque_constant">${torque_constant}</param>
           <param name="left_spring_joint">${left_spring_joint}</param>
           <param name="right_spring_joint">${right_spring_joint}</param>
@@ -50,5 +54,7 @@
                         reduction="40.273862263"
                         drive_mode="5"
-                        velocity_limit="1.0"/>
+                        velocity_limit="1.0"
+                        gear_ratio="0.002407705"
+                        torque_constant="0.0174"/>
       <xacro:hsrb_joint name="arm_flex_joint"
                         min_angle="-2.62"
@@ -57,5 +63,7 @@
                         reduction="1.0"
                         drive_mode="5"
-                        velocity_limit="1.0"/>
+                        velocity_limit="1.0"
+                        gear_ratio="0.00128576"
+                        torque_constant="0.0208"/>
       <xacro:hsrb_joint name="arm_roll_joint"
                         min_angle="-2.09"
@@ -64,5 +72,7 @@
                         reduction="1.0"
                         drive_mode="5"
-                        velocity_limit="1.0"/>
+                        velocity_limit="1.0"
+                        gear_ratio="0.003333333"
+                        torque_constant="0.0184"/>
       <xacro:hsrb_joint name="wrist_flex_joint"
                         min_angle="-1.92"
@@ -71,5 +81,7 @@
                         reduction="1.0"
                         drive_mode="5"
-                        velocity_limit="1.0"/>
+                        velocity_limit="1.0"
+                        gear_ratio="0.0035"
+                        torque_constant="0.0184"/>
       <xacro:hsrb_joint name="wrist_roll_joint"
                         min_angle="-1.92"
@@ -78,5 +90,7 @@
                         reduction="-1.0"
                         drive_mode="5"
-                        velocity_limit="1.0"/>
+                        velocity_limit="1.0"
+                        gear_ratio="0.0035"
+                        torque_constant="0.0184"/>
       <xacro:hsrb_joint name="head_pan_joint"
                         min_angle="-3.84"
@@ -85,5 +99,7 @@
                         reduction="1.0"
                         drive_mode="5"
-                        velocity_limit="1.0"/>
+                        velocity_limit="1.0"
+                        gear_ratio="0.01"
+                        torque_constant="0.0184"/>
       <xacro:hsrb_joint name="head_tilt_joint"
                         min_angle="-1.57"
@@ -92,5 +108,7 @@
                         reduction="-1.0"
                         drive_mode="5"
-                        velocity_limit="1.0"/>
+                        velocity_limit="1.0"
+                        gear_ratio="0.0028"
+                        torque_constant="0.0184"/>
       <xacro:gripper_active_joint name="hand_motor_joint"
                                   min_angle="-0.798"
@@ -100,4 +118,6 @@
                                   drive_mode="0"
                                   velocity_limit="1.0"
+                                  gear_ratio="0.005090909"
+                                  torque_constant="0.0184"
                                   left_spring_joint="hand_l_spring_proximal_joint"
                                   right_spring_joint="hand_r_spring_proximal_joint"/>
@@ -108,5 +128,8 @@
                         reduction="1.0"
                         drive_mode="3"
-                        velocity_limit="20.8"/>
+                        velocity_limit="20.8"
+                        gear_ratio="0.006451613"
+                        torque_constant="0.0174"
+                        control_type="Wheel"/>
       <xacro:hsrb_joint name="base_r_drive_wheel_joint"
                         min_angle="-999999"
@@ -115,5 +138,8 @@
                         reduction="1.0"
                         drive_mode="3"
-                        velocity_limit="20.8"/>
+                        velocity_limit="20.8"
+                        gear_ratio="0.006451613"
+                        torque_constant="0.0174"
+                        control_type="Wheel"/>
       <xacro:hsrb_joint name="base_roll_joint"
                         min_angle="-999999"
@@ -122,5 +148,7 @@
                         reduction="-1.0"
                         drive_mode="5"
-                        velocity_limit="2.5"/>
+                        velocity_limit="2.5"
+                        gear_ratio="0.003333333"
+                        torque_constant="0.0368"/>
     </ros2_control>
   </xacro:macro>

Commit message: Add acceleration_limit

File: hsrb_description/urdf/ros2_control.robot.xacro (robot description, xacro)
@@ -6,5 +6,5 @@
         <plugin>hsrb_robot_hardware/HsrbHW</plugin>
       </hardware>
-      <xacro:macro name="hsrb_joint" params="name min_angle max_angle motor_id reduction drive_mode velocity_limit gear_ratio torque_constant control_type:=ActiveJoint">
+      <xacro:macro name="hsrb_joint" params="name min_angle max_angle motor_id reduction drive_mode velocity_limit gear_ratio torque_constant control_type:=ActiveJoint acceleration_limit:=1000.0">
         <joint name="${name}">
           <command_interface name="position">
@@ -24,4 +24,5 @@
           <param name="drive_mode">${drive_mode}</param>
           <param name="velocity_limit">${velocity_limit}</param>
+          <param name="acceleration_limit">${acceleration_limit}</param>
           <param name="gear_ratio">${gear_ratio}</param>
           <param name="torque_constant">${torque_constant}</param>
@@ -42,4 +43,5 @@
           <param name="drive_mode">${drive_mode}</param>
           <param name="velocity_limit">${velocity_limit}</param>
+          <param name="acceleration_limit">1000.0</param>
           <param name="gear_ratio">${gear_ratio}</param>
           <param name="torque_constant">${torque_constant}</param>
@@ -131,5 +133,6 @@
                         gear_ratio="0.006451613"
                         torque_constant="0.0174"
-                        control_type="Wheel"/>
+                        control_type="Wheel"
+                        acceleration_limit="41.7"/>
       <xacro:hsrb_joint name="base_r_drive_wheel_joint"
                         min_angle="-999999"
@@ -141,5 +144,6 @@
                         gear_ratio="0.006451613"
                         torque_constant="0.0174"
-                        control_type="Wheel"/>
+                        control_type="Wheel"
+                        acceleration_limit="41.7"/>
       <xacro:hsrb_joint name="base_roll_joint"
                         min_angle="-999999"
@@ -150,5 +154,6 @@
                         velocity_limit="2.5"
                         gear_ratio="0.003333333"
-                        torque_constant="0.0368"/>
+                        torque_constant="0.0368"
+                        acceleration_limit="5.0"/>
     </ros2_control>
   </xacro:macro>

File: hsrc_description/urdf/ros2_control.robot.xacro (robot description, xacro)
@@ -6,5 +6,5 @@
         <plugin>hsrb_robot_hardware/HsrbHW</plugin>
       </hardware>
-      <xacro:macro name="hsrb_joint" params="name min_angle max_angle motor_id reduction drive_mode velocity_limit gear_ratio torque_constant control_type:=ActiveJoint">
+      <xacro:macro name="hsrb_joint" params="name min_angle max_angle motor_id reduction drive_mode velocity_limit gear_ratio torque_constant control_type:=ActiveJoint acceleration_limit:=1000.0">
         <joint name="${name}">
           <command_interface name="position">
@@ -24,4 +24,5 @@
           <param name="drive_mode">${drive_mode}</param>
           <param name="velocity_limit">${velocity_limit}</param>
+          <param name="acceleration_limit">${acceleration_limit}</param>
           <param name="gear_ratio">${gear_ratio}</param>
           <param name="torque_constant">${torque_constant}</param>
@@ -42,4 +43,5 @@
           <param name="drive_mode">${drive_mode}</param>
           <param name="velocity_limit">${velocity_limit}</param>
+          <param name="acceleration_limit">1000.0</param>
           <param name="gear_ratio">${gear_ratio}</param>
           <param name="torque_constant">${torque_constant}</param>
@@ -131,5 +133,6 @@
                         gear_ratio="0.006451613"
                         torque_constant="0.0174"
-                        control_type="Wheel"/>
+                        control_type="Wheel"
+                        acceleration_limit="41.7"/>
       <xacro:hsrb_joint name="base_r_drive_wheel_joint"
                         min_angle="-999999"
@@ -141,5 +144,6 @@
                         gear_ratio="0.006451613"
                         torque_constant="0.0174"
-                        control_type="Wheel"/>
+                        control_type="Wheel"
+                        acceleration_limit="41.7"/>
       <xacro:hsrb_joint name="base_roll_joint"
                         min_angle="-999999"
@@ -150,5 +154,6 @@
                         velocity_limit="2.5"
                         gear_ratio="0.003333333"
-                        torque_constant="0.0368"/>
+                        torque_constant="0.0368"
+                        acceleration_limit="5.0"/>
     </ros2_control>
     <ros2_control name="hsrb_gpio" type="system">
