Commit message: fix hsrc stereo_camera position

File: hsrc_description/urdf/head_v0/head.urdf.xacro (robot description, xacro)
@@ -67,8 +67,8 @@
         <!-- cameras -->
         <xacro:pointgrey_chameleon prefix="${prefix}_l_stereo" parent="${prefix}_tilt_link" robot_namespace="${robot_name}" baseline="0.00">
-            <origin xyz="0.0312 0.07 0.08" rpy="${-pi/2.0} 0.0 ${-pi/2.0}"/>
+            <origin xyz="0.0262 0.07 0.08" rpy="${-pi/2.0} 0.0 ${-pi/2.0}"/>
         </xacro:pointgrey_chameleon>
         <xacro:pointgrey_chameleon prefix="${prefix}_r_stereo" parent="${prefix}_tilt_link" robot_namespace="${robot_name}" baseline="0.14">
-            <origin xyz="0.0312 -0.07 0.08" rpy="${-pi/2.0} 0.0 ${-pi/2.0}"/>
+            <origin xyz="0.0262 -0.07 0.08" rpy="${-pi/2.0} 0.0 ${-pi/2.0}"/>
         </xacro:pointgrey_chameleon>
         <xacro:asus_xtion prefix="${prefix}" parent="${prefix}_tilt_link" robot_namespace="${robot_name}" sensor_name="rgbd_sensor">

Commit message: delete hsrc's head_dummy.stl

File: hsrc_description/urdf/head_v0/head.urdf.xacro (robot description, xacro)
@@ -59,9 +59,4 @@
                 </geometry>
             </collision>
-            <collision>
-                <geometry>
-                    <mesh filename="package://hsrc_description/meshes/head_v0/head_dummy.stl" />
-                </geometry>
-            </collision>
         </link>
         <!-- cameras -->
