Commit message: Separate bumper from base

File: hsrb_description/urdf/base_v2/base.gazebo.xacro (robot description, xacro)
@@ -10,4 +10,6 @@
         <gazebo_link name="${prefix}_range_sensor_link" gravity="true" collide="false" friction="0.9"/>
         <gazebo_link name="${prefix}_imu_frame" gravity="true" collide="false" friction="0.9"/>
+        <gazebo_link_bumper name="${prefix}_f_bumper" gravity="true" collide="false" friction="0.9"/>
+        <gazebo_link_bumper name="${prefix}_b_bumper" gravity="true" collide="false" friction="0.9"/>
     </xacro:macro>
 </robot>

File: hsrb_description/urdf/base_v2/base.urdf.xacro (robot description, xacro)
@@ -188,4 +188,54 @@
             <origin xyz="0.0005 0.1296 0.181" rpy="0.0 0.0 0.0" />
         </xacro:imu_sensor>
+        <!-- base front bumper -->
+        <joint name="${prefix}_f_bumper_joint" type="revolute">
+            <limit effort="0" velocity="0" lower="0" upper="0"/>
+            <parent link="${prefix}_link" />
+            <child link="${prefix}_f_bumper_link" />
+        </joint>
+        <link name="${prefix}_f_bumper_link">
+            <inertial>
+                <origin xyz="0.0 0.0 0.0" />
+                <mass value="0.50"/>
+                <inertia
+                    ixx="0.07671000"  ixy="-0.01005000"  ixz="0.00174900"
+                    iyy="0.09057000" iyz="0.00154900" izz="0.14500000" />
+            </inertial>
+            <visual>
+                <geometry>
+                    <mesh filename="package://hsrb_description/meshes/base_v2/front_bumper.dae" />
+                </geometry>
+            </visual>
+            <collision>
+                <geometry>
+                    <mesh filename="package://hsrb_description/meshes/base_v2/front_bumper.stl" />
+                </geometry>
+            </collision>
+        </link>
+       <!-- base rear bumper -->
+        <joint name="${prefix}_b_bumper_joint" type="revolute">
+            <parent link="${prefix}_link" />
+            <child link="${prefix}_b_bumper_link" />
+            <limit effort="0" velocity="0" lower="0" upper="0"/>
+        </joint>
+        <link name="${prefix}_b_bumper_link">
+            <inertial>
+                <origin xyz="0.0 0.0 0.0" />
+                <mass value="0.50"/>
+                <inertia
+                    ixx="0.07671000"  ixy="-0.01005000"  ixz="0.00174900"
+                    iyy="0.09057000" iyz="0.00154900" izz="0.14500000" />
+            </inertial>
+            <visual>
+                <geometry>
+                    <mesh filename="package://hsrb_description/meshes/base_v2/rear_bumper.dae" />
+                </geometry>
+            </visual>
+            <collision>
+                <geometry>
+                    <mesh filename="package://hsrb_description/meshes/base_v2/rear_bumper.stl" />
+                </geometry>
+            </collision>
+        </link>
         <xacro:hsrb_base_gazebo prefix="${prefix}"/>
         <xacro:hsrb_base_transmission prefix="${prefix}"/>

File: hsrb_description/urdf/common/kinetic/common.xacro (robot description, xacro)
@@ -79,4 +79,24 @@
     </gazebo>
   </xacro:macro>
+  <xacro:macro name="gazebo_link_bumper" params="name gravity collide friction">
+    <gazebo reference="${name}_link">
+      <selfCollide>${collide}</selfCollide>
+      <gravity>${gravity}</gravity>
+      <mu1>${friction}</mu1>
+      <mu2>${friction}</mu2>
+      <sensor name="${name}_contact" type="contact">
+        <always_on>true</always_on>
+        <update_rate>10</update_rate>
+        <contact>
+          <collision>${name}_link_collision</collision>
+        </contact>
+        <plugin name="hsrb_gazebo_ros_bumper_controller" filename="libhsrb_bumper.so">
+          <robotNamespace>hsrb</robotNamespace>
+          <bumperTopicName>${name}_sensor</bumperTopicName>
+          <frameName>${name}_link</frameName>
+        </plugin>
+      </sensor>
+    </gazebo>
+  </xacro:macro>
   <xacro:macro name="gazebo_joint" params="name">
     <gazebo reference="${name}">

File: hsrc_description/urdf/base_v0/base.urdf.xacro (robot description, xacro)
@@ -185,4 +185,54 @@
             <origin xyz="0.167 0.0 0.1904" rpy="0.0 0.0 0.0" />
         </xacro:hokuyo_laser>
+        <!-- base front bumper -->
+        <joint name="${prefix}_f_bumper_joint" type="revolute">
+            <limit effort="0" velocity="0" lower="0" upper="0"/>
+            <parent link="${prefix}_link" />
+            <child link="${prefix}_f_bumper_link" />
+        </joint>
+        <link name="${prefix}_f_bumper_link">
+            <inertial>
+                <origin xyz="0.0 0.0 0.0" />
+                <mass value="0.50"/>
+                <inertia
+                    ixx="0.07671000"  ixy="-0.01005000"  ixz="0.00174900"
+                    iyy="0.09057000" iyz="0.00154900" izz="0.14500000" />
+            </inertial>
+            <visual>
+                <geometry>
+                    <mesh filename="package://hsrc_description/meshes/base_v0/front_bumper.dae" />
+                </geometry>
+            </visual>
+            <collision>
+                <geometry>
+                    <mesh filename="package://hsrc_description/meshes/base_v0/front_bumper.stl" />
+                </geometry>
+            </collision>
+        </link>
+       <!-- base rear bumper -->
+        <joint name="${prefix}_b_bumper_joint" type="revolute">
+            <parent link="${prefix}_link" />
+            <child link="${prefix}_b_bumper_link" />
+            <limit effort="0" velocity="0" lower="0" upper="0"/>
+        </joint>
+        <link name="${prefix}_b_bumper_link">
+            <inertial>
+                <origin xyz="0.0 0.0 0.0" />
+                <mass value="0.50"/>
+                <inertia
+                    ixx="0.07671000"  ixy="-0.01005000"  ixz="0.00174900"
+                    iyy="0.09057000" iyz="0.00154900" izz="0.14500000" />
+            </inertial>
+            <visual>
+                <geometry>
+                    <mesh filename="package://hsrc_description/meshes/base_v0/rear_bumper.dae" />
+                </geometry>
+            </visual>
+            <collision>
+                <geometry>
+                    <mesh filename="package://hsrc_description/meshes/base_v0/rear_bumper.stl" />
+                </geometry>
+            </collision>
+        </link>
         <xacro:imu_sensor prefix="${prefix}" robot_namespace="${robot_namespace}" parent="${prefix}_link">
             <origin xyz="0.003 -0.08594 0.203" rpy="0.0 0.0 0.0" />

Commit message: Use valid bumper plugin

File: hsrb_description/urdf/base_v2/base.gazebo.xacro (robot description, xacro)
@@ -1,5 +1,5 @@
 <?xml version="1.0"?>
 <robot xmlns:xacro="http://ros.org/wiki/xacro">
-    <xacro:macro name="hsrb_base_gazebo" params="personal_name prefix robot_name">
+    <xacro:macro name="hsrb_base_gazebo" params="prefix robot_namespace">
         <xacro:gazebo_link name="${prefix}_link" gravity="true" collide="false" friction="0.9"/>
         <xacro:gazebo_link name="${prefix}_roll_link" gravity="true" collide="false" friction="0.9"/>
@@ -10,6 +10,6 @@
         <xacro:gazebo_link name="${prefix}_range_sensor_link" gravity="true" collide="false" friction="0.9"/>
         <xacro:gazebo_link name="${prefix}_imu_frame" gravity="true" collide="false" friction="0.9"/>
-        <xacro:gazebo_link_bumper name="${prefix}_f_bumper" personal_name="${personal_name}" robot_name="${robot_name}" gravity="true" collide="false" friction="0.9"/>
-        <xacro:gazebo_link_bumper name="${prefix}_b_bumper" personal_name="${personal_name}" robot_name="${robot_name}" gravity="true" collide="false" friction="0.9"/>
+        <xacro:gazebo_link_bumper name="${prefix}_f_bumper" robot_namespace="${robot_namespace}" gravity="true" collide="false" friction="0.9"/>
+        <xacro:gazebo_link_bumper name="${prefix}_b_bumper" robot_namespace="${robot_namespace}" gravity="true" collide="false" friction="0.9"/>
     </xacro:macro>
 </robot>

File: hsrb_description/urdf/base_v2/base.urdf.xacro (robot description, xacro)
@@ -227,5 +227,5 @@
                 rpy="0.0 0.0 ${pi}" />
         </xacro:hsrb_bumper>
-        <xacro:hsrb_base_gazebo personal_name="${personal_name}" prefix="${prefix}" robot_name="${robot_name}"/>
+        <xacro:hsrb_base_gazebo prefix="${prefix}" robot_namespace="${robot_namespace}"/>
     </xacro:macro>
 </robot>

File: hsrb_description/urdf/common.xacro (robot description, xacro)
@@ -43,5 +43,5 @@
     </gazebo>
   </xacro:macro>
-  <xacro:macro name="gazebo_link_bumper" params="name personal_name robot_name gravity collide friction">
+  <xacro:macro name="gazebo_link_bumper" params="name robot_namespace gravity collide friction">
     <gazebo reference="${name}_link">
       <selfCollide>${collide}</selfCollide>
@@ -55,8 +55,9 @@
           <collision>${name}_link_collision</collision>
         </contact>
-        <plugin name="hsrb_gazebo_ros_bumper_controller" filename="libhsrb_gazebo_ros_bumper.so">
-          <robotNamespace>${personal_name}/${robot_name}</robotNamespace>
-          <bumperTopicName>${name}_sensor</bumperTopicName>
-          <frameName>${name}_link</frameName>
+        <plugin name="${name}_bumper_controller" filename="libtmc_gazebo_ros_bumper.so">
+          <ros>
+            <namespace>${robot_namespace}</namespace>
+            <remapping>bumper_states:=${name}_sensor</remapping>
+          </ros>
         </plugin>
       </sensor>

File: hsrc_description/urdf/base_v0/base.urdf.xacro (robot description, xacro)
@@ -224,5 +224,5 @@
                 rpy="0.0 0.0 ${pi}" />
         </xacro:hsrb_bumper>
-        <xacro:hsrb_base_gazebo personal_name="${personal_name}" prefix="${prefix}" robot_name="${robot_name}"/>
+        <xacro:hsrb_base_gazebo prefix="${prefix}" robot_namespace="${robot_namespace}"/>
     </xacro:macro>
 </robot>

File: hsrc_description/urdf/common.xacro (robot description, xacro)
@@ -79,5 +79,5 @@
     </gazebo>
   </xacro:macro>
-  <xacro:macro name="gazebo_link_bumper" params="name personal_name robot_name gravity collide friction">
+  <xacro:macro name="gazebo_link_bumper" params="name robot_namespace gravity collide friction">
     <gazebo reference="${name}_link">
       <selfCollide>${collide}</selfCollide>
@@ -91,8 +91,9 @@
           <collision>${name}_link_collision</collision>
         </contact>
-        <plugin name="hsrb_gazebo_ros_bumper_controller" filename="libhsrb_gazebo_ros_bumper.so">
-          <robotNamespace>${personal_name}/${robot_name}</robotNamespace>
-          <bumperTopicName>${name}_sensor</bumperTopicName>
-          <frameName>${name}_link</frameName>
+        <plugin name="${name}_bumper_controller" filename="libtmc_gazebo_ros_bumper.so">
+          <ros>
+            <namespace>${robot_namespace}</namespace>
+            <remapping>bumper_states:=${name}_sensor</remapping>
+          </ros>
         </plugin>
       </sensor>
