Commit message: delete some material items in base_v2 and head_v2

File: hsrb_description/urdf/base_v2/base.urdf.xacro (robot description, xacro)
@@ -121,5 +121,4 @@
                     <mesh filename="package://hsrb_description/meshes/base_v2/base_light.dae" />
                 </geometry>
-                <material name="body_main" />
             </visual>
             <visual>
@@ -127,5 +126,4 @@
                     <mesh filename="package://hsrb_description/meshes/base_v2/body_light.dae" />
                 </geometry>
-                <material name="body_main" />
             </visual>
             <visual>
@@ -133,5 +131,4 @@
                     <mesh filename="package://hsrb_description/meshes/base_v2/torso_base.dae" />
                 </geometry>
-                <material name="body_sub" />
             </visual>
             <collision>

File: hsrb_description/urdf/head_v2/head.urdf.xacro (robot description, xacro)
@@ -27,5 +27,4 @@
                     <mesh filename="package://hsrb_description/meshes/head_v1/head_pan.dae" />
                 </geometry>
-                <material name="body_main" />
             </visual>
             <collision>
@@ -54,5 +53,4 @@
                     <mesh filename="package://hsrb_description/meshes/head_v1/head_upper.dae" />
                 </geometry>
-                <material name="body_sub" />
             </visual>
             <visual>
@@ -60,5 +58,4 @@
                     <mesh filename="package://hsrb_description/meshes/head_v1/head_tilt.dae" />
                 </geometry>
-                <material name="body_main" />
             </visual>
             <visual>
@@ -66,5 +63,4 @@
                     <mesh filename="package://hsrb_description/meshes/head_v1/tablet_base.dae" />
                 </geometry>
-                <material name="body_sub" />
             </visual>
             <collision>

Commit message: Change gazebo IMU plugin

File: hsrb_description/urdf/base_v2/base.urdf.xacro (robot description, xacro)
@@ -185,5 +185,5 @@
         </xacro:hokuyo_laser>
         <xacro:imu_sensor prefix="${prefix}" robot_namespace="${robot_namespace}" parent="${prefix}_link">
-            <origin xyz="0.0005 0.1296 0.181" rpy="${pi} 0.0 0.0" />
+            <origin xyz="0.0005 0.1296 0.181" rpy="0.0 0.0 0.0" />
         </xacro:imu_sensor>
         <xacro:hsrb_base_gazebo prefix="${prefix}"/>

File: hsrb_description/urdf/sensors/imu.gazebo.xacro (robot description, xacro)
@@ -25,13 +25,18 @@
         </gazebo>
         <gazebo>
-            <!-- IMU Plugin is a model plugin. Then it should be atached to HSR-B model. -->
-            <plugin name="${sensor_name}_plugin" filename="libgazebo_ros_imu.so">
-                <imuName>${sensor_name}</imuName>
-                <topicName>${sensor_name}/data</topicName>
-                <serviceName>${sensor_name}/calibrate</serviceName>
-                <frameName>${frame_name}</frameName>
-                <bodyName>base_link</bodyName>
-                <robotNamespace>${robot_namespace}</robotNamespace>
-            </plugin>
+	    <!-- IMU Plugin is a model plugin. Then it should be atached to HSR-B model. -->
+	    <plugin name="${sensor_name}_plugin" filename="libhector_gazebo_ros_imu.so">
+		<robotNamespace>${robot_namespace}</robotNamespace>
+		<updateRate>50.0</updateRate>
+		<bodyName>base_link</bodyName>
+		<topicName>${sensor_name}/data</topicName>
+		<serviceName>${sensor_name}/calibrate</serviceName>
+		<accelDrift>0.000 0.000 0.000</accelDrift>
+		<accelGaussianNoise>0.000 0.000 0.000</accelGaussianNoise>
+		<rateDrift>0.000 0.000 0.000 </rateDrift>
+		<rateGaussianNoise>0.000 0.000 0.000 </rateGaussianNoise>
+		<headingDrift>0.000</headingDrift>
+		<headingGaussianNoise>0.000</headingGaussianNoise>
+	    </plugin>
         </gazebo>
     </xacro:macro>

Commit message: add dummy weight

File: hsrb_description/urdf/base_v2/base.urdf.xacro (robot description, xacro)
@@ -105,5 +105,11 @@
     <!-- base -->
     <xacro:macro name="hsrb_base" params="prefix robot_namespace">
-        <link name="base_footprint"/>
+        <link name="base_footprint">
+            <inertial>
+                <origin xyz="0 0 0"/>
+                <mass value="0.01"/>
+                <inertia ixx="0.001" ixy="0" ixz="0" iyy="0.001" iyz="0" izz="0.001"/>
+            </inertial>
+        </link>
         <joint name="${prefix}_footprint_joint" type="fixed">
             <parent link="base_footprint" />

File: hsrb_description/urdf/hand_v0/hand.urdf.xacro (robot description, xacro)
@@ -17,8 +17,8 @@
         <link name="${name}">
             <inertial>
-                <mass value="0.001"/>
-                <inertia
-                    ixx="0.00015" ixy="0.0" ixz="0.0"
-                    iyy="0.00015" iyz="0.0" izz="0.00015"/>
+                <mass value="0.01"/>
+                <inertia
+                    ixx="0.0015" ixy="0.0" ixz="0.0"
+                    iyy="0.0015" iyz="0.0" izz="0.0015"/>
             </inertial>
         </link>
@@ -127,5 +127,5 @@
             <parent link="${prefix}_${suffix}_mimic_distal_link" />
             <child link="${prefix}_${suffix}_distal_link" />
-            <mimic joint="${prefix}_motor_joint" multiplier="-1.0" offset="${-distal_joint_angle_offset}"/>
+	    <mimic joint="${prefix}_motor_joint" multiplier="-1.0" offset="${-distal_joint_angle_offset}"/>
             <dynamics damping="0.0001"/>
         </joint>
@@ -194,8 +194,8 @@
         <link name="${prefix}_${suffix}_finger_vacuum_frame">
             <inertial>
-                <mass value="0.001"/>
-                <inertia
-                    ixx="0.00015" ixy="0.0" ixz="0.0"
-                    iyy="0.00015" iyz="0.0" izz="0.00015"/>
+                <mass value="0.01"/>
+                <inertia
+                    ixx="0.0015" ixy="0.0" ixz="0.0"
+                    iyy="0.0015" iyz="0.0" izz="0.0015"/>
             </inertial>
             <visual>

File: hsrb_parts_description/urdf/sensors/hokuyo_laser.urdf.xacro (robot description, xacro)
@@ -20,4 +20,9 @@
                 </geometry>
             </collision>
+            <inertial>
+                <origin xyz="0 0 0"/>
+                <mass value="0.01"/>
+                <inertia ixx="0.001" ixy="0" ixz="0" iyy="0.001" iyz="0" izz="0.001"/>
+            </inertial>
         </link>
         <xacro:hokuyo_laser_gazebo

File: hsrb_parts_description/urdf/sensors/imu.urdf.xacro (robot description, xacro)
@@ -9,5 +9,11 @@
             <child link="${prefix}_imu_frame" />
         </joint>
-        <link name="${prefix}_imu_frame"/>
+        <link name="${prefix}_imu_frame">
+            <inertial>
+                <origin xyz="0 0 0"/>
+                <mass value="0.01"/>
+                <inertia ixx="0.001" ixy="0" ixz="0" iyy="0.001" iyz="0" izz="0.001"/>
+            </inertial>
+        </link>
         <xacro:imu_gazebo
             sensor_name="${prefix}_imu"

File: hsrb_parts_description/urdf/sensors/minebea_ft_sensor.urdf.xacro (robot description, xacro)
@@ -18,5 +18,5 @@
         <xacro:minebea_ft_sensor_gazebo
             robot_namespace="${robot_namespace}"
-            joint_name="${prefix}_ft_sensor_frame_joint" ros_topic="${prefix}_wrench/raw" />
+            joint_name="${prefix}_ft_sensor_frame_joint" ros_topic="${prefix}_wrench" />
     </xacro:macro>
 </robot>

File: hsrb_parts_description/urdf/sensors/pointgrey_chameleon.urdf.xacro (robot description, xacro)
@@ -15,4 +15,9 @@
                 </geometry>
             </visual>
+            <inertial>
+                <origin xyz="0 0 0"/>
+                <mass value="0.01"/>
+                <inertia ixx="0.001" ixy="0" ixz="0" iyy="0.001" iyz="0" izz="0.001"/>
+            </inertial>
         </link>
         <joint name="${prefix}_camera_gazebo_frame_joint" type="fixed">
@@ -21,5 +26,11 @@
             <child link="${prefix}_camera_gazebo_frame" />
         </joint>
-        <link name="${prefix}_camera_gazebo_frame"></link>
+        <link name="${prefix}_camera_gazebo_frame">
+            <inertial>
+                <origin xyz="0 0 0"/>
+                <mass value="0.01"/>
+                <inertia ixx="0.001" ixy="0" ixz="0" iyy="0.001" iyz="0" izz="0.001"/>
+            </inertial>
+        </link>
         <xacro:pointgrey_chameleon_gazebo
             sensor_name="${prefix}_camera"

File: hsrb_parts_description/urdf/sensors/wide_camera.urdf.xacro (robot description, xacro)
@@ -9,5 +9,11 @@
             <child link="${prefix}_camera_frame" />
         </joint>
-        <link name="${prefix}_camera_frame"></link>
+        <link name="${prefix}_camera_frame">
+            <inertial>
+                <origin xyz="0 0 0"/>
+                <mass value="0.01"/>
+                <inertia ixx="0.001" ixy="0" ixz="0" iyy="0.001" iyz="0" izz="0.001"/>
+            </inertial>
+        </link>
         <joint name="${prefix}_camera_gazebo_frame_joint" type="fixed">
             <origin xyz="0 0 0" rpy="${rpy}"/>
@@ -15,5 +21,11 @@
             <child link="${prefix}_camera_gazebo_frame" />
         </joint>
-        <link name="${prefix}_camera_gazebo_frame"></link>
+        <link name="${prefix}_camera_gazebo_frame">
+            <inertial>
+                <origin xyz="0 0 0"/>
+                <mass value="0.01"/>
+                <inertia ixx="0.001" ixy="0" ixz="0" iyy="0.001" iyz="0" izz="0.001"/>
+            </inertial>
+        </link>
         <xacro:wide_camera_gazebo
             robot_namespace="${robot_namespace}"

Commit message: Update model files

File: hsrb_description/urdf/base_v2/base.urdf.xacro (robot description, xacro)
@@ -106,9 +106,4 @@
     <xacro:macro name="hsrb_base" params="prefix robot_namespace">
         <link name="base_footprint">
-            <inertial>
-                <origin xyz="0 0 0"/>
-                <mass value="0.01"/>
-                <inertia ixx="0.001" ixy="0" ixz="0" iyy="0.001" iyz="0" izz="0.001"/>
-            </inertial>
         </link>
         <joint name="${prefix}_footprint_joint" type="fixed">

File: hsrc_description/urdf/base_v0/base.urdf.xacro (robot description, xacro)
@@ -106,9 +106,4 @@
     <xacro:macro name="hsrb_base" params="prefix robot_namespace">
         <link name="base_footprint">
-            <inertial>
-                <origin xyz="0 0 0"/>
-                <mass value="0.01"/>
-                <inertia ixx="0.001" ixy="0" ixz="0" iyy="0.001" iyz="0" izz="0.001"/>
-            </inertial>
         </link>
         <joint name="${prefix}_footprint_joint" type="fixed">

File: hsrc_description/urdf/hand_v0/hand.urdf.xacro (robot description, xacro)
@@ -188,5 +188,5 @@
         <xacro:hsrb_gripper_dummy_link name="${prefix}_${suffix}_finger_tip_frame" />
         <joint name="${prefix}_${suffix}_finger_vacuum_frame_joint" type="fixed">
-            <origin xyz="0.0075 -0.010 0.0362" rpy="${pi*50/180.0} 0.0 0.0" />
+            <origin xyz="0.0065 -0.00953 0.035577" rpy="${pi*40/180.0} 0.0 0.0" />
             <parent link="${prefix}_${suffix}_distal_link" />
             <child link="${prefix}_${suffix}_finger_vacuum_frame" />

File: hsrc_description/urdf/head_v0/head.urdf.xacro (robot description, xacro)
@@ -73,5 +73,5 @@
         </xacro:pointgrey_chameleon>
         <xacro:asus_xtion prefix="${prefix}" parent="${prefix}_tilt_link" robot_namespace="${robot_name}" sensor_name="rgbd_sensor">
-            <origin xyz="-0.076822 0.022 0.248" rpy="${-pi/2.0} 0.0 ${-pi/2.0}"/>
+            <origin xyz="-0.0786 0.022 0.248" rpy="${-pi/2.0} 0.0 ${-pi/2.0}"/>
         </xacro:asus_xtion>
         <xacro:hsrb_head_gazebo prefix="${prefix}"/>

Commit message: Fix bumper weight

File: hsrb_description/urdf/base_v2/base.urdf.xacro (robot description, xacro)
@@ -103,4 +103,32 @@
         </link>
     </xacro:macro>
+    <!-- bumper -->
+    <xacro:macro name="hsrb_bumper" params="prefix suffix parent *origin">
+        <joint name="${prefix}_${suffix}_bumper_joint" type="revolute">
+            <xacro:insert_block name="origin" />
+            <parent link="${parent}" />
+            <child link="${prefix}_${suffix}_bumper_link" />
+            <limit effort="0" velocity="0" lower="0" upper="0"/>
+        </joint>
+        <link name="${prefix}_${suffix}_bumper_link">
+            <inertial>
+                <origin xyz="0.0 0.0 0.0" />
+                <mass value="0.06"/>
+                <inertia
+                    ixx="0.001437"  ixy="0.0"  ixz="0.0"
+                    iyy="0.001437" iyz="0.0" izz="0.002875" />
+            </inertial>
+            <visual>
+                <geometry>
+                    <mesh filename="package://hsrb_description/meshes/base_v2/bumper.dae" />
+                </geometry>
+            </visual>
+            <collision>
+                <geometry>
+                    <mesh filename="package://hsrb_description/meshes/base_v2/bumper.stl" />
+                </geometry>
+            </collision>
+        </link>
+    </xacro:macro>
     <!-- base -->
     <xacro:macro name="hsrb_base" params="prefix robot_namespace">
@@ -188,54 +216,15 @@
             <origin xyz="0.0005 0.1296 0.181" rpy="0.0 0.0 0.0" />
         </xacro:imu_sensor>
-        <!-- base front bumper -->
-        <joint name="${prefix}_f_bumper_joint" type="revolute">
-            <limit effort="0" velocity="0" lower="0" upper="0"/>
-            <parent link="${prefix}_link" />
-            <child link="${prefix}_f_bumper_link" />
-        </joint>
-        <link name="${prefix}_f_bumper_link">
-            <inertial>
-                <origin xyz="0.0 0.0 0.0" />
-                <mass value="0.50"/>
-                <inertia
-                    ixx="0.07671000"  ixy="-0.01005000"  ixz="0.00174900"
-                    iyy="0.09057000" iyz="0.00154900" izz="0.14500000" />
-            </inertial>
-            <visual>
-                <geometry>
-                    <mesh filename="package://hsrb_description/meshes/base_v2/front_bumper.dae" />
-                </geometry>
-            </visual>
-            <collision>
-                <geometry>
-                    <mesh filename="package://hsrb_description/meshes/base_v2/front_bumper.stl" />
-                </geometry>
-            </collision>
-        </link>
-       <!-- base rear bumper -->
-        <joint name="${prefix}_b_bumper_joint" type="revolute">
-            <parent link="${prefix}_link" />
-            <child link="${prefix}_b_bumper_link" />
-            <limit effort="0" velocity="0" lower="0" upper="0"/>
-        </joint>
-        <link name="${prefix}_b_bumper_link">
-            <inertial>
-                <origin xyz="0.0 0.0 0.0" />
-                <mass value="0.50"/>
-                <inertia
-                    ixx="0.07671000"  ixy="-0.01005000"  ixz="0.00174900"
-                    iyy="0.09057000" iyz="0.00154900" izz="0.14500000" />
-            </inertial>
-            <visual>
-                <geometry>
-                    <mesh filename="package://hsrb_description/meshes/base_v2/rear_bumper.dae" />
-                </geometry>
-            </visual>
-            <collision>
-                <geometry>
-                    <mesh filename="package://hsrb_description/meshes/base_v2/rear_bumper.stl" />
-                </geometry>
-            </collision>
-        </link>
+        <!-- bumper -->
+        <xacro:hsrb_bumper prefix="${prefix}" suffix="f" parent="${prefix}_link">
+            <origin
+                xyz="0.0 0.0 0.0"
+                rpy="0.0 0.0 0.0" />
+        </xacro:hsrb_bumper>
+        <xacro:hsrb_bumper prefix="${prefix}" suffix="b" parent="${prefix}_link">
+            <origin
+                xyz="0.0 0.0013 0.0"
+                rpy="0.0 0.0 ${pi}" />
+        </xacro:hsrb_bumper>
         <xacro:hsrb_base_gazebo prefix="${prefix}"/>
         <xacro:hsrb_base_transmission prefix="${prefix}"/>

File: hsrc_description/urdf/base_v0/base.urdf.xacro (robot description, xacro)
@@ -103,4 +103,32 @@
         </link>
     </xacro:macro>
+    <!-- bumper -->
+    <xacro:macro name="hsrb_bumper" params="prefix suffix parent *origin">
+        <joint name="${prefix}_${suffix}_bumper_joint" type="revolute">
+            <xacro:insert_block name="origin" />
+            <parent link="${parent}" />
+            <child link="${prefix}_${suffix}_bumper_link" />
+            <limit effort="0" velocity="0" lower="0" upper="0"/>
+        </joint>
+        <link name="${prefix}_${suffix}_bumper_link">
+            <inertial>
+                <origin xyz="0.0 0.0 0.0" />
+                <mass value="0.06"/>
+                <inertia
+                    ixx="0.001437"  ixy="0.0"  ixz="0.0"
+                    iyy="0.001437" iyz="0.0" izz="0.002875" />
+            </inertial>
+            <visual>
+                <geometry>
+                    <mesh filename="package://hsrc_description/meshes/base_v0/bumper.dae" />
+                </geometry>
+            </visual>
+            <collision>
+                <geometry>
+                    <mesh filename="package://hsrc_description/meshes/base_v0/bumper.stl" />
+                </geometry>
+            </collision>
+        </link>
+    </xacro:macro>
     <!-- base -->
     <xacro:macro name="hsrb_base" params="prefix robot_namespace">
@@ -185,54 +213,15 @@
             <origin xyz="0.167 0.0 0.1904" rpy="0.0 0.0 0.0" />
         </xacro:hokuyo_laser>
-        <!-- base front bumper -->
-        <joint name="${prefix}_f_bumper_joint" type="revolute">
-            <limit effort="0" velocity="0" lower="0" upper="0"/>
-            <parent link="${prefix}_link" />
-            <child link="${prefix}_f_bumper_link" />
-        </joint>
-        <link name="${prefix}_f_bumper_link">
-            <inertial>
-                <origin xyz="0.0 0.0 0.0" />
-                <mass value="0.50"/>
-                <inertia
-                    ixx="0.07671000"  ixy="-0.01005000"  ixz="0.00174900"
-                    iyy="0.09057000" iyz="0.00154900" izz="0.14500000" />
-            </inertial>
-            <visual>
-                <geometry>
-                    <mesh filename="package://hsrc_description/meshes/base_v0/front_bumper.dae" />
-                </geometry>
-            </visual>
-            <collision>
-                <geometry>
-                    <mesh filename="package://hsrc_description/meshes/base_v0/front_bumper.stl" />
-                </geometry>
-            </collision>
-        </link>
-       <!-- base rear bumper -->
-        <joint name="${prefix}_b_bumper_joint" type="revolute">
-            <parent link="${prefix}_link" />
-            <child link="${prefix}_b_bumper_link" />
-            <limit effort="0" velocity="0" lower="0" upper="0"/>
-        </joint>
-        <link name="${prefix}_b_bumper_link">
-            <inertial>
-                <origin xyz="0.0 0.0 0.0" />
-                <mass value="0.50"/>
-                <inertia
-                    ixx="0.07671000"  ixy="-0.01005000"  ixz="0.00174900"
-                    iyy="0.09057000" iyz="0.00154900" izz="0.14500000" />
-            </inertial>
-            <visual>
-                <geometry>
-                    <mesh filename="package://hsrc_description/meshes/base_v0/rear_bumper.dae" />
-                </geometry>
-            </visual>
-            <collision>
-                <geometry>
-                    <mesh filename="package://hsrc_description/meshes/base_v0/rear_bumper.stl" />
-                </geometry>
-            </collision>
-        </link>
+        <!-- bumper -->
+        <xacro:hsrb_bumper prefix="${prefix}" suffix="f" parent="${prefix}_link">
+            <origin
+                xyz="0.0 0.0 0.0"
+                rpy="0.0 0.0 0.0" />
+        </xacro:hsrb_bumper>
+        <xacro:hsrb_bumper prefix="${prefix}" suffix="b" parent="${prefix}_link">
+            <origin
+                xyz="0.0 0.0 0.0"
+                rpy="0.0 0.0 ${pi}" />
+        </xacro:hsrb_bumper>
         <xacro:imu_sensor prefix="${prefix}" robot_namespace="${robot_namespace}" parent="${prefix}_link">
             <origin xyz="0.003 -0.08594 0.203" rpy="0.0 0.0 0.0" />

Commit message: Change wheel max effort

File: hsrb_description/urdf/base_v2/base.urdf.xacro (robot description, xacro)
@@ -12,5 +12,5 @@
     <xacro:property name="passive_wheel_offset_x" value="0.1495" />
     <xacro:property name="passive_wheel_offset_y" value="0.055" />
-    <xacro:property name="drive_wheel_max_effort" value="11.067" />
+    <xacro:property name="drive_wheel_max_effort" value="28.0" />
     <xacro:property name="drive_wheel_max_velocity" value="20.8" />
     <xacro:property name="roll_joint_max_effort" value="34.46" />

File: hsrc_description/urdf/base_v0/base.urdf.xacro (robot description, xacro)
@@ -12,5 +12,5 @@
     <xacro:property name="passive_wheel_offset_x" value="0.1665" />
     <xacro:property name="passive_wheel_offset_y" value="0.055" />
-    <xacro:property name="drive_wheel_max_effort" value="11.067" />
+    <xacro:property name="drive_wheel_max_effort" value="28.0" />
     <xacro:property name="drive_wheel_max_velocity" value="20.8" />
     <xacro:property name="roll_joint_max_effort" value="34.46" />
