Commit message: [Mod] Change from “file” to “package”

File: hsrc_parts_description/urdf/sensors/intel_d405.urdf.xacro (robot description, xacro)
@@ -68,5 +68,5 @@
         <origin xyz="${d405_zero_depth_to_glass + d405_glass_to_front} ${-d405_cam_depth_py} 0" rpy="${M_PI/2} 0 ${M_PI/2}"/>
         <geometry>
-	        <mesh filename="file://$(find hsrc_parts_description)/meshes/sensors/d405.stl" scale="0.001 0.001 0.001" />
+	        <mesh filename="package://hsrc_parts_description/meshes/sensors/d405.stl" scale="0.001 0.001 0.001" />
         </geometry>
         <material name="aluminum"/>
