Commit message: [Fix] bug fix

File: hsrc_ex_description/urdf/arm_v0/arm.urdf.xacro (robot description, xacro)
@@ -42,5 +42,5 @@
                 <mass value="1.339295"/>
                 <origin xyz="0.000632 0.006404 0.118529"/>
-                <inertia ixx="7.528" ixy="-0.000020284207" ixz="-0.000022947194"
+                <inertia ixx="0.007528" ixy="-0.000020284207" ixz="-0.000022947194"
                     iyy="0.007102" iyz="-0.000091796075" izz="0.001552"/>
             </inertial>

File: hsrc_ex_description/urdf/base_v0/base.urdf.xacro (robot description, xacro)
@@ -125,6 +125,6 @@
                 <mass value="0.06"/>
                 <inertia
-                    ixx="0.001437"  ixy="0.0"  ixz="0.0"
-                    iyy="0.001437" iyz="0.0" izz="0.002875" />
+                    ixx="0.001537"  ixy="0.0"  ixz="0.0"
+                    iyy="0.001537" iyz="0.0" izz="0.002875" />
             </inertial>
             <visual>

File: hsrc_ex_description/urdf/hand_v0/hand.urdf.xacro (robot description, xacro)
@@ -22,6 +22,6 @@
                 <mass value="0.01"/>
                 <inertia
-                    ixx="0.0" ixy="0.0" ixz="0.0"
-                    iyy="0.0" iyz="0.0" izz="0.0"/>
+                    ixx="0.001" ixy="0.0" ixz="0.0"
+                    iyy="0.001" iyz="0.0" izz="0.001"/>
             </inertial>
         </link>
@@ -148,6 +148,6 @@
                 <origin xyz="0.021418 0.00248 0.022688"/>
                 <inertia
-                    ixx="0.0" ixy="0.0" ixz="0.0"
-                    iyy="0.0" iyz="0.0" izz="0.0"/>
+                    ixx="0.001" ixy="0.0" ixz="0.0"
+                    iyy="0.001" iyz="0.0" izz="0.001"/>
             </inertial>
             <visual>
@@ -157,4 +157,8 @@
             </visual>
             <collision>
+                <origin xyz="0.0205 -0.0075 0.04" rpy="0.0 0.0 0.0" />
+                <geometry>
+                    <box size="0.032 0.015 0.05"/>
+                </geometry>
                 <geometry>
                     <mesh filename="package://hsrc_ex_description/meshes/hand_v0/l_proximal.stl" />
@@ -171,6 +175,6 @@
                 <origin xyz="0.011116 0.005679 0.017532"/>
                 <inertia
-                    ixx="0.0" ixy="0.0" ixz="0.0"
-                    iyy="0.0" iyz="0.0" izz="0.0"/>
+                    ixx="0.001" ixy="0.0" ixz="0.0"
+                    iyy="0.001" iyz="0.0" izz="0.001"/>
             </inertial>
             <visual>
@@ -180,7 +184,7 @@
             </visual>
             <collision>
-                <geometry>
+                <!-- <geometry>
                     <mesh filename="package://hsrc_ex_description/meshes/hand_v0/l_distal.stl" />
-                </geometry>
+                </geometry> -->
             </collision>
         </link>
@@ -202,6 +206,6 @@
                 <mass value="0.001"/>
                 <inertia
-                    ixx="0.0" ixy="0.0" ixz="0.0"
-                    iyy="0.0" iyz="0.0" izz="0.0"/>
+                    ixx="0.001" ixy="0.0" ixz="0.0"
+                    iyy="0.001" iyz="0.0" izz="0.001"/>
             </inertial>
             <visual>
@@ -225,6 +229,6 @@
                 <origin xyz="0.013203 0.002096 0.023311"/>
                 <inertia
-                    ixx="0.0" ixy="0.0" ixz="0.0"
-                    iyy="0.0" iyz="0.0" izz="0.0"/>
+                    ixx="0.001" ixy="0.0" ixz="0.0"
+                    iyy="0.001" iyz="0.0" izz="0.001"/>
             </inertial>
             <visual>
@@ -248,6 +252,6 @@
                 <origin xyz="0.014256 -0.008321 0.015591"/>
                 <inertia
-                    ixx="0.0" ixy="0.0" ixz="0.0"
-                    iyy="0.0" iyz="0.0" izz="0.0"/>
+                    ixx="0.001" ixy="0.0" ixz="0.0"
+                    iyy="0.001" iyz="0.0" izz="0.001"/>
             </inertial>
             <visual>
