Commit message: [Mod] Modify the hand camera orientation, Color Change

File: hsrc_ex_description/urdf/head_v0/head.urdf.xacro (robot description, xacro)
@@ -71,5 +71,5 @@
         </xacro:asus_xtion> -->
         <xacro:gemini336l parent="${prefix}_tilt_link" robot_namespace="${personal_name}" sensor_name="head_rgbd_sensor">
-            <origin xyz="-0.09542 0.0 0.23299" rpy="-0.01742 0.05987 0.01117"/>
+            <origin xyz="-0.09542 0.0 0.23299" rpy="0.0 0.0 0.0"/>
         </xacro:gemini336l>
         <xacro:hsrb_head_gazebo prefix="${prefix}"/>

File: hsrc_parts_description/urdf/sensors/gemini_336l.urdf.xacro (robot description, xacro)
@@ -29,5 +29,5 @@
                 </geometry>
                 <material name="">
-                <color rgba="0.1 0.1 0.1 1.0" />
+                <color rgba="0.0 0.0 0.0 1.0" />
                 </material>
             </visual>
