Commit message: [Mod] update

File: hsrc_ex_description/robots/hsrc1s.urdf.xacro (robot description, xacro)
@@ -16,4 +16,5 @@
     <xacro:include filename="$(find hsrc_ex_description)/urdf/hand_v0/hand.urdf.xacro" />
     <xacro:arg name="gazebo_sim" default="False"/>
+    <xacro:arg name="ignition_gazebo_sim" default="False"/>
     <xacro:arg name="rviz_sim" default="False"/>
     <xacro:arg name="personal_name" default=""/>
@@ -41,5 +42,5 @@
     </xacro:hsrb_hand>
     <!-- Import ros2_control description -->
-    <xacro:if value="${not $(arg gazebo_sim) and not $(arg ignition_gazebo_sim) and not $(arg rviz_sim)}">
+    <xacro:if value="${'false' == $(arg gazebo_sim) and 'false' == $(arg ignition_gazebo_sim) and 'false' == $(arg rviz_sim)}">
       <xacro:include filename="$(find hsrc_ex_description)/urdf/ros2_control.robot.xacro" />
       <xacro:ros2_contorl_robot/>

File: hsrc_ex_description/urdf/head_v0/head.urdf.xacro (robot description, xacro)
@@ -3,5 +3,5 @@
     <xacro:include filename="$(find hsrc_ex_description)/urdf/head_v0/head.gazebo.xacro"/>
     <!-- <xacro:include filename="$(find hsrb_parts_description)/urdf/sensors/asus_xtion.urdf.xacro"/> -->
-    <xacro:include filename="$(find hsrc_parts_description)/urdf/sensors/Gemini336L.urdf.xacro"/>
+    <xacro:include filename="$(find hsrc_parts_description)/urdf/sensors/gemini_336l.urdf.xacro"/>
     <xacro:include filename="$(find hsrb_parts_description)/urdf/sensors/pointgrey_chameleon.urdf.xacro"/>
     <xacro:include filename="$(find hsrb_parts_description)/urdf/sensors/wide_camera.urdf.xacro"/>
@@ -71,5 +71,5 @@
         </xacro:asus_xtion> -->
         <xacro:gemini336l parent="${prefix}_tilt_link" robot_namespace="${personal_name}/${robot_name}" sensor_name="head_rgbd_sensor">
-            <origin xyz="-0.09542 0.06168 0.23299" rpy="-0.01742 0.05987 0.01117"/>
+            <origin xyz="-0.09542 0.0 0.23299" rpy="-0.01742 0.05987 0.01117"/>
         </xacro:gemini336l>
         <xacro:hsrb_head_gazebo prefix="${prefix}"/>

File: hsrc_ex_description/urdf/ros2_control.robot.xacro (robot description, xacro)
@@ -157,5 +157,5 @@
                         acceleration_limit="5.0"/>
     </ros2_control>
-    <!-- <ros2_control name="hsrb_gpio" type="system">
+    <ros2_control name="hsrb_gpio" type="system">
       <hardware>
         <plugin>hsrb_cgos_driver/HsrbCgosHw</plugin>
@@ -171,5 +171,5 @@
         <param name="direction">out</param>
       </gpio>
-    </ros2_control> -->
+    </ros2_control>
   </xacro:macro>
 </robot>

File: hsrc_parts_description/urdf/sensors/intel_d405.urdf.xacro (robot description, xacro)
@@ -23,4 +23,6 @@
   <xacro:include filename="$(find hsrc_parts_description)/urdf/sensors/realsense/_materials.urdf.xacro" />
   <xacro:include filename="$(find hsrc_parts_description)/urdf/sensors/realsense/_usb_plug.urdf.xacro" />
+  <xacro:include filename="$(find hsrc_parts_description)/urdf/sensors/intel_d405.urdf.gazebo.xacro"/>
+  <xacro:arg name="ignition_gazebo_sim" default="false" />
   <xacro:macro name="d405" params="parent robot_namespace sensor_name *origin use_nominal_extrinsics:=false">
     <xacro:arg name="add_plug" default="false" />
@@ -143,4 +145,18 @@
       </xacro:usb_plug>
     </xacro:if>
+    <xacro:if value="$(arg ignition_gazebo_sim)">
+      <xacro:intel_realsense_d405_gazebo_ignition
+        robot_namespace="${robot_namespace}"
+        sensor_name="${sensor_name}"
+        parent_frame="${sensor_name}_color_frame"
+        topic_frame_id="${sensor_name}_color_optical_frame" />
+    </xacro:if>
+    <xacro:unless value="$(arg ignition_gazebo_sim)">
+      <xacro:intel_realsense_d405_gazebo
+        robot_namespace="${robot_namespace}"
+        sensor_name="${sensor_name}"
+        parent_frame="${sensor_name}_color_frame"
+        topic_frame_id="${sensor_name}_color_optical_frame" />
+    </xacro:unless>
   </xacro:macro>
 </robot>

Commit message: [Mod] Adjust the head position offset

File: hsrc_ex_description/robots/hsrc1s.urdf.xacro (robot description, xacro)
@@ -30,5 +30,5 @@
     </xacro:hsrb_torso>
     <xacro:hsrb_head prefix="head" parent="torso_lift_link">
-        <origin xyz="0.0 0.0 0.0" rpy="0.0 0.0 0.0"/>
+        <origin xyz="-0.04 0.0 0.0" rpy="0.0 0.0 0.0"/>
     </xacro:hsrb_head>
     <xacro:hsrb_arm prefix="arm" parent="base_link">
