Commit message: [Mod] bug fix

File: hsrc_ex_description/urdf/hand_v0/hand.urdf.xacro (robot description, xacro)
@@ -80,5 +80,5 @@
             <origin xyz="0.026 0.0 0.0034" rpy="0.0 0.0 0.0"/>
         </xacro:wide_camera> -->
-        <xacro:d405 parent="${prefix}_palm_link" robot_namespace="${personal_name}/${robot_name}" sensor_name="${prefix}_camera">
+        <xacro:d405 parent="${prefix}_palm_link" robot_namespace="${personal_name}/${robot_name}" sensor_name="hand_camera">
             <!-- <origin xyz="0.06280 -0.00789 -0.00690" rpy="0.03170 -1.55148 0.03736"/> -->
             <origin xyz="0.05123 -0.00880 0.00109" rpy="-0.01478 -1.60225 -0.00722"/>

File: hsrc_parts_description/urdf/sensors/gemini_336l.urdf.gazebo.xacro (robot description, xacro)
@@ -8,5 +8,5 @@
     <xacro:property name="Gemini336LImageHeight" value="480"/>
     <xacro:property name="Gemini336LMinDistance" value="0.17"/>
-    <xacro:property name="Gemini336LMaxDistance" value="0.20"/>
+    <xacro:property name="Gemini336LMaxDistance" value="20.0"/>
     <xacro:property name="Gemini336LFrameRate" value="30"/>
     <xacro:property name="Gemini336LHorizontalFov" value="1.5708"/>
@@ -40,5 +40,5 @@
                     <cy>0.0</cy>
                     <ros>
-                        <namespace>${robot_namespace}</namespace>
+                        <!-- <namespace>${robot_namespace}</namespace> -->
                         <remapping>${sensor_name}/image_raw:=${sensor_name}/color/image_rect_color</remapping>
                         <remapping>${sensor_name}/camera_info:=${sensor_name}/color/camera_info</remapping>
@@ -70,5 +70,6 @@
                 </camera>
                 <gz_frame_id>${topic_frame_id}</gz_frame_id>
-                <topic>${robot_namespace}/${sensor_name}/color/image_image</topic>
+                <topic>${sensor_name}/color/image_raw</topic>
+                <!-- <topic>${robot_namespace}/${sensor_name}/color/image_raw</topic> -->
             </sensor>
             <sensor type="depth_camera" name="${sensor_name}_camera_depth">
@@ -90,5 +91,6 @@
                 </camera>
                 <gz_frame_id>${topic_frame_id}</gz_frame_id>
-                <topic>${robot_namespace}/${sensor_name}/depth/image_raw</topic>
+                <topic>${sensor_name}/depth/image_raw</topic>
+                <!-- <topic>${robot_namespace}/${sensor_name}/depth/image_raw</topic> -->
             </sensor>
         </gazebo>

File: hsrc_parts_description/urdf/sensors/intel_d405.urdf.gazebo.xacro (robot description, xacro)
@@ -40,5 +40,5 @@
                     <cy>0.0</cy>
                     <ros>
-                        <namespace>${robot_namespace}</namespace>
+                        <!-- <namespace>${robot_namespace}</namespace> -->
                         <remapping>${sensor_name}/image_raw:=${sensor_name}/color/image_rect_raw</remapping>
                         <remapping>${sensor_name}/camera_info:=${sensor_name}/color/camera_info</remapping>
@@ -70,5 +70,6 @@
                 </camera>
                 <gz_frame_id>${topic_frame_id}</gz_frame_id>
-                <topic>${robot_namespace}/${sensor_name}/color/image_rect_raw</topic>
+                <!-- <topic>${robot_namespace}/${sensor_name}/color/image_rect_raw</topic> -->
+                <topic>${sensor_name}/color/image_rect_raw</topic>
             </sensor>
             <sensor type="depth_camera" name="${sensor_name}_camera_depth">
@@ -90,5 +91,6 @@
                 </camera>
                 <gz_frame_id>${topic_frame_id}</gz_frame_id>
-                <topic>${robot_namespace}/${sensor_name}/depth/image_rect_raw</topic>
+                <topic>${sensor_name}/depth/image_rect_raw</topic>
+                <!-- <topic>${robot_namespace}/${sensor_name}/depth/image_rect_raw</topic> -->
             </sensor>
         </gazebo>

File: hsrc_parts_description/urdf/sensors/intel_d405.urdf.xacro (robot description, xacro)
@@ -19,5 +19,5 @@
 aluminum peripherial evaluation case.
 -->
-<robot name="hsrc" xmlns:xacro="http://ros.org/wiki/xacro">
+<robot name="d405" xmlns:xacro="http://ros.org/wiki/xacro">
   <!-- Includes -->
   <xacro:include filename="$(find hsrc_parts_description)/urdf/sensors/realsense/_materials.urdf.xacro" />

Commit message: [fix] bug fix

File: hsrc_ex_description/urdf/hand_v0/hand.urdf.xacro (robot description, xacro)
@@ -157,11 +157,11 @@
             </visual>
             <collision>
-                <origin xyz="0.0205 -0.0075 0.04" rpy="0.0 0.0 0.0" />
-                <geometry>
-                    <box size="0.032 0.015 0.05"/>
-                </geometry>
-                <geometry>
+                <origin xyz="0.0205 -0.0075 0.035" rpy="0.0 0.0 0.0" />
+                <geometry>
+                    <box size="0.032 0.015 0.050"/>
+                </geometry>
+                <!-- <geometry>
                     <mesh filename="package://hsrc_ex_description/meshes/hand_v0/l_proximal.stl" />
-                </geometry>
+                </geometry> -->
             </collision>
         </link>
@@ -184,7 +184,7 @@
             </visual>
             <collision>
-                <!-- <geometry>
+                <geometry>
                     <mesh filename="package://hsrc_ex_description/meshes/hand_v0/l_distal.stl" />
-                </geometry> -->
+                </geometry>
             </collision>
         </link>
@@ -238,7 +238,11 @@
             </visual>
             <collision>
-                <geometry>
+                <origin xyz="0.0205 0.0075 0.035" rpy="0.0 0.0 0.0" />
+                <geometry>
+                    <box size="0.032 0.015 0.050"/>
+                </geometry>
+                <!-- <geometry>
                     <mesh filename="package://hsrc_ex_description/meshes/hand_v0/r_proximal.stl" />
-                </geometry>
+                </geometry> -->
             </collision>
         </link>

File: hsrc_parts_description/urdf/sensors/intel_d405.urdf.xacro (robot description, xacro)
@@ -65,6 +65,7 @@
     <link name="${sensor_name}_link">
       <visual>
+        <origin xyz="0 0 0" rpy="${M_PI/2} 0 ${M_PI/2}"/>
         <!-- the mesh origin is at front plate in between the two infrared camera axes -->
-        <origin xyz="${d405_zero_depth_to_glass + d405_glass_to_front} ${-d405_cam_depth_py} 0" rpy="${M_PI/2} 0 ${M_PI/2}"/>
+        <!-- <origin xyz="${d405_zero_depth_to_glass + d405_glass_to_front} ${-d405_cam_depth_py} 0" rpy="${M_PI/2} 0 ${M_PI/2}"/> -->
         <geometry>
 	        <mesh filename="package://hsrc_parts_description/meshes/sensors/d405.stl" scale="0.001 0.001 0.001" />
@@ -73,5 +74,5 @@
       </visual>
       <collision>
-        <origin xyz="${d405_zero_depth_to_glass-d405_cam_depth/2} ${-d405_cam_depth_py} 0" rpy="0 0 0"/>
+        <origin xyz="${-d405_cam_depth/2} 0 0" rpy="0 0 0"/>
         <geometry>
           <box size="${d405_cam_depth} ${d405_cam_width} ${d405_cam_height}"/>

Commit message: [Mod] update

File: hsrc_ex_description/urdf/hand_v0/hand.urdf.xacro (robot description, xacro)
@@ -82,5 +82,6 @@
         <xacro:d405 parent="${prefix}_palm_link" robot_namespace="${personal_name}" sensor_name="hand_camera" use_nominal_extrinsics="true">
             <!-- <origin xyz="0.06280 -0.00789 -0.00690" rpy="0.03170 -1.55148 0.03736"/> -->
-            <origin xyz="0.05123 -0.00880 0.00109" rpy="-0.01478 -1.60225 -0.00722"/>
+            <!-- <origin xyz="0.05123 -0.00880 0.00109" rpy="-0.01478 -1.60225 -0.00722"/> -->
+            <origin xyz="0.03846 0.00629 -0.0469" rpy="0.0311676 -0.9649463 3.087223"/>
         </xacro:d405>
         <xacro:hsrb_hand_gazebo prefix="${prefix}"/>

Commit message: Correction due to change to HSRC-EX hand camera

File: hsrc_ex_description/urdf/hand_v0/hand.urdf.xacro (robot description, xacro)
@@ -83,5 +83,6 @@
             <!-- <origin xyz="0.06280 -0.00789 -0.00690" rpy="0.03170 -1.55148 0.03736"/> -->
             <!-- <origin xyz="0.05123 -0.00880 0.00109" rpy="-0.01478 -1.60225 -0.00722"/> -->
-            <origin xyz="0.03846 0.00629 -0.0469" rpy="0.0311676 -0.9649463 3.087223"/>
+            <origin xyz="0.03846 0.01529 -0.0469" rpy="0.0311676 -0.9649463 3.087223"/>
+            <!-- <origin xyz="0.03846 0.00629 -0.0469" rpy="0.0311676 -0.9649463 3.087223"/> -->
         </xacro:d405>
         <xacro:hsrb_hand_gazebo prefix="${prefix}"/>
