Commit message: Port hsrc_description to ROS2

File: hsrc_description/robots/hsrc1s.urdf.xacro (robot description, xacro)
@@ -15,4 +15,6 @@
     <xacro:include filename="$(find hsrc_description)/urdf/wrist_v0/wrist.urdf.xacro" />
     <xacro:include filename="$(find hsrc_description)/urdf/hand_v0/hand.urdf.xacro" />
+    <xacro:arg name="gazebo_sim" default="False"/>
+    <xacro:arg name="rviz_sim" default="False"/>
     <xacro:arg name="personal_name" default=""/>
     <xacro:arg name="ground_truth_xyz_offset" default="0.0\ 0.0\ 0.0"/>
@@ -38,18 +40,12 @@
         <origin xyz="0.0 0.0 0.155" rpy="0.0 0.0 ${pi}"/>
     </xacro:hsrb_hand>
-    <gazebo>
-        <plugin name="${robot_name}_ros_control" filename="lib${robot_name}_gazebo_ros_control.so">
-            <robotNamespace>${personal_name}/${robot_name}</robotNamespace>
-            <legacyModeNS>false</legacyModeNS>
-        </plugin>
-        <plugin name="${robot_name}_p3d_ground_truth" filename="lib${robot_name}_gazebo_ros_p3d.so">
-            <robotNamespace>${personal_name}/${robot_name}</robotNamespace>
-            <bodyName>base_footprint</bodyName>
-            <topicName>odom_ground_truth</topicName>
-            <frameName>map</frameName>
-            <updateRate>30</updateRate>
-	    <xyzOffset>$(arg ground_truth_xyz_offset)</xyzOffset>
-	    <rpyOffset>$(arg ground_truth_rpy_offset)</rpyOffset>
-        </plugin>
-    </gazebo>
+    <!-- Import ros2_control description -->
+    <xacro:if value="${not $(arg gazebo_sim) and not $(arg rviz_sim)}">
+      <xacro:include filename="$(find hsrc_description)/urdf/ros2_control.robot.xacro" />
+      <xacro:ros2_contorl_robot/>
+    </xacro:if>
+    <xacro:if value="$(arg gazebo_sim)">
+      <xacro:include filename="$(find hsrb_description)/urdf/ros2_control.gazebo.xacro" />
+      <xacro:ros2_contorl_gazebo/>
+    </xacro:if>
 </robot>

File: hsrc_description/urdf/arm_v0/arm.urdf.xacro (robot description, xacro)
@@ -1,5 +1,4 @@
 <?xml version="1.0"?>
 <robot name="arm" xmlns:xacro="http://ros.org/wiki/xacro">
-    <xacro:include filename="$(find hsrc_description)/urdf/arm_v0/arm.transmission.xacro"/>
     <xacro:include filename="$(find hsrc_description)/urdf/arm_v0/arm.gazebo.xacro"/>
     <!-- arm -->
@@ -84,5 +83,4 @@
         </link>
         <xacro:hsrb_arm_gazebo prefix="${prefix}"/>
-        <xacro:hsrb_arm_transmission prefix="${prefix}"/>
     </xacro:macro>
 </robot>

File: hsrc_description/urdf/base_v0/base.urdf.xacro (robot description, xacro)
@@ -1,5 +1,4 @@
 <?xml version="1.0"?>
 <robot name="base" xmlns:xacro="http://ros.org/wiki/xacro">
-    <xacro:include filename="$(find hsrc_description)/urdf/base_v0/base.transmission.xacro"/>
     <xacro:include filename="$(find hsrc_description)/urdf/base_v0/base.gazebo.xacro"/>
     <xacro:include filename="$(find hsrb_parts_description)/urdf/sensors/hokuyo_laser.urdf.xacro"/>
@@ -141,5 +140,5 @@
         <link name="${prefix}_link">
             <inertial>
-                <mass value="50.00"/>  <!-- use dummy weight to stabilize gazebo move base (real value: 11.017971)-->
+                <mass value="50.00"/>  <!-- use dummy weight to stabilize gazebo move base (real value is 11.017971)-->
                 <origin xyz="-0.025978 -0.005498 0.17633"/>
                 <inertia ixx="0.3742" ixy="0.000434172172" ixz="0.03088"
@@ -225,9 +224,5 @@
                 rpy="0.0 0.0 ${pi}" />
         </xacro:hsrb_bumper>
-        <xacro:imu_sensor prefix="${prefix}" robot_namespace="${robot_namespace}" parent="${prefix}_link" topic_name="data">
-            <origin xyz="0.003 -0.08594 0.203" rpy="0.0 0.0 0.0" />
-        </xacro:imu_sensor>
         <xacro:hsrb_base_gazebo personal_name="${personal_name}" prefix="${prefix}" robot_name="${robot_name}"/>
-        <xacro:hsrb_base_transmission prefix="${prefix}"/>
     </xacro:macro>
 </robot>

File: hsrc_description/urdf/hand_v0/hand.gazebo.xacro (robot description, xacro)
@@ -26,28 +26,27 @@
         <xacro:gazebo_joint name="${prefix}_r_distal_joint"/>
         <gazebo>
-            <plugin name="hsrb_hrh_gripper_plugin" filename="libtmc_gazebo_hrh_gripper.so">
-                <sensitiveness>0.05</sensitiveness>
-                <update_rate>1000.0</update_rate>
-                <max_torque>8.0</max_torque>
-                <!-- 5[deg] -->
-                <error_tolerance>0.0872</error_tolerance>
-                <stall_timeout>2.0</stall_timeout>
-                <robot_namespace>${personal_name}/${robot_name}</robot_namespace>
-            </plugin>
-            <plugin name="hsrb_grasp_hack_plugin" filename="libhsrb_grasp_hack.so">
-                <grasp_check>
-                    <attach_steps>1</attach_steps>
-                    <detach_steps>2</detach_steps>
-                    <min_contact_count>1</min_contact_count>
-                    <max_attach_weight>1.2</max_attach_weight>
-                </grasp_check>
-                <gripper_link>${prefix}_r_distal_link</gripper_link>
-                <gripper_link>${prefix}_l_distal_link</gripper_link>
-                <gripper_link>${prefix}_r_spring_proximal_link</gripper_link>
-                <gripper_link>${prefix}_l_spring_proximal_link</gripper_link>
-		<!-- hand_palm_link is merged with wrist_ft_sensor_frame by fixed joint  -->
-		<palm_link>wrist_ft_sensor_frame</palm_link>
-                <robot_namespace>${personal_name}/${robot_name}</robot_namespace>
-            </plugin>
+          <plugin name="hsrb_hrh_gripper_plugin" filename="libtmc_gazebo_ros_hrh_gripper.so">
+            <sensitiveness>0.05</sensitiveness>
+            <update_rate>1000.0</update_rate>
+            <max_torque>8.0</max_torque>
+            <error_tolerance>0.0872</error_tolerance>
+            <stall_timeout>2.0</stall_timeout>
+            <robot_namespace>${personal_name}/${robot_name}</robot_namespace>
+          </plugin>
+          <!-- <plugin name="hsrb_grasp_hack_plugin" filename="libhsrb_grasp_hack.so">
+            <grasp_check>
+              <attach_steps>1</attach_steps>
+              <detach_steps>2</detach_steps>
+              <min_contact_count>1</min_contact_count>
+              <max_attach_weight>1.2</max_attach_weight>
+            </grasp_check>
+            <gripper_link>${prefix}_r_distal_link</gripper_link>
+            <gripper_link>${prefix}_l_distal_link</gripper_link>
+            <gripper_link>${prefix}_r_spring_proximal_link</gripper_link>
+            <gripper_link>${prefix}_l_spring_proximal_link</gripper_link> -->
+	    <!-- hand_palm_link is merged with wrist_ft_sensor_frame by fixed joint  -->
+            <!-- <palm_link>wrist_ft_sensor_frame</palm_link>
+            <robot_namespace>${personal_name}/${robot_name}</robot_namespace>
+          </plugin> -->
         </gazebo>
     </xacro:macro>

File: hsrc_description/urdf/hand_v0/hand.urdf.xacro (robot description, xacro)
@@ -1,5 +1,4 @@
 <?xml version="1.0"?>
 <robot name="hand" xmlns:xacro="http://ros.org/wiki/xacro">
-    <xacro:include filename="$(find hsrc_description)/urdf/hand_v0/hand.transmission.xacro"/>
     <xacro:include filename="$(find hsrc_description)/urdf/hand_v0/hand.gazebo.xacro"/>
     <xacro:include filename="$(find hsrb_parts_description)/urdf/sensors/wide_camera.urdf.xacro"/>
@@ -78,5 +77,4 @@
         </xacro:wide_camera>
         <xacro:hsrb_hand_gazebo prefix="${prefix}"/>
-        <xacro:hsrb_hand_transmission prefix="${prefix}"/>
     </xacro:macro>
     <!-- gripper finger proximal base -->

File: hsrc_description/urdf/head_v0/head.urdf.xacro (robot description, xacro)
@@ -1,5 +1,4 @@
 <?xml version="1.0"?>
 <robot name="head" xmlns:xacro="http://ros.org/wiki/xacro">
-    <xacro:include filename="$(find hsrc_description)/urdf/head_v0/head.transmission.xacro"/>
     <xacro:include filename="$(find hsrc_description)/urdf/head_v0/head.gazebo.xacro"/>
     <xacro:include filename="$(find hsrb_parts_description)/urdf/sensors/asus_xtion.urdf.xacro"/>
@@ -71,5 +70,4 @@
         </xacro:asus_xtion>
         <xacro:hsrb_head_gazebo prefix="${prefix}"/>
-        <xacro:hsrb_head_transmission prefix="${prefix}"/>
     </xacro:macro>
 </robot>

File: hsrc_description/urdf/ros2_control.robot.xacro (robot description, xacro)
@@ -54,5 +54,5 @@
                         reduction="40.273862263"
                         drive_mode="5"
-                        velocity_limit="1.0"
+                        velocity_limit="6.28"
                         gear_ratio="0.002407705"
                         torque_constant="0.0174"/>
@@ -63,23 +63,23 @@
                         reduction="1.0"
                         drive_mode="5"
-                        velocity_limit="1.0"
+                        velocity_limit="1.58"
                         gear_ratio="0.00128576"
                         torque_constant="0.0208"/>
       <xacro:hsrb_joint name="arm_roll_joint"
-                        min_angle="-2.09"
-                        max_angle="3.84"
+                        min_angle="-1.92"
+                        max_angle="3.67"
                         motor_id="23"
                         reduction="1.0"
                         drive_mode="5"
-                        velocity_limit="1.0"
+                        velocity_limit="2.0"
                         gear_ratio="0.003333333"
                         torque_constant="0.0184"/>
       <xacro:hsrb_joint name="wrist_flex_joint"
-                        min_angle="-1.92"
+                        min_angle="-1.75"
                         max_angle="1.22"
                         motor_id="24"
                         reduction="1.0"
                         drive_mode="5"
-                        velocity_limit="1.0"
+                        velocity_limit="2.0"
                         gear_ratio="0.0035"
                         torque_constant="0.0184"/>
@@ -89,6 +89,6 @@
                         motor_id="25"
                         reduction="1.0"
-                        drive_mode="5"
-                        velocity_limit="1.0"
+                        drive_mode="7"
+                        velocity_limit="2.0"
                         gear_ratio="0.0035"
                         torque_constant="0.0184"/>
@@ -99,5 +99,5 @@
                         reduction="1.0"
                         drive_mode="5"
-                        velocity_limit="1.0"
+                        velocity_limit="2.0"
                         gear_ratio="0.01"
                         torque_constant="0.0184"/>
@@ -108,5 +108,5 @@
                         reduction="-1.0"
                         drive_mode="5"
-                        velocity_limit="1.0"
+                        velocity_limit="2.0"
                         gear_ratio="0.0028"
                         torque_constant="0.0184"/>

File: hsrc_description/urdf/torso_v0/torso.gazebo.xacro (robot description, xacro)
@@ -5,5 +5,5 @@
         <xacro:gazebo_joint_mimic name="${prefix}_lift_joint"/>
         <gazebo>
-            <plugin name="torso_mimic_plugin" filename="libtmc_gazebo_mimic_plugin.so">
+            <plugin name="torso_mimic_plugin" filename="libtmc_gazebo_ros_mimic_joint.so">
                 <joint>${prefix}_lift_joint</joint>
                 <mimicJoint>${mimic_joint}</mimicJoint>

File: hsrc_description/urdf/wrist_v0/wrist.urdf.xacro (robot description, xacro)
@@ -1,5 +1,4 @@
 <?xml version="1.0"?>
 <robot name="wrist" xmlns:xacro="http://ros.org/wiki/xacro">
-    <xacro:include filename="$(find hsrc_description)/urdf/wrist_v0/wrist.transmission.xacro"/>
     <xacro:include filename="$(find hsrc_description)/urdf/wrist_v0/wrist.gazebo.xacro"/>
     <xacro:include filename="$(find hsrb_parts_description)/urdf/sensors/minebea_ft_sensor.urdf.xacro"/>
@@ -88,5 +87,4 @@
         </xacro:minebea_ft_sensor>
         <xacro:hsrb_wrist_gazebo prefix="${prefix}"/>
-        <xacro:hsrb_wrist_transmission prefix="${prefix}"/>
     </xacro:macro>
 </robot>
