Commit message: add discription hsrc_ex

File: hsrc_description/robots/hsrc1s.urdf.xacro (robot description, xacro)
@@ -29,5 +29,5 @@
     </xacro:hsrb_torso>
     <xacro:hsrb_head prefix="head" parent="torso_lift_link">
-        <origin xyz="0.0 0.0 0.0" rpy="0.0 0.0 0.0"/>
+        <origin xyz="-0.04 0.0 0.0" rpy="0.0 0.0 0.0"/>
     </xacro:hsrb_head>
     <xacro:hsrb_arm prefix="arm" parent="base_link">

File: hsrc_description/urdf/arm_v0/arm.urdf.xacro (robot description, xacro)
@@ -42,5 +42,5 @@
                 <mass value="1.339295"/>
                 <origin xyz="0.000632 0.006404 0.118529"/>
-                <inertia ixx="7.528" ixy="-0.000020284207" ixz="-0.000022947194"
+                <inertia ixx="0.007528" ixy="-0.000020284207" ixz="-0.000022947194"
                     iyy="0.007102" iyz="-0.000091796075" izz="0.001552"/>
             </inertial>
@@ -52,5 +52,5 @@
             <collision>
                 <geometry>
-                    <mesh filename="package://hsrc_description/meshes/arm_v0/arm_flex.stl" />
+                    <mesh filename="package://hsrc_description/meshes/arm_v0/arm_flex.stl" scale="1000.0 1000.0 1000.0"/>
                 </geometry>
             </collision>
@@ -81,4 +81,33 @@
                 </geometry>
             </collision>
+            <!-- for enhanced -->
+            <visual>
+                <origin xyz="-0.020 -0.0434 -0.067888" rpy="1.5707963267948966 0.0 0.0"/>
+                <geometry>
+                    <cylinder radius="0.013" length="0.0568" />
+                </geometry>
+                <material name="body_sub" />
+            </visual>
+            <visual>
+                <origin xyz="0.000 0.0484 -0.070588" rpy="-1.5707963267948966 0.0 0.0"/>
+                <geometry>
+                    <cylinder radius="0.013" length="0.0468" />
+                </geometry>
+                <material name="body_sub" />
+            </visual>
+            <collision>
+                <origin xyz="-0.020 -0.0444 -0.067888" rpy="1.5707963267948966 0.0 0.0"/>
+                <geometry>
+                    <cylinder radius="0.014" length="0.0568" />
+                </geometry>
+                <material name="body_sub" />
+            </collision>
+            <collision>
+                <origin xyz="0.0065 0.0494 -0.070588" rpy="-1.5707963267948966 0.0 0.0"/>
+                <geometry>
+                    <cylinder radius="0.014" length="0.0468" />
+                </geometry>
+                <material name="body_sub" />
+            </collision>
         </link>
         <xacro:hsrb_arm_gazebo prefix="${prefix}"/>

File: hsrc_description/urdf/base_v0/base.urdf.xacro (robot description, xacro)
@@ -6,14 +6,24 @@
     <!-- constant -->
     <xacro:property name="drive_wheel_width" value="0.03" />
-    <xacro:property name="drive_wheel_radius" value="0.0445" />
-    <xacro:property name="drive_wheel_offset_x" value="0.110" />
-    <xacro:property name="drive_wheel_offset_y" value="0.133" />
-    <xacro:property name="passive_wheel_radius" value="0.0245" />
+    <!-- <xacro:property name="drive_wheel_radius" value="0.0445" /> -->
+    <xacro:property name="drive_wheel_radius" value="0.04725" />
+    <!-- <xacro:property name="drive_wheel_offset_x" value="0.110" />
+    <xacro:property name="drive_wheel_offset_y" value="0.133" /> -->
+    <xacro:property name="drive_wheel_offset_x" value="0.114" />
+    <xacro:property name="drive_wheel_offset_y" value="0.1245" />
+    <!-- <xacro:property name="passive_wheel_radius" value="0.0245" />
     <xacro:property name="passive_wheel_offset_x" value="0.1665" />
+    <xacro:property name="passive_wheel_offset_y" value="0.055" /> -->
+    <xacro:property name="passive_wheel_radius" value="0.025" />
+    <xacro:property name="passive_wheel_offset_x" value="0.1495" />
     <xacro:property name="passive_wheel_offset_y" value="0.055" />
-    <xacro:property name="drive_wheel_max_effort" value="28.0" />
-    <xacro:property name="drive_wheel_max_velocity" value="20.8" />
-    <xacro:property name="roll_joint_max_effort" value="34.46" />
-    <xacro:property name="roll_joint_max_velocity" value="2.5" />
+    <!-- <xacro:property name="drive_wheel_max_effort" value="28.0" />
+    <xacro:property name="drive_wheel_max_velocity" value="20.8" /> -->
+    <xacro:property name="drive_wheel_max_effort" value="20.0"/>
+    <xacro:property name="drive_wheel_max_velocity" value="35.0" />
+    <!-- <xacro:property name="roll_joint_max_effort" value="34.46" />
+    <xacro:property name="roll_joint_max_velocity" value="2.5" /> -->
+    <xacro:property name="roll_joint_max_effort" value="50.0"/>
+    <xacro:property name="roll_joint_max_velocity" value="11.6" />
     <!-- drive wheel -->
     <xacro:macro name="hsrb_drive_wheel" params="prefix suffix parent *origin">
@@ -115,6 +125,6 @@
                 <mass value="0.06"/>
                 <inertia
-                    ixx="0.001437"  ixy="0.0"  ixz="0.0"
-                    iyy="0.001437" iyz="0.0" izz="0.002875" />
+                    ixx="0.001537"  ixy="0.0"  ixz="0.0"
+                    iyy="0.001537" iyz="0.0" izz="0.002875" />
             </inertial>
             <visual>

File: hsrc_description/urdf/hand_v0/hand.urdf.xacro (robot description, xacro)
@@ -2,5 +2,6 @@
 <robot name="hand" xmlns:xacro="http://ros.org/wiki/xacro">
     <xacro:include filename="$(find hsrc_description)/urdf/hand_v0/hand.gazebo.xacro"/>
-    <xacro:include filename="$(find hsrb_parts_description)/urdf/sensors/wide_camera.urdf.xacro"/>
+    <!-- <xacro:include filename="$(find hsrb_parts_description)/urdf/sensors/wide_camera.urdf.xacro"/> -->
+    <xacro:include filename="$(find hsrc_parts_description)/urdf/sensors/intel_d405.urdf.xacro"/>
     <xacro:property name="palm_to_proximal_x" value="-0.031" />
     <xacro:property name="palm_to_proximal_y" value="-0.0245" />
@@ -21,6 +22,6 @@
                 <mass value="0.01"/>
                 <inertia
-                    ixx="0.0" ixy="0.0" ixz="0.0"
-                    iyy="0.0" iyz="0.0" izz="0.0"/>
+                    ixx="0.001" ixy="0.0" ixz="0.0"
+                    iyy="0.001" iyz="0.0" izz="0.001"/>
             </inertial>
         </link>
@@ -76,7 +77,12 @@
         </xacro:hsrb_finger_without_vacuum>
         <!-- camera -->
-        <xacro:wide_camera prefix="${prefix}" parent="${prefix}_palm_link" robot_namespace="${personal_name}" rpy="${pi/2.0} ${-pi/2.0} 0" >
+        <!-- <xacro:wide_camera prefix="${prefix}" parent="${prefix}_palm_link" robot_namespace="${personal_name}" rpy="${pi/2.0} ${-pi/2.0} 0" >
             <origin xyz="0.026 0.0 0.0034" rpy="0.0 0.0 0.0"/>
-        </xacro:wide_camera>
+        </xacro:wide_camera> -->
+        <xacro:d405 parent="${prefix}_palm_link" robot_namespace="${personal_name}/${robot_name}" sensor_name="${prefix}_camera">
+            <!-- <origin xyz="0.05846 0.00629 -0.00169" rpy="0.031 -0.964 3.087"/> -->
+	    <origin xyz="0.03846 0.01529 -0.0469" rpy="0.0311676 -0.9649463 3.087223"/>
+            <!-- <origin xyz="0.03846 0.00629 -0.0469" rpy="0.0311676 -0.9649463 3.087223"/> -->
+        </xacro:d405>
         <xacro:hsrb_hand_gazebo prefix="${prefix}"/>
     </xacro:macro>
@@ -143,6 +149,6 @@
                 <origin xyz="0.021418 0.00248 0.022688"/>
                 <inertia
-                    ixx="0.0" ixy="0.0" ixz="0.0"
-                    iyy="0.0" iyz="0.0" izz="0.0"/>
+                    ixx="0.001" ixy="0.0" ixz="0.0"
+                    iyy="0.001" iyz="0.0" izz="0.001"/>
             </inertial>
             <visual>
@@ -152,6 +158,7 @@
             </visual>
             <collision>
-                <geometry>
-                    <mesh filename="package://hsrc_description/meshes/hand_v0/l_proximal.stl" />
+                <origin xyz="0.0169 -0.004125 0.035" rpy="0.0 0.0 0.0" />
+                <geometry>
+                    <box size="0.0362 0.01575 0.04"/>
                 </geometry>
             </collision>
@@ -166,6 +173,6 @@
                 <origin xyz="0.011116 0.005679 0.017532"/>
                 <inertia
-                    ixx="0.0" ixy="0.0" ixz="0.0"
-                    iyy="0.0" iyz="0.0" izz="0.0"/>
+                    ixx="0.001" ixy="0.0" ixz="0.0"
+                    iyy="0.001" iyz="0.0" izz="0.001"/>
             </inertial>
             <visual>
@@ -175,6 +182,7 @@
             </visual>
             <collision>
-                <geometry>
-                    <mesh filename="package://hsrc_description/meshes/hand_v0/l_distal.stl" />
+                <origin xyz="0.02 0.014 0.025" rpy="0.0 0.0 0.0" />
+                <geometry>
+                    <box size="0.04 0.01 0.032"/>
                 </geometry>
             </collision>
@@ -220,6 +228,6 @@
                 <origin xyz="0.013203 0.002096 0.023311"/>
                 <inertia
-                    ixx="0.0" ixy="0.0" ixz="0.0"
-                    iyy="0.0" iyz="0.0" izz="0.0"/>
+                    ixx="0.001" ixy="0.0" ixz="0.0"
+                    iyy="0.001" iyz="0.0" izz="0.001"/>
             </inertial>
             <visual>
@@ -229,6 +237,7 @@
             </visual>
             <collision>
-                <geometry>
-                    <mesh filename="package://hsrc_description/meshes/hand_v0/r_proximal.stl" />
+                <origin xyz="0.0169 0.004125 0.035" rpy="0.0 0.0 0.0" />
+                <geometry>
+                    <box size="0.0362 0.01575 0.04"/>
                 </geometry>
             </collision>
@@ -243,6 +252,6 @@
                 <origin xyz="0.014256 -0.008321 0.015591"/>
                 <inertia
-                    ixx="0.0" ixy="0.0" ixz="0.0"
-                    iyy="0.0" iyz="0.0" izz="0.0"/>
+                    ixx="0.001" ixy="0.0" ixz="0.0"
+                    iyy="0.001" iyz="0.0" izz="0.001"/>
             </inertial>
             <visual>
@@ -252,6 +261,7 @@
             </visual>
             <collision>
-                <geometry>
-                    <mesh filename="package://hsrc_description/meshes/hand_v0/r_distal.stl" />
+                <origin xyz="0.02 -0.0015 0.02" rpy="0.0 0.0 0.0" />
+                <geometry>
+                    <box size="0.04 0.023 0.04"/>
                 </geometry>
             </collision>

File: hsrc_description/urdf/head_v0/head.urdf.xacro (robot description, xacro)
@@ -2,5 +2,6 @@
 <robot name="head" xmlns:xacro="http://ros.org/wiki/xacro">
     <xacro:include filename="$(find hsrc_description)/urdf/head_v0/head.gazebo.xacro"/>
-    <xacro:include filename="$(find hsrb_parts_description)/urdf/sensors/asus_xtion.urdf.xacro"/>
+    <!-- <xacro:include filename="$(find hsrb_parts_description)/urdf/sensors/asus_xtion.urdf.xacro"/> -->
+    <xacro:include filename="$(find hsrc_parts_description)/urdf/sensors/Gemini336L.urdf.xacro"/>
     <xacro:include filename="$(find hsrb_parts_description)/urdf/sensors/pointgrey_chameleon.urdf.xacro"/>
     <xacro:include filename="$(find hsrb_parts_description)/urdf/sensors/wide_camera.urdf.xacro"/>
@@ -36,5 +37,6 @@
             <origin xyz="0.02 0.0 0.0" rpy="0.0 0.0 0.0" />
             <axis xyz="0.0 -1.0 0.0" />
-            <limit effort="100.0" velocity="1.0" lower="-1.57" upper="0.52" />
+            <!-- <limit effort="100.0" velocity="1.0" lower="-1.57" upper="0.52" /> -->
+            <limit effort="100.0" velocity="1.0" lower="-1.58" upper="0.55" />
             <parent link="${prefix}_pan_link" />
             <child link="${prefix}_tilt_link" />
@@ -66,7 +68,11 @@
             <origin xyz="0.0262 -0.07 0.08" rpy="${-pi/2.0} 0.0 ${-pi/2.0}"/>
         </xacro:pointgrey_chameleon>
-        <xacro:asus_xtion prefix="${prefix}" parent="${prefix}_tilt_link" robot_namespace="${personal_name}" sensor_name="rgbd_sensor">
+        <!-- <xacro:asus_xtion prefix="${prefix}" parent="${prefix}_tilt_link" robot_namespace="${personal_name}" sensor_name="rgbd_sensor">
             <origin xyz="-0.0786 0.022 0.248" rpy="${-pi/2.0} 0.0 ${-pi/2.0}"/>
-        </xacro:asus_xtion>
+        </xacro:asus_xtion> -->
+        <xacro:gemini336l parent="${prefix}_tilt_link" robot_namespace="${personal_name}/${robot_name}" sensor_name="head_rgbd_sensor">
+            <origin xyz="-0.09542 0.0 0.23299" rpy="0.0 0.0 0.0"/>
+            <!-- <origin xyz="-0.07550 0.05367 0.23223" rpy="0.00785 0.00571 -0.00718"/> -->
+        </xacro:gemini336l>
         <xacro:hsrb_head_gazebo prefix="${prefix}"/>
     </xacro:macro>

File: hsrc_description/urdf/ros2_control.robot.xacro (robot description, xacro)
@@ -56,5 +56,5 @@
                         reduction="40.273862263"
                         drive_mode="5"
-                        velocity_limit="6.05"
+                        velocity_limit="30.0"
                         gear_ratio="0.002407705"
                         torque_constant="0.0174"/>
@@ -65,5 +65,5 @@
                         reduction="1.0"
                         drive_mode="5"
-                        velocity_limit="1.58"
+                        velocity_limit="6.0"
                         gear_ratio="0.00128576"
                         torque_constant="0.0208"/>
@@ -74,5 +74,5 @@
                         reduction="1.0"
                         drive_mode="5"
-                        velocity_limit="2.0"
+                        velocity_limit="4.0"
                         gear_ratio="0.003333333"
                         torque_constant="0.0184"/>
@@ -83,5 +83,5 @@
                         reduction="1.0"
                         drive_mode="5"
-                        velocity_limit="2.0"
+                        velocity_limit="6.0"
                         gear_ratio="0.0035"
                         torque_constant="0.0184"/>
@@ -92,5 +92,5 @@
                         reduction="1.0"
                         drive_mode="7"
-                        velocity_limit="2.0"
+                        velocity_limit="6.0"
                         gear_ratio="0.0035"
                         torque_constant="0.0184"/>
@@ -101,14 +101,14 @@
                         reduction="1.0"
                         drive_mode="5"
-                        velocity_limit="2.0"
+                        velocity_limit="9.0"
                         gear_ratio="0.01"
                         torque_constant="0.0184"/>
       <xacro:hsrb_joint name="head_tilt_joint"
-                        min_angle="-1.57"
-                        max_angle="0.52"
+                        min_angle="-1.58"
+                        max_angle="0.55"
                         motor_id="32"
                         reduction="-1.0"
                         drive_mode="5"
-                        velocity_limit="2.0"
+                        velocity_limit="2.6"
                         gear_ratio="0.0028"
                         torque_constant="0.0184"/>
@@ -130,9 +130,9 @@
                         reduction="1.0"
                         drive_mode="3"
-                        velocity_limit="20.8"
+                        velocity_limit="35.0"
                         gear_ratio="0.006451613"
                         torque_constant="0.0174"
                         control_type="Wheel"
-                        acceleration_limit="41.7"/>
+                        acceleration_limit="20.0"/>
       <xacro:hsrb_joint name="base_r_drive_wheel_joint"
                         min_angle="-999999"
@@ -141,9 +141,9 @@
                         reduction="1.0"
                         drive_mode="3"
-                        velocity_limit="20.8"
+                        velocity_limit="35.0"
                         gear_ratio="0.006451613"
                         torque_constant="0.0174"
                         control_type="Wheel"
-                        acceleration_limit="41.7"/>
+                        acceleration_limit="20.0"/>
       <xacro:hsrb_joint name="base_roll_joint"
                         min_angle="-999999"
@@ -152,10 +152,10 @@
                         reduction="-1.0"
                         drive_mode="3"
-                        velocity_limit="2.5"
+                        velocity_limit="11.6"
                         gear_ratio="0.003333333"
                         torque_constant="0.0368"
                         acceleration_limit="5.0"/>
     </ros2_control>
-    <ros2_control name="hsrb_gpio" type="system">
+    <!-- <ros2_control name="hsrb_gpio" type="system">
       <hardware>
         <plugin>hsrb_cgos_driver/HsrbCgosHw</plugin>
@@ -171,5 +171,5 @@
         <param name="direction">out</param>
       </gpio>
-    </ros2_control>
+    </ros2_control> -->
   </xacro:macro>
 </robot>

File: hsrc_description/urdf/wrist_v0/wrist.urdf.xacro (robot description, xacro)
@@ -58,5 +58,6 @@
         </link>
         <joint name="${prefix}_ft_sensor_frame_inverse_joint" type="fixed">
-            <origin xyz="0.0 0.0 0.1" rpy="-${pi} 0.0 0.0"/>
+            <!-- <origin xyz="0.0 0.0 0.1" rpy="-${pi} 0.0 0.0"/> -->
+            <origin xyz="0.0 0.0 -0.1" rpy="0.0 0.0 -1.57"/>
             <parent link="${prefix}_ft_sensor_frame" />
             <child link="${prefix}_roll_link" />
@@ -84,5 +85,6 @@
             robot_namespace="${robot_namespace}"
 	    parent="${prefix}_ft_sensor_mount_link">
-	  <origin xyz="0.0 0.0 0.1" rpy="${pi} 0.0 0.0"/>
+	  <!-- <origin xyz="0.0 0.0 0.1" rpy="${pi} 0.0 0.0"/> -->
+            <origin xyz="0.0 0.0 0.1" rpy="0.0 0.0 1.57"/>
         </xacro:minebea_ft_sensor>
         <xacro:hsrb_wrist_gazebo prefix="${prefix}"/>
